File: KICAD_Project/sub_circuits/efi-drivers.sch (KiCad schematic (older format))
At the start: 26 parts, among them Q501 IRGB14C40LPBF, Q502 IRGB14C40LPBF, Q503 IRGB14C40LPBF, Q504 IRGB14C40LPBF, Q505 IRGB14C40LPBF, Q506 IRGB14C40LPBF, Q507 IRGB14C40LPBF, Q508 IRGB14C40LPBF, U723 74HCT244_THRU

Commit message: Looks like the bulk components are golden now, there are still a couple straglers, mostly switch mode power supply stuff.
Signed-off-by: Jared Harvey <TortiseGIT@jaredharvey.com>
Parts:
- R1448: footprint (none) -> SM0805; construct (none) -> thick film; mfg,mfg# (none) -> BOURNS,CR0805-FX-1002ELF; misc (none) -> other,more,stuff; tolerance (none) -> 1%; vend1,vend1# (none) -> newark,02J2368; w (none) -> 125mW
- R511, R512, R513, R514, R515, R516, R517, R518: footprint R3_SM0805 -> SM0805; SM mfg># SM>> -> (none); SM vend1># SM>digikey>RHM1.00KCRCT-ND -> (none); construct Thick film -> thick film; mfg,mfg# (none) -> vishay,CRCW08051K00FKTA; power .125w -> (none); thru mfg># TH>> -> (none); thru vend1># TH>digikey> -> (none); tolerance 5% -> 1%; vend1,vend1# (none) -> newark,05F1507; w (none) -> 125mW
Changed lines of the file:
@@
 F 0 "R1448" V 5430 10600 50  0000 C CNN
 F 1 "10K" V 5350 10600 50  0000 C CNN
+F 2 "SM0805" V 1130 2600 60  0001 C CNN
+F 4 "BOURNS,CR0805-FX-1002ELF" V 1130 2600 60  0001 C CNN "mfg,mfg#"
+F 5 "newark,02J2368" V 1130 2600 60  0001 C CNN "vend1,vend1#"
+F 6 "" V 1130 2600 60  0001 C CNN ""
+F 7 "" V 1130 2600 60  0001 C CNN ""
+F 8 "125mW" V 1130 2600 60  0001 C CNN "w"
+F 9 "1%" V 1130 2600 60  0001 C CNN "tolerance"
+F 10 "thick film" V 1130 2600 60  0001 C CNN "construct"
+F 11 "other,more,stuff" V 1130 2600 60  0001 C CNN "misc"
 	1    5350 10600
 	-1   0    0    1
@@
 F 0 "R518" V 8980 9950 50  0000 C CNN
 F 1 "1K" V 8900 9950 50  0000 C CNN
-F 2 "R3_SM0805" V 1130 2600 60  0001 C CNN
-F 4 "SM>>" V 1130 2600 60  0001 C CNN "SM mfg>#"
-F 5 "TH>>" V 1130 2600 60  0001 C CNN "thru mfg>#"
-F 6 "SM>digikey>RHM1.00KCRCT-ND" V 1130 2600 60  0001 C CNN "SM vend1>#"
-F 7 "TH>digikey>" V 1130 2600 60  0001 C CNN "thru vend1>#"
-F 8 ".125w" V 1130 2600 60  0001 C CNN "power"
-F 9 "5%" V 1130 2600 60  0001 C CNN "tolerance"
-F 10 "Thick film" V 1130 2600 60  0001 C CNN "construct"
+F 2 "SM0805" V 1130 2600 60  0001 C CNN
+F 4 "vishay,CRCW08051K00FKTA" V 1130 2600 60  0001 C CNN "mfg,mfg#"
+F 5 "newark,05F1507" V 1130 2600 60  0001 C CNN "vend1,vend1#"
+F 6 "" V 1130 2600 60  0001 C CNN ""
+F 7 "" V 1130 2600 60  0001 C CNN ""
+F 8 "125mW" V 1130 2600 60  0001 C CNN "w"
+F 9 "1%" V 1130 2600 60  0001 C CNN "tolerance"
+F 10 "thick film" V 1130 2600 60  0001 C CNN "construct"
 F 11 "other,more,stuff" V 1130 2600 60  0001 C CNN "misc"
 	1    8900 9950
@@
 F 0 "R517" V 8980 8700 50  0000 C CNN
 F 1 "1K" V 8900 8700 50  0000 C CNN
-F 2 "R3_SM0805" V 1130 2600 60  0001 C CNN
-F 4 "SM>>" V 1130 2600 60  0001 C CNN "SM mfg>#"
-F 5 "TH>>" V 1130 2600 60  0001 C CNN "thru mfg>#"
-F 6 "SM>digikey>RHM1.00KCRCT-ND" V 1130 2600 60  0001 C CNN "SM vend1>#"
-F 7 "TH>digikey>" V 1130 2600 60  0001 C CNN "thru vend1>#"
-F 8 ".125w" V 1130 2600 60  0001 C CNN "power"
-F 9 "5%" V 1130 2600 60  0001 C CNN "tolerance"
-F 10 "Thick film" V 1130 2600 60  0001 C CNN "construct"
+F 2 "SM0805" V 1130 2600 60  0001 C CNN
+F 4 "vishay,CRCW08051K00FKTA" V 1130 2600 60  0001 C CNN "mfg,mfg#"
+F 5 "newark,05F1507" V 1130 2600 60  0001 C CNN "vend1,vend1#"
+F 6 "" V 1130 2600 60  0001 C CNN ""
+F 7 "" V 1130 2600 60  0001 C CNN ""
+F 8 "125mW" V 1130 2600 60  0001 C CNN "w"
+F 9 "1%" V 1130 2600 60  0001 C CNN "tolerance"
+F 10 "thick film" V 1130 2600 60  0001 C CNN "construct"
 F 11 "other,more,stuff" V 1130 2600 60  0001 C CNN "misc"
 	1    8900 8700
@@
 F 0 "R516" V 8980 7450 50  0000 C CNN
 F 1 "1K" V 8900 7450 50  0000 C CNN
-F 2 "R3_SM0805" V 1130 2600 60  0001 C CNN
-F 4 "SM>>" V 1130 2600 60  0001 C CNN "SM mfg>#"
-F 5 "TH>>" V 1130 2600 60  0001 C CNN "thru mfg>#"
-F 6 "SM>digikey>RHM1.00KCRCT-ND" V 1130 2600 60  0001 C CNN "SM vend1>#"
-F 7 "TH>digikey>" V 1130 2600 60  0001 C CNN "thru vend1>#"
-F 8 ".125w" V 1130 2600 60  0001 C CNN "power"
-F 9 "5%" V 1130 2600 60  0001 C CNN "tolerance"
-F 10 "Thick film" V 1130 2600 60  0001 C CNN "construct"
+F 2 "SM0805" V 1130 2600 60  0001 C CNN
+F 4 "vishay,CRCW08051K00FKTA" V 1130 2600 60  0001 C CNN "mfg,mfg#"
+F 5 "newark,05F1507" V 1130 2600 60  0001 C CNN "vend1,vend1#"
+F 6 "" V 1130 2600 60  0001 C CNN ""
+F 7 "" V 1130 2600 60  0001 C CNN ""
+F 8 "125mW" V 1130 2600 60  0001 C CNN "w"
+F 9 "1%" V 1130 2600 60  0001 C CNN "tolerance"
+F 10 "thick film" V 1130 2600 60  0001 C CNN "construct"
 F 11 "other,more,stuff" V 1130 2600 60  0001 C CNN "misc"
 	1    8900 7450
@@
 F 0 "R515" V 8980 6200 50  0000 C CNN
 F 1 "1K" V 8900 6200 50  0000 C CNN
-F 2 "R3_SM0805" V 1130 2600 60  0001 C CNN
-F 4 "SM>>" V 1130 2600 60  0001 C CNN "SM mfg>#"
-F 5 "TH>>" V 1130 2600 60  0001 C CNN "thru mfg>#"
-F 6 "SM>digikey>RHM1.00KCRCT-ND" V 1130 2600 60  0001 C CNN "SM vend1>#"
-F 7 "TH>digikey>" V 1130 2600 60  0001 C CNN "thru vend1>#"
-F 8 ".125w" V 1130 2600 60  0001 C CNN "power"
-F 9 "5%" V 1130 2600 60  0001 C CNN "tolerance"
-F 10 "Thick film" V 1130 2600 60  0001 C CNN "construct"
+F 2 "SM0805" V 1130 2600 60  0001 C CNN
+F 4 "vishay,CRCW08051K00FKTA" V 1130 2600 60  0001 C CNN "mfg,mfg#"
+F 5 "newark,05F1507" V 1130 2600 60  0001 C CNN "vend1,vend1#"
+F 6 "" V 1130 2600 60  0001 C CNN ""
+F 7 "" V 1130 2600 60  0001 C CNN ""
+F 8 "125mW" V 1130 2600 60  0001 C CNN "w"
+F 9 "1%" V 1130 2600 60  0001 C CNN "tolerance"
+F 10 "thick film" V 1130 2600 60  0001 C CNN "construct"
 F 11 "other,more,stuff" V 1130 2600 60  0001 C CNN "misc"
 	1    8900 6200
@@
 F 0 "R514" V 8980 4950 50  0000 C CNN
 F 1 "1K" V 8900 4950 50  0000 C CNN
-F 2 "R3_SM0805" V 1130 2600 60  0001 C CNN
-F 4 "SM>>" V 1130 2600 60  0001 C CNN "SM mfg>#"
-F 5 "TH>>" V 1130 2600 60  0001 C CNN "thru mfg>#"
-F 6 "SM>digikey>RHM1.00KCRCT-ND" V 1130 2600 60  0001 C CNN "SM vend1>#"
-F 7 "TH>digikey>" V 1130 2600 60  0001 C CNN "thru vend1>#"
-F 8 ".125w" V 1130 2600 60  0001 C CNN "power"
-F 9 "5%" V 1130 2600 60  0001 C CNN "tolerance"
-F 10 "Thick film" V 1130 2600 60  0001 C CNN "construct"
+F 2 "SM0805" V 1130 2600 60  0001 C CNN
+F 4 "vishay,CRCW08051K00FKTA" V 1130 2600 60  0001 C CNN "mfg,mfg#"
+F 5 "newark,05F1507" V 1130 2600 60  0001 C CNN "vend1,vend1#"
+F 6 "" V 1130 2600 60  0001 C CNN ""
+F 7 "" V 1130 2600 60  0001 C CNN ""
+F 8 "125mW" V 1130 2600 60  0001 C CNN "w"
+F 9 "1%" V 1130 2600 60  0001 C CNN "tolerance"
+F 10 "thick film" V 1130 2600 60  0001 C CNN "construct"
 F 11 "other,more,stuff" V 1130 2600 60  0001 C CNN "misc"
 	1    8900 4950
@@
 F 0 "R513" V 8980 3700 50  0000 C CNN
 F 1 "1K" V 8900 3700 50  0000 C CNN
-F 2 "R3_SM0805" V 1130 2600 60  0001 C CNN
-F 4 "SM>>" V 1130 2600 60  0001 C CNN "SM mfg>#"
-F 5 "TH>>" V 1130 2600 60  0001 C CNN "thru mfg>#"
-F 6 "SM>digikey>RHM1.00KCRCT-ND" V 1130 2600 60  0001 C CNN "SM vend1>#"
-F 7 "TH>digikey>" V 1130 2600 60  0001 C CNN "thru vend1>#"
-F 8 ".125w" V 1130 2600 60  0001 C CNN "power"
-F 9 "5%" V 1130 2600 60  0001 C CNN "tolerance"
-F 10 "Thick film" V 1130 2600 60  0001 C CNN "construct"
+F 2 "SM0805" V 1130 2600 60  0001 C CNN
+F 4 "vishay,CRCW08051K00FKTA" V 1130 2600 60  0001 C CNN "mfg,mfg#"
+F 5 "newark,05F1507" V 1130 2600 60  0001 C CNN "vend1,vend1#"
+F 6 "" V 1130 2600 60  0001 C CNN ""
+F 7 "" V 1130 2600 60  0001 C CNN ""
+F 8 "125mW" V 1130 2600 60  0001 C CNN "w"
+F 9 "1%" V 1130 2600 60  0001 C CNN "tolerance"
+F 10 "thick film" V 1130 2600 60  0001 C CNN "construct"
 F 11 "other,more,stuff" V 1130 2600 60  0001 C CNN "misc"
 	1    8900 3700
@@
 F 0 "R512" V 8980 2450 50  0000 C CNN
 F 1 "1K" V 8900 2450 50  0000 C CNN
-F 2 "R3_SM0805" V 1130 2600 60  0001 C CNN
-F 4 "SM>>" V 1130 2600 60  0001 C CNN "SM mfg>#"
-F 5 "TH>>" V 1130 2600 60  0001 C CNN "thru mfg>#"
-F 6 "SM>digikey>RHM1.00KCRCT-ND" V 1130 2600 60  0001 C CNN "SM vend1>#"
-F 7 "TH>digikey>" V 1130 2600 60  0001 C CNN "thru vend1>#"
-F 8 ".125w" V 1130 2600 60  0001 C CNN "power"
-F 9 "5%" V 1130 2600 60  0001 C CNN "tolerance"
-F 10 "Thick film" V 1130 2600 60  0001 C CNN "construct"
+F 2 "SM0805" V 1130 2600 60  0001 C CNN
+F 4 "vishay,CRCW08051K00FKTA" V 1130 2600 60  0001 C CNN "mfg,mfg#"
+F 5 "newark,05F1507" V 1130 2600 60  0001 C CNN "vend1,vend1#"
+F 6 "" V 1130 2600 60  0001 C CNN ""
+F 7 "" V 1130 2600 60  0001 C CNN ""
+F 8 "125mW" V 1130 2600 60  0001 C CNN "w"
+F 9 "1%" V 1130 2600 60  0001 C CNN "tolerance"
+F 10 "thick film" V 1130 2600 60  0001 C CNN "construct"
 F 11 "other,more,stuff" V 1130 2600 60  0001 C CNN "misc"
 	1    8900 2450
@@
 F 0 "R511" V 8980 1200 50  0000 C CNN
 F 1 "1K" V 8900 1200 50  0000 C CNN
-F 2 "R3_SM0805" V 1130 2600 60  0001 C CNN
-F 4 "SM>>" V 1130 2600 60  0001 C CNN "SM mfg>#"
-F 5 "TH>>" V 1130 2600 60  0001 C CNN "thru mfg>#"
-F 6 "SM>digikey>RHM1.00KCRCT-ND" V 1130 2600 60  0001 C CNN "SM vend1>#"
-F 7 "TH>digikey>" V 1130 2600 60  0001 C CNN "thru vend1>#"
-F 8 ".125w" V 1130 2600 60  0001 C CNN "power"
-F 9 "5%" V 1130 2600 60  0001 C CNN "tolerance"
-F 10 "Thick film" V 1130 2600 60  0001 C CNN "construct"
+F 2 "SM0805" V 1130 2600 60  0001 C CNN
+F 4 "vishay,CRCW08051K00FKTA" V 1130 2600 60  0001 C CNN "mfg,mfg#"
+F 5 "newark,05F1507" V 1130 2600 60  0001 C CNN "vend1,vend1#"
+F 6 "" V 1130 2600 60  0001 C CNN ""
+F 7 "" V 1130 2600 60  0001 C CNN ""
+F 8 "125mW" V 1130 2600 60  0001 C CNN "w"
+F 9 "1%" V 1130 2600 60  0001 C CNN "tolerance"
+F 10 "thick film" V 1130 2600 60  0001 C CNN "construct"
 F 11 "other,more,stuff" V 1130 2600 60  0001 C CNN "misc"
 	1    8900 1200
