File: KICAD_Project/sub_circuits/CAN_TJA1054.sch (KiCad schematic (older format))
At the start: 7 parts

Commit message: About to runs scripts to scrub the BOM's, so here's a backup copy in case it goes wrong.
Signed-off-by: Jared Harvey <TortiseGIT@jaredharvey.com>
Parts:
- removed C?: 100nF, SM0805-C1, symbol C
- removed C?: 10uF, SM0805-C1, symbol C
- removed P? (x2): CONN_1, PINTST, symbol CONN_1
- removed R?: 511, SM0805-R4, symbol R
- added C1001: 100nF, SM0805-C1, symbol C
- added C1002: 10uF, SM0805-C1, symbol C
- added P1001, P1002: CONN_1, PINTST, symbol CONN_1
- added R1001: 511, SM0805, symbol R
- R1002: renamed from R?; footprint SM0805-R4 -> SM0805
- gave numbers to parts that had none: 1
Changed lines of the file:
@@
-EESchema Schematic File Version 2  date 8/7/2011 7:33:15 PM
+EESchema Schematic File Version 2  date 8/14/2011 3:32:15 PM
 LIBS:power
 LIBS:device
@@
 $Descr User 11000 8500
 encoding utf-8
-Sheet 10 14
+Sheet 10 13
 Title "freeEMS PLUS from Cinch template "
-Date "7 aug 2011"
+Date "14 aug 2011"
 Rev "A"
 Comp "diyefi.org/openecu.info"
@@
 $EndDescr
 $Comp
-L R R?
+L R R1002
 U 1 1 4C313BED
 P 9400 6700
-F 0 "R?" V 9300 6700 50  0000 C CNN
+F 0 "R1002" V 9300 6700 50  0000 C CNN
 F 1 "511" V 9400 6700 50  0000 C CNN
-F 2 "SM0805-R4" V 9580 6800 60  0001 C CNN
+F 2 "SM0805" V 9580 6800 60  0001 C CNN
 F 4 "multicomp,MC0805S8F5110T5E" V 5580 8350 60  0001 C CNN "mfg,#"
 F 5 "newark,04P0624" V 5580 8350 60  0001 C CNN "vend,#"
@@
 $EndComp
 Wire Wire Line
-	9725 6200 9800 6200
+	9800 6200 9725 6200
 Wire Wire Line
 	9725 6200 9725 6600
@@
 TJA1054_TXD
 $Comp
-L CONN_1 P?
-U 1 1 4C0A3402
+L CONN_1 P1002
+U 1 1 4E467E0E
 P 9950 6400
-F 0 "P?" H 10030 6400 40  0000 L CNN
+F 0 "P1002" H 10030 6400 40  0000 L CNN
 F 1 "CONN_1" H 9950 6455 30  0001 C CNN
 F 2 "PINTST" H 9950 6400 60  0001 C CNN
@@
 $EndComp
 $Comp
-L TJA1054A U??
+L TJA1054A U1001
 U 1 1 4C0A33D8
 P 7975 6400
-F 0 "U??" H 7975 6800 60  0000 C CNN
+F 0 "U1001" H 7975 6800 60  0000 C CNN
 F 1 "TJA1054A" H 7975 6000 50  0000 C CNN
 F 2 "SO14E" H 7975 6400 60  0001 C CNN
@@
 $EndComp
 $Comp
-L CONN_1 P?
-U 1 1 4C0A2746
+L CONN_1 P1001
+U 1 1 4E467E0C
 P 9950 6300
-F 0 "P?" H 10030 6300 40  0000 L CNN
+F 0 "P1001" H 10030 6300 40  0000 L CNN
 F 1 "CONN_1" H 9950 6355 30  0001 C CNN
 F 2 "PINTST" H 9950 6300 60  0001 C CNN
@@
 $EndComp
 $Comp
-L GND #PWR?
-U 1 1 4C09CD98
+L GND #PWR0146
+U 1 1 4E467E0B
 P 8650 6200
-F 0 "#PWR?" H 8650 6200 30  0001 C CNN
+F 0 "#PWR0146" H 8650 6200 30  0001 C CNN
 F 1 "GND" H 8650 6130 30  0001 C CNN
 	1    8650 6200
@@
 VBAT
 $Comp
-L GND #PWR?
-U 1 1 4C09CCDD
+L GND #PWR0147
+U 1 1 4E467E0A
 P 9350 6150
-F 0 "#PWR?" H 9350 6150 30  0001 C CNN
+F 0 "#PWR0147" H 9350 6150 30  0001 C CNN
 F 1 "GND" H 9350 6080 30  0001 C CNN
 	1    9350 6150
@@
 $EndComp
 $Comp
-L R R?
-U 1 1 4C09CAFD
+L R R1001
+U 1 1 4E467E09
 P 9400 6600
-F 0 "R?" V 9500 6600 50  0000 C CNN
+F 0 "R1001" V 9500 6600 50  0000 C CNN
 F 1 "511" V 9400 6600 50  0000 C CNN
-F 2 "SM0805-R4" V 9580 6700 60  0001 C CNN
+F 2 "SM0805" V 9580 6700 60  0001 C CNN
 F 4 "multicomp,MC0805S8F5110T5E" V 5580 8350 60  0001 C CNN "mfg,#"
 F 5 "newark,04P0624" V 5580 8350 60  0001 C CNN "vend,#"
@@
 $EndComp
 $Comp
-L GND #PWR?
-U 1 1 4BF65418
+L GND #PWR0148
+U 1 1 4E467E07
 P 8775 7225
-F 0 "#PWR?" H 8775 7225 30  0001 C CNN
+F 0 "#PWR0148" H 8775 7225 30  0001 C CNN
 F 1 "GND" H 8775 7155 30  0001 C CNN
 	1    8775 7225
@@
 $EndComp
 $Comp
-L C C?
-U 1 1 4BF507DC
+L C C1002
+U 1 1 4E467E01
 P 9050 6100
-F 0 "C?" V 9100 6325 50  0000 L CNN
+F 0 "C1002" V 9100 6325 50  0000 L CNN
 F 1 "10uF" V 8975 5900 50  0000 L CNN
 F 2 "SM0805-C1" V 6130 7200 60  0001 C CNN
@@
 $EndComp
 $Comp
-L C C?
-U 1 1 4BF507A3
+L C C1001
+U 1 1 4E467DFE
 P 8775 6975
-F 0 "C?" H 8800 7075 50  0000 L CNN
+F 0 "C1001" H 8800 7075 50  0000 L CNN
 F 1 "100nF" H 8525 7075 50  0000 L CNN
 F 2 "SM0805-C1" V 5855 8075 60  0001 C CNN

Commit message: caps have been done with the scripts next up is the resistors.
Signed-off-by: Jared Harvey <TortiseGIT@jaredharvey.com>
Parts:
- C1001: Field3 - -> (none); Field4 - -> (none); Field5 50,V -> (none); Field6 10,% -> (none); Field7 ceramic -> (none); Field8 other,more,stuff -> (none); V (none) -> 100V; construct (none) -> ceramic; mfg,# murata,GRM21BR71H104KA01L -> (none); mfg,mfg# (none) -> avx,08051C104KAT2A; misc (none) -> other,more,stuff; tolerance (none) -> 10%; vend,# newark,38K1694 -> (none); vend1,vend1# (none) -> newark,96M1354
Changed lines of the file:
@@
-EESchema Schematic File Version 2  date 8/14/2011 3:32:15 PM
+EESchema Schematic File Version 2  date 8/14/2011 7:31:25 PM
 LIBS:power
 LIBS:device
@@
 F 0 "C1001" H 8800 7075 50  0000 L CNN
 F 1 "100nF" H 8525 7075 50  0000 L CNN
-F 2 "SM0805-C1" V 5855 8075 60  0001 C CNN
-F 4 "murata,GRM21BR71H104KA01L" V 5855 8075 60  0001 C CNN "mfg,#"
-F 5 "newark,38K1694" V 5855 8075 60  0001 C CNN "vend,#"
-F 6 "-" V 5855 8075 60  0001 C CNN "Field3"
-F 7 "-" V 5855 8075 60  0001 C CNN "Field4"
-F 8 "50,V" V 5855 8075 60  0001 C CNN "Field5"
-F 9 "10,%" V 5855 8075 60  0001 C CNN "Field6"
-F 10 "ceramic" V 5855 8075 60  0001 C CNN "Field7"
-F 11 "other,more,stuff" V 5855 8075 60  0001 C CNN "Field8"
+F 2 "SM0805-C1" V 1130 2600 60  0001 C CNN
+F 4 "avx,08051C104KAT2A" V 1130 2600 60  0001 C CNN "mfg,mfg#"
+F 5 "newark,96M1354" V 1130 2600 60  0001 C CNN "vend1,vend1#"
+F 6 "" V 1130 2600 60  0001 C CNN ""
+F 7 "" V 1130 2600 60  0001 C CNN ""
+F 8 "100V" V 1130 2600 60  0001 C CNN "V"
+F 9 "10%" V 1130 2600 60  0001 C CNN "tolerance"
+F 10 "ceramic" V 1130 2600 60  0001 C CNN "construct"
+F 11 "other,more,stuff" V 1130 2600 60  0001 C CNN "misc"
 	1    8775 6975
 	1    0    0    1

Commit message: several pins on the SOM are now connected.
Signed-off-by: Jared Harvey <TortiseGIT@jaredharvey.com>
Parts:
- renumbered C1001 to C1101, C1002 to C1102, P1001 to P1101, P1002 to P1102, R1001 to R1101, R1002 to R1102, U1001 to U1101
Other:
- moved on the sheet: C1101, C1102, R1101, R1102
