File: KICAD_Project/sub_circuits/CAN_TJA1054.sch (KiCad schematic (older format))
At the start: 7 parts, among them P1101 CONN_1, P1102 CONN_1, U1101 TJA1054A

Commit message: Made more progress on the AN protects and LS drive 33800
Signed-off-by: Jared Harvey <TortiseGIT@jaredharvey.com>
Parts:
- C1101: footprint SM0805-C1 -> SM0805; TOL (none) -> 10%; V 100V -> 200V; construct ceramic -> CERAMIC; mfg,mfg# avx,08051C104KAT2A -> AVX,08055C104KAT2A; tolerance 10% -> (none); vend1,vend1# newark,96M1354 -> newark,27C8438
Changed lines of the file:
@@
-EESchema Schematic File Version 2  date 10/14/2011 5:26:22 AM
+EESchema Schematic File Version 2  date 10/16/2011 7:32:22 AM
 LIBS:power
 LIBS:device
@@
 $Descr User 11000 8500
 encoding utf-8
-Sheet 11 12
+Sheet 10 12
 Title "Open5xxxECU (o5e), an ECU that is no longer affiliated with freeEMS."
-Date "14 oct 2011"
+Date "16 oct 2011"
 Rev "A-DRAFT5"
 Comp "http://open5xxxecu.org/"
@@
 F 0 "C1101" H 8800 6925 50  0000 L CNN
 F 1 "100nF" H 8525 6925 50  0000 L CNN
-F 2 "SM0805-C1" V 1130 2450 60  0001 C CNN
-F 4 "avx,08051C104KAT2A" V 1130 2450 60  0001 C CNN "mfg,mfg#"
-F 5 "newark,96M1354" V 1130 2450 60  0001 C CNN "vend1,vend1#"
-F 6 "" V 1130 2450 60  0001 C CNN "Field6"
-F 7 "" V 1130 2450 60  0001 C CNN "Field7"
-F 8 "100V" V 1130 2450 60  0001 C CNN "V"
-F 9 "10%" V 1130 2450 60  0001 C CNN "tolerance"
-F 10 "ceramic" V 1130 2450 60  0001 C CNN "construct"
-F 11 "other,more,stuff" V 1130 2450 60  0001 C CNN "misc"
+F 2 "SM0805" V 1130 2600 60  0001 C CNN
+F 4 "AVX,08055C104KAT2A" V 1130 2600 60  0001 C CNN "mfg,mfg#"
+F 5 "newark,27C8438" V 1130 2600 60  0001 C CNN "vend1,vend1#"
+F 6 "" V 1130 2600 60  0001 C CNN "Field6"
+F 7 "" V 1130 2600 60  0001 C CNN "Field7"
+F 8 "200V" V 1130 2600 60  0001 C CNN "V"
+F 9 "10%" V 1130 2600 60  0001 C CNN "TOL"
+F 10 "CERAMIC" V 1130 2600 60  0001 C CNN "construct"
+F 11 "other,more,stuff" V 1130 2600 60  0001 C CNN "misc"
 	1    8775 6825
 	1    0    0    1

Commit message: about to position the regulators, save it as a backup copy
Signed-off-by: Jared Harvey <TortiseGIT@jaredharvey.com>
Parts:
- C1102: footprint SM0805-C1 -> SM0805
Changed lines of the file:
@@
-EESchema Schematic File Version 2  date 10/20/2011 5:18:40 AM
+EESchema Schematic File Version 2  date 10/21/2011 6:23:35 AM
 LIBS:power
 LIBS:device
@@
 Sheet 10 12
 Title "Open5xxxECU (o5e), an ECU that is no longer affiliated with freeEMS."
-Date "20 oct 2011"
-Rev "A-DRAFT6"
+Date "21 oct 2011"
+Rev "A-DRAFT7"
 Comp "http://open5xxxecu.org/"
 Comment1 "comms CAN/USB/Other"
@@
 F 0 "C1102" V 9100 6175 50  0000 L CNN
 F 1 "10uF" V 8975 5750 50  0000 L CNN
-F 2 "SM0805-C1" V 1130 2600 60  0001 C CNN
+F 2 "SM0805" V 1130 2600 60  0001 C CNN
 F 4 "AVX,08053C104KAT2A" V 1130 2600 60  0001 C CNN "mfg,mfg#"
 F 5 "newark,96M1381" V 1130 2600 60  0001 C CNN "vend1,vend1#"
-F 6 "" V 1130 2600 60  0001 C CNN "Field6"
-F 7 "" V 1130 2600 60  0001 C CNN "Field7"
-F 8 "25V" V 1130 2600 60  0001 C CNN "V"
-F 9 "10%" V 1130 2600 60  0001 C CNN "tolerance"
-F 10 "multi layer ceramic" V 1130 2600 60  0001 C CNN "construct"
-F 11 "other,more,stuff" V 1130 2600 60  0001 C CNN "misc"
+F 6 "25V" V 1130 2600 60  0001 C CNN "V"
+F 7 "10%" V 1130 2600 60  0001 C CNN "tolerance"
+F 8 "multi layer ceramic" V 1130 2600 60  0001 C CNN "construct"
+F 9 "other,more,stuff" V 1130 2600 60  0001 C CNN "misc"
 	1    9050 5950
 	0    1    -1   0
