File: KICAD_Project/sub_circuits/CPU.sch (KiCad schematic (older format))
At the start: 1 part

Commit message: More work to capture, also I need it up there for collaboration purposes.
Signed-off-by: Jared Harvey <TortiseGIT@jaredharvey.com>
Connections:
- net labels added: MAX9924_2_CRANK_DIGI
- net labels removed: MC33800_EN_DIGI, MC33810_1,2_OUT-EN_DIGI, MC33810_1_MAXI_DIGI, MC33810_1_NOMI_DIGI, MC33810_1_SDUR_DIGI, MC33810_1_SPI-CS, MC33810_2_MAXI_DIGI, MC33810_2_NOMI_DIGI, MC33810_2_SDUR_DIGI, MC33810_2_SPI-CS, MC33810_3_MAXI_DIGI, MC33810_3_NOMI_DIGI, MC33810_3_OUT-EN_DIGI, MC33810_3_SDUR_DIGI, MC33810_3_SPI-CS, RPM_CRANK_AN
- wire segments 291 -> 279
- no-connect marks 192 -> 191

Commit message: About to runs scripts to scrub the BOM's, so here's a backup copy in case it goes wrong.
Signed-off-by: Jared Harvey <TortiseGIT@jaredharvey.com>
Parts:
- gave numbers to parts that had none: 1

Commit message: several pins on the SOM are now connected.
Signed-off-by: Jared Harvey <TortiseGIT@jaredharvey.com>
Parts:
- renumbered P301 to P201
Connections:
- net labels added: 01_IGN_DIGI, 01_INJ_DIGI, 02_IGN_DIGI, 02_INJ_DIGI, 03_IGN_DIGI, 03_INJ_DIGI, 04_IGN_DIGI, 04_INJ_DIGI, 05_IGN_DIGI, 05_INJ_DIGI, 06_IGN_DIGI, 06_INJ_DIGI, 07_IGN_DIGI, 07_INJ_DIGI, 08_IGN_DIGI, 08_INJ_DIGI, 09_INJ_DIGI, 10_IGN_DIGI, 10_INJ_DIGI, 11_IGN_DIGI, 11_INJ_DIGI, 12_IGN_DIGI, 12_INJ_DIGI, 13_INJ_DIGI, 14_INJ_DIGI, 15_INJ_DIGI, 16_INJ_DIGI, 17_INJ_DIGI, 18_INJ_DIGI, 19_INJ_DIGI, 20_INJ_DIGI, 21_INJ_DIGI, 22_INJ_DIGI, 23_INJ_DIGI, 24_INJ_DIGI, 9_IGN_DIGI, AN_26, AN_27, AN_27_CSNS, AN_28, AN_29, AN_30, AN_31, CS-TCPL1, CS-TCPL2, MC33800_EN
- net labels removed: MC33810_1_1_IGN_DIGI, MC33810_1_1_INJ_DIGI, MC33810_1_2_IGN_DIGI, MC33810_1_2_INJ_DIGI, MC33810_1_3_IGN_DIGI, MC33810_1_3_INJ_DIGI, MC33810_1_4_IGN_DIGI, MC33810_1_4_INJ_DIGI, MC33810_2_5_IGN_DIGI, MC33810_2_5_INJ_DIGI, MC33810_2_6_IGN_DIGI, MC33810_2_6_INJ_DIGI, MC33810_2_7_IGN_DIGI, MC33810_2_7_INJ_DIGI, MC33810_2_8_IGN_DIGI, MC33810_2_8_INJ_DIGI, MC33810_3_10_IGN_DIGI, MC33810_3_10_INJ_DIGI, MC33810_3_11_IGN_DIGI, MC33810_3_11_INJ_DIGI, MC33810_3_12_IGN_DIGI, MC33810_3_12_INJ_DIGI, MC33810_3_9_IGN_DIGI, MC33810_3_9_INJ_DIGI, MISC1_AIR_TEMP_AN, MISC2_AIR_TEMP_AN
- wire segments 279 -> 281
- no-connect marks 191 -> 216
