File: KICAD_Project/sub_circuits/CPU.sch (KiCad schematic (older format))
At the start: 1 part, among them P201 MPC5554

Commit message: routing has started
Signed-off-by: Jared Harvey <TortiseGIT@jaredharvey.com>
Connections:
- net labels added: 09_IGN_DIGI, 3412_CSNS, P01, P02, P03, P04, P05, P06, P07, P08, P09, P10, P11, P12, P13, P14
- net labels removed: 9_IGN_DIGI, AN_26, AN_27, AN_27_CSNS, AN_28, AN_29, AN_30, AN_31, AN_32, AN_33, AN_34, AN_35, AN_36, AN_37, AN_38, AN_39
- wire segments 281 -> 227
- no-connect marks 216 -> 186

Commit message: Errr, routing doesn't begin yet. Still need to iron our CPU sheet.
Signed-off-by: Jared Harvey <TortiseGIT@jaredharvey.com>
Parts:
- added D201: LED, symbol LED
- added R201: 470R, symbol R
- added SW201: SWITCH_INV, symbol SWITCH_INV
- added SW202: SW_PUSH, symbol SW_PUSH
Connections:
- net labels added: RS232_2_RX, RS232_2_TX
- wire segments 227 -> 273
- no-connect marks 186 -> 166

Commit message: Changed over voltage protected MOSFETs to SO8 footprints.
Signed-off-by: Jared Harvey <TortiseGIT@jaredharvey.com>
Connections:
- net labels added: L297_CCW, L297_CLK, L297_EN
- net labels removed: MC33879_EN_DIGI, MC33879_IN5_DIGI, MC33879_IN6_DIGI, MC33879_SPI-CS
- wire segments 273 -> 272
- no-connect marks 166 -> 167
Changed lines of the file:
@@
-EESchema Schematic File Version 2  date 8/30/2011 5:58:28 AM
+EESchema Schematic File Version 2  date 9/1/2011 7:35:06 PM
 LIBS:power
 LIBS:device
@@
 Sheet 2 13
 Title "freeEMS PLUS from Cinch template "
-Date "30 aug 2011"
+Date "1 sep 2011"
 Rev "A-DRAF"
 Comp "diyefi.org/openecu.info"
@@
 Comment4 ""
 $EndDescr
+NoConn ~ 25300 6100
 Wire Wire Line
 	22750 21000 23050 21000
@@
 Wire Wire Line
 	23875 6000 23875 6025
-Wire Wire Line
-	25350 6100 25300 6100
 Wire Wire Line
 	25300 5700 25325 5700
@@
 MC10XS3412_IN0_DIGI
 Text HLabel 23850 2300 0    60   Input ~ 0
-MC33879_IN6_DIGI
+L297_CLK
 Text HLabel 25350 2100 2    60   Input ~ 0
-MC33879_IN5_DIGI
+L297_CCW
 Text HLabel 23850 2200 0    60   Input ~ 0
 MC33800_PWM6_DIGI
@@
 MC33926_EN_DIGI
 Text HLabel 23850 17600 0    60   Input ~ 0
-MC33879_EN_DIGI
+L297_EN
 Text HLabel 25300 20000 2    60   Input ~ 0
 12_IGN_DIGI
@@
 Text HLabel 23850 6400 0    60   Input ~ 0
 MC10XS3412_SPI-CS
-Text HLabel 25350 6100 2    60   Input ~ 0
-MC33879_SPI-CS
 Text HLabel 23850 6300 0    60   Input ~ 0
 MC33800_SPI-CS
