File: KICAD_Project/sub_circuits/O2_input_CJ125.sch (KiCad schematic (older format))
At the start: 27 parts

Commit message: I did a fiar bit of work, and I want to be able to step back if I can, so this is a misc check in.
Signed-off-by: Jared Harvey <TortiseGIT@jaredharvey.com>
Parts:
- added C? (x3): 33nF, SM0805-C1, symbol C
- added C? (x2): 100nF, SM0805-C1, symbol C
- added C?: 2.2nF, SM0805-C1, symbol C
- added C?: 1nF, SM0805-C1, symbol C
- added C?: 10nF, SM0805-C1, symbol C
- added P? (x6): CONN_1, PINTST, symbol CONN_1
- added R?: 4.7k, SM0805-R4, symbol R
- added R?: 470k, SM0805-R4, symbol R
- added R?: 82.5, SM0805-R4, symbol R
- added R?: 27k, SM0805-R4, symbol R
- added R? (x2): 10k, SM0805-R4, symbol R
- added R?: 6.8k, SM0805-R4, symbol R
- added R? (x2): 100k, SM0805-R4, symbol R
- added R?: 61.9, SM0805-R4, symbol R
- added R? (x2): 1k, SM0805-R4, symbol R
- added U?: CJ125, SOIC24, symbol CJ125
Connections:
- net labels added: CJ125-1_SCK, CJ125-1_SI, CJ125-1_SO, CJ125-1_SS, CJ125-1_UA, CJ125-1_UR, CJ125-2_SCK, CJ125-2_SI, CJ125-2_SO, CJ125-2_SS, CJ125-2_UA, CJ125-2_UR, DIAHD-1?, DIAHD-2?, DIAHG-1?, DIAHG-2?, IA-1?, IA-2?, IP-1?, IP-2?, O2-1_DIAHD_PIN, O2-1_DIAHG_PIN, O2-1_IA_PIN, O2-1_IP_PIN, O2-1_UN_PIN, O2-1_VM_PIN, O2-2_DIAHD_PIN, O2-2_DIAHG_PIN, O2-2_IA_PIN, O2-2_IP_PIN, O2-2_UN_PIN, O2-2_VM_PIN, UN-1?, UN-2?
- net labels removed: CJ125_SCK, CJ125_SI, CJ125_SO, CJ125_SS, CJ125_UA, CJ125_UR, DIAHD?, DIAHG?, IA?, IP?, O2_DIAHD_PIN, O2_DIAHG_PIN, O2_IA_PIN, O2_IP_PIN, O2_UN_PIN, O2_VM_PIN, UN?
- wire segments 65 -> 145
Other:
- moved on the sheet: C?, R?

Commit message: About to runs scripts to scrub the BOM's, so here's a backup copy in case it goes wrong.
Signed-off-by: Jared Harvey <TortiseGIT@jaredharvey.com>
Parts:
- removed C?: 10nF, SM0805-C1, symbol C
- removed C? (x2): 33nF, SM0805-C1, symbol C
- removed P?: CONN_1, PINTST, symbol CONN_1
- removed R? (x2): 1k, SM0805-R4, symbol R
- removed R?: 100k, SM0805-R4, symbol R
- removed R?: 10k, SM0805-R4, symbol R
- added C1104, C1110: 33nF, SM0805-C1, symbol C
- added C1116: 10nF, SM0805-C1, symbol C
- added P1112: CONN_1, PINTST, symbol CONN_1
- added R1109: 10k, SM0805, symbol R
- added R1112, R1124: 1k, SM0805, symbol R
- added R1121: 100k, SM0805, symbol R
- R1101, R1102, R1103, R1104, R1105, R1106, R1107, R1108, R1110, R1111, R1113, R1114, R1115, R1116, R1117, R1118, R1119, R1120, R1122, R1123: renamed from R?; footprint SM0805-R4 -> SM0805
- gave numbers to parts that had none: 26
Connections:
- wire segments 145 -> 129
Other:
- moved on the sheet: C1101, C1102, C1103, C1105, C1106, C1107, C1108, C1109, C1111, C1112, C1113, C1114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

Commit message: caps have been done with the scripts next up is the resistors.
Signed-off-by: Jared Harvey <TortiseGIT@jaredharvey.com>
Parts:
- C1103, C1104, C1109, C1110, C1113, C1114: Field3 -,- -> (none); Field4 -,- -> (none); Field5 25,V -> (none); Field6 10,% -> (none); Field7 Ceramic -> (none); Field8 other,more,stuff -> (none); V (none) -> 25V; construct (none) -> ceramic; mfg,# yageo,CC0805KRX7R8BB333 -> (none); mfg,mfg# (none) -> yageo,CC0805KRX7R8BB333; misc (none) -> other,more,stuff; tolerance (none) -> 10%; vend,# newark,69C9599 -> (none); vend1,vend1# (none) -> newark,69C9599
- C1105, C1106, C1111, C1112: Field3 -,- -> (none); Field4 -,- -> (none); Field5 50,V -> (none); Field6 10,% -> (none); Field7 Ceramic -> (none); Field8 other,more,stuff -> (none); V (none) -> 100V; construct (none) -> ceramic; mfg,# murata,GRM21BR71H104KA01L -> (none); mfg,mfg# (none) -> avx,08051C104KAT2A; misc (none) -> other,more,stuff; tolerance (none) -> 10%; vend,# newark,38K1694 -> (none); vend1,vend1# (none) -> newark,96M1354
- C1115, C1116: Field3 -,- -> (none); Field4 -,- -> (none); Field5 50,V -> (none); Field6 5,% -> (none); Field7 Ceramic -> (none); Field8 other,more,stuff -> (none); V (none) -> 200V; construct (none) -> alum elec; mfg,# murata,GRM216R71H103JA01D -> (none); mfg,mfg# (none) -> ill cap,106CKE200M; misc (none) -> other,more,stuff; tolerance (none) -> 10%; vend,# newark,38K1697 -> (none); vend1,vend1# (none) -> newark,69K7896

Commit message: Looks like the bulk components are golden now, there are still a couple straglers, mostly switch mode power supply stuff.
Signed-off-by: Jared Harvey <TortiseGIT@jaredharvey.com>
Parts:
- R1101, R1102, R1106, R1109: Field3 -,- -> (none); Field4 -,- -> (none); Field5 125,mW -> (none); Field6 1,% -> (none); Field7 thick film -> (none); Field8 other,more,stuff -> (none); construct (none) -> thick film; mfg,# bourns,CR0805-FX-1002ELF -> (none); mfg,mfg# (none) -> BOURNS,CR0805-FX-1002ELF; misc (none) -> other,more,stuff; tolerance (none) -> 1%; vend,# newark,02J2368 -> (none); vend1,vend1# (none) -> newark,02J2368; w (none) -> 125mW
- R1111, R1112, R1123, R1124: Field3 -,- -> (none); Field4 -,- -> (none); Field5 125,mW -> (none); Field6 1,% -> (none); Field7 thick film -> (none); Field8 other,more,stuff -> (none); construct (none) -> thick film; mfg,# vishay,CRCW08051K00FKTA -> (none); mfg,mfg# (none) -> vishay,CRCW08051K00FKTA; misc (none) -> other,more,stuff; tolerance (none) -> 1%; vend,# newark,05F1507 -> (none); vend1,vend1# (none) -> newark,05F1507; w (none) -> 125mW
- R1117, R1118, R1119, R1121: Field3 -,- -> (none); Field4 -,- -> (none); Field5 125,mW -> (none); Field6 1,% -> (none); Field7 thick film -> (none); Field8 other,more,stuff -> (none); construct (none) -> thick film; mfg,# bourns,CR0805-FX-1003ELF -> (none); mfg,mfg# (none) -> vishay,CRCW0805100KFKEA; misc (none) -> other,more,stuff; tolerance (none) -> 1%; vend,# newark,32K2766 -> (none); vend1,vend1# (none) -> newark,52K9808; w (none) -> 125mW

Commit message: several pins on the SOM are now connected.
Signed-off-by: Jared Harvey <TortiseGIT@jaredharvey.com>
Parts:
- renumbered C1101 to C1201, C1102 to C1202, C1103 to C1203, C1104 to C1204, C1105 to C1205, C1106 to C1206, C1107 to C1207, C1108 to C1208, C1109 to C1209, C1110 to C1210, C1111 to C1211, C1112 to C1212, C1113 to C1213, C1114 to C1214, C1115 to C1215, C1116 to C1216, P1101 to P1201, P1102 to P1202, P1103 to P1203, P1104 to P1204, P1105 to P1205, P1106 to P1206, P1107 to P1207, P1108 to P1208, P1109 to P1209, P1110 to P1210, P1111 to P1211, P1112 to P1212, R1101 to R1201, R1102 to R1202, R1103 to R1203, R1104 to R1204, R1105 to R1205, R1106 to R1206, R1107 to R1207, R1108 to R1208, R1109 to R1209, R1110 to R1210, R1111 to R1211, R1112 to R1212, R1113 to R1213, R1114 to R1214, R1115 to R1215, R1116 to R1216, R1117 to R1217, R1118 to R1218, R1119 to R1219, R1120 to R1220, R1121 to R1221, R1122 to R1222, R1123 to R1223, R1124 to R1224, U1101 to U1201, U1102 to U1202
