File: KICAD_Project/sub_circuits/O2_input_CJ125.sch (KiCad schematic (older format))
At the start: 54 parts, among them P1201 CONN_1, P1202 CONN_1, P1203 CONN_1, P1204 CONN_1, P1205 CONN_1, P1206 CONN_1, P1207 CONN_1, P1208 CONN_1, P1209 CONN_1, P1210 CONN_1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

Commit message: routing has started
Signed-off-by: Jared Harvey <TortiseGIT@jaredharvey.com>
Changed lines of the file:
@@
-EESchema Schematic File Version 2  date 8/20/2011 7:18:56 AM
+EESchema Schematic File Version 2  date 8/20/2011 7:59:51 PM
 LIBS:power
 LIBS:device
@@
 $Descr User 11000 8500
 encoding utf-8
-Sheet 11 13
+Sheet 12 13
 Title "freeEMS PLUS from Cinch template "
 Date "20 aug 2011"
@@
 	5500 5500 5500 5575
 Wire Wire Line
-	5500 5500 5175 5500
+	5500 5500 5125 5500
 Wire Wire Line
 	5775 5150 5775 5200
 Wire Wire Line
-	5775 5150 5450 5150
+	5775 5150 5300 5150
 Connection ~ 9775 5375
 Wire Wire Line
@@
 	5775 5100 5775 5050
 Wire Wire Line
-	5775 5050 5450 5050
+	5775 5050 5300 5050
 Wire Wire Line
 	6550 5375 5450 5375
 Connection ~ 5775 5375
 Wire Wire Line
-	5175 5625 5500 5625
+	5125 5625 5500 5625
 Wire Wire Line
 	5500 5625 5500 5675
@@
 	5500 3025 5500 3075
 Wire Wire Line
-	5500 3025 5175 3025
+	5500 3025 5100 3025
 Connection ~ 5775 2775
 Wire Wire Line
 	5450 2775 6550 2775
 Wire Wire Line
-	5450 2450 5775 2450
+	5350 2450 5775 2450
 Wire Wire Line
 	5775 2450 5775 2500
@@
 Connection ~ 9750 2775
 Wire Wire Line
-	5450 2550 5775 2550
+	5350 2550 5775 2550
 Wire Wire Line
 	5775 2550 5775 2600
 Wire Wire Line
-	5175 2900 5500 2900
+	5100 2900 5500 2900
 Wire Wire Line
 	5500 2900 5500 2975
@@
 P 8375 2675
 F 0 "C1211" V 8400 2850 50  0000 L CNN
-F 1 "100nF" V 8400 2525 50  0000 L CNN
+F 1 "100nF" V 8400 2500 50  0000 L CNN
 F 2 "SM0805-C1" V 1130 2600 60  0001 C CNN
 F 4 "avx,08051C104KAT2A" V 1130 2600 60  0001 C CNN "mfg,mfg#"
@@
 U 1 1 4E39E9D1
 P 8550 2875
-F 0 "R1219" V 8500 3150 50  0000 C CNN
+F 0 "R1219" V 8500 2575 50  0000 C CNN
 F 1 "100k" V 8550 2875 50  0000 C CNN
 F 2 "SM0805" V 1130 2600 60  0001 C CNN
@@
 U 1 1 4E39E9CC
 P 6250 2675
-F 0 "R1205" V 6200 2925 50  0000 C CNN
+F 0 "R1205" V 6200 2975 50  0000 C CNN
 F 1 "61.9" V 6250 2675 50  0000 C CNN
 F 2 "SM0805" V 6430 2775 60  0001 C CNN
@@
 U 1 1 4E39E9CB
 P 6250 2875
-F 0 "R1206" V 6300 2625 50  0000 C CNN
+F 0 "R1206" V 6300 2575 50  0000 C CNN
 F 1 "10k" V 6250 2875 50  0000 C CNN
 F 2 "SM0805" V 1130 2600 60  0001 C CNN
@@
 U 1 1 4E39E9C6
 P 6250 3075
-F 0 "R1207" V 6300 3325 50  0000 C CNN
+F 0 "R1207" V 6300 3375 50  0000 C CNN
 F 1 "6.8k" V 6250 3075 50  0000 C CNN
 F 2 "SM0805" V 6430 3175 60  0001 C CNN
@@
 U 1 1 4E39E9C5
 P 6400 2375
-F 0 "C1207" H 6200 2475 50  0000 L CNN
+F 0 "C1207" H 6150 2475 50  0000 L CNN
 F 1 "2.2nF" H 6150 2275 50  0000 L CNN
 F 2 "SM0805-C1" V 3480 3475 60  0001 C CNN
@@
 U 1 1 4E39E9C3
 P 4500 3175
-F 0 "R1201" V 4550 3425 50  0000 C CNN
+F 0 "R1201" V 4600 3175 50  0000 C CNN
 F 1 "10k" V 4500 3175 50  0000 C CNN
 F 2 "SM0805" V 1130 2600 60  0001 C CNN
@@
 P 6100 3525
 F 0 "C1205" V 6000 3350 50  0000 L CNN
-F 1 "100nF" V 6000 3675 50  0000 L CNN
+F 1 "100nF" V 6000 3700 50  0000 L CNN
 F 2 "SM0805-C1" V 1130 2600 60  0001 C CNN
 F 4 "avx,08051C104KAT2A" V 1130 2600 60  0001 C CNN "mfg,mfg#"
@@
 U 1 1 4E39E9C1
 P 6150 3375
-F 0 "R1203" V 6200 3625 50  0000 C CNN
+F 0 "R1203" V 6200 3675 50  0000 C CNN
 F 1 "27k" V 6150 3375 50  0000 C CNN
 F 2 "SM0805" V 6330 3475 60  0001 C CNN
@@
 U 1 1 4E39E9BB
 P 7950 2975
-F 0 "R1215" V 8000 3200 50  0000 C CNN
+F 0 "R1215" V 8000 3250 50  0000 C CNN
 F 1 "4.7k" V 7950 2975 50  0000 C CNN
 F 2 "SM0805" V 8130 3075 60  0001 C CNN
@@
 U 1 1 4E39E9B9
 P 8825 3375
-F 0 "C1213" H 8900 3475 50  0000 L CNN
+F 0 "C1213" H 8550 3275 50  0000 L CNN
 F 1 "33nF" H 8625 3475 50  0000 L CNN
 F 2 "SM0805-C1" V 1130 2600 60  0001 C CNN
@@
 U 1 1 4E39E9B6
 P 5625 2675
-F 0 "P1207" H 5705 2675 40  0000 L CNN
+F 0 "P1207" H 5675 2675 40  0000 L CNN
 F 1 "CONN_1" H 5625 2730 30  0001 C CNN
 F 2 "PINTST" H 5625 2675 60  0001 C CNN
@@
 U 1 1 4E39E9B5
 P 5625 2600
-F 0 "P1206" H 5705 2600 40  0000 L CNN
+F 0 "P1206" H 5675 2600 40  0000 L CNN
 F 1 "CONN_1" H 5625 2655 30  0001 C CNN
 F 2 "PINTST" H 5625 2600 60  0001 C CNN
@@
 U 1 1 4E39E9B3
 P 5625 2500
-F 0 "P1205" H 5705 2500 40  0000 L CNN
+F 0 "P1205" H 5675 2500 40  0000 L CNN
 F 1 "CONN_1" H 5625 2555 30  0001 C CNN
 F 2 "PINTST" H 5625 2500 60  0001 C CNN
@@
 U 1 1 4E39E9B2
 P 5350 2975
-F 0 "P1201" H 5430 2975 40  0000 L CNN
+F 0 "P1201" H 5400 2975 40  0000 L CNN
 F 1 "CONN_1" H 5350 3030 30  0001 C CNN
 F 2 "PINTST" H 5350 2975 60  0001 C CNN
@@
 U 1 1 4E39E9B1
 P 5350 3075
-F 0 "P1202" H 5430 3075 40  0000 L CNN
+F 0 "P1202" H 5400 3075 40  0000 L CNN
 F 1 "CONN_1" H 5350 3130 30  0001 C CNN
 F 2 "PINTST" H 5350 3075 60  0001 C CNN
@@
 Text HLabel 5450 2775 0    60   Input ~ 0
 O2-1_IA_PIN
-Text HLabel 5450 2550 0    60   Input ~ 0
+Text HLabel 5350 2550 0    60   Input ~ 0
 O2-1_IP_PIN
-Text HLabel 5450 2450 0    60   Input ~ 0
+Text HLabel 5350 2450 0    60   Input ~ 0
 O2-1_UN_PIN
-Text HLabel 5175 2900 0    60   Input ~ 0
+Text HLabel 5100 2900 0    60   Input ~ 0
 O2-1_DIAHG_PIN
-Text HLabel 5175 3025 0    60   Input ~ 0
+Text HLabel 5100 3025 0    60   Input ~ 0
 O2-1_DIAHD_PIN
 Text HLabel 9025 4275 2    60   Input ~ 0
@@
 Text HLabel 9025 6875 2    60   Input ~ 0
 O2-2_VM_PIN
-Text HLabel 5175 5625 0    60   Input ~ 0
+Text HLabel 5125 5625 0    60   Input ~ 0
 O2-2_DIAHD_PIN
-Text HLabel 5175 5500 0    60   Input ~ 0
+Text HLabel 5125 5500 0    60   Input ~ 0
 O2-2_DIAHG_PIN
-Text HLabel 5450 5050 0    60   Input ~ 0
+Text HLabel 5300 5050 0    60   Input ~ 0
 O2-2_UN_PIN
-Text HLabel 5450 5150 0    60   Input ~ 0
+Text HLabel 5300 5150 0    60   Input ~ 0
 O2-2_IP_PIN
 Text HLabel 5450 5375 0    60   Input ~ 0
@@
 U 1 1 4C0A2A7C
 P 5350 5675
-F 0 "P1204" H 5430 5675 40  0000 L CNN
+F 0 "P1204" H 5400 5675 40  0000 L CNN
 F 1 "CONN_1" H 5350 5730 30  0001 C CNN
 F 2 "PINTST" H 5350 5675 60  0001 C CNN
@@
 U 1 1 4C0A2A79
 P 5350 5575
-F 0 "P1203" H 5430 5575 40  0000 L CNN
+F 0 "P1203" H 5400 5575 40  0000 L CNN
 F 1 "CONN_1" H 5350 5630 30  0001 C CNN
 F 2 "PINTST" H 5350 5575 60  0001 C CNN
@@
 U 1 1 4C0A2881
 P 5625 5100
-F 0 "P1208" H 5705 5100 40  0000 L CNN
+F 0 "P1208" H 5675 5100 40  0000 L CNN
 F 1 "CONN_1" H 5625 5155 30  0001 C CNN
 F 2 "PINTST" H 5625 5100 60  0001 C CNN
@@
 U 1 1 4C0A2733
 P 5625 5200
-F 0 "P1209" H 5705 5200 40  0000 L CNN
+F 0 "P1209" H 5675 5200 40  0000 L CNN
 F 1 "CONN_1" H 5625 5255 30  0001 C CNN
 F 2 "PINTST" H 5625 5200 60  0001 C CNN
@@
 U 1 1 4C0A271E
 P 5625 5275
-F 0 "P1210" H 5705 5275 40  0000 L CNN
+F 0 "P1210" H 5675 5275 40  0000 L CNN
 F 1 "CONN_1" H 5625 5330 30  0001 C CNN
 F 2 "PINTST" H 5625 5275 60  0001 C CNN
@@
 U 1 1 4C09CCDE
 P 8825 5975
-F 0 "C1214" H 8900 6075 50  0000 L CNN
+F 0 "C1214" H 8575 5875 50  0000 L CNN
 F 1 "33nF" H 8625 6075 50  0000 L CNN
 F 2 "SM0805-C1" V 1130 2600 60  0001 C CNN
@@
 U 1 1 4C09C82A
 P 6150 5975
-F 0 "R1204" V 6200 6225 50  0000 C CNN
+F 0 "R1204" V 6200 6275 50  0000 C CNN
 F 1 "27k" V 6150 5975 50  0000 C CNN
 F 2 "SM0805" V 6330 6075 60  0001 C CNN
@@
 P 6100 6125
 F 0 "C1206" V 6000 5950 50  0000 L CNN
-F 1 "100nF" V 6000 6275 50  0000 L CNN
+F 1 "100nF" V 6000 6300 50  0000 L CNN
 F 2 "SM0805-C1" V 1130 2600 60  0001 C CNN
 F 4 "avx,08051C104KAT2A" V 1130 2600 60  0001 C CNN "mfg,mfg#"
@@
 U 1 1 4C09C812
 P 4500 5775
-F 0 "R1202" V 4550 6025 50  0000 C CNN
+F 0 "R1202" V 4600 5775 50  0000 C CNN
 F 1 "10k" V 4500 5775 50  0000 C CNN
 F 2 "SM0805" V 1130 2600 60  0001 C CNN
@@
 U 1 1 4C09C77F
 P 6400 4975
-F 0 "C1208" H 6200 5075 50  0000 L CNN
+F 0 "C1208" H 6150 5050 50  0000 L CNN
 F 1 "2.2nF" H 6150 4875 50  0000 L CNN
 F 2 "SM0805-C1" V 3480 6075 60  0001 C CNN
@@
 U 1 1 4C09C74A
 P 6250 5675
-F 0 "R1210" V 6300 5925 50  0000 C CNN
+F 0 "R1210" V 6300 5975 50  0000 C CNN
 F 1 "6.8k" V 6250 5675 50  0000 C CNN
 F 2 "SM0805" V 6430 5775 60  0001 C CNN
@@
 U 1 1 4C09C749
 P 4950 5975
-F 0 "C1202" H 5025 5875 50  0000 L CNN
+F 0 "C1202" H 4950 6100 50  0000 L CNN
 F 1 "1nF" H 4750 5875 50  0000 L CNN
 F 2 "SM0805-C1" V 2030 7075 60  0001 C CNN
@@
 U 1 1 4E467E05
 P 6250 5475
-F 0 "R1209" V 6300 5225 50  0000 C CNN
+F 0 "R1209" V 6300 5175 50  0000 C CNN
 F 1 "10k" V 6250 5475 50  0000 C CNN
 F 2 "SM0805" V 1130 2600 60  0001 C CNN
@@
 U 1 1 4BF6512C
 P 6250 5275
-F 0 "R1208" V 6200 5525 50  0000 C CNN
+F 0 "R1208" V 6200 5575 50  0000 C CNN
 F 1 "61.9" V 6250 5275 50  0000 C CNN
 F 2 "SM0805" V 6430 5375 60  0001 C CNN
@@
 U 1 1 4E467DFB
 P 8550 5475
-F 0 "R1221" V 8500 5750 50  0000 C CNN
+F 0 "R1221" V 8500 5200 50  0000 C CNN
 F 1 "100k" V 8550 5475 50  0000 C CNN
 F 2 "SM0805" V 1130 2600 60  0001 C CNN

Commit message: more stepper updates
Signed-off-by: Jared Harvey <TortiseGIT@jaredharvey.com>
Parts:
- R1217, R1218, R1219, R1221: W (none) -> 125mW; w 125mW -> (none)
Changed lines of the file:
@@
-EESchema Schematic File Version 2  date 8/27/2011 10:55:19 AM
+EESchema Schematic File Version 2  date 8/30/2011 5:58:29 AM
 LIBS:power
 LIBS:device
@@
 Sheet 12 13
 Title "freeEMS PLUS from Cinch template "
-Date "27 aug 2011"
+Date "30 aug 2011"
 Rev "A-DRAF"
 Comp "diyefi.org/openecu.info"
@@
 F 4 "vishay,CRCW0805100KFKEA" V 1130 2600 60  0001 C CNN "mfg,mfg#"
 F 5 "newark,52K9808" V 1130 2600 60  0001 C CNN "vend1,vend1#"
-F 6 "" V 1130 2600 60  0001 C CNN "Field6"
-F 7 "" V 1130 2600 60  0001 C CNN "Field7"
-F 8 "125mW" V 1130 2600 60  0001 C CNN "w"
+F 6 "" V 1130 2600 60  0001 C CNN ""
+F 7 "" V 1130 2600 60  0001 C CNN ""
+F 8 "125mW" V 1130 2600 60  0001 C CNN "W"
 F 9 "1%" V 1130 2600 60  0001 C CNN "tolerance"
 F 10 "thick film" V 1130 2600 60  0001 C CNN "construct"
@@
 F 4 "vishay,CRCW0805100KFKEA" V 1130 2600 60  0001 C CNN "mfg,mfg#"
 F 5 "newark,52K9808" V 1130 2600 60  0001 C CNN "vend1,vend1#"
-F 6 "" V 1130 2600 60  0001 C CNN "Field6"
-F 7 "" V 1130 2600 60  0001 C CNN "Field7"
-F 8 "125mW" V 1130 2600 60  0001 C CNN "w"
+F 6 "" V 1130 2600 60  0001 C CNN ""
+F 7 "" V 1130 2600 60  0001 C CNN ""
+F 8 "125mW" V 1130 2600 60  0001 C CNN "W"
 F 9 "1%" V 1130 2600 60  0001 C CNN "tolerance"
 F 10 "thick film" V 1130 2600 60  0001 C CNN "construct"
@@
 F 4 "vishay,CRCW0805100KFKEA" V 1130 2600 60  0001 C CNN "mfg,mfg#"
 F 5 "newark,52K9808" V 1130 2600 60  0001 C CNN "vend1,vend1#"
-F 6 "" V 1130 2600 60  0001 C CNN "Field6"
-F 7 "" V 1130 2600 60  0001 C CNN "Field7"
-F 8 "125mW" V 1130 2600 60  0001 C CNN "w"
+F 6 "" V 1130 2600 60  0001 C CNN ""
+F 7 "" V 1130 2600 60  0001 C CNN ""
+F 8 "125mW" V 1130 2600 60  0001 C CNN "W"
 F 9 "1%" V 1130 2600 60  0001 C CNN "tolerance"
 F 10 "thick film" V 1130 2600 60  0001 C CNN "construct"
@@
 F 4 "vishay,CRCW0805100KFKEA" V 1130 2600 60  0001 C CNN "mfg,mfg#"
 F 5 "newark,52K9808" V 1130 2600 60  0001 C CNN "vend1,vend1#"
-F 6 "" V 1130 2600 60  0001 C CNN "Field6"
-F 7 "" V 1130 2600 60  0001 C CNN "Field7"
-F 8 "125mW" V 1130 2600 60  0001 C CNN "w"
+F 6 "" V 1130 2600 60  0001 C CNN ""
+F 7 "" V 1130 2600 60  0001 C CNN ""
+F 8 "125mW" V 1130 2600 60  0001 C CNN "W"
 F 9 "1%" V 1130 2600 60  0001 C CNN "tolerance"
 F 10 "thick film" V 1130 2600 60  0001 C CNN "construct"
