File: KICAD_Project/sub_circuits/O2_input_CJ125.sch (KiCad schematic (older format))
At the start: 42 parts, among them U1201 CJ125, U1202 CJ125

Commit message: Made more progress on the AN protects and LS drive 33800
Signed-off-by: Jared Harvey <TortiseGIT@jaredharvey.com>
Parts:
- C1205, C1206, C1211, C1212: TOL (none) -> 10%; V 100V -> 200V; construct ceramic -> CERAMIC; mfg,mfg# avx,08051C104KAT2A -> AVX,08055C104KAT2A; tolerance 10% -> (none); vend1,vend1# newark,96M1354 -> newark,27C8438
- C1215, C1216: TOL (none) -> 10%; V 200V -> 50V; construct alum elec -> CERAMIC; mfg,mfg# ill cap,106CKE200M -> AVX,08055C103KAT2A; tolerance 10% -> (none); vend1,vend1# newark,69K7896 -> newark,07J3575
Changed lines of the file:
@@
-EESchema Schematic File Version 2  date 10/14/2011 5:26:22 AM
+EESchema Schematic File Version 2  date 10/16/2011 7:32:23 AM
 LIBS:power
 LIBS:device
@@
 Sheet 11 12
 Title "Open5xxxECU (o5e), an ECU that is no longer affiliated with freeEMS."
-Date "14 oct 2011"
+Date "16 oct 2011"
 Rev "A-DRAFT5"
 Comp "http://open5xxxecu.org/"
@@
 F 1 "100nF" V 8400 2500 50  0000 L CNN
 F 2 "SM0805" V 1130 2600 60  0001 C CNN
-F 4 "avx,08051C104KAT2A" V 1130 2600 60  0001 C CNN "mfg,mfg#"
-F 5 "newark,96M1354" V 1130 2600 60  0001 C CNN "vend1,vend1#"
-F 6 "100V" V 1130 2600 60  0001 C CNN "V"
-F 7 "10%" V 1130 2600 60  0001 C CNN "tolerance"
-F 8 "ceramic" V 1130 2600 60  0001 C CNN "construct"
-F 9 "other,more,stuff" V 1130 2600 60  0001 C CNN "misc"
+F 4 "AVX,08055C104KAT2A" V 1130 2600 60  0001 C CNN "mfg,mfg#"
+F 5 "newark,27C8438" V 1130 2600 60  0001 C CNN "vend1,vend1#"
+F 6 "" V 1130 2600 60  0001 C CNN "Field6"
+F 7 "" V 1130 2600 60  0001 C CNN "Field7"
+F 8 "200V" V 1130 2600 60  0001 C CNN "V"
+F 9 "10%" V 1130 2600 60  0001 C CNN "TOL"
+F 10 "CERAMIC" V 1130 2600 60  0001 C CNN "construct"
+F 11 "other,more,stuff" V 1130 2600 60  0001 C CNN "misc"
 	1    8375 2675
 	0    1    1    0
@@
 F 1 "10nF" H 9550 3150 50  0000 L CNN
 F 2 "SM0805" V 1130 2600 60  0001 C CNN
-F 4 "ill cap,106CKE200M" V 1130 2600 60  0001 C CNN "mfg,mfg#"
-F 5 "newark,69K7896" V 1130 2600 60  0001 C CNN "vend1,vend1#"
-F 6 "200V" V 1130 2600 60  0001 C CNN "V"
-F 7 "10%" V 1130 2600 60  0001 C CNN "tolerance"
-F 8 "alum elec" V 1130 2600 60  0001 C CNN "construct"
-F 9 "other,more,stuff" V 1130 2600 60  0001 C CNN "misc"
+F 4 "AVX,08055C103KAT2A" V 1130 2600 60  0001 C CNN "mfg,mfg#"
+F 5 "newark,07J3575" V 1130 2600 60  0001 C CNN "vend1,vend1#"
+F 6 "" V 1130 2600 60  0001 C CNN "Field6"
+F 7 "" V 1130 2600 60  0001 C CNN "Field7"
+F 8 "50V" V 1130 2600 60  0001 C CNN "V"
+F 9 "10%" V 1130 2600 60  0001 C CNN "TOL"
+F 10 "CERAMIC" V 1130 2600 60  0001 C CNN "construct"
+F 11 "other,more,stuff" V 1130 2600 60  0001 C CNN "misc"
 	1    9750 3050
 	1    0    0    1
@@
 F 1 "100nF" V 6000 3700 50  0000 L CNN
 F 2 "SM0805" V 1130 2600 60  0001 C CNN
-F 4 "avx,08051C104KAT2A" V 1130 2600 60  0001 C CNN "mfg,mfg#"
-F 5 "newark,96M1354" V 1130 2600 60  0001 C CNN "vend1,vend1#"
-F 6 "100V" V 1130 2600 60  0001 C CNN "V"
-F 7 "10%" V 1130 2600 60  0001 C CNN "tolerance"
-F 8 "ceramic" V 1130 2600 60  0001 C CNN "construct"
-F 9 "other,more,stuff" V 1130 2600 60  0001 C CNN "misc"
+F 4 "AVX,08055C104KAT2A" V 1130 2600 60  0001 C CNN "mfg,mfg#"
+F 5 "newark,27C8438" V 1130 2600 60  0001 C CNN "vend1,vend1#"
+F 6 "" V 1130 2600 60  0001 C CNN "Field6"
+F 7 "" V 1130 2600 60  0001 C CNN "Field7"
+F 8 "200V" V 1130 2600 60  0001 C CNN "V"
+F 9 "10%" V 1130 2600 60  0001 C CNN "TOL"
+F 10 "CERAMIC" V 1130 2600 60  0001 C CNN "construct"
+F 11 "other,more,stuff" V 1130 2600 60  0001 C CNN "misc"
 	1    6100 3525
 	0    -1   -1   0
@@
 F 1 "100nF" V 6000 6300 50  0000 L CNN
 F 2 "SM0805" V 1130 2600 60  0001 C CNN
-F 4 "avx,08051C104KAT2A" V 1130 2600 60  0001 C CNN "mfg,mfg#"
-F 5 "newark,96M1354" V 1130 2600 60  0001 C CNN "vend1,vend1#"
-F 6 "100V" V 1130 2600 60  0001 C CNN "V"
-F 7 "10%" V 1130 2600 60  0001 C CNN "tolerance"
-F 8 "ceramic" V 1130 2600 60  0001 C CNN "construct"
-F 9 "other,more,stuff" V 1130 2600 60  0001 C CNN "misc"
+F 4 "AVX,08055C104KAT2A" V 1130 2600 60  0001 C CNN "mfg,mfg#"
+F 5 "newark,27C8438" V 1130 2600 60  0001 C CNN "vend1,vend1#"
+F 6 "" V 1130 2600 60  0001 C CNN "Field6"
+F 7 "" V 1130 2600 60  0001 C CNN "Field7"
+F 8 "200V" V 1130 2600 60  0001 C CNN "V"
+F 9 "10%" V 1130 2600 60  0001 C CNN "TOL"
+F 10 "CERAMIC" V 1130 2600 60  0001 C CNN "construct"
+F 11 "other,more,stuff" V 1130 2600 60  0001 C CNN "misc"
 	1    6100 6125
 	0    -1   -1   0
@@
 F 1 "10nF" H 9575 5750 50  0000 L CNN
 F 2 "SM0805" V 1130 2600 60  0001 C CNN
-F 4 "ill cap,106CKE200M" V 1130 2600 60  0001 C CNN "mfg,mfg#"
-F 5 "newark,69K7896" V 1130 2600 60  0001 C CNN "vend1,vend1#"
-F 6 "200V" V 1130 2600 60  0001 C CNN "V"
-F 7 "10%" V 1130 2600 60  0001 C CNN "tolerance"
-F 8 "alum elec" V 1130 2600 60  0001 C CNN "construct"
-F 9 "other,more,stuff" V 1130 2600 60  0001 C CNN "misc"
+F 4 "AVX,08055C103KAT2A" V 1130 2600 60  0001 C CNN "mfg,mfg#"
+F 5 "newark,07J3575" V 1130 2600 60  0001 C CNN "vend1,vend1#"
+F 6 "" V 1130 2600 60  0001 C CNN "Field6"
+F 7 "" V 1130 2600 60  0001 C CNN "Field7"
+F 8 "50V" V 1130 2600 60  0001 C CNN "V"
+F 9 "10%" V 1130 2600 60  0001 C CNN "TOL"
+F 10 "CERAMIC" V 1130 2600 60  0001 C CNN "construct"
+F 11 "other,more,stuff" V 1130 2600 60  0001 C CNN "misc"
 	1    9775 5650
 	1    0    0    1
@@
 F 1 "100nF" V 8400 5125 50  0000 L CNN
 F 2 "SM0805" V 1130 2600 60  0001 C CNN
-F 4 "avx,08051C104KAT2A" V 1130 2600 60  0001 C CNN "mfg,mfg#"
-F 5 "newark,96M1354" V 1130 2600 60  0001 C CNN "vend1,vend1#"
-F 6 "100V" V 1130 2600 60  0001 C CNN "V"
-F 7 "10%" V 1130 2600 60  0001 C CNN "tolerance"
-F 8 "ceramic" V 1130 2600 60  0001 C CNN "construct"
-F 9 "other,more,stuff" V 1130 2600 60  0001 C CNN "misc"
+F 4 "AVX,08055C104KAT2A" V 1130 2600 60  0001 C CNN "mfg,mfg#"
+F 5 "newark,27C8438" V 1130 2600 60  0001 C CNN "vend1,vend1#"
+F 6 "" V 1130 2600 60  0001 C CNN "Field6"
+F 7 "" V 1130 2600 60  0001 C CNN "Field7"
+F 8 "200V" V 1130 2600 60  0001 C CNN "V"
+F 9 "10%" V 1130 2600 60  0001 C CNN "TOL"
+F 10 "CERAMIC" V 1130 2600 60  0001 C CNN "construct"
+F 11 "other,more,stuff" V 1130 2600 60  0001 C CNN "misc"
 	1    8375 5275
 	0    1    1    0
