File: KICAD_Project/sub_circuits/RPM_input_MAX9926.sch (KiCad schematic (older format))
At the start: 15 parts

Commit message: I did a fiar bit of work, and I want to be able to step back if I can, so this is a misc check in.
Signed-off-by: Jared Harvey <TortiseGIT@jaredharvey.com>
Parts:
- removed R? (x4): 10k, SM0805-R4, symbol R
- added C? (x3): .1uF, SM0805-C1, symbol C
- added C? (x6): 1nF, SM0805-C1, symbol C
- added C? (x3): 10uF, SM0805-C1, symbol C
- added P? (x12): CONN_1, PINTST, symbol CONN_1
- added R? (x48): 5k, SM0805, symbol R
- added R? (x6): 10k, SM0805-R4, symbol R
- added U? (x3): MAX9926/9927, MAXIM-10-QSOP16, symbol MAX9926/9927
Connections:
- net labels added: CAM1+, CAM1-, CAM2+, CAM2-, CRK1+, CRK2+, CRK2-, LB_SIG+, LB_SIG-, LF_SIG+, LF_SIG-, RB_SIG+, RB_SIG-, RF_SIG+, RF_SIG-, RPM-CK1, RPM-CK2, RPM-CM1, RPM-CM2, RPM-LB, RPM-LF, RPM-RB, RPM-RF
- net labels removed: EXT1, EXT2, RPM1, RPM2, VR_1+, VR_1-, VR_2+, VR_2-
- wire segments 46 -> 240
- no-connect marks 0 -> 8
Other:
- note added: "CAM 1&2, HALL OR VR"
- note added: "CRANK 1&2, HALL OR VR"
- note added: "WHEEL, HALL OR VR"
- moved on the sheet: C?, R?

Commit message: About to runs scripts to scrub the BOM's, so here's a backup copy in case it goes wrong.
Signed-off-by: Jared Harvey <TortiseGIT@jaredharvey.com>
Parts:
- R401, R402, R403, R404, R429, R430, R431, R432: renamed from R?; footprint SM0805-R4 -> SM0805
- gave numbers to parts that had none: 84
Connections:
- wire segments 240 -> 157

Commit message: caps have been done with the scripts next up is the resistors.
Signed-off-by: Jared Harvey <TortiseGIT@jaredharvey.com>
Parts:
- C401, C402, C409, C410: value .1uF -> 0.1uF; Field3 -,- -> (none); Field4 -,- -> (none); Field5 100,V -> (none); Field6 10,% -> (none); Field7 ceramic -> (none); Field8 other,more,stuff -> (none); V (none) -> 100V; construct (none) -> ceramic; mfg,# avx,08051C104KAT2A -> (none); mfg,mfg# (none) -> avx,08051C104KAT2A; misc (none) -> other,more,stuff; tolerance (none) -> 10%; vend,# newark,96M1354 -> (none); vend1,vend1# (none) -> newark,96M1354
Changed lines of the file:
@@
-EESchema Schematic File Version 2  date 8/14/2011 3:32:14 PM
+EESchema Schematic File Version 2  date 8/14/2011 7:31:24 PM
 LIBS:power
 LIBS:device
@@
 U 1 1 4E39DFBE
 P 7625 800
-F 0 "C411" H 7675 900 50  0000 L CNN
+F 0 "C411" H 7650 700 50  0000 L CNN
 F 1 "10uF" H 7400 900 50  0000 L CNN
 F 2 "SM0805-C1" V 4155 800 60  0001 C CNN
@@
 U 1 1 4E39DFB7
 P 7175 800
-F 0 "C409" H 7225 900 50  0000 L CNN
-F 1 ".1uF" H 7025 900 50  0000 L CNN
-F 2 "SM0805-C1" V 3705 800 60  0001 C CNN
-F 4 "avx,08051C104KAT2A" V 3705 800 60  0001 C CNN "mfg,#"
-F 5 "newark,96M1354" V 3705 800 60  0001 C CNN "vend,#"
-F 6 "-,-" V 3705 800 60  0001 C CNN "Field3"
-F 7 "-,-" V 3705 800 60  0001 C CNN "Field4"
-F 8 "100,V" V 3705 800 60  0001 C CNN "Field5"
-F 9 "10,%" V 3705 800 60  0001 C CNN "Field6"
-F 10 "ceramic" V 3705 800 60  0001 C CNN "Field7"
-F 11 "other,more,stuff" V 3705 800 60  0001 C CNN "Field8"
+F 0 "C409" H 7200 700 50  0000 L CNN
+F 1 "0.1uF" H 6950 900 50  0000 L CNN
+F 2 "SM0805-C1" V 1130 2600 60  0001 C CNN
+F 4 "avx,08051C104KAT2A" V 1130 2600 60  0001 C CNN "mfg,mfg#"
+F 5 "newark,96M1354" V 1130 2600 60  0001 C CNN "vend1,vend1#"
+F 6 "" V 1130 2600 60  0001 C CNN ""
+F 7 "" V 1130 2600 60  0001 C CNN ""
+F 8 "100V" V 1130 2600 60  0001 C CNN "V"
+F 9 "10%" V 1130 2600 60  0001 C CNN "tolerance"
+F 10 "ceramic" V 1130 2600 60  0001 C CNN "construct"
+F 11 "other,more,stuff" V 1130 2600 60  0001 C CNN "misc"
 	1    7175 800
 	-1   0    0    1
@@
 U 1 1 4E39DF39
 P 7175 2800
-F 0 "C410" H 7225 2900 50  0000 L CNN
-F 1 ".1uF" H 7025 2900 50  0000 L CNN
-F 2 "SM0805-C1" V 3705 2800 60  0001 C CNN
-F 4 "avx,08051C104KAT2A" V 3705 2800 60  0001 C CNN "mfg,#"
-F 5 "newark,96M1354" V 3705 2800 60  0001 C CNN "vend,#"
-F 6 "-,-" V 3705 2800 60  0001 C CNN "Field3"
-F 7 "-,-" V 3705 2800 60  0001 C CNN "Field4"
-F 8 "100,V" V 3705 2800 60  0001 C CNN "Field5"
-F 9 "10,%" V 3705 2800 60  0001 C CNN "Field6"
-F 10 "ceramic" V 3705 2800 60  0001 C CNN "Field7"
-F 11 "other,more,stuff" V 3705 2800 60  0001 C CNN "Field8"
+F 0 "C410" H 7250 2700 50  0000 L CNN
+F 1 "0.1uF" H 6950 2900 50  0000 L CNN
+F 2 "SM0805-C1" V 1130 2600 60  0001 C CNN
+F 4 "avx,08051C104KAT2A" V 1130 2600 60  0001 C CNN "mfg,mfg#"
+F 5 "newark,96M1354" V 1130 2600 60  0001 C CNN "vend1,vend1#"
+F 6 "" V 1130 2600 60  0001 C CNN ""
+F 7 "" V 1130 2600 60  0001 C CNN ""
+F 8 "100V" V 1130 2600 60  0001 C CNN "V"
+F 9 "10%" V 1130 2600 60  0001 C CNN "tolerance"
+F 10 "ceramic" V 1130 2600 60  0001 C CNN "construct"
+F 11 "other,more,stuff" V 1130 2600 60  0001 C CNN "misc"
 	1    7175 2800
 	-1   0    0    1
@@
 U 1 1 4E39DF32
 P 7625 2800
-F 0 "C412" H 7675 2900 50  0000 L CNN
+F 0 "C412" H 7700 2700 50  0000 L CNN
 F 1 "10uF" H 7400 2900 50  0000 L CNN
 F 2 "SM0805-C1" V 4155 2800 60  0001 C CNN
@@
 U 1 1 4E39DF0D
 P 2775 2800
-F 0 "C404" H 2825 2900 50  0000 L CNN
+F 0 "C404" H 2850 2700 50  0000 L CNN
 F 1 "10uF" H 2550 2900 50  0000 L CNN
 F 2 "SM0805-C1" V -695 2800 60  0001 C CNN
@@
 U 1 1 4E39DF06
 P 2250 2800
-F 0 "C402" H 2300 2900 50  0000 L CNN
-F 1 ".1uF" H 2100 2900 50  0000 L CNN
-F 2 "SM0805-C1" V -1220 2800 60  0001 C CNN
-F 4 "avx,08051C104KAT2A" V -1220 2800 60  0001 C CNN "mfg,#"
-F 5 "newark,96M1354" V -1220 2800 60  0001 C CNN "vend,#"
-F 6 "-,-" V -1220 2800 60  0001 C CNN "Field3"
-F 7 "-,-" V -1220 2800 60  0001 C CNN "Field4"
-F 8 "100,V" V -1220 2800 60  0001 C CNN "Field5"
-F 9 "10,%" V -1220 2800 60  0001 C CNN "Field6"
-F 10 "ceramic" V -1220 2800 60  0001 C CNN "Field7"
-F 11 "other,more,stuff" V -1220 2800 60  0001 C CNN "Field8"
+F 0 "C402" H 2350 2700 50  0000 L CNN
+F 1 "0.1uF" H 2000 2900 50  0000 L CNN
+F 2 "SM0805-C1" V 1130 2600 60  0001 C CNN
+F 4 "avx,08051C104KAT2A" V 1130 2600 60  0001 C CNN "mfg,mfg#"
+F 5 "newark,96M1354" V 1130 2600 60  0001 C CNN "vend1,vend1#"
+F 6 "" V 1130 2600 60  0001 C CNN ""
+F 7 "" V 1130 2600 60  0001 C CNN ""
+F 8 "100V" V 1130 2600 60  0001 C CNN "V"
+F 9 "10%" V 1130 2600 60  0001 C CNN "tolerance"
+F 10 "ceramic" V 1130 2600 60  0001 C CNN "construct"
+F 11 "other,more,stuff" V 1130 2600 60  0001 C CNN "misc"
 	1    2250 2800
 	-1   0    0    1
@@
 U 1 1 4ADA0C57
 P 2250 800
-F 0 "C401" H 2300 900 50  0000 L CNN
-F 1 ".1uF" H 2100 900 50  0000 L CNN
-F 2 "SM0805-C1" V -1220 800 60  0001 C CNN
-F 4 "avx,08051C104KAT2A" V -1220 800 60  0001 C CNN "mfg,#"
-F 5 "newark,96M1354" V -1220 800 60  0001 C CNN "vend,#"
-F 6 "-,-" V -1220 800 60  0001 C CNN "Field3"
-F 7 "-,-" V -1220 800 60  0001 C CNN "Field4"
-F 8 "100,V" V -1220 800 60  0001 C CNN "Field5"
-F 9 "10,%" V -1220 800 60  0001 C CNN "Field6"
-F 10 "ceramic" V -1220 800 60  0001 C CNN "Field7"
-F 11 "other,more,stuff" V -1220 800 60  0001 C CNN "Field8"
+F 0 "C401" H 2300 700 50  0000 L CNN
+F 1 "0.1uF" H 2000 900 50  0000 L CNN
+F 2 "SM0805-C1" V 1130 2600 60  0001 C CNN
+F 4 "avx,08051C104KAT2A" V 1130 2600 60  0001 C CNN "mfg,mfg#"
+F 5 "newark,96M1354" V 1130 2600 60  0001 C CNN "vend1,vend1#"
+F 6 "" V 1130 2600 60  0001 C CNN ""
+F 7 "" V 1130 2600 60  0001 C CNN ""
+F 8 "100V" V 1130 2600 60  0001 C CNN "V"
+F 9 "10%" V 1130 2600 60  0001 C CNN "tolerance"
+F 10 "ceramic" V 1130 2600 60  0001 C CNN "construct"
+F 11 "other,more,stuff" V 1130 2600 60  0001 C CNN "misc"
 	1    2250 800
 	-1   0    0    1
@@
 U 1 1 4AD9CB8E
 P 2775 800
-F 0 "C403" H 2825 900 50  0000 L CNN
+F 0 "C403" H 2850 700 50  0000 L CNN
 F 1 "10uF" H 2550 900 50  0000 L CNN
 F 2 "SM0805-C1" V -695 800 60  0001 C CNN

Commit message: Looks like the bulk components are golden now, there are still a couple straglers, mostly switch mode power supply stuff.
Signed-off-by: Jared Harvey <TortiseGIT@jaredharvey.com>
Parts:
- R401, R402, R403, R404, R429, R430, R431, R432: Field3 -,- -> (none); Field4 -,- -> (none); Field5 125,mW -> (none); Field6 1,% -> (none); Field7 thick film -> (none); Field8 other,more,stuff -> (none); construct (none) -> thick film; mfg,# bourns,CR0805-FX-1002ELF -> (none); mfg,mfg# (none) -> BOURNS,CR0805-FX-1002ELF; misc (none) -> other,more,stuff; tolerance (none) -> 1%; vend,# newark,02J2368 -> (none); vend1,vend1# (none) -> newark,02J2368; w (none) -> 125mW

Commit message: several pins on the SOM are now connected.
Signed-off-by: Jared Harvey <TortiseGIT@jaredharvey.com>
Parts:
- renumbered C401 to C601, C402 to C602, C403 to C603, C404 to C604, C405 to C605, C406 to C606, C407 to C607, C408 to C608, C409 to C609, C410 to C610, C411 to C611, C412 to C612, C413 to C613, C414 to C614, C415 to C615, C416 to C616, P401 to P601, P402 to P602, P403 to P603, P404 to P604, P405 to P605, P406 to P606, P407 to P607, P408 to P608, P409 to P609, P410 to P610, P411 to P611, P412 to P612, P413 to P613, P414 to P614, P415 to P615, P416 to P616, R401 to R681, R402 to R682, R403 to R683, R404 to R684, R405 to R685, R406 to R686, R407 to R687, R408 to R688, R409 to R689, R410 to R690, R411 to R691, R412 to R692, R413 to R693, R414 to R694, R415 to R695, R416 to R696, R417 to R697, R418 to R698, R419 to R699, R420 to R700, R421 to R701, R422 to R702, R423 to R703, R424 to R704, R425 to R705, R426 to R706, R427 to R707, R428 to R708, R429 to R709, R430 to R710, R431 to R711, R432 to R712, R433 to R713, R434 to R714, R435 to R715, R436 to R716, R437 to R717, R438 to R718, R439 to R719, R440 to R720, R441 to R721, R442 to R722, R443 to R723, R444 to R724, R445 to R725, R446 to R726, R447 to R727, R448 to R728, R449 to R729, R450 to R730, R451 to R731, R452 to R732, R453 to R733, R454 to R734, R455 to R735, R456 to R736, U401 to U601, U402 to U602, U403 to U603, U404 to U604
