File: KICAD_Project/sub_circuits/RPM_input_MAX9926.sch (KiCad schematic (older format))
At the start: 92 parts, among them P601 CONN_1, P602 CONN_1, P603 CONN_1, P604 CONN_1, P605 CONN_1, P606 CONN_1, P607 CONN_1, P608 CONN_1, P609 CONN_1, P610 CONN_1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

Commit message: more stepper updates
Signed-off-by: Jared Harvey <TortiseGIT@jaredharvey.com>
Parts:
- C603, C604, C611, C612: Field3 -,- -> (none); Field4 -,- -> (none); Field5 200,V -> (none); Field6 20,% -> (none); Field7 alum electro -> (none); Field8 other,more,stuff -> (none); V (none) -> 25V; construct (none) -> multi layer ceramic; mfg,# ill cap,106CKE200M -> (none); mfg,mfg# (none) -> AVX,08053C104KAT2A; misc (none) -> other,more,stuff; tolerance (none) -> 10%; vend,# newark,69K7896 -> (none); vend1,vend1# (none) -> newark,96M1381
Changed lines of the file:
@@
-EESchema Schematic File Version 2  date 8/27/2011 10:55:18 AM
+EESchema Schematic File Version 2  date 8/30/2011 5:58:29 AM
 LIBS:power
 LIBS:device
@@
 Sheet 6 13
 Title "freeEMS PLUS from Cinch template "
-Date "27 aug 2011"
+Date "30 aug 2011"
 Rev "A-DRAF"
 Comp "diyefi.org/openecu.info"
@@
 F 0 "C611" H 7650 700 50  0000 L CNN
 F 1 "10uF" H 7400 900 50  0000 L CNN
-F 2 "SM0805-C1" V 4155 800 60  0001 C CNN
-F 4 "ill cap,106CKE200M" V 4155 800 60  0001 C CNN "mfg,#"
-F 5 "newark,69K7896" V 4155 800 60  0001 C CNN "vend,#"
-F 6 "-,-" V 4155 800 60  0001 C CNN "Field3"
-F 7 "-,-" V 4155 800 60  0001 C CNN "Field4"
-F 8 "200,V" V 4155 800 60  0001 C CNN "Field5"
-F 9 "20,%" V 4155 800 60  0001 C CNN "Field6"
-F 10 "alum electro" V 4155 800 60  0001 C CNN "Field7"
-F 11 "other,more,stuff" V 4155 800 60  0001 C CNN "Field8"
+F 2 "SM0805-C1" V 1130 2600 60  0001 C CNN
+F 4 "AVX,08053C104KAT2A" V 1130 2600 60  0001 C CNN "mfg,mfg#"
+F 5 "newark,96M1381" V 1130 2600 60  0001 C CNN "vend1,vend1#"
+F 6 "" V 1130 2600 60  0001 C CNN ""
+F 7 "" V 1130 2600 60  0001 C CNN ""
+F 8 "25V" V 1130 2600 60  0001 C CNN "V"
+F 9 "10%" V 1130 2600 60  0001 C CNN "tolerance"
+F 10 "multi layer ceramic" V 1130 2600 60  0001 C CNN "construct"
+F 11 "other,more,stuff" V 1130 2600 60  0001 C CNN "misc"
 	1    7625 800
 	-1   0    0    1
@@
 F 0 "C612" H 7700 2700 50  0000 L CNN
 F 1 "10uF" H 7400 2900 50  0000 L CNN
-F 2 "SM0805-C1" V 4155 2800 60  0001 C CNN
-F 4 "ill cap,106CKE200M" V 4155 2800 60  0001 C CNN "mfg,#"
-F 5 "newark,69K7896" V 4155 2800 60  0001 C CNN "vend,#"
-F 6 "-,-" V 4155 2800 60  0001 C CNN "Field3"
-F 7 "-,-" V 4155 2800 60  0001 C CNN "Field4"
-F 8 "200,V" V 4155 2800 60  0001 C CNN "Field5"
-F 9 "20,%" V 4155 2800 60  0001 C CNN "Field6"
-F 10 "alum electro" V 4155 2800 60  0001 C CNN "Field7"
-F 11 "other,more,stuff" V 4155 2800 60  0001 C CNN "Field8"
+F 2 "SM0805-C1" V 1130 2600 60  0001 C CNN
+F 4 "AVX,08053C104KAT2A" V 1130 2600 60  0001 C CNN "mfg,mfg#"
+F 5 "newark,96M1381" V 1130 2600 60  0001 C CNN "vend1,vend1#"
+F 6 "" V 1130 2600 60  0001 C CNN ""
+F 7 "" V 1130 2600 60  0001 C CNN ""
+F 8 "25V" V 1130 2600 60  0001 C CNN "V"
+F 9 "10%" V 1130 2600 60  0001 C CNN "tolerance"
+F 10 "multi layer ceramic" V 1130 2600 60  0001 C CNN "construct"
+F 11 "other,more,stuff" V 1130 2600 60  0001 C CNN "misc"
 	1    7625 2800
 	-1   0    0    1
@@
 F 0 "C604" H 2850 2700 50  0000 L CNN
 F 1 "10uF" H 2550 2900 50  0000 L CNN
-F 2 "SM0805-C1" V -695 2800 60  0001 C CNN
-F 4 "ill cap,106CKE200M" V -695 2800 60  0001 C CNN "mfg,#"
-F 5 "newark,69K7896" V -695 2800 60  0001 C CNN "vend,#"
-F 6 "-,-" V -695 2800 60  0001 C CNN "Field3"
-F 7 "-,-" V -695 2800 60  0001 C CNN "Field4"
-F 8 "200,V" V -695 2800 60  0001 C CNN "Field5"
-F 9 "20,%" V -695 2800 60  0001 C CNN "Field6"
-F 10 "alum electro" V -695 2800 60  0001 C CNN "Field7"
-F 11 "other,more,stuff" V -695 2800 60  0001 C CNN "Field8"
+F 2 "SM0805-C1" V 1130 2600 60  0001 C CNN
+F 4 "AVX,08053C104KAT2A" V 1130 2600 60  0001 C CNN "mfg,mfg#"
+F 5 "newark,96M1381" V 1130 2600 60  0001 C CNN "vend1,vend1#"
+F 6 "" V 1130 2600 60  0001 C CNN ""
+F 7 "" V 1130 2600 60  0001 C CNN ""
+F 8 "25V" V 1130 2600 60  0001 C CNN "V"
+F 9 "10%" V 1130 2600 60  0001 C CNN "tolerance"
+F 10 "multi layer ceramic" V 1130 2600 60  0001 C CNN "construct"
+F 11 "other,more,stuff" V 1130 2600 60  0001 C CNN "misc"
 	1    2775 2800
 	-1   0    0    1
@@
 F 0 "C603" H 2850 700 50  0000 L CNN
 F 1 "10uF" H 2550 900 50  0000 L CNN
-F 2 "SM0805-C1" V -695 800 60  0001 C CNN
-F 4 "ill cap,106CKE200M" V -695 800 60  0001 C CNN "mfg,#"
-F 5 "newark,69K7896" V -695 800 60  0001 C CNN "vend,#"
-F 6 "-,-" V -695 800 60  0001 C CNN "Field3"
-F 7 "-,-" V -695 800 60  0001 C CNN "Field4"
-F 8 "200,V" V -695 800 60  0001 C CNN "Field5"
-F 9 "20,%" V -695 800 60  0001 C CNN "Field6"
-F 10 "alum electro" V -695 800 60  0001 C CNN "Field7"
-F 11 "other,more,stuff" V -695 800 60  0001 C CNN "Field8"
+F 2 "SM0805-C1" V 1130 2600 60  0001 C CNN
+F 4 "AVX,08053C104KAT2A" V 1130 2600 60  0001 C CNN "mfg,mfg#"
+F 5 "newark,96M1381" V 1130 2600 60  0001 C CNN "vend1,vend1#"
+F 6 "" V 1130 2600 60  0001 C CNN ""
+F 7 "" V 1130 2600 60  0001 C CNN ""
+F 8 "25V" V 1130 2600 60  0001 C CNN "V"
+F 9 "10%" V 1130 2600 60  0001 C CNN "tolerance"
+F 10 "multi layer ceramic" V 1130 2600 60  0001 C CNN "construct"
+F 11 "other,more,stuff" V 1130 2600 60  0001 C CNN "misc"
 	1    2775 800
 	-1   0    0    1
