File: KICAD_Project/sub_circuits/amp_connector.sch (KiCad schematic (older format))
At the start: 30 parts

Commit message: More work to capture, also I need it up there for collaboration purposes.
Signed-off-by: Jared Harvey <TortiseGIT@jaredharvey.com>
Parts:
- added J?: MOLEX_HARNESS_SD-64333-100, symbol MOLEX_HARNESS_SD-64333-100
Changed lines of the file:
@@
-EESchema Schematic File Version 2  date 8/6/2011 9:18:51 PM
+EESchema Schematic File Version 2  date 8/6/2011 11:05:38 PM
 LIBS:power
 LIBS:device
@@
 $Descr A 11000 8500
 encoding utf-8
-Sheet 8 16
-Title "freeEMS PLUS"
+Sheet 6 14
+Title "freeEMS PLUS from Cinch template "
 Date "7 aug 2011"
 Rev "A"
@@
 Comment4 ""
 $EndDescr
+$Comp
+L MOLEX_HARNESS_SD-64333-100 J?
+U 1 1 4E3DF531
+P 3850 3900
+F 0 "J?" H 3850 5650 70  0000 C CNN
+F 1 "MOLEX_HARNESS_SD-64333-100" H 3900 1900 70  0000 C CNN
+	1    3850 3900
+	1    0    0    -1
+$EndComp
 Wire Wire Line
 	7975 2250 8050 2250

Commit message: About to runs scripts to scrub the BOM's, so here's a backup copy in case it goes wrong.
Signed-off-by: Jared Harvey <TortiseGIT@jaredharvey.com>
Parts:
- J601: renamed from J?; footprint (none) -> Molex_SD-64333-100_on_Cinch_ModICE_w_5554_SOM
- P601: renamed from P?; footprint AMP35 -> (none)
- P602: renamed from P??; footprint AMP35 -> (none)
- gave numbers to parts that had none: 28
Changed lines of the file:
@@
-EESchema Schematic File Version 2  date 8/7/2011 7:33:14 PM
+EESchema Schematic File Version 2  date 8/14/2011 3:32:14 PM
 LIBS:power
 LIBS:device
@@
 $Descr A 11000 8500
 encoding utf-8
-Sheet 6 14
+Sheet 6 13
 Title "freeEMS PLUS from Cinch template "
-Date "7 aug 2011"
+Date "14 aug 2011"
 Rev "A"
 Comp "diyefi.org/openecu.info"
@@
 $EndDescr
 $Comp
-L MOLEX_HARNESS_SD-64333-100 J?
+L MOLEX_HARNESS_SD-64333-100 J601
 U 1 1 4E3DF531
 P 3850 3900
-F 0 "J?" H 3850 5650 70  0000 C CNN
+F 0 "J601" H 3850 5650 70  0000 C CNN
 F 1 "MOLEX_HARNESS_SD-64333-100" H 3900 1900 70  0000 C CNN
+F 2 "Molex_SD-64333-100_on_Cinch_ModICE_w_5554_SOM" H 3850 3900 60  0001 C CNN
 	1    3850 3900
 	1    0    0    -1
@@
 AN/GPI_1
 $Comp
-L R R?
+L R R622
 U 1 1 4C255D9A
 P 9575 2650
-F 0 "R?" V 9550 2975 50  0000 C CNN
+F 0 "R622" V 9550 2975 50  0000 C CNN
 F 1 "0R" V 9575 2650 50  0000 C CNN
 F 2 "SM0805-C1" H 9575 2650 60  0001 C CNN
@@
 $EndComp
 $Comp
-L R R?
+L R R621
 U 1 1 4C255D99
 P 9575 2550
-F 0 "R?" V 9550 2875 50  0000 C CNN
+F 0 "R621" V 9550 2875 50  0000 C CNN
 F 1 "0R" V 9575 2550 50  0000 C CNN
 F 2 "SM0805-C1" H 9575 2550 60  0001 C CNN
@@
 AN/GPI_3
 $Comp
-L R R?
+L R R623
 U 1 1 4C255D95
 P 9575 2750
-F 0 "R?" V 9550 3075 50  0000 C CNN
+F 0 "R623" V 9550 3075 50  0000 C CNN
 F 1 "0R" V 9575 2750 50  0000 C CNN
 F 2 "SM0805-C1" H 9575 2750 60  0001 C CNN
@@
 $EndComp
 $Comp
-L R R?
+L R R624
 U 1 1 4C255D94
 P 9575 2850
-F 0 "R?" V 9550 3175 50  0000 C CNN
+F 0 "R624" V 9550 3175 50  0000 C CNN
 F 1 "0R" V 9575 2850 50  0000 C CNN
 F 2 "SM0805-C1" H 9575 2850 60  0001 C CNN
@@
 $EndComp
 $Comp
-L R R?
+L R R626
 U 1 1 4C255D32
 P 9575 3050
-F 0 "R?" V 9550 3375 50  0000 C CNN
+F 0 "R626" V 9550 3375 50  0000 C CNN
 F 1 "0R" V 9575 3050 50  0000 C CNN
 F 2 "SM0805-C1" H 9575 3050 60  0001 C CNN
@@
 $EndComp
 $Comp
-L R R?
+L R R625
 U 1 1 4C255D31
 P 9575 2950
-F 0 "R?" V 9550 3275 50  0000 C CNN
+F 0 "R625" V 9550 3275 50  0000 C CNN
 F 1 "0R" V 9575 2950 50  0000 C CNN
 F 2 "SM0805-C1" H 9575 2950 60  0001 C CNN
@@
 AN/GPI_5
 $Comp
-L R R?
+L R R627
 U 1 1 4C255D18
 P 9575 3150
-F 0 "R?" V 9550 3475 50  0000 C CNN
+F 0 "R627" V 9550 3475 50  0000 C CNN
 F 1 "0R" V 9575 3150 50  0000 C CNN
 F 2 "SM0805-C1" H 9575 3150 60  0001 C CNN
@@
 $EndComp
 $Comp
-L R R?
+L R R628
 U 1 1 4C255D17
 P 9575 3250
-F 0 "R?" V 9550 3575 50  0000 C CNN
+F 0 "R628" V 9550 3575 50  0000 C CNN
 F 1 "0R" V 9575 3250 50  0000 C CNN
 F 2 "SM0805-C1" H 9575 3250 60  0001 C CNN
@@
 MISC_6
 $Comp
-L R R?
+L R R617
 U 1 1 4C255AD4
 P 9525 4750
-F 0 "R?" V 9500 5075 50  0000 C CNN
+F 0 "R617" V 9500 5075 50  0000 C CNN
 F 1 "0R" V 9525 4750 50  0000 C CNN
 F 2 "SM0805-C1" H 9525 4750 60  0001 C CNN
@@
 $EndComp
 $Comp
-L R R?
+L R R619
 U 1 1 4C255AD3
 P 9525 4950
-F 0 "R?" V 9500 5275 50  0000 C CNN
+F 0 "R619" V 9500 5275 50  0000 C CNN
 F 1 "0R" V 9525 4950 50  0000 C CNN
 F 2 "SM0805-C1" H 9525 4950 60  0001 C CNN
@@
 $EndComp
 $Comp
-L R R?
+L R R620
 U 1 1 4C255AD2
 P 9525 5050
-F 0 "R?" V 9500 5375 50  0000 C CNN
+F 0 "R620" V 9500 5375 50  0000 C CNN
 F 1 "0R" V 9525 5050 50  0000 C CNN
 F 2 "SM0805-C1" H 9525 5050 60  0001 C CNN
@@
 $EndComp
 $Comp
-L R R?
+L R R618
 U 1 1 4C255AD1
 P 9525 4850
-F 0 "R?" V 9500 5175 50  0000 C CNN
+F 0 "R618" V 9500 5175 50  0000 C CNN
 F 1 "0R" V 9525 4850 50  0000 C CNN
 F 2 "SM0805-C1" H 9525 4850 60  0001 C CNN
@@
 $EndComp
 $Comp
-L R R?
+L R R614
 U 1 1 4C255A92
 P 9525 4450
-F 0 "R?" V 9500 4775 50  0000 C CNN
+F 0 "R614" V 9500 4775 50  0000 C CNN
 F 1 "0R" V 9525 4450 50  0000 C CNN
 F 2 "SM0805-C1" H 9525 4450 60  0001 C CNN
@@
 $EndComp
 $Comp
-L R R?
+L R R616
 U 1 1 4C255A91
 P 9525 4650
-F 0 "R?" V 9500 4975 50  0000 C CNN
+F 0 "R616" V 9500 4975 50  0000 C CNN
 F 1 "0R" V 9525 4650 50  0000 C CNN
 F 2 "SM0805-C1" H 9525 4650 60  0001 C CNN
@@
 $EndComp
 $Comp
-L R R?
+L R R615
 U 1 1 4C255A90
 P 9525 4550
-F 0 "R?" V 9500 4875 50  0000 C CNN
+F 0 "R615" V 9500 4875 50  0000 C CNN
 F 1 "0R" V 9525 4550 50  0000 C CNN
 F 2 "SM0805-C1" H 9525 4550 60  0001 C CNN
@@
 $EndComp
 $Comp
-L R R?
+L R R613
 U 1 1 4C255A8F
 P 9525 4350
-F 0 "R?" V 9500 4675 50  0000 C CNN
+F 0 "R613" V 9500 4675 50  0000 C CNN
 F 1 "0R" V 9525 4350 50  0000 C CNN
 F 2 "SM0805-C1" H 9525 4350 60  0001 C CNN
@@
 232_RX
 $Comp
-L R R?
+L R R601
 U 1 1 4C2559AC
 P 6775 4750
-F 0 "R?" V 6725 5025 50  0000 C CNN
+F 0 "R601" V 6725 5025 50  0000 C CNN
 F 1 "0R" V 6775 4750 50  0000 C CNN
 F 2 "SM0805-C1" H 6775 4750 60  0001 C CNN
@@
 $EndComp
 $Comp
-L R R?
+L R R603
 U 1 1 4C2559AB
 P 6775 4950
-F 0 "R?" V 6725 5225 50  0000 C CNN
+F 0 "R603" V 6725 5225 50  0000 C CNN
 F 1 "0R" V 6775 4950 50  0000 C CNN
 F 2 "SM0805-C1" H 6775 4950 60  0001 C CNN
@@
 $EndComp
 $Comp
-L R R?
+L R R604
 U 1 1 4C2559A9
 P 6775 5050
-F 0 "R?" V 6725 5325 50  0000 C CNN
+F 0 "R604" V 6725 5325 50  0000 C CNN
 F 1 "0R" V 6775 5050 50  0000 C CNN
 F 2 "SM0805-C1" H 6775 5050 60  0001 C CNN
@@
 $EndComp
 $Comp
-L R R?
+L R R602
 U 1 1 4C2559A8
 P 6775 4850
-F 0 "R?" V 6725 5125 50  0000 C CNN
+F 0 "R602" V 6725 5125 50  0000 C CNN
 F 1 "0R" V 6775 4850 50  0000 C CNN
 F 2 "SM0805-C1" H 6775 4850 60  0001 C CNN
@@
 $EndComp
 $Comp
-L R R?
+L R R606
 U 1 1 4C255811
 P 6775 5950
-F 0 "R?" V 6725 6200 50  0000 C CNN
+F 0 "R606" V 6725 6200 50  0000 C CNN
 F 1 "0R" V 6775 5950 50  0000 C CNN
 F 2 "SM0805-C1" H 6775 5950 60  0001 C CNN
@@
 $EndComp
 $Comp
-L R R?
+L R R608
 U 1 1 4C255810
 P 6775 6150
-F 0 "R?" V 6725 6400 50  0000 C CNN
+F 0 "R608" V 6725 6400 50  0000 C CNN
 F 1 "0R" V 6775 6150 50  0000 C CNN
 F 2 "SM0805-C1" H 6775 6150 60  0001 C CNN
@@
 $EndComp
 $Comp
-L R R?
+L R R612
 U 1 1 4C25580F
 P 6775 6550
-F 0 "R?" V 6725 6800 50  0000 C CNN
+F 0 "R612" V 6725 6800 50  0000 C CNN
 F 1 "0R" V 6775 6550 50  0000 C CNN
 F 2 "SM0805-C1" H 6775 6550 60  0001 C CNN
@@
 $EndComp
 $Comp
-L R R?
+L R R610
 U 1 1 4C25580E
 P 6775 6350
-F 0 "R?" V 6725 6600 50  0000 C CNN
+F 0 "R610" V 6725 6600 50  0000 C CNN
 F 1 "0R" V 6775 6350 50  0000 C CNN
 F 2 "SM0805-C1" H 6775 6350 60  0001 C CNN
@@
 $EndComp
 $Comp
-L R R?
+L R R609
 U 1 1 4C2557BE
 P 6775 6250
-F 0 "R?" V 6725 6500 50  0000 C CNN
+F 0 "R609" V 6725 6500 50  0000 C CNN
 F 1 "0R" V 6775 6250 50  0000 C CNN
 F 2 "SM0805-C1" H 6775 6250 60  0001 C CNN
@@
 $EndComp
 $Comp
-L R R?
+L R R611
 U 1 1 4C2557BD
 P 6775 6450
-F 0 "R?" V 6725 6700 50  0000 C CNN
+F 0 "R611" V 6725 6700 50  0000 C CNN
 F 1 "0R" V 6775 6450 50  0000 C CNN
 F 2 "SM0805-C1" H 6775 6450 60  0001 C CNN
@@
 $EndComp
 $Comp
-L R R?
+L R R607
 U 1 1 4C2557B4
 P 6775 6050
-F 0 "R?" V 6725 6300 50  0000 C CNN
+F 0 "R607" V 6725 6300 50  0000 C CNN
 F 1 "0R" V 6775 6050 50  0000 C CNN
 F 2 "SM0805-C1" H 6775 6050 60  0001 C CNN
@@
 $EndComp
 $Comp
-L R R?
+L R R605
 U 1 1 4C25578F
 P 6775 5850
-F 0 "R?" V 6725 6100 50  0000 C CNN
+F 0 "R605" V 6725 6100 50  0000 C CNN
 F 1 "0R" V 6775 5850 50  0000 C CNN
 F 2 "SM0805-C1" H 6775 5850 60  0001 C CNN
@@
 GND_PWR1
 $Comp
-L AMP35 P?
+L AMP35 P601
 U 1 1 4C215770
 P 8450 5450
-F 0 "P?" H 8500 6800 70  0000 C CNN
+F 0 "P601" H 8500 6800 70  0000 C CNN
 F 1 "AMP35" H 8400 4100 70  0000 C CNN
-F 2 "AMP35" H 8450 5450 60  0001 C CNN
 	1    8450 5450
 	1    0    0    -1
 $EndComp
 $Comp
-L AMP35 P??
+L AMP35 P602
 U 1 1 4C21576A
 P 8500 2450
-F 0 "P??" H 8550 3800 70  0000 C CNN
+F 0 "P602" H 8550 3800 70  0000 C CNN
 F 1 "AMP35" H 8450 1100 70  0000 C CNN
-F 2 "AMP35" H 8500 2450 60  0001 C CNN
 	1    8500 2450
 	1    0    0    -1

Commit message: Looks like the bulk components are golden now, there are still a couple straglers, mostly switch mode power supply stuff.
Signed-off-by: Jared Harvey <TortiseGIT@jaredharvey.com>
Parts:
- R601, R602, R603, R604, R605, R606, R607, R608, R609, R610, R611, R612, R613, R614, R615, R616, R617, R618, R619, R620, R621, R622, R623, R624, R625, R626, R627, R628: footprint SM0805-C1 -> SM0805; mfg,# vishay,CRCW08050000ZSTA -> (none); mfg,mfg# (none) -> vishay,CRCW08050000Z0EA; misc (none) -> other,more,stuff; tolerance (none) -> %; vend,# newark,36C9353 -> (none); vend1,vend1# (none) -> newark,52K9721; w (none) -> mW

Commit message: harness connector is much more ironed out now. CPU is not connected.
Signed-off-by: Jared Harvey <TortiseGIT@jaredharvey.com>
Parts:
- removed P601, P602: AMP35, symbol AMP35
- removed R601, R602, R603, R604, R605, R606, R607, R608, R609, R610, R611, R612, R613, R614, R615, R616, R617, R618, R619, R620, R621, R622, R623, R624, R625, R626, R627, R628: 0R, SM0805, symbol R
Connections:
- net labels added: 12V_BAT, 12V_ECU, CAM+, CAM-, CANH, CANL, CRANK+, CRANK-, ENG_TEMP, EXTRA, GND, GND1_INJIGN, GND2_INJIGN, GND3_INJIGN, GND4_STAGED8, GND5_STAGED4, HS2, HS3, IGN01_HARN, IGN02_HARN, IGN03_HARN, IGN04_HARN, IGN05_HARN, IGN06_HARN, IGN07_HARN, IGN08_HARN, IGN09_HARN, IGN10_HARN, IGN11_HARN, IGN12_HARN, INJ01_HARN, INJ02_HARN, INJ03_HARN, INJ04_HARN, INJ05_HARN, INJ06_HARN, INJ07_HARN, INJ08_HARN, INJ09_HARN, INJ10_HARN, INJ11_HARN, INJ12_HARN, INJ13_HARN, INJ14_HARN, INJ15_HARN, INJ16_HARN, INJ17_HARN, INJ18_HARN, INJ19_HARN, INJ20_HARN, INJ21_HARN, INJ22_HARN, INJ23_HARN, INJ24_HARN, KNCK1+, KNCK1-, KNCK2+, KNCK2-, MAP+_5V, MAP_GND, MIAT, MIL_LS-1A, MISC_1A, O2_HD1_PWR, O2_HD2_PWR, O2_IA1, O2_IA2, O2_IP1, O2_IP2, O2_UN1, O2_UN2, O2_VM1, O2_VM2, P01, P02, P03, P04, P05, P06, P07, P08, P09, P10, P11, P12, P13, P14, PUMP_LS-1A, RPM_LB+, RPM_LB-, RPM_LF+, RPM_LF-, RPM_RB+, RPM_RB-, RPM_RF+, RPM_RF-, STEP_GND, TPS+_5V, TPS-_GND, TPS_SIG
- net labels removed: 5VREG_PWR, 5VREG_SENSE, AN/GPI_1, AN/GPI_2, AN/GPI_3, AN/GPI_4, AN/GPI_5, CANH-PIN, CANL-PIN, GND_PWR1, GND_PWR2, GND_PWR3, GND_SENSE, IGN10_PIN, IGN11_PIN, IGN12_PIN, IGN1_PIN, IGN2_PIN, IGN3_PIN, IGN4_PIN, IGN5_PIN, IGN6_PIN, IGN7_PIN, IGN8_PIN, IGN9_PIN, INJ10_PIN, INJ11_PIN, INJ12_PIN, INJ1_PIN, INJ2_PIN, INJ3_PIN, INJ4_PIN, INJ5_PIN, INJ6_PIN, INJ7_PIN, INJ8_PIN, INJ9_PIN, KNCK1+PIN, KNCK1-PIN, KNCK2+PIN, KNCK2-PIN, MIL_33800, MISC_3, MISC_4, MISC_5, MISC_6, O2_HD1-PIN, O2_HD2-PIN, O2_IA1-PIN, O2_IA2-PIN, O2_IP1-PIN, O2_IP2-PIN, O2_UN1-PIN, O2_UN2-PIN, O2_VM1-PIN, O2_VM2-PIN, PUMP_33800, THERM1, THERM2, THERM_AIR, THERM_ENG, TPS_AN, VBAT_SW, VR+_CAM1_PIN, VR+_CAM2_PIN, VR+_CR_PIN, VR+_WHBL_PIN, VR+_WHBR_PIN, VR+_WHFL_PIN, VR+_WHFR_PIN, VR-_CAM1_PIN, VR-_CAM2_PIN, VR-_CR_PIN, VR-_WH_COMMON
- wire segments 126 -> 6

Commit message: several pins on the SOM are now connected.
Signed-off-by: Jared Harvey <TortiseGIT@jaredharvey.com>
Parts:
- renumbered J601 to J301
Changed lines of the file:
@@
-EESchema Schematic File Version 2  date 8/19/2011 6:13:40 AM
+EESchema Schematic File Version 2  date 8/20/2011 7:18:54 AM
 LIBS:power
 LIBS:device
@@
 $Descr A 11000 8500
 encoding utf-8
-Sheet 2 13
+Sheet 3 13
 Title "freeEMS PLUS from Cinch template "
-Date "19 aug 2011"
+Date "20 aug 2011"
 Rev "A-DRAF"
 Comp "diyefi.org/openecu.info"
@@
 GND
 $Comp
-L MOLEX_HARNESS_SD-64333-100 J601
+L MOLEX_HARNESS_SD-64333-100 J301
 U 1 1 4E3DF531
 P 7825 5275
-F 0 "J601" H 9350 5275 70  0000 C CNN
+F 0 "J301" H 9350 5275 70  0000 C CNN
 F 1 "MOLEX_HARNESS_SD-64333-100" H 6950 5275 70  0000 C CNN
 F 2 "Molex_SD-64333-100_on_Cinch_ModICE_w_5554_SOM" H 7825 5275 60  0001 C CNN
