File: KICAD_Project/sub_circuits/amp_connector.sch (KiCad schematic (older format))
At the start: 1 part, among them J301 MOLEX_HARNESS_SD-64333-100

Commit message: corrected con2 1-4 arrangement, updated SOM pin out, made draft attempt at ball park placement of critical components.
Signed-off-by: Jared Harvey <TortiseGIT@jaredharvey.com>
Parts:
- J301: footprint Molex_SD-64333-100_on_Cinch_ModICE_w_5554_SOM -> Molex_SD-64333-100_on_Cinch_ModICE_w_5554_SOM_con-only
Connections:
- wire segments 6 -> 5

Commit message: updated harness pin out per layout preferences
Signed-off-by: Jared Harvey <TortiseGIT@jaredharvey.com>
Changed lines of the file:
@@
-EESchema Schematic File Version 2  date 8/21/2011 9:23:44 AM
+EESchema Schematic File Version 2  date 8/21/2011 7:46:53 PM
 LIBS:power
 LIBS:device
@@
 Text HLabel 8225 3975 2    60   Input ~ 0
 INJ18_HARN
-Text HLabel 9425 5275 2    60   Input ~ 0
+Text HLabel 9425 5375 2    60   Input ~ 0
 12V_ECU
 Text HLabel 9425 5175 2    60   Input ~ 0
@@
 Text HLabel 8225 3675 2    60   Input ~ 0
 GND4_STAGED8
-Text HLabel 6225 5275 0    60   Input ~ 0
+Text HLabel 9425 5475 2    60   Input ~ 0
 STEP_GND
 Text Label 8875 5825 0    60   ~ 0
 GND
-Text HLabel 7425 5575 0    60   Input ~ 0
+Text HLabel 6225 5475 0    60   Input ~ 0
 CRANK+
 Text HLabel 7425 5275 0    60   Input ~ 0
@@
 Text HLabel 8225 4975 2    60   Input ~ 0
 P04
-Text HLabel 8225 5375 2    60   Input ~ 0
+Text HLabel 8225 5275 2    60   Input ~ 0
 232_TX
+Text HLabel 9425 5275 2    60   Input ~ 0
+232_RX
+Text HLabel 7425 5575 0    60   Input ~ 0
+STEP_S1
 Text HLabel 8225 5475 2    60   Input ~ 0
-232_RX
-Text HLabel 6225 5075 0    60   Input ~ 0
-STEP_S1
-Text HLabel 6225 5175 0    60   Input ~ 0
 STEP_S4
-Text HLabel 6225 5375 0    60   Input ~ 0
+Text HLabel 8225 5575 2    60   Input ~ 0
 STEP_D5
-Text HLabel 6225 5475 0    60   Input ~ 0
+Text HLabel 9425 5575 2    60   Input ~ 0
 STEP_D8
 Text HLabel 7425 3675 0    60   Input ~ 0
@@
 Text HLabel 8225 4075 2    60   Input ~ 0
 RPM_RF-
-Text HLabel 8225 5275 2    60   Input ~ 0
+Text HLabel 8225 5375 2    60   Input ~ 0
 MIL_LS-1A
 Text HLabel 6225 5575 0    60   Input ~ 0
@@
 Text HLabel 8225 4175 2    60   Input ~ 0
 RPM_RF+
-Text HLabel 9425 5575 2    60   Input ~ 0
+Text HLabel 6225 5275 0    60   Input ~ 0
 CAM+
-Text HLabel 8225 5575 2    60   Input ~ 0
+Text HLabel 6225 5375 0    60   Input ~ 0
 CAM-
 Text HLabel 8225 5175 2    60   Input ~ 0
@@
 Text HLabel 6225 5875 0    60   Input ~ 0
 INJ04_HARN
-Text HLabel 9425 5475 2    60   Input ~ 0
+Text HLabel 6225 5175 0    60   Input ~ 0
 CANL
-Text HLabel 9425 5375 2    60   Input ~ 0
+Text HLabel 6225 5075 0    60   Input ~ 0
 CANH
 Text HLabel 6225 4275 0    60   Input ~ 0

Commit message: Changed over voltage protected MOSFETs to SO8 footprints.
Signed-off-by: Jared Harvey <TortiseGIT@jaredharvey.com>
Changed lines of the file:
@@
-EESchema Schematic File Version 2  date 8/30/2011 5:58:28 AM
+EESchema Schematic File Version 2  date 9/1/2011 7:35:06 PM
 LIBS:power
 LIBS:device
@@
 Sheet 3 13
 Title "freeEMS PLUS from Cinch template "
-Date "30 aug 2011"
+Date "1 sep 2011"
 Rev "A-DRAF"
 Comp "diyefi.org/openecu.info"
@@
 $EndDescr
 Wire Wire Line
-	6225 3700 6225 3675
-Wire Wire Line
-	8225 5775 8225 5825
-Wire Wire Line
-	8225 5825 8875 5825
+	9425 3700 9425 3675
 Wire Wire Line
 	6200 5825 6225 5825
 Wire Wire Line
 	6225 5825 6225 5775
+Wire Wire Line
+	7160 5820 7425 5820
+Wire Wire Line
+	7425 5820 7425 5775
 $Comp
 L MOLEX_HARNESS_SD-64333-100 J301
@@
 	0    -1   -1   0
 $EndComp
-Text Label 6225 3700 2    60   ~ 0
+Text Label 9425 3700 0    60   ~ 0
 GND
 Text HLabel 9425 6425 2    60   Input ~ 0
@@
 Text Label 6200 5825 2    60   ~ 0
 GND
-Text HLabel 8225 6925 2    60   Input ~ 0
+Text HLabel 7425 6925 0    60   Input ~ 0
 GND5_STAGED4
-Text HLabel 8225 3675 2    60   Input ~ 0
+Text HLabel 7425 3675 0    60   Input ~ 0
 GND4_STAGED8
 Text HLabel 9425 5475 2    60   Input ~ 0
 STEP_GND
-Text Label 8875 5825 0    60   ~ 0
+Text Label 7160 5820 2    60   ~ 0
 GND
 Text HLabel 6225 5475 0    60   Input ~ 0
@@
 Text HLabel 9425 5575 2    60   Input ~ 0
 STEP_D8
-Text HLabel 7425 3675 0    60   Input ~ 0
+Text HLabel 8225 3675 2    60   Input ~ 0
 GND2_INJIGN
 Text HLabel 8225 6525 2    60   Input ~ 0
@@
 Text HLabel 7425 5375 0    60   Input ~ 0
 TPS_SIG
-Text HLabel 8225 5775 2    60   Input ~ 0
+Text HLabel 7425 5775 0    60   Input ~ 0
 GND
 Text HLabel 9425 5775 2    60   Input ~ 0
 12V_BAT
-Text HLabel 7425 6925 0    60   Input ~ 0
+Text HLabel 8225 6925 2    60   Input ~ 0
 GND3_INJIGN
 Text HLabel 9425 5075 2    60   Input ~ 0
@@
 Text HLabel 7425 3975 0    60   Input ~ 0
 INJ19_HARN
-Text HLabel 7425 5775 0    60   Input ~ 0
+Text HLabel 8225 5775 2    60   Input ~ 0
 GND1_INJIGN
 Text HLabel 9425 6825 2    60   Input ~ 0
@@
 Text HLabel 7425 5075 0    60   Input ~ 0
 ENG_TEMP
-Text HLabel 9425 3675 2    60   Input ~ 0
+Text HLabel 6225 3675 0    60   Input ~ 0
 EXTRA
 $EndSCHEMATC
