File: KICAD_Project/sub_circuits/amp_connector.sch (KiCad schematic (older format))
At the start: 1 part, among them J301 MOLEX_HARNESS_SD-64333-100

Commit message: changed stepper from L297 to A4988 from pololu
Signed-off-by: Jared Harvey <TortiseGIT@jaredharvey.com>
Connections:
- net labels added: STEP_1A, STEP_1B, STEP_2B
- net labels removed: STEP_D5, STEP_D8, STEP_S1, STEP_S4
Changed lines of the file:
@@
-EESchema Schematic File Version 2  date 9/27/2011 11:45:22 AM
+EESchema Schematic File Version 2  date 10/2/2011 8:46:35 AM
 LIBS:power
 LIBS:device
@@
 $Descr A 11000 8500
 encoding utf-8
-Sheet 3 13
+Sheet 3 12
 Title "freeEMS PLUS from Cinch template "
-Date "27 sep 2011"
+Date "2 oct 2011"
 Rev "A-DRAFT5"
 Comp "diyefi.org/openecu.info"
@@
 232_RX
 Text HLabel 7425 5575 0    60   Input ~ 0
-STEP_S1
+STEP_1A
 Text HLabel 8225 5475 2    60   Input ~ 0
-STEP_S4
+STEP_1B
 Text HLabel 8225 5575 2    60   Input ~ 0
-STEP_D5
+STEP_1B
 Text HLabel 9425 5575 2    60   Input ~ 0
-STEP_D8
+STEP_2B
 Text HLabel 6225 3575 0    60   Input ~ 0
 GND2_INJIGN

Commit message: Added some simulations for the AN protect lines
Signed-off-by: Jared Harvey <TortiseGIT@jaredharvey.com>
Connections:
- net labels added: STEP_2A
Changed lines of the file:
@@
-EESchema Schematic File Version 2  date 10/2/2011 8:46:35 AM
+EESchema Schematic File Version 2  date 10/4/2011 8:27:03 PM
 LIBS:power
 LIBS:device
@@
 Sheet 3 12
 Title "freeEMS PLUS from Cinch template "
-Date "2 oct 2011"
+Date "5 oct 2011"
 Rev "A-DRAFT5"
 Comp "diyefi.org/openecu.info"
@@
 Text HLabel 9425 5275 2    60   Input ~ 0
 232_RX
-Text HLabel 7425 5575 0    60   Input ~ 0
+Text HLabel 8225 5575 2    60   Input ~ 0
 STEP_1A
 Text HLabel 8225 5475 2    60   Input ~ 0
 STEP_1B
-Text HLabel 8225 5575 2    60   Input ~ 0
-STEP_1B
 Text HLabel 9425 5575 2    60   Input ~ 0
+STEP_2A
+Text HLabel 7425 5575 0    60   Input ~ 0
 STEP_2B
 Text HLabel 6225 3575 0    60   Input ~ 0

Commit message: Made more progress on the AN protects and LS drive 33800
Signed-off-by: Jared Harvey <TortiseGIT@jaredharvey.com>
Changed lines of the file:
@@
-EESchema Schematic File Version 2  date 10/14/2011 5:26:21 AM
+EESchema Schematic File Version 2  date 10/16/2011 7:32:21 AM
 LIBS:power
 LIBS:device
@@
 Sheet 3 12
 Title "Open5xxxECU (o5e), an ECU that is no longer affiliated with freeEMS."
-Date "14 oct 2011"
+Date "16 oct 2011"
 Rev "A-DRAFT5"
 Comp "http://open5xxxecu.org/"
@@
 Text Label 7425 3700 2    60   ~ 0
 GND
-Text HLabel 9425 6425 2    60   Input ~ 0
+Text HLabel 7425 6425 0    60   Input ~ 0
 P09
+Text HLabel 8225 6325 2    60   Input ~ 0
+P05
+Text HLabel 6225 6425 0    60   Input ~ 0
+P10
+Text HLabel 7425 6325 0    60   Input ~ 0
+P06
+Text HLabel 7425 6625 0    60   Input ~ 0
+P13
+Text HLabel 7425 6525 0    60   Input ~ 0
+P11
+Text HLabel 6225 6325 0    60   Input ~ 0
+P07
 Text HLabel 9425 6325 2    60   Input ~ 0
-P05
+MISC_1A
 Text HLabel 8225 6425 2    60   Input ~ 0
-P10
-Text HLabel 8225 6325 2    60   Input ~ 0
-P06
-Text HLabel 7425 6525 0    60   Input ~ 0
-P13
-Text HLabel 7425 6425 0    60   Input ~ 0
-P11
-Text HLabel 7425 6325 0    60   Input ~ 0
-P07
-Text HLabel 6225 6625 0    60   Input ~ 0
-MISC_1A
-Text HLabel 6225 6325 0    60   Input ~ 0
 P08
 Text HLabel 9425 6725 2    60   Input ~ 0
@@
 Text HLabel 8225 6525 2    60   Input ~ 0
 FLEX_CAN_L
-Text HLabel 6225 6525 0    60   Input ~ 0
+Text HLabel 6225 6625 0    60   Input ~ 0
 P14
-Text HLabel 9425 6525 2    60   Input ~ 0
+Text HLabel 8225 6625 2    60   Input ~ 0
 FLEX_CAN_H
 Text HLabel 8225 3975 2    60   Input ~ 0
@@
 Text HLabel 9425 4075 2    60   Input ~ 0
 RPM_LB-
-Text HLabel 7425 6625 0    60   Input ~ 0
+Text HLabel 9425 6425 2    60   Input ~ 0
 PUMP_LS-1A
 Text HLabel 9425 4175 2    60   Input ~ 0
@@
 Text HLabel 9425 3975 2    60   Input ~ 0
 RPM_RB+
-Text HLabel 6225 6425 0    60   Input ~ 0
+Text HLabel 6225 6525 0    60   Input ~ 0
 P12
 Text HLabel 8225 4175 2    60   Input ~ 0
@@
 Text HLabel 6225 4275 0    60   Input ~ 0
 O2_UN2
-Text HLabel 8225 6625 2    60   Input ~ 0
+Text HLabel 9425 6525 2    60   Input ~ 0
 O2_HD2_PWR
 Text HLabel 7425 4275 0    60   Input ~ 0
