File: KICAD_Project/sub_circuits/efi-drivers_sub_circuits.sch (KiCad schematic (older format))
At the start: 0 parts

Commit message: I did a fiar bit of work, and I want to be able to step back if I can, so this is a misc check in.
Signed-off-by: Jared Harvey <TortiseGIT@jaredharvey.com>
Parts:
- added C? (x8): CP1, symbol CP1
- added Q? (x24): IRGS14C40L, DPAK2, symbol IRGS14C40L
- added R? (x24): 1K, SM0805, symbol R
- added U? (x4): TCMT410, symbol TCMT410
- added U? (x4): 7805, symbol 7805
Connections:
- net labels added: 12v_bat, EFI_OUT0-0, EFI_OUT0-1, EFI_OUT0-2, EFI_OUT0-3, EFI_OUT1-0, EFI_OUT1-1, EFI_OUT1-2, EFI_OUT1-3, EFI_OUT2-0, EFI_OUT2-1, EFI_OUT2-2, EFI_OUT2-3, EFI_OUT3-0, EFI_OUT3-1, EFI_OUT3-2, EFI_OUT3-3, EFI_OUT4-0, EFI_OUT4-1, EFI_OUT4-2, EFI_OUT4-3, EFI_OUT5-0, EFI_OUT5-1, EFI_OUT5-2, EFI_OUT5-3, EFI_SIG0-0, EFI_SIG0-1, EFI_SIG0-2, EFI_SIG0-3, EFI_SIG1-0, EFI_SIG1-1, EFI_SIG1-2, EFI_SIG1-3, EFI_SIG2-0, EFI_SIG2-1, EFI_SIG2-2, EFI_SIG2-3, EFI_SIG3-0, EFI_SIG3-1, EFI_SIG3-2, EFI_SIG3-3, EFI_SIG4-0, EFI_SIG4-1, EFI_SIG4-2, EFI_SIG4-3, EFI_SIG5-0, EFI_SIG5-1, EFI_SIG5-2, EFI_SIG5-3, GND, GND0_4, GND1_4, GND2_4, GND3_4, GND4_1, GND5_4
- wire segments 0 -> 234

Commit message: Started laying out the harness in DXF, initial schematic capture complete, except for harness.
Signed-off-by: Jared Harvey <TortiseGIT@jaredharvey.com>
Parts:
- removed C? (x8): CP1, symbol CP1
- removed Q? (x24): IRGS14C40L, DPAK2, symbol IRGS14C40L
- removed R? (x24): 1K, SM0805, symbol R
- removed U? (x4): TCMT410, symbol TCMT410
- removed U? (x4): 7805, symbol 7805
- added C? (x18): 1uF, SM0805, symbol CP1
- added Q? (x36): IRGS14C40L, DPAK2, symbol IRGS14C40L
- added R? (x72): 0R, SM0805, symbol R
- added R? (x36): 100K, SM0805, symbol R
- added R? (x72): 1K, SM0805, symbol R
- added U? (x36): VO1400, symbol VO1400
- added U? (x9): 7805, symbol 7805
Connections:
- net labels added: GND_IGN1, IGN_OUT0-0, IGN_OUT0-1, IGN_OUT0-2, IGN_OUT0-3, IGN_OUT1-0, IGN_OUT1-1, IGN_OUT1-2, IGN_OUT1-3, IGN_OUT2-0, IGN_OUT2-1, IGN_OUT2-2, IGN_OUT2-3, IGN_SIG0-0, IGN_SIG0-1, IGN_SIG0-2, IGN_SIG0-3, IGN_SIG1-0, IGN_SIG1-1, IGN_SIG1-2, IGN_SIG1-3, IGN_SIG2-0, IGN_SIG2-1, IGN_SIG2-2, IGN_SIG2-3
- wire segments 234 -> 594
Other:
- note added: "IGNITION"
- note added: "INJECTION"

Commit message: About to runs scripts to scrub the BOM's, so here's a backup copy in case it goes wrong.
Signed-off-by: Jared Harvey <TortiseGIT@jaredharvey.com>
Parts:
- removed U? (x35): VO1400, symbol VO1400
- removed U? (x8): 7805, symbol 7805
- added U202, U203, U204, U205, U206, U210, U211, U212, U213, U214, U215, U216, U217, U218, U219, U220, U221, U225, U226, U227, U228, U229, U230, U231, U232, U233, U234, U235, U236, U240, U241, U242, U243, U244, U245: VO1400, relay-SOP04, symbol VO1400
- added U208, U209, U222, U223, U224, U237, U238, U239: LP2951, MSOP_8, symbol 7805
- U201: renamed from U?; footprint (none) -> relay-SOP04; mfg # VO1400AEFTR -> SFH690ABT; sm vend 1 newark -> digi; sm vend 1 # 46M5888 -> 751-1367-2-ND
- U207: renamed from U?; value 7805 -> LP2951; footprint (none) -> MSOP_8; MFG # LP2951CM/NOPB -> LP2951CMM/NOPB; VEND1 NEWARK -> digi; VEND1 # 26K2433 -> LP2951CMMCT-ND
- gave numbers to parts that had none: 234
Connections:
- net labels added: GND0, GND1, GND2, GND3
- net labels removed: GND0_4, GND1_4, GND2_4, GND3_4, GND4_1, GND5_4, GND_IGN1

Commit message: Looks like the bulk components are golden now, there are still a couple straglers, mostly switch mode power supply stuff.
Signed-off-by: Jared Harvey <TortiseGIT@jaredharvey.com>
Parts:
- R201, R202, R203, R210, R211, R212, R219, R220, R221, R222, R223, R224, R237, R238, R239, R240, R241, R242, R249, R250, R251, R258, R259, R260, R261, R262, R263, R270, R271, R272, R279, R280, R281, R282, R283, R284, R297, R298, R299, R300, R301, R302, R309, R310, R311, R318, R319, R320, R321, R322, R323, R330, R331, R332, R339, R340, R341, R342, R343, R344, R357, R358, R359, R360, R361, R362, R369, R370, R371, R378, R379, R380: construct Thick film -> thick film; mfg Rohm Semiconductor -> (none); mfg # MCR10EZPF1001 -> (none); mfg,mfg# (none) -> vishay,CRCW08051K00FKTA; power .125w -> (none); sm vend1 digi -> (none); sm vend1 # RHM1.00KCRCT-ND -> (none); tolerance 5% -> 1%; vend1,vend1# (none) -> newark,05F1507; w (none) -> 125mW
- R204, R205, R206, R207, R208, R209, R213, R214, R215, R216, R217, R218, R243, R244, R245, R246, R247, R248, R252, R253, R254, R255, R256, R257, R264, R265, R266, R267, R268, R269, R273, R274, R275, R276, R277, R278, R303, R304, R305, R306, R307, R308, R312, R313, R314, R315, R316, R317, R324, R325, R326, R327, R328, R329, R333, R334, R335, R336, R337, R338, R363, R364, R365, R366, R367, R368, R372, R373, R374, R375, R376, R377: mfg vishay -> (none); mfg # CRCW08050000Z0EA -> (none); mfg,mfg# (none) -> vishay,CRCW08050000Z0EA; misc (none) -> other,more,stuff; tolerance (none) -> %; vend1 newark -> (none); vend1 # 52K9721 -> (none); vend1,vend1# (none) -> newark,52K9721; w (none) -> mW
- R225, R226, R227, R228, R229, R230, R231, R232, R233, R234, R235, R236, R285, R286, R287, R288, R289, R290, R291, R292, R293, R294, R295, R296, R345, R346, R347, R348, R349, R350, R351, R352, R353, R354, R355, R356: construct Thick film -> thick film; mfg Rohm Semiconductor -> (none); mfg,mfg# (none) -> vishay,CRCW0805100KFKEA; power .125w -> (none); sm vend1 digi -> (none); tolerance 5% -> 1%; vend1,vend1# (none) -> newark,52K9808; w (none) -> 125mW

Commit message: harness connector is much more ironed out now. CPU is not connected.
Signed-off-by: Jared Harvey <TortiseGIT@jaredharvey.com>
Connections:
- net labels added: GND4, GND5
- net labels removed: GND0
- wire segments 594 -> 597

Commit message: several pins on the SOM are now connected.
Signed-off-by: Jared Harvey <TortiseGIT@jaredharvey.com>
Parts:
- renumbered C201 to C501, C202 to C502, C203 to C503, C204 to C504, C205 to C505, C206 to C506, C207 to C507, C208 to C508, C209 to C509, C210 to C510, C211 to C511, C212 to C512, C213 to C513, C214 to C514, C215 to C515, C216 to C516, C217 to C517, C218 to C518, Q201 to Q501, Q202 to Q502, Q203 to Q503, Q204 to Q504, Q205 to Q505, Q206 to Q506, Q207 to Q507, Q208 to Q508, Q209 to Q509, Q210 to Q510, Q211 to Q511, Q212 to Q512, Q213 to Q513, Q214 to Q514, Q215 to Q515, Q216 to Q516, Q217 to Q517, Q218 to Q518, Q219 to Q519, Q220 to Q520, Q221 to Q521, Q222 to Q522, Q223 to Q523, Q224 to Q524, Q225 to Q525, Q226 to Q526, Q227 to Q527, Q228 to Q528, Q229 to Q529, Q230 to Q530, Q231 to Q531, Q232 to Q532, Q233 to Q533, Q234 to Q534, Q235 to Q535, Q236 to Q536, R201 to R501, R202 to R502, R203 to R503, R204 to R504, R205 to R505, R206 to R506, R207 to R507, R208 to R508, R209 to R509, R210 to R510, R211 to R511, R212 to R512, R213 to R513, R214 to R514, R215 to R515, R216 to R516, R217 to R517, R218 to R518, R219 to R519, R220 to R520, R221 to R521, R222 to R522, R223 to R523, R224 to R524, R225 to R525, R226 to R526, R227 to R527, R228 to R528, R229 to R529, R230 to R530, R231 to R531, R232 to R532, R233 to R533, R234 to R534, R235 to R535, R236 to R536, R237 to R537, R238 to R538, R239 to R539, R240 to R540, R241 to R541, R242 to R542, R243 to R543, R244 to R544, R245 to R545, R246 to R546, R247 to R547, R248 to R548, R249 to R549, R250 to R550, R251 to R551, R252 to R552, R253 to R553, R254 to R554, R255 to R555, R256 to R556, R257 to R557, R258 to R558, R259 to R559, R260 to R560, R261 to R561, R262 to R562, R263 to R563, R264 to R564, R265 to R565, R266 to R566, R267 to R567, R268 to R568, R269 to R569, R270 to R570, R271 to R571, R272 to R572, R273 to R573, R274 to R574, R275 to R575, R276 to R576, R277 to R577, R278 to R578, R279 to R579, R280 to R580, R281 to R581, R282 to R582, R283 to R583, R284 to R584, R285 to R585, R286 to R586, R287 to R587, R288 to R588, R289 to R589, R290 to R590, R291 to R591, R292 to R592, R293 to R593, R294 to R594, R295 to R595, R296 to R596, R297 to R597, R298 to R598, R299 to R599, R300 to R600, R301 to R601, R302 to R602, R303 to R603, R304 to R604, R305 to R605, R306 to R606, R307 to R607, R308 to R608, R309 to R609, R310 to R610, R311 to R611, R312 to R612, R313 to R613, R314 to R614, R315 to R615, R316 to R616, R317 to R617, R318 to R618, R319 to R619, R320 to R620, R321 to R621, R322 to R622, R323 to R623, R324 to R624, R325 to R625, R326 to R626, R327 to R627, R328 to R628, R329 to R629, R330 to R630, R331 to R631, R332 to R632, R333 to R633, R334 to R634, R335 to R635, R336 to R636, R337 to R637, R338 to R638, R339 to R639, R340 to R640, R341 to R641, R342 to R642, R343 to R643, R344 to R644, R345 to R645, R346 to R646, R347 to R647, R348 to R648, R349 to R649, R350 to R650, R351 to R651, R352 to R652, R353 to R653, R354 to R654, R355 to R655, R356 to R656, R357 to R657, R358 to R658, R359 to R659, R360 to R660, R361 to R661, R362 to R662, R363 to R663, R364 to R664, R365 to R665, R366 to R666, R367 to R667, R368 to R668, R369 to R669, R370 to R670, R371 to R671, R372 to R672, R373 to R673, R374 to R674, R375 to R675, R376 to R676, R377 to R677, R378 to R678, R379 to R679, R380 to R680, U201 to U501, U202 to U502, U203 to U503, U204 to U504, U205 to U505, U206 to U506, U207 to U507, U208 to U508, U209 to U509, U210 to U510, U211 to U511, U212 to U512, U213 to U513, U214 to U514, U215 to U515, U216 to U516, U217 to U517, U218 to U518, U219 to U519, U220 to U520, U221 to U521, U222 to U522, U223 to U523, U224 to U524, U225 to U525, U226 to U526, U227 to U527, U228 to U528, U229 to U529, U230 to U530, U231 to U531, U232 to U532, U233 to U533, U234 to U534, U235 to U535, U236 to U536, U237 to U537, U238 to U538, U239 to U539, U240 to U540, U241 to U541, U242 to U542, U243 to U543, U244 to U544, U245 to U545
