File: KICAD_Project/sub_circuits/efi-drivers_sub_circuits.sch (KiCad schematic (older format))
At the start: 279 parts, among them Q501 IRGS14C40L, Q502 IRGS14C40L, Q503 IRGS14C40L, Q504 IRGS14C40L, Q505 IRGS14C40L, Q506 IRGS14C40L, Q507 IRGS14C40L, Q508 IRGS14C40L, Q509 IRGS14C40L, Q510 IRGS14C40L, Q511 IRGS14C40L, Q512 IRGS14C40L, Q513 IRGS14C40L, Q514 IRGS14C40L, Q515 IRGS14C40L, Q516 IRGS14C40L, Q517 IRGS14C40L, Q518 IRGS14C40L, Q519 IRGS14C40L, Q520 IRGS14C40L, Q521 IRGS14C40L, Q522 IRGS14C40L, Q523 IRGS14C40L, Q524 IRGS14C40L, Q525 IRGS14C40L, Q526 IRGS14C40L, Q527 IRGS14C40L, Q528 IRGS14C40L, Q529 IRGS14C40L, Q530 IRGS14C40L, Q531 IRGS14C40L, Q532 IRGS14C40L, Q533 IRGS14C40L, Q534 IRGS14C40L, Q535 IRGS14C40L, Q536 IRGS14C40L, U501 VO1400, U502 VO1400, U503 VO1400, U504 VO1400, U505 VO1400, U506 VO1400, U507 LP2951, U508 LP2951, U509 LP2951, U510 VO1400, U511 VO1400, U512 VO1400, U513 VO1400, U514 VO1400, U515 VO1400, U516 VO1400, U517 VO1400, U518 VO1400, U519 VO1400, U520 VO1400, U521 VO1400, U522 LP2951, U523 LP2951, U524 LP2951, U525 VO1400, U526 VO1400, U527 VO1400, U528 VO1400, U529 VO1400, U530 VO1400, U531 VO1400, U532 VO1400, U533 VO1400, U534 VO1400, U535 VO1400, U536 VO1400, U537 LP2951, U538 LP2951, U539 LP2951, U540 VO1400, U541 VO1400, U542 VO1400, U543 VO1400, U544 VO1400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

Commit message: routing has started
Signed-off-by: Jared Harvey <TortiseGIT@jaredharvey.com>
Parts:
- removed U507, U508, U509, U522, U523, U524, U537, U538, U539: LP2951, MSOP_8, symbol 7805
- added U507, U508, U509, U522, U523, U524, U537, U538, U539: LM3480, SOT23-3, symbol LM3480

Commit message: corrected con2 1-4 arrangement, updated SOM pin out, made draft attempt at ball park placement of critical components.
Signed-off-by: Jared Harvey <TortiseGIT@jaredharvey.com>
Parts:
- U501, U502, U503, U504, U505, U506, U510, U511, U512, U513, U514, U515, U516, U517, U518, U519, U520, U521, U525, U526, U527, U528, U529, U530, U531, U532, U533, U534, U535, U536, U540, U541, U542, U543, U544, U545: value VO1400 -> OPTO
Connections:
- no-connect marks 0 -> 1

Commit message: Changed over voltage protected MOSFETs to SO8 footprints.
Signed-off-by: Jared Harvey <TortiseGIT@jaredharvey.com>
Parts:
- Q501, Q502, Q503, Q504, Q505, Q506, Q507, Q508, Q509, Q510, Q511, Q512, Q513, Q514, Q515, Q516, Q517, Q518, Q519, Q520, Q521, Q522, Q523, Q524, Q525, Q526, Q527, Q528, Q529, Q530, Q531, Q532, Q533, Q534, Q535, Q536: value IRGS14C40L -> OVP_DRIVER; footprint DPAK2 -> SO8E_ST; A (none) -> 12A; OVP (none) -> 40V; construct (none) -> OVP MOSFET; mfg irf -> (none); mfg # IRGS14C40L -> (none); mfg,mfg# (none) -> ST,VNS14NV04; misc (none) -> other,more,stuff; sm vend1 digi -> (none); sm vend1 # IRGS14C40LPBF-ND -> (none); vend1,vend1# (none) -> newark,33R1503
