File: KICAD_Project/sub_circuits/efi-drivers_sub_circuits.sch (KiCad schematic (older format))
At the start: 217 parts, among them P501 CONN_1, P502 CONN_1, P503 CONN_1, P504 CONN_1, Q501 OVP_DRIVER, Q502 OVP_DRIVER, Q503 OVP_DRIVER, Q504 OVP_DRIVER, Q505 OVP_DRIVER, Q506 OVP_DRIVER, Q507 OVP_DRIVER, Q508 OVP_DRIVER, Q509 OVP_DRIVER, Q510 OVP_DRIVER, Q511 OVP_DRIVER, Q512 OVP_DRIVER, Q513 OVP_DRIVER, Q514 OVP_DRIVER, Q515 OVP_DRIVER, Q516 OVP_DRIVER, Q517 OVP_DRIVER, Q518 OVP_DRIVER, Q519 OVP_DRIVER, Q520 OVP_DRIVER, Q521 OVP_DRIVER, Q522 OVP_DRIVER, Q523 OVP_DRIVER, Q524 OVP_DRIVER, Q525 OVP_DRIVER, Q526 OVP_DRIVER, Q527 OVP_DRIVER, Q528 OVP_DRIVER, Q529 OVP_DRIVER, Q530 OVP_DRIVER, Q531 OVP_DRIVER, Q532 OVP_DRIVER, Q533 OVP_DRIVER, Q534 OVP_DRIVER, Q535 OVP_DRIVER, Q536 OVP_DRIVER, U501 OPTO, U502 OPTO, U503 OPTO, U504 OPTO, U505 OPTO, U506 OPTO, U507 LM3480, U508 LM3480, U509 LM3480, U510 OPTO, U511 OPTO, U512 OPTO, U513 OPTO, U514 OPTO, U515 OPTO, U516 OPTO, U517 OPTO, U518 OPTO, U519 OPTO, U520 OPTO, U521 OPTO, U522 LM3480, U524 LM3480, U525 OPTO, U526 OPTO, U527 OPTO, U528 OPTO, U529 OPTO, U530 OPTO, U531 OPTO, U532 OPTO, U533 OPTO, U534 OPTO, U535 OPTO, U536 OPTO, U540 OPTO, U541 OPTO, U542 OPTO, U543 OPTO, U544 OPTO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

Commit message: Added some simulations for the AN protect lines
Signed-off-by: Jared Harvey <TortiseGIT@jaredharvey.com>
Changed lines of the file:
@@
-EESchema Schematic File Version 2  date 10/2/2011 8:46:35 AM
+EESchema Schematic File Version 2  date 10/4/2011 8:27:04 PM
 LIBS:power
 LIBS:device
@@
 Sheet 5 12
 Title "freeEMS PLUS from Cinch template "
-Date "2 oct 2011"
+Date "5 oct 2011"
 Rev "A-DRAFT5"
 Comp "diyefi.org/openecu.info"
@@
 Text HLabel 8875 2850 0    60   Output ~ 0
 IGN_SIG0-0
-Text HLabel 9975 2800 0    60   Output ~ 0
+Text HLabel 9975 1300 0    60   Output ~ 0
 IGN_OUT0-0
 Text HLabel 10225 2800 2    60   Output ~ 0
@@
 Text HLabel 10225 1300 2    60   Output ~ 0
 IGN_OUT0-2
-Text HLabel 9975 1300 0    60   Output ~ 0
+Text HLabel 9975 2800 0    60   Output ~ 0
 IGN_OUT0-1
 Text HLabel 11325 1050 2    60   Output ~ 0
