File: KICAD_Project/sub_circuits/high_side_drive.sch (KiCad schematic (older format))
At the start: 28 parts

Commit message: About to runs scripts to scrub the BOM's, so here's a backup copy in case it goes wrong.
Signed-off-by: Jared Harvey <TortiseGIT@jaredharvey.com>
Parts:
- removed C?: 22nF, SM0805-C1, symbol C
- removed C?: 10uF, SM0805-C1, symbol C
- added C802: 10uF, SM0805-C1, symbol C
- added C808: 22nF, SM0805-C1, symbol C
- R801, R802, R803, R804, R805, R806, R807, R808, R809, R810, R811, R812, R813, R814: renamed from R?; footprint SM0805-R4 -> SM0805
- gave numbers to parts that had none: 12

Commit message: caps have been done with the scripts next up is the resistors.
Signed-off-by: Jared Harvey <TortiseGIT@jaredharvey.com>
Parts:
- C803: Field3 - -> (none); Field4 - -> (none); Field5 50,V -> (none); Field6 10,% -> (none); Field7 Ceramic -> (none); Field8 other,more,stuff -> (none); V (none) -> 100V; construct (none) -> ceramic; mfg,# murata,GRM21BR71H104KA01L -> (none); mfg,mfg# (none) -> avx,08051C104KAT2A; misc (none) -> other,more,stuff; tolerance (none) -> 10%; vend,# newark,38K1694 -> (none); vend1,vend1# (none) -> newark,96M1354
- C806: Field3 - -> (none); Field4 - -> (none); Field5 50,V -> (none); Field6 10,% -> (none); Field7 ceramic -> (none); Field8 other,more,stuff -> (none); V (none) -> 100V; construct (none) -> ceramic; mfg,# murata,GRM21BR71H104KA01L -> (none); mfg,mfg# (none) -> avx,08051C104KAT2A; misc (none) -> other,more,stuff; tolerance (none) -> 10%; vend,# newark,38K1694 -> (none); vend1,vend1# (none) -> newark,96M1354
Changed lines of the file:
@@
-EESchema Schematic File Version 2  date 8/14/2011 3:32:15 PM
+EESchema Schematic File Version 2  date 8/14/2011 7:31:25 PM
 LIBS:power
 LIBS:device
@@
 F 0 "C806" V 10125 5600 50  0000 L CNN
 F 1 "100nF" V 10050 5575 50  0000 L CNN
-F 2 "SM0805-C1" V 7180 7000 60  0001 C CNN
-F 4 "murata,GRM21BR71H104KA01L " V 7180 7000 60  0001 C CNN "mfg,#"
-F 5 "newark,38K1694" V 7180 7000 60  0001 C CNN "vend,#"
-F 6 "-" V 7180 7000 60  0001 C CNN "Field3"
-F 7 "-" V 7180 7000 60  0001 C CNN "Field4"
-F 8 "50,V" V 7180 7000 60  0001 C CNN "Field5"
-F 9 "10,%" V 7180 7000 60  0001 C CNN "Field6"
-F 10 "ceramic" V 7180 7000 60  0001 C CNN "Field7"
-F 11 "other,more,stuff" V 7180 7000 60  0001 C CNN "Field8"
+F 2 "SM0805-C1" V 1130 2600 60  0001 C CNN
+F 4 "avx,08051C104KAT2A" V 1130 2600 60  0001 C CNN "mfg,mfg#"
+F 5 "newark,96M1354" V 1130 2600 60  0001 C CNN "vend1,vend1#"
+F 6 "" V 1130 2600 60  0001 C CNN ""
+F 7 "" V 1130 2600 60  0001 C CNN ""
+F 8 "100V" V 1130 2600 60  0001 C CNN "V"
+F 9 "10%" V 1130 2600 60  0001 C CNN "tolerance"
+F 10 "ceramic" V 1130 2600 60  0001 C CNN "construct"
+F 11 "other,more,stuff" V 1130 2600 60  0001 C CNN "misc"
 	1    10100 5900
 	0    -1   -1   0
@@
 F 0 "C803" V 8750 6350 50  0000 L CNN
 F 1 "100nF" V 8675 5825 50  0000 L CNN
-F 2 "SM0805-C1" V 5780 7275 60  0001 C CNN
-F 4 "murata,GRM21BR71H104KA01L" V 5780 7275 60  0001 C CNN "mfg,#"
-F 5 "newark,38K1694" V 5780 7275 60  0001 C CNN "vend,#"
-F 6 "-" V 5780 7275 60  0001 C CNN "Field3"
-F 7 "-" V 5780 7275 60  0001 C CNN "Field4"
-F 8 "50,V" V 5780 7275 60  0001 C CNN "Field5"
-F 9 "10,%" V 5780 7275 60  0001 C CNN "Field6"
-F 10 "Ceramic" V 5780 7275 60  0001 C CNN "Field7"
-F 11 "other,more,stuff" V 5780 7275 60  0001 C CNN "Field8"
+F 2 "SM0805-C1" V 1130 2600 60  0001 C CNN
+F 4 "avx,08051C104KAT2A" V 1130 2600 60  0001 C CNN "mfg,mfg#"
+F 5 "newark,96M1354" V 1130 2600 60  0001 C CNN "vend1,vend1#"
+F 6 "" V 1130 2600 60  0001 C CNN ""
+F 7 "" V 1130 2600 60  0001 C CNN ""
+F 8 "100V" V 1130 2600 60  0001 C CNN "V"
+F 9 "10%" V 1130 2600 60  0001 C CNN "tolerance"
+F 10 "ceramic" V 1130 2600 60  0001 C CNN "construct"
+F 11 "other,more,stuff" V 1130 2600 60  0001 C CNN "misc"
 	1    8700 6175
 	0    1    1    0

Commit message: Looks like the bulk components are golden now, there are still a couple straglers, mostly switch mode power supply stuff.
Signed-off-by: Jared Harvey <TortiseGIT@jaredharvey.com>
Parts:
- R801: Field3 - -> (none); Field4 - -> (none); Field5 125,mW -> (none); Field6 1,% -> (none); Field7 ? film -> (none); Field8 other,more,stuff -> (none); construct (none) -> thin film; mfg,# -,- -> (none); mfg,mfg# (none) -> vishay,TNPW08052K49BEEA; misc (none) -> other,more,stuff; tolerance (none) -> .1%; vend,# -,- -> (none); vend1,vend1# (none) -> newark,05R1646; w (none) -> 125mW
- R802, R805, R806, R807: Field3 - -> (none); Field4 - -> (none); Field5 125,mW -> (none); Field6 1,% -> (none); Field7 thick film -> (none); Field8 other,more,stuff -> (none); construct (none) -> thick film; mfg,# bourns,CR0805-FX-1003ELF -> (none); mfg,mfg# (none) -> vishay,CRCW0805100KFKEA; misc (none) -> other,more,stuff; tolerance (none) -> 1%; vend,# newark,32K2766 -> (none); vend1,vend1# (none) -> newark,52K9808; w (none) -> 125mW
- R803, R804: Field3 - -> (none); Field4 - -> (none); Field5 125,mW -> (none); Field6 1,% -> (none); Field7 carbon film -> (none); Field8 other,more,stuff -> (none); construct (none) -> thick film; mfg,# bourns,CR0805-FX-1003ELF -> (none); mfg,mfg# (none) -> vishay,CRCW0805100KFKEA; misc (none) -> other,more,stuff; tolerance (none) -> 1%; vend,# newark,32K2766 -> (none); vend1,vend1# (none) -> newark,52K9808; w (none) -> 125mW
- R808, R809: Field3 - -> (none); Field4 - -> (none); Field5 125,mW -> (none); Field6 1,% -> (none); Field7 thick film -> (none); Field8 other,more,stuff -> (none); construct (none) -> thick film; mfg,# bourns,CR0805-FX-1002ELF -> (none); mfg,mfg# (none) -> BOURNS,CR0805-FX-1002ELF; misc (none) -> other,more,stuff; tolerance (none) -> 1%; vend,# newark,02J2368 -> (none); vend1,vend1# (none) -> newark,02J2368; w (none) -> 125mW
- R810, R811, R812, R814: Field3 - -> (none); Field4 - -> (none); Field5 125,mW -> (none); Field6 -,% -> (none); Field7 na -> (none); Field8 other,more,stuff -> (none); mfg,# vishay,CRCW08050000ZSTA -> (none); mfg,mfg# (none) -> vishay,CRCW08050000Z0EA; misc (none) -> other,more,stuff; tolerance (none) -> %; vend,# newark,36C9353 -> (none); vend1,vend1# (none) -> newark,52K9721; w (none) -> mW
- R813: Field3 - -> (none); Field4 - -> (none); Field5 ?,mW -> (none); Field6 ?,% -> (none); Field7 ? film -> (none); Field8 other,more,stuff -> (none); construct (none) -> thick film; mfg,# -,- -> (none); mfg,mfg# (none) -> vishay,CRCW08056K65FKEA; misc (none) -> other,more,stuff; tolerance (none) -> 1%; vend,# -,- -> (none); vend1,vend1# (none) -> newark,53K0371; w (none) -> 125mW

Commit message: harness connector is much more ironed out now. CPU is not connected.
Signed-off-by: Jared Harvey <TortiseGIT@jaredharvey.com>
Other:
- moved on the sheet: C801, C802, C803, C804, C805, C806, C807, C808, C809, R801, R802, R803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

Commit message: several pins on the SOM are now connected.
Signed-off-by: Jared Harvey <TortiseGIT@jaredharvey.com>
Parts:
- renumbered C801 to C901, C802 to C902, C803 to C903, C804 to C904, C805 to C905, C806 to C906, C807 to C907, C808 to C908, C809 to C909, P801 to P901, P802 to P902, P803 to P903, P804 to P904, R801 to R901, R802 to R902, R803 to R903, R804 to R904, R805 to R905, R806 to R906, R807 to R907, R808 to R908, R809 to R909, R810 to R910, R811 to R911, R812 to R912, R813 to R913, R814 to R914, U801 to U901
Changed lines of the file:
@@
-EESchema Schematic File Version 2  date 8/19/2011 6:13:41 AM
+EESchema Schematic File Version 2  date 8/20/2011 7:18:56 AM
 LIBS:power
 LIBS:device
@@
 Sheet 9 13
 Title "freeEMS PLUS from Cinch template "
-Date "19 aug 2011"
+Date "20 aug 2011"
 Rev "A-DRAF"
 Comp "diyefi.org/openecu.info"
@@
 NoConn ~ 10300 4875
 $Comp
-L C C805
+L C C905
 U 1 1 4C09B5F3
 P 9900 6325
-F 0 "C805" V 9800 6500 50  0000 L CNN
+F 0 "C905" V 9800 6500 50  0000 L CNN
 F 1 "22nF" V 9800 6175 50  0000 L CNN
 F 2 "SM0805-C1" V 6980 7425 60  0001 C CNN
@@
 $EndComp
 $Comp
-L CONN_1 P802
+L CONN_1 P902
 U 1 1 4C09B5F2
 P 9700 6525
-F 0 "P802" H 9780 6525 40  0000 L CNN
+F 0 "P902" H 9780 6525 40  0000 L CNN
 F 1 "CONN_1" H 9700 6580 30  0001 C CNN
 F 2 "PINTST" V 3180 7125 60  0001 C CNN
@@
 $EndComp
 $Comp
-L C C804
+L C C904
 U 1 1 4C09B5A3
 P 9900 3925
-F 0 "C804" V 9950 4125 50  0000 L CNN
+F 0 "C904" V 9950 4125 50  0000 L CNN
 F 1 "22nF" V 9950 3775 50  0000 L CNN
 F 2 "SM0805-C1" V 6980 5025 60  0001 C CNN
@@
 $EndComp
 $Comp
-L CONN_1 P801
+L CONN_1 P901
 U 1 1 4C09B5A2
 P 9700 3725
-F 0 "P801" H 9780 3725 40  0000 L CNN
+F 0 "P901" H 9780 3725 40  0000 L CNN
 F 1 "CONN_1" H 9700 3780 30  0001 C CNN
 F 2 "PINTST" V 3180 4325 60  0001 C CNN
@@
 $EndComp
 $Comp
-L C C809
+L C C909
 U 1 1 4C09B57D
 P 10650 5325
-F 0 "C809" V 10700 5475 50  0000 L CNN
+F 0 "C909" V 10700 5475 50  0000 L CNN
 F 1 "22nF" V 10700 5175 50  0000 L CNN
 F 2 "SM0805-C1" V 7730 6425 60  0001 C CNN
@@
 $EndComp
 $Comp
-L R R805
+L R R905
 U 1 1 4C09B3BB
 P 8250 4675
-F 0 "R805" V 8200 4400 50  0000 C CNN
+F 0 "R905" V 8200 4400 50  0000 C CNN
 F 1 "100k" V 8250 4675 50  0000 C CNN
 F 2 "SM0805" V 1130 2300 60  0001 C CNN
@@
 $EndComp
 $Comp
-L R R807
+L R R907
 U 1 1 4C09B3BA
 P 8250 4875
-F 0 "R807" V 8200 4600 50  0000 C CNN
+F 0 "R907" V 8200 4600 50  0000 C CNN
 F 1 "100k" V 8250 4875 50  0000 C CNN
 F 2 "SM0805" V 1130 2300 60  0001 C CNN
@@
 $EndComp
 $Comp
-L R R808
+L R R908
 U 1 1 4C09B3B6
 P 8250 4975
-F 0 "R808" V 8200 4700 50  0000 C CNN
+F 0 "R908" V 8200 4700 50  0000 C CNN
 F 1 "10k" V 8250 4975 50  0000 C CNN
 F 2 "SM0805" V 1130 2300 60  0001 C CNN
@@
 $EndComp
 $Comp
-L C C801
+L C C901
 U 1 1 4BF942A5
 P 8300 4125
-F 0 "C801" V 8225 4300 50  0000 L CNN
+F 0 "C901" V 8225 4300 50  0000 L CNN
 F 1 "22nF" V 8225 3975 50  0000 L CNN
 F 2 "SM0805-C1" V 5380 5225 60  0001 C CNN
@@
 $EndComp
 $Comp
-L R R801
+L R R901
 U 1 1 4BF94282
 P 8250 3925
-F 0 "R801" V 8200 3600 50  0000 C CNN
+F 0 "R901" V 8200 3600 50  0000 C CNN
 F 1 "2.5k 1%" V 8250 3925 50  0000 C CNN
 F 2 "SM0805" V 1130 2300 60  0001 C CNN
@@
 $EndComp
 $Comp
-L R R802
+L R R902
 U 1 1 4BF94278
 P 8250 4275
-F 0 "R802" V 8300 4000 50  0000 C CNN
+F 0 "R902" V 8300 4000 50  0000 C CNN
 F 1 "100k" V 8250 4275 50  0000 C CNN
 F 2 "SM0805" V 1130 2300 60  0001 C CNN
@@
 3412_CSNS
 $Comp
-L R R809
+L R R909
 U 1 1 4BF9425C
 P 8250 5075
-F 0 "R809" V 8200 4800 50  0000 C CNN
+F 0 "R909" V 8200 4800 50  0000 C CNN
 F 1 "10k" V 8250 5075 50  0000 C CNN
 F 2 "SM0805" V 1130 2300 60  0001 C CNN
@@
 3412_RST
 $Comp
-L R R814
+L R R914
 U 1 1 4BF94241
 P 9000 6100
-F 0 "R814" V 9050 5825 50  0000 C CNN
+F 0 "R914" V 9050 5825 50  0000 C CNN
 F 1 "0R" V 9000 6100 50  0000 C CNN
 F 2 "SM0805" V 1130 2300 60  0001 C CNN
@@
 3412_SO
 $Comp
-L R R813
+L R R913
 U 1 1 4BF94234
 P 9000 3775
-F 0 "R813" V 8925 3500 50  0000 C CNN
+F 0 "R913" V 8925 3500 50  0000 C CNN
 F 1 "6.6k 1%" V 9000 3775 50  0000 C CNN
 F 2 "SM0805" V 1130 2300 60  0001 C CNN
@@
 3412_IN1
 $Comp
-L R R804
+L R R904
 U 1 1 4BF94215
 P 8250 4475
-F 0 "R804" V 8300 4200 50  0000 C CNN
+F 0 "R904" V 8300 4200 50  0000 C CNN
 F 1 "100k" V 8250 4475 50  0000 C CNN
 F 2 "SM0805" V 1130 2300 60  0001 C CNN
@@
 $EndComp
 $Comp
-L R R806
+L R R906
 U 1 1 4BF94213
 P 8250 4775
-F 0 "R806" V 8200 4500 50  0000 C CNN
+F 0 "R906" V 8200 4500 50  0000 C CNN
 F 1 "100k" V 8250 4775 50  0000 C CNN
 F 2 "SM0805" V 1130 2300 60  0001 C CNN
@@
 3412_IN0
 $Comp
-L R R803
+L R R903
 U 1 1 4BF94207
 P 8250 4375
-F 0 "R803" V 8300 4100 50  0000 C CNN
+F 0 "R903" V 8300 4100 50  0000 C CNN
 F 1 "100k" V 8250 4375 50  0000 C CNN
 F 2 "SM0805" V 1130 2300 60  0001 C CNN
@@
 $EndComp
 $Comp
-L R R812
+L R R912
 U 1 1 4BF941B3
 P 8250 5375
-F 0 "R812" V 8200 5100 50  0000 C CNN
+F 0 "R912" V 8200 5100 50  0000 C CNN
 F 1 "0R" V 8250 5375 50  0000 C CNN
 F 2 "SM0805" V 1130 2300 60  0001 C CNN
@@
 $EndComp
 $Comp
-L R R811
+L R R911
 U 1 1 4BF941B0
 P 8250 5275
-F 0 "R811" V 8200 5000 50  0000 C CNN
+F 0 "R911" V 8200 5000 50  0000 C CNN
 F 1 "0R" V 8250 5275 50  0000 C CNN
 F 2 "SM0805" V 1130 2300 60  0001 C CNN
@@
 $EndComp
 $Comp
-L R R810
+L R R910
 U 1 1 4BF941AD
 P 8250 5175
-F 0 "R810" V 8200 4900 50  0000 C CNN
+F 0 "R910" V 8200 4900 50  0000 C CNN
 F 1 "0R" V 8250 5175 50  0000 C CNN
 F 2 "SM0805" V 1130 2300 60  0001 C CNN
@@
 $EndComp
 $Comp
-L C C807
+L C C907
 U 1 1 4BF9411C
 P 10100 5825
-F 0 "C807" V 10150 5525 50  0000 L CNN
+F 0 "C907" V 10150 5525 50  0000 L CNN
 F 1 "100uF" V 10075 5500 50  0000 L CNN
 F 2 "SM0805-C1" V 7180 6925 60  0001 C CNN
@@
 $EndComp
 $Comp
-L C C806
+L C C906
 U 1 1 4BF940FB
 P 10100 5600
-F 0 "C806" V 10125 5300 50  0000 L CNN
+F 0 "C906" V 10125 5300 50  0000 L CNN
 F 1 "100nF" V 10050 5275 50  0000 L CNN
 F 2 "SM0805-C1" V 1130 2300 60  0001 C CNN
@@
 $EndComp
 $Comp
-L C C803
+L C C903
 U 1 1 4BF94010
 P 8700 5875
-F 0 "C803" V 8750 6050 50  0000 L CNN
+F 0 "C903" V 8750 6050 50  0000 L CNN
 F 1 "100nF" V 8675 5525 50  0000 L CNN
 F 2 "SM0805-C1" V 1130 2300 60  0001 C CNN
@@
 $EndComp
 $Comp
-L MC10XS3412 U801
+L MC10XS3412 U901
 U 1 1 4BF93CA3
 P 9450 4875
-F 0 "U801" H 9450 4775 60  0000 C CNN
+F 0 "U901" H 9450 4775 60  0000 C CNN
 F 1 "MC10XS3412" H 9450 4875 50  0000 C CNN
 F 2 "PQFN_24" H 9450 4875 60  0001 C CNN
@@
 $EndComp
 $Comp
-L CONN_1 P803
+L CONN_1 P903
 U 1 1 4BF650D4
 P 10450 4225
-F 0 "P803" H 10530 4225 40  0000 L CNN
+F 0 "P903" H 10530 4225 40  0000 L CNN
 F 1 "CONN_1" H 10450 4280 30  0001 C CNN
 F 2 "PINTST" V 3930 4825 60  0001 C CNN
@@
 $EndComp
 $Comp
-L CONN_1 P804
+L CONN_1 P904
 U 1 1 4BF3BED1
 P 10450 5125
-F 0 "P804" H 10530 5125 40  0000 L CNN
+F 0 "P904" H 10530 5125 40  0000 L CNN
 F 1 "CONN_1" H 10450 5180 30  0001 C CNN
 F 2 "PINTST" V 3930 5725 60  0001 C CNN
@@
 3.3V
 $Comp
-L C C802
+L C C902
 U 1 1 4E467DF7
 P 8700 5625
-F 0 "C802" V 8625 5800 50  0000 L CNN
+F 0 "C902" V 8625 5800 50  0000 L CNN
 F 1 "10uF" V 8675 5300 50  0000 L CNN
 F 2 "SM0805-C1" V 5780 6725 60  0001 C CNN
@@
 $EndComp
 $Comp
-L C C808
+L C C908
 U 1 1 4E467DEE
 P 10650 4425
-F 0 "C808" V 10700 4525 50  0000 L CNN
+F 0 "C908" V 10700 4525 50  0000 L CNN
 F 1 "22nF" V 10700 4275 50  0000 L CNN
 F 2 "SM0805-C1" V 7730 5525 60  0001 C CNN
