File: KICAD_Project/sub_circuits/high_side_drive.sch (KiCad schematic (older format))
At the start: 28 parts, among them P901 CONN_1, P902 CONN_1, P903 CONN_1, P904 CONN_1, U901 MC10XS3412

Commit message: more stepper updates
Signed-off-by: Jared Harvey <TortiseGIT@jaredharvey.com>
Parts:
- C902: Field3 - -> (none); Field4 - -> (none); Field5 200,V -> (none); Field6 20,% -> (none); Field7 alum electro -> (none); Field8 other,more,stuff -> (none); V (none) -> 25V; construct (none) -> multi layer ceramic; mfg,# ill cap,106CKE200M -> (none); mfg,mfg# (none) -> AVX,08053C104KAT2A; misc (none) -> other,more,stuff; tolerance (none) -> 10%; vend,# newark,69K7896 -> (none); vend1,vend1# (none) -> newark,96M1381
- C907: Field3 - -> (none); Field4 - -> (none); Field5 35,V -> (none); Field6 20,% -> (none); Field7 alum electro -> (none); Field8 other,more,stuff -> (none); V (none) -> 100V; construct (none) -> ceramic; mfg,# ill cap,107CKE035M -> (none); mfg,mfg# (none) -> avx,08051C104KAT2A; misc (none) -> other,more,stuff; tolerance (none) -> 10%; vend,# newark,69K7903 -> (none); vend1,vend1# (none) -> newark,96M1354
- R902, R903, R904, R905, R906, R907: W (none) -> 125mW; w 125mW -> (none)
Changed lines of the file:
@@
-EESchema Schematic File Version 2  date 8/27/2011 10:55:18 AM
+EESchema Schematic File Version 2  date 8/30/2011 5:58:29 AM
 LIBS:power
 LIBS:device
@@
 Sheet 9 13
 Title "freeEMS PLUS from Cinch template "
-Date "27 aug 2011"
+Date "30 aug 2011"
 Rev "A-DRAF"
 Comp "diyefi.org/openecu.info"
@@
 F 0 "R905" V 8200 4400 50  0000 C CNN
 F 1 "100k" V 8250 4675 50  0000 C CNN
-F 2 "SM0805" V 1130 2300 60  0001 C CNN
-F 4 "vishay,CRCW0805100KFKEA" V 1130 2300 60  0001 C CNN "mfg,mfg#"
-F 5 "newark,52K9808" V 1130 2300 60  0001 C CNN "vend1,vend1#"
-F 6 "" V 1130 2300 60  0001 C CNN "Field6"
-F 7 "" V 1130 2300 60  0001 C CNN "Field7"
-F 8 "125mW" V 1130 2300 60  0001 C CNN "w"
-F 9 "1%" V 1130 2300 60  0001 C CNN "tolerance"
-F 10 "thick film" V 1130 2300 60  0001 C CNN "construct"
-F 11 "other,more,stuff" V 1130 2300 60  0001 C CNN "misc"
+F 2 "SM0805" V 1130 2600 60  0001 C CNN
+F 4 "vishay,CRCW0805100KFKEA" V 1130 2600 60  0001 C CNN "mfg,mfg#"
+F 5 "newark,52K9808" V 1130 2600 60  0001 C CNN "vend1,vend1#"
+F 6 "" V 1130 2600 60  0001 C CNN ""
+F 7 "" V 1130 2600 60  0001 C CNN ""
+F 8 "125mW" V 1130 2600 60  0001 C CNN "W"
+F 9 "1%" V 1130 2600 60  0001 C CNN "tolerance"
+F 10 "thick film" V 1130 2600 60  0001 C CNN "construct"
+F 11 "other,more,stuff" V 1130 2600 60  0001 C CNN "misc"
 	1    8250 4675
 	0    -1   1    0
@@
 F 0 "R907" V 8200 4600 50  0000 C CNN
 F 1 "100k" V 8250 4875 50  0000 C CNN
-F 2 "SM0805" V 1130 2300 60  0001 C CNN
-F 4 "vishay,CRCW0805100KFKEA" V 1130 2300 60  0001 C CNN "mfg,mfg#"
-F 5 "newark,52K9808" V 1130 2300 60  0001 C CNN "vend1,vend1#"
-F 6 "" V 1130 2300 60  0001 C CNN "Field6"
-F 7 "" V 1130 2300 60  0001 C CNN "Field7"
-F 8 "125mW" V 1130 2300 60  0001 C CNN "w"
-F 9 "1%" V 1130 2300 60  0001 C CNN "tolerance"
-F 10 "thick film" V 1130 2300 60  0001 C CNN "construct"
-F 11 "other,more,stuff" V 1130 2300 60  0001 C CNN "misc"
+F 2 "SM0805" V 1130 2600 60  0001 C CNN
+F 4 "vishay,CRCW0805100KFKEA" V 1130 2600 60  0001 C CNN "mfg,mfg#"
+F 5 "newark,52K9808" V 1130 2600 60  0001 C CNN "vend1,vend1#"
+F 6 "" V 1130 2600 60  0001 C CNN ""
+F 7 "" V 1130 2600 60  0001 C CNN ""
+F 8 "125mW" V 1130 2600 60  0001 C CNN "W"
+F 9 "1%" V 1130 2600 60  0001 C CNN "tolerance"
+F 10 "thick film" V 1130 2600 60  0001 C CNN "construct"
+F 11 "other,more,stuff" V 1130 2600 60  0001 C CNN "misc"
 	1    8250 4875
 	0    -1   1    0
@@
 F 0 "R902" V 8300 4000 50  0000 C CNN
 F 1 "100k" V 8250 4275 50  0000 C CNN
-F 2 "SM0805" V 1130 2300 60  0001 C CNN
-F 4 "vishay,CRCW0805100KFKEA" V 1130 2300 60  0001 C CNN "mfg,mfg#"
-F 5 "newark,52K9808" V 1130 2300 60  0001 C CNN "vend1,vend1#"
-F 6 "" V 1130 2300 60  0001 C CNN "Field6"
-F 7 "" V 1130 2300 60  0001 C CNN "Field7"
-F 8 "125mW" V 1130 2300 60  0001 C CNN "w"
-F 9 "1%" V 1130 2300 60  0001 C CNN "tolerance"
-F 10 "thick film" V 1130 2300 60  0001 C CNN "construct"
-F 11 "other,more,stuff" V 1130 2300 60  0001 C CNN "misc"
+F 2 "SM0805" V 1130 2600 60  0001 C CNN
+F 4 "vishay,CRCW0805100KFKEA" V 1130 2600 60  0001 C CNN "mfg,mfg#"
+F 5 "newark,52K9808" V 1130 2600 60  0001 C CNN "vend1,vend1#"
+F 6 "" V 1130 2600 60  0001 C CNN ""
+F 7 "" V 1130 2600 60  0001 C CNN ""
+F 8 "125mW" V 1130 2600 60  0001 C CNN "W"
+F 9 "1%" V 1130 2600 60  0001 C CNN "tolerance"
+F 10 "thick film" V 1130 2600 60  0001 C CNN "construct"
+F 11 "other,more,stuff" V 1130 2600 60  0001 C CNN "misc"
 	1    8250 4275
 	0    -1   1    0
@@
 F 0 "R904" V 8300 4200 50  0000 C CNN
 F 1 "100k" V 8250 4475 50  0000 C CNN
-F 2 "SM0805" V 1130 2300 60  0001 C CNN
-F 4 "vishay,CRCW0805100KFKEA" V 1130 2300 60  0001 C CNN "mfg,mfg#"
-F 5 "newark,52K9808" V 1130 2300 60  0001 C CNN "vend1,vend1#"
-F 6 "" V 1130 2300 60  0001 C CNN "Field6"
-F 7 "" V 1130 2300 60  0001 C CNN "Field7"
-F 8 "125mW" V 1130 2300 60  0001 C CNN "w"
-F 9 "1%" V 1130 2300 60  0001 C CNN "tolerance"
-F 10 "thick film" V 1130 2300 60  0001 C CNN "construct"
-F 11 "other,more,stuff" V 1130 2300 60  0001 C CNN "misc"
+F 2 "SM0805" V 1130 2600 60  0001 C CNN
+F 4 "vishay,CRCW0805100KFKEA" V 1130 2600 60  0001 C CNN "mfg,mfg#"
+F 5 "newark,52K9808" V 1130 2600 60  0001 C CNN "vend1,vend1#"
+F 6 "" V 1130 2600 60  0001 C CNN ""
+F 7 "" V 1130 2600 60  0001 C CNN ""
+F 8 "125mW" V 1130 2600 60  0001 C CNN "W"
+F 9 "1%" V 1130 2600 60  0001 C CNN "tolerance"
+F 10 "thick film" V 1130 2600 60  0001 C CNN "construct"
+F 11 "other,more,stuff" V 1130 2600 60  0001 C CNN "misc"
 	1    8250 4475
 	0    -1   1    0
@@
 F 0 "R906" V 8200 4500 50  0000 C CNN
 F 1 "100k" V 8250 4775 50  0000 C CNN
-F 2 "SM0805" V 1130 2300 60  0001 C CNN
-F 4 "vishay,CRCW0805100KFKEA" V 1130 2300 60  0001 C CNN "mfg,mfg#"
-F 5 "newark,52K9808" V 1130 2300 60  0001 C CNN "vend1,vend1#"
-F 6 "" V 1130 2300 60  0001 C CNN "Field6"
-F 7 "" V 1130 2300 60  0001 C CNN "Field7"
-F 8 "125mW" V 1130 2300 60  0001 C CNN "w"
-F 9 "1%" V 1130 2300 60  0001 C CNN "tolerance"
-F 10 "thick film" V 1130 2300 60  0001 C CNN "construct"
-F 11 "other,more,stuff" V 1130 2300 60  0001 C CNN "misc"
+F 2 "SM0805" V 1130 2600 60  0001 C CNN
+F 4 "vishay,CRCW0805100KFKEA" V 1130 2600 60  0001 C CNN "mfg,mfg#"
+F 5 "newark,52K9808" V 1130 2600 60  0001 C CNN "vend1,vend1#"
+F 6 "" V 1130 2600 60  0001 C CNN ""
+F 7 "" V 1130 2600 60  0001 C CNN ""
+F 8 "125mW" V 1130 2600 60  0001 C CNN "W"
+F 9 "1%" V 1130 2600 60  0001 C CNN "tolerance"
+F 10 "thick film" V 1130 2600 60  0001 C CNN "construct"
+F 11 "other,more,stuff" V 1130 2600 60  0001 C CNN "misc"
 	1    8250 4775
 	0    -1   1    0
@@
 F 0 "R903" V 8300 4100 50  0000 C CNN
 F 1 "100k" V 8250 4375 50  0000 C CNN
-F 2 "SM0805" V 1130 2300 60  0001 C CNN
-F 4 "vishay,CRCW0805100KFKEA" V 1130 2300 60  0001 C CNN "mfg,mfg#"
-F 5 "newark,52K9808" V 1130 2300 60  0001 C CNN "vend1,vend1#"
-F 6 "" V 1130 2300 60  0001 C CNN "Field6"
-F 7 "" V 1130 2300 60  0001 C CNN "Field7"
-F 8 "125mW" V 1130 2300 60  0001 C CNN "w"
-F 9 "1%" V 1130 2300 60  0001 C CNN "tolerance"
-F 10 "thick film" V 1130 2300 60  0001 C CNN "construct"
-F 11 "other,more,stuff" V 1130 2300 60  0001 C CNN "misc"
+F 2 "SM0805" V 1130 2600 60  0001 C CNN
+F 4 "vishay,CRCW0805100KFKEA" V 1130 2600 60  0001 C CNN "mfg,mfg#"
+F 5 "newark,52K9808" V 1130 2600 60  0001 C CNN "vend1,vend1#"
+F 6 "" V 1130 2600 60  0001 C CNN ""
+F 7 "" V 1130 2600 60  0001 C CNN ""
+F 8 "125mW" V 1130 2600 60  0001 C CNN "W"
+F 9 "1%" V 1130 2600 60  0001 C CNN "tolerance"
+F 10 "thick film" V 1130 2600 60  0001 C CNN "construct"
+F 11 "other,more,stuff" V 1130 2600 60  0001 C CNN "misc"
 	1    8250 4375
 	0    -1   1    0
@@
 F 0 "C907" V 10150 5525 50  0000 L CNN
 F 1 "100uF" V 10075 5500 50  0000 L CNN
-F 2 "SM0805-C1" V 7180 6925 60  0001 C CNN
-F 4 "ill cap,107CKE035M" V 7180 6925 60  0001 C CNN "mfg,#"
-F 5 "newark,69K7903" V 7180 6925 60  0001 C CNN "vend,#"
-F 6 "-" V 7180 6925 60  0001 C CNN "Field3"
-F 7 "-" V 7180 6925 60  0001 C CNN "Field4"
-F 8 "35,V" V 7180 6925 60  0001 C CNN "Field5"
-F 9 "20,%" V 7180 6925 60  0001 C CNN "Field6"
-F 10 "alum electro" V 7180 6925 60  0001 C CNN "Field7"
-F 11 "other,more,stuff" V 7180 6925 60  0001 C CNN "Field8"
+F 2 "SM0805-C1" V 1130 2600 60  0001 C CNN
+F 4 "avx,08051C104KAT2A" V 1130 2600 60  0001 C CNN "mfg,mfg#"
+F 5 "newark,96M1354" V 1130 2600 60  0001 C CNN "vend1,vend1#"
+F 6 "" V 1130 2600 60  0001 C CNN ""
+F 7 "" V 1130 2600 60  0001 C CNN ""
+F 8 "100V" V 1130 2600 60  0001 C CNN "V"
+F 9 "10%" V 1130 2600 60  0001 C CNN "tolerance"
+F 10 "ceramic" V 1130 2600 60  0001 C CNN "construct"
+F 11 "other,more,stuff" V 1130 2600 60  0001 C CNN "misc"
 	1    10100 5825
 	0    -1   -1   0
@@
 F 0 "C902" V 8625 5800 50  0000 L CNN
 F 1 "10uF" V 8675 5300 50  0000 L CNN
-F 2 "SM0805-C1" V 5780 6725 60  0001 C CNN
-F 4 "ill cap,106CKE200M" V 5780 6725 60  0001 C CNN "mfg,#"
-F 5 "newark,69K7896" V 5780 6725 60  0001 C CNN "vend,#"
-F 6 "-" V 5780 6725 60  0001 C CNN "Field3"
-F 7 "-" V 5780 6725 60  0001 C CNN "Field4"
-F 8 "200,V" V 5780 6725 60  0001 C CNN "Field5"
-F 9 "20,%" V 5780 6725 60  0001 C CNN "Field6"
-F 10 "alum electro" V 5780 6725 60  0001 C CNN "Field7"
-F 11 "other,more,stuff" V 5780 6725 60  0001 C CNN "Field8"
+F 2 "SM0805-C1" V 1130 2600 60  0001 C CNN
+F 4 "AVX,08053C104KAT2A" V 1130 2600 60  0001 C CNN "mfg,mfg#"
+F 5 "newark,96M1381" V 1130 2600 60  0001 C CNN "vend1,vend1#"
+F 6 "" V 1130 2600 60  0001 C CNN ""
+F 7 "" V 1130 2600 60  0001 C CNN ""
+F 8 "25V" V 1130 2600 60  0001 C CNN "V"
+F 9 "10%" V 1130 2600 60  0001 C CNN "tolerance"
+F 10 "multi layer ceramic" V 1130 2600 60  0001 C CNN "construct"
+F 11 "other,more,stuff" V 1130 2600 60  0001 C CNN "misc"
 	1    8700 5625
 	0    1    1    0
