File: KICAD_Project/sub_circuits/high_side_drive.sch (KiCad schematic (older format))
At the start: 28 parts, among them P901 CONN_1, P902 CONN_1, P903 CONN_1, P904 CONN_1, U901 MC10XS3412

Commit message: Added some simulations for the AN protect lines
Signed-off-by: Jared Harvey <TortiseGIT@jaredharvey.com>
Parts:
- removed C908: 22nF, SM0805-C1, symbol C
- removed P901, P902, P903, P904: CONN_1, PINTST, symbol CONN_1
- C901, C902, C903, C904, C906, C907, C909: footprint SM0805-C1 -> SM0805
Connections:
- net labels removed: HS0_PIN
- wire segments 60 -> 56
- no-connect marks 2 -> 3

Commit message: Made more progress on the AN protects and LS drive 33800
Signed-off-by: Jared Harvey <TortiseGIT@jaredharvey.com>
Parts:
- C903, C906: TOL (none) -> 10%; V 100V -> 200V; construct ceramic -> CERAMIC; mfg,mfg# avx,08051C104KAT2A -> AVX,08055C104KAT2A; tolerance 10% -> (none); vend1,vend1# newark,96M1354 -> newark,27C8438
Changed lines of the file:
@@
-EESchema Schematic File Version 2  date 10/14/2011 5:26:22 AM
+EESchema Schematic File Version 2  date 10/16/2011 7:32:22 AM
 LIBS:power
 LIBS:device
@@
 Sheet 8 12
 Title "Open5xxxECU (o5e), an ECU that is no longer affiliated with freeEMS."
-Date "14 oct 2011"
+Date "16 oct 2011"
 Rev "A-DRAFT5"
 Comp "http://open5xxxecu.org/"
@@
 3412_WAKE
 $Comp
-L GND #PWR0141
+L GND #PWR0149
 U 1 1 4C1CA88F
 P 7750 4900
-F 0 "#PWR0141" H 7750 4900 30  0001 C CNN
+F 0 "#PWR0149" H 7750 4900 30  0001 C CNN
 F 1 "GND" H 7750 4830 30  0001 C CNN
 	1    7750 4900
@@
 HS2_PIN
 $Comp
-L GND #PWR0142
+L GND #PWR0150
 U 1 1 4C09B719
 P 8500 4175
-F 0 "#PWR0142" H 8500 4175 30  0001 C CNN
+F 0 "#PWR0150" H 8500 4175 30  0001 C CNN
 F 1 "GND" H 8500 4105 30  0001 C CNN
 	1    8500 4175
@@
 $EndComp
 $Comp
-L GND #PWR0143
+L GND #PWR0151
 U 1 1 4BF94289
 P 8000 3975
-F 0 "#PWR0143" H 8000 3975 30  0001 C CNN
+F 0 "#PWR0151" H 8000 3975 30  0001 C CNN
 F 1 "GND" H 8000 3905 30  0001 C CNN
 	1    8000 3975
@@
 $EndComp
 $Comp
-L GND #PWR0144
+L GND #PWR0152
 U 1 1 4BF94163
 P 10300 5875
-F 0 "#PWR0144" H 10300 5875 30  0001 C CNN
+F 0 "#PWR0152" H 10300 5875 30  0001 C CNN
 F 1 "GND" H 10300 5805 30  0001 C CNN
 	1    10300 5875
@@
 F 0 "C906" V 10125 5300 50  0000 L CNN
 F 1 "100nF" V 10050 5275 50  0000 L CNN
-F 2 "SM0805" V 1130 2300 60  0001 C CNN
-F 4 "avx,08051C104KAT2A" V 1130 2300 60  0001 C CNN "mfg,mfg#"
-F 5 "newark,96M1354" V 1130 2300 60  0001 C CNN "vend1,vend1#"
-F 6 "100V" V 1130 2300 60  0001 C CNN "V"
-F 7 "10%" V 1130 2300 60  0001 C CNN "tolerance"
-F 8 "ceramic" V 1130 2300 60  0001 C CNN "construct"
-F 9 "other,more,stuff" V 1130 2300 60  0001 C CNN "misc"
+F 2 "SM0805" V 1130 2600 60  0001 C CNN
+F 4 "AVX,08055C104KAT2A" V 1130 2600 60  0001 C CNN "mfg,mfg#"
+F 5 "newark,27C8438" V 1130 2600 60  0001 C CNN "vend1,vend1#"
+F 6 "" V 1130 2600 60  0001 C CNN "Field6"
+F 7 "" V 1130 2600 60  0001 C CNN "Field7"
+F 8 "200V" V 1130 2600 60  0001 C CNN "V"
+F 9 "10%" V 1130 2600 60  0001 C CNN "TOL"
+F 10 "CERAMIC" V 1130 2600 60  0001 C CNN "construct"
+F 11 "other,more,stuff" V 1130 2600 60  0001 C CNN "misc"
 	1    10100 5600
 	0    -1   -1   0
@@
 F 0 "C903" V 8750 6050 50  0000 L CNN
 F 1 "100nF" V 8675 5525 50  0000 L CNN
-F 2 "SM0805" V 1130 2300 60  0001 C CNN
-F 4 "avx,08051C104KAT2A" V 1130 2300 60  0001 C CNN "mfg,mfg#"
-F 5 "newark,96M1354" V 1130 2300 60  0001 C CNN "vend1,vend1#"
-F 6 "100V" V 1130 2300 60  0001 C CNN "V"
-F 7 "10%" V 1130 2300 60  0001 C CNN "tolerance"
-F 8 "ceramic" V 1130 2300 60  0001 C CNN "construct"
-F 9 "other,more,stuff" V 1130 2300 60  0001 C CNN "misc"
+F 2 "SM0805" V 1130 2600 60  0001 C CNN
+F 4 "AVX,08055C104KAT2A" V 1130 2600 60  0001 C CNN "mfg,mfg#"
+F 5 "newark,27C8438" V 1130 2600 60  0001 C CNN "vend1,vend1#"
+F 6 "" V 1130 2600 60  0001 C CNN "Field6"
+F 7 "" V 1130 2600 60  0001 C CNN "Field7"
+F 8 "200V" V 1130 2600 60  0001 C CNN "V"
+F 9 "10%" V 1130 2600 60  0001 C CNN "TOL"
+F 10 "CERAMIC" V 1130 2600 60  0001 C CNN "construct"
+F 11 "other,more,stuff" V 1130 2600 60  0001 C CNN "misc"
 	1    8700 5875
 	0    1    1    0
 $EndComp
 $Comp
-L GND #PWR0145
+L GND #PWR0153
 U 1 1 4BF93FBA
 P 9450 3875
-F 0 "#PWR0145" H 9450 3875 30  0001 C CNN
+F 0 "#PWR0153" H 9450 3875 30  0001 C CNN
 F 1 "GND" H 9450 3805 30  0001 C CNN
 	1    9450 3875
@@
 $EndComp
 $Comp
-L GND #PWR0146
+L GND #PWR0154
 U 1 1 4BF93FB3
 P 9150 5875
-F 0 "#PWR0146" H 9150 5875 30  0001 C CNN
+F 0 "#PWR0154" H 9150 5875 30  0001 C CNN
 F 1 "GND" H 9150 5805 30  0001 C CNN
 	1    9150 5875
@@
 BATV
 $Comp
-L GND #PWR0147
+L GND #PWR0155
 U 1 1 4BF50953
 P 9450 5875
-F 0 "#PWR0147" H 9450 5875 30  0001 C CNN
+F 0 "#PWR0155" H 9450 5875 30  0001 C CNN
 F 1 "GND" H 9450 5805 30  0001 C CNN
 	1    9450 5875
@@
 $EndComp
 $Comp
-L GND #PWR0148
+L GND #PWR0156
 U 1 1 4BF5090D
 P 10950 6375
-F 0 "#PWR0148" H 10950 6375 30  0001 C CNN
+F 0 "#PWR0156" H 10950 6375 30  0001 C CNN
 F 1 "GND" H 10950 6305 30  0001 C CNN
 	1    10950 6375
