File: KICAD_Project/sub_circuits/low_side_drive.sch (KiCad schematic (older format))
At the start: 82 parts

Commit message: Started laying out the harness in DXF, initial schematic capture complete, except for harness.
Signed-off-by: Jared Harvey <TortiseGIT@jaredharvey.com>
Connections:
- net labels added: GND_PWR8
- net labels removed: GND_PWR1, GND_PWR3
- wire segments 217 -> 216
Changed lines of the file:
@@
-EESchema Schematic File Version 2  date 8/6/2011 11:05:39 PM
+EESchema Schematic File Version 2  date 8/7/2011 7:33:14 PM
 LIBS:power
 LIBS:device
@@
 	6650 3550 7150 3550
 Wire Wire Line
-	6400 1300 5900 1300
-Wire Wire Line
 	5900 1400 6400 1400
 Wire Wire Line
@@
 $EndComp
 Text Label 3950 2650 0    60   ~ 0
-GND_PWR1
+GND_PWR8
 $Comp
 L CONN_1 P?
@@
 $EndComp
 Text Label 1925 2550 0    60   ~ 0
-GND_PWR1
+GND_PWR8
 Text Label 2350 2150 0    60   ~ 0
-GND_PWR1
+GND_PWR8
 Text Label 2950 1850 0    60   ~ 0
-GND_PWR1
+GND_PWR8
 $Comp
 L GND #PWR?
@@
 $EndComp
 Text Label 8075 2700 2    60   ~ 0
-GND_PWR1
+GND_PWR8
 Text Label 9650 2550 2    60   ~ 0
-GND_PWR3
+GND_PWR8
 Text Label 9225 2150 2    60   ~ 0
-GND_PWR3
+GND_PWR8
 Text Label 8625 1850 2    60   ~ 0
-GND_PWR1
+GND_PWR8
 Text Label 9200 4425 2    60   ~ 0
-GND_PWR1
+GND_PWR8
 Text HLabel 5900 1400 0    60   Input ~ 0
-GND_PWR3
+GND_PWR8
 Text Label 6400 1400 2    60   ~ 0
-GND_PWR3
-Text Label 6400 1300 2    60   ~ 0
-GND_PWR1
-Text HLabel 5900 1300 0    60   Input ~ 0
-GND_PWR1
+GND_PWR8
 Text HLabel 3350 1650 1    60   Input ~ 0
 misc2_drv_LO
@@
 misc1_drv_LO
 Text Label 7150 3550 2    60   ~ 0
-GND_PWR1
+GND_PWR8
 Text Label 7150 3050 2    60   ~ 0
-GND_PWR1
+GND_PWR8
 Text Label 7150 2850 2    60   ~ 0
-GND_PWR1
+GND_PWR8
 Text HLabel 8700 1950 1    60   Input ~ 0
 up_O2_heat_LO

Commit message: About to runs scripts to scrub the BOM's, so here's a backup copy in case it goes wrong.
Signed-off-by: Jared Harvey <TortiseGIT@jaredharvey.com>
Parts:
- removed C?: 100nF, SM0805-C1, symbol C
- removed C? (x2): 10nF, SM0805-C1, symbol C
- removed P? (x2): CONN_1, PINTST, symbol CONN_1
- removed R?: NA, SM0805-R4, symbol R
- removed R?: 0R, SM0805-R4, symbol R
- added C914: 100nF, SM0805-C1, symbol C
- added C916, C919: 10nF, SM0805-C1, symbol C
- added P929, P931: CONN_1, PINTST, symbol CONN_1
- added R905: NA, SM0805, symbol R
- added R912: 0R, SM0805, symbol R
- R901, R902, R903, R904, R906, R907, R908, R909, R910, R911, R913, R914, R915, R916, R917, R918: renamed from R?; footprint SM0805-R4 -> SM0805
- gave numbers to parts that had none: 56

Commit message: caps have been done with the scripts next up is the resistors.
Signed-off-by: Jared Harvey <TortiseGIT@jaredharvey.com>
Parts:
- C901, C902, C903, C904, C905, C906, C907, C908, C909, C910, C911, C912, C913, C916, C917, C918, C919, C920, C921, C922, C923, C924: Field3 -,- -> (none); Field4 -,- -> (none); Field5 200,V -> (none); Field6 10,% -> (none); Field7 alum electro -> (none); Field8 other,more,stuff -> (none); V (none) -> 200V; construct (none) -> alum elec; mfg,# ill cap,106CKE200M -> (none); mfg,mfg# (none) -> ill cap,106CKE200M; misc (none) -> other,more,stuff; tolerance (none) -> 10%; vend,# newark,69K7896 -> (none); vend1,vend1# (none) -> newark,69K7896
- C914, C915: Field3 -,- -> (none); Field4 -,- -> (none); Field5 50,V -> (none); Field6 10,% -> (none); Field7 Ceramic -> (none); Field8 other,more,stuff -> (none); V (none) -> 100V; construct (none) -> ceramic; mfg,# mutata,GRM21BR71H104KA01L -> (none); mfg,mfg# (none) -> avx,08051C104KAT2A; misc (none) -> other,more,stuff; tolerance (none) -> 10%; vend,# newark,38K1694 -> (none); vend1,vend1# (none) -> newark,96M1354

Commit message: Looks like the bulk components are golden now, there are still a couple straglers, mostly switch mode power supply stuff.
Signed-off-by: Jared Harvey <TortiseGIT@jaredharvey.com>
Parts:
- R901, R906, R908, R909, R910, R911, R912, R913, R915: Field3 -,- -> (none); Field4 -,- -> (none); Field5 -,mW -> (none); Field6 -,% -> (none); Field7 na -> (none); Field8 other,more,stuff -> (none); mfg,# wishay,CRCW08050000ZSTA -> (none); mfg,mfg# (none) -> vishay,CRCW08050000Z0EA; misc (none) -> other,more,stuff; tolerance (none) -> %; vend,# newark,36C9353 -> (none); vend1,vend1# (none) -> newark,52K9721; w (none) -> mW
- R903: Field3 -,- -> (none); Field4 -,- -> (none); Field5 125,mW -> (none); Field6 1,% -> (none); Field7 thick film -> (none); Field8 other,more,stuff -> (none); construct (none) -> thick film; mfg,# vishay,CRCW08051K00FKTA -> (none); mfg,mfg# (none) -> vishay,CRCW08051K00FKTA; misc (none) -> other,more,stuff; tolerance (none) -> 1%; vend,# newark,05F1507 -> (none); vend1,vend1# (none) -> newark,05F1507; w (none) -> 125mW

Commit message: harness connector is much more ironed out now. CPU is not connected.
Signed-off-by: Jared Harvey <TortiseGIT@jaredharvey.com>
Connections:
- net labels added: GND_MC33800
Changed lines of the file:
@@
-EESchema Schematic File Version 2  date 8/14/2011 8:37:17 PM
+EESchema Schematic File Version 2  date 8/19/2011 6:13:41 AM
 LIBS:power
 LIBS:device
@@
 Sheet 9 13
 Title "freeEMS PLUS from Cinch template "
-Date "14 aug 2011"
-Rev "A"
+Date "19 aug 2011"
+Rev "A-DRAF"
 Comp "diyefi.org/openecu.info"
 Comment1 "misc high side and low side drives"
@@
 Comment4 ""
 $EndDescr
+$Comp
+L GND #PWR0152
+U 1 1 4C2B134E
+P 6400 1425
+F 0 "#PWR0152" H 6400 1425 30  0001 C CNN
+F 1 "GND" H 6400 1355 30  0001 C CNN
+	1    6400 1425
+	1    0    0    -1
+$EndComp
+Wire Wire Line
+	6400 1425 6400 1400
 $Comp
 L IRF7341 Q903
@@
 Connection ~ 2400 3200
 Wire Wire Line
-	2400 3200 3525 3200
-Wire Wire Line
-	3525 4000 2400 4000
+	3525 3200 2400 3200
+Wire Wire Line
+	2400 4000 3525 4000
 Wire Wire Line
 	4950 3450 4400 3450
@@
 	6650 3550 7150 3550
 Wire Wire Line
-	5900 1400 6400 1400
+	6400 1400 5750 1400
 Wire Wire Line
 	8125 2350 8800 2350
@@
 Wire Wire Line
 	9200 2800 9200 4425
-Wire Wire Line
-	6400 1400 6400 1425
 Wire Wire Line
 	3850 2050 3400 2050
@@
 Text Label 2950 1850 0    60   ~ 0
 GND_PWR8
-$Comp
-L GND #PWR0138
-U 1 1 4C2B134E
-P 6400 1425
-F 0 "#PWR0138" H 6400 1425 30  0001 C CNN
-F 1 "GND" H 6400 1355 30  0001 C CNN
-	1    6400 1425
-	1    0    0    -1
-$EndComp
 Text Label 8075 2700 2    60   ~ 0
 GND_PWR8
@@
 Text Label 9200 4425 2    60   ~ 0
 GND_PWR8
-Text HLabel 5900 1400 0    60   Input ~ 0
-GND_PWR8
+Text HLabel 5750 1400 0    60   Input ~ 0
+GND_MC33800
 Text Label 6400 1400 2    60   ~ 0
-GND_PWR8
+GND_MC33800
 Text HLabel 3350 1650 1    60   Input ~ 0
 misc2_drv_LO
@@
 $EndComp
 $Comp
-L GND #PWR0139
+L GND #PWR0153
 U 1 1 4BF50AC9
 P 4875 4175
-F 0 "#PWR0139" H 4875 4175 30  0001 C CNN
+F 0 "#PWR0153" H 4875 4175 30  0001 C CNN
 F 1 "GND" H 4875 4105 30  0001 C CNN
 	1    4875 4175
@@
 $EndComp
 $Comp
-L GND #PWR0140
+L GND #PWR0154
 U 1 1 4BF5091E
 P 6725 4575
-F 0 "#PWR0140" H 6725 4575 30  0001 C CNN
+F 0 "#PWR0154" H 6725 4575 30  0001 C CNN
 F 1 "GND" H 6725 4505 30  0001 C CNN
 	1    6725 4575
@@
 $EndComp
 $Comp
-L GND #PWR0141
+L GND #PWR0155
 U 1 1 4BF50915
 P 6700 4375
-F 0 "#PWR0141" H 6700 4375 30  0001 C CNN
+F 0 "#PWR0155" H 6700 4375 30  0001 C CNN
 F 1 "GND" H 6700 4305 30  0001 C CNN
 	1    6700 4375
@@
 $EndComp
 $Comp
-L GND #PWR0142
+L GND #PWR0156
 U 1 1 4BF3BCE7
 P 4150 4600
-F 0 "#PWR0142" H 4150 4600 30  0001 C CNN
+F 0 "#PWR0156" H 4150 4600 30  0001 C CNN
 F 1 "GND" H 4150 4530 30  0001 C CNN
 	1    4150 4600
@@
 $EndComp
 $Comp
-L GND #PWR0143
+L GND #PWR0157
 U 1 1 4BF3BCD4
 P 2575 2975
-F 0 "#PWR0143" H 2575 2975 30  0001 C CNN
+F 0 "#PWR0157" H 2575 2975 30  0001 C CNN
 F 1 "GND" H 2575 2905 30  0001 C CNN
 	1    2575 2975
@@
 $EndComp
 $Comp
-L GND #PWR0144
+L GND #PWR0158
 U 1 1 4BF34837
 P 7650 4150
-F 0 "#PWR0144" H 7650 4150 30  0001 C CNN
+F 0 "#PWR0158" H 7650 4150 30  0001 C CNN
 F 1 "GND" H 7650 4080 30  0001 C CNN
 	1    7650 4150
@@
 $EndComp
 $Comp
-L GND #PWR0145
+L GND #PWR0159
 U 1 1 4BF34814
 P 7650 4450
-F 0 "#PWR0145" H 7650 4450 30  0001 C CNN
+F 0 "#PWR0159" H 7650 4450 30  0001 C CNN
 F 1 "GND" H 7650 4380 30  0001 C CNN
 	1    7650 4450

Commit message: several pins on the SOM are now connected.
Signed-off-by: Jared Harvey <TortiseGIT@jaredharvey.com>
Parts:
- renumbered C901 to C1001, C902 to C1002, C903 to C1003, C904 to C1004, C905 to C1005, C906 to C1006, C907 to C1007, C908 to C1008, C909 to C1009, C910 to C1010, C911 to C1011, C912 to C1012, C913 to C1013, C914 to C1014, C915 to C1015, C916 to C1016, C917 to C1017, C918 to C1018, C919 to C1019, C920 to C1020, C921 to C1021, C922 to C1022, C923 to C1023, C924 to C1024, D901 to D1001, D902 to D1002, P901 to P1001, P902 to P1002, P903 to P1003, P904 to P1004, P905 to P1005, P906 to P1006, P907 to P1007, P908 to P1008, P909 to P1009, P910 to P1010, P911 to P1011, P912 to P1012, P913 to P1013, P914 to P1014, P915 to P1015, P916 to P1016, P917 to P1017, P918 to P1018, P919 to P1019, P920 to P1020, P921 to P1021, P922 to P1022, P923 to P1023, P924 to P1024, P925 to P1025, P926 to P1026, P927 to P1027, P928 to P1028, P929 to P1029, P930 to P1030, P931 to P1031, Q901 to Q1001, Q902 to Q1002, Q903 to Q1003, R901 to R1001, R902 to R1002, R903 to R1003, R904 to R1004, R905 to R1005, R906 to R1006, R907 to R1007, R908 to R1008, R909 to R1009, R910 to R1010, R911 to R1011, R912 to R1012, R913 to R1013, R914 to R1014, R915 to R1015, R916 to R1016, R917 to R1017, R918 to R1018, U901 to U1001
