File: KICAD_Project/sub_circuits/low_side_drive.sch (KiCad schematic (older format))
At the start: 79 parts, among them P1001 CONN_1, P1002 CONN_1, P1003 CONN_1, P1004 CONN_1, P1005 CONN_1, P1006 CONN_1, P1007 CONN_1, P1008 CONN_1, P1009 CONN_1, P1010 CONN_1, P1011 CONN_1, P1012 CONN_1, P1013 CONN_1, P1014 CONN_1, P1015 CONN_1, P1016 CONN_1, P1017 CONN_1, P1018 CONN_1, P1019 CONN_1, P1020 CONN_1, P1021 CONN_1, P1022 CONN_1, P1023 CONN_1, P1024 CONN_1, P1025 CONN_1, P1026 CONN_1, P1027 CONN_1, P1028 CONN_1, P1029 CONN_1, P1030 CONN_1, P1031 CONN_1, Q1001 IRF7341, Q1002 IRF7341, Q1003 IRF7341, U1001 MC33800

Commit message: routing has started
Signed-off-by: Jared Harvey <TortiseGIT@jaredharvey.com>
Changed lines of the file:
@@
-EESchema Schematic File Version 2  date 8/20/2011 7:18:56 AM
+EESchema Schematic File Version 2  date 8/20/2011 7:59:51 PM
 LIBS:power
 LIBS:device
@@
 U 2 1 4C3E5656
 P 9100 2550
-F 0 "Q1003" H 9050 2700 60  0000 R CNN
+F 0 "Q1003" H 9250 2800 60  0000 R CNN
 F 1 "IRF7341" H 9075 2400 60  0000 R CNN
 F 2 "SO8E" H 9100 2550 60  0001 C CNN
@@
 U 1 1 4C3E5179
 P 2500 2550
-F 0 "Q1001" H 2450 2700 60  0000 R CNN
-F 1 "IRF7341" H 2475 2400 60  0000 R CNN
+F 0 "Q1001" H 2725 2800 60  0000 R CNN
+F 1 "IRF7341" H 2375 2450 60  0000 R CNN
 F 2 "SO8E" H 2500 2550 60  0001 C CNN
 F 4 "irf,IRF7341PBF" H 2500 2550 60  0001 C CNN "mfg,#"
@@
 U 1 1 4BF3BCD7
 P 2925 2750
-F 0 "P1003" H 3005 2750 40  0000 L CNN
+F 0 "P1003" H 2975 2750 40  0000 L CNN
 F 1 "CONN_1" H 2925 2805 30  0001 C CNN
 F 2 "PINTST" V -3595 3350 60  0001 C CNN
@@
 U 1 1 4BF654C5
 P 4600 2650
-F 0 "R1009" V 4650 2450 50  0000 C CNN
+F 0 "R1009" V 4650 2350 50  0000 C CNN
 F 1 "0R" V 4600 2650 50  0000 C CNN
 F 2 "SM0805" V 1130 2600 60  0001 C CNN
@@
 U 1 1 4E467E08
 P 7200 2650
-F 0 "R1012" V 7150 2900 50  0000 C CNN
+F 0 "R1012" V 7150 2925 50  0000 C CNN
 F 1 "0R" V 7200 2650 50  0000 C CNN
 F 2 "SM0805" V 1130 2600 60  0001 C CNN
@@
 U 1 1 4BF65288
 P 4250 3850
-F 0 "P1012" H 4375 3850 40  0000 L CNN
+F 0 "P1012" H 4300 3850 40  0000 L CNN
 F 1 "CONN_1" H 4250 3905 30  0001 C CNN
 F 2 "PINTST" V -2270 4450 60  0001 C CNN
@@
 U 1 1 4BF65287
 P 2600 3900
-F 0 "C1002" V 2520 4020 50  0000 L CNN
+F 0 "C1002" V 2575 4250 50  0000 L CNN
 F 1 "10nF" V 2525 3700 50  0000 L CNN
 F 2 "SM0805-C1" V 1130 2600 60  0001 C CNN
@@
 U 1 1 4BF65286
 P 4250 3750
-F 0 "P1011" H 4375 3750 40  0000 L CNN
+F 0 "P1011" H 4300 3750 40  0000 L CNN
 F 1 "CONN_1" H 4250 3805 30  0001 C CNN
 F 2 "PINTST" V -2270 4350 60  0001 C CNN
@@
 U 1 1 4BF65284
 P 4250 3650
-F 0 "P1010" H 4375 3650 40  0000 L CNN
+F 0 "P1010" H 4300 3650 40  0000 L CNN
 F 1 "CONN_1" H 4250 3705 30  0001 C CNN
 F 2 "PINTST" V -2270 4250 60  0001 C CNN
@@
 U 1 1 4BF65282
 P 4250 3550
-F 0 "P1009" H 4375 3550 40  0000 L CNN
+F 0 "P1009" H 4300 3550 40  0000 L CNN
 F 1 "CONN_1" H 4250 3605 30  0001 C CNN
 F 2 "PINTST" V -2270 4150 60  0001 C CNN
@@
 P 3725 3600
 F 0 "C1010" V 3745 3805 50  0000 L CNN
-F 1 "10nF" V 3650 3400 50  0000 L CNN
+F 1 "10nF" V 3650 3450 50  0000 L CNN
 F 2 "SM0805-C1" V 1130 2600 60  0001 C CNN
 F 4 "ill cap,106CKE200M" V 1130 2600 60  0001 C CNN "mfg,mfg#"
@@
 U 1 1 4BF6521E
 P 4250 4050
-F 0 "P1014" H 4375 4050 40  0000 L CNN
+F 0 "P1014" H 4300 4050 40  0000 L CNN
 F 1 "CONN_1" H 4250 4105 30  0001 C CNN
 F 2 "PINTST" V -2270 4650 60  0001 C CNN
@@
 U 1 1 4BF6521C
 P 4250 3950
-F 0 "P1013" H 4375 3950 40  0000 L CNN
+F 0 "P1013" H 4300 3950 40  0000 L CNN
 F 1 "CONN_1" H 4250 4005 30  0001 C CNN
 F 2 "PINTST" V -2270 4550 60  0001 C CNN
@@
 P 3725 4000
 F 0 "C1011" V 3745 4205 50  0000 L CNN
-F 1 "10nF" V 3650 3800 50  0000 L CNN
+F 1 "10nF" V 3650 3850 50  0000 L CNN
 F 2 "SM0805-C1" V 1130 2600 60  0001 C CNN
 F 4 "ill cap,106CKE200M" V 1130 2600 60  0001 C CNN "mfg,mfg#"
@@
 P 3725 3200
 F 0 "C1009" V 3755 3405 50  0000 L CNN
-F 1 "10nF" V 3650 3000 50  0000 L CNN
+F 1 "10nF" V 3650 3050 50  0000 L CNN
 F 2 "SM0805-C1" V 1130 2600 60  0001 C CNN
 F 4 "ill cap,106CKE200M" V 1130 2600 60  0001 C CNN "mfg,mfg#"
@@
 U 1 1 4BF65219
 P 4250 3150
-F 0 "P1005" H 4375 3150 40  0000 L CNN
+F 0 "P1005" H 4300 3150 40  0000 L CNN
 F 1 "CONN_1" H 4250 3205 30  0001 C CNN
 F 2 "PINTST" V -2270 3750 60  0001 C CNN
@@
 U 1 1 4BF65217
 P 4250 3250
-F 0 "P1006" H 4375 3250 40  0000 L CNN
+F 0 "P1006" H 4300 3250 40  0000 L CNN
 F 1 "CONN_1" H 4250 3305 30  0001 C CNN
 F 2 "PINTST" V -2270 3850 60  0001 C CNN
@@
 U 1 1 4BF65215
 P 4250 3350
-F 0 "P1007" H 4375 3350 40  0000 L CNN
+F 0 "P1007" H 4300 3350 40  0000 L CNN
 F 1 "CONN_1" H 4250 3405 30  0001 C CNN
 F 2 "PINTST" V -2270 3950 60  0001 C CNN
@@
 U 1 1 4BF65214
 P 2600 3500
-F 0 "C1001" V 2520 3620 50  0000 L CNN
+F 0 "C1001" V 2575 3825 50  0000 L CNN
 F 1 "10nF" V 2525 3300 50  0000 L CNN
 F 2 "SM0805-C1" V 1130 2600 60  0001 C CNN
@@
 U 1 1 4BF65213
 P 4250 3450
-F 0 "P1008" H 4375 3450 40  0000 L CNN
+F 0 "P1008" H 4300 3450 40  0000 L CNN
 F 1 "CONN_1" H 4250 3505 30  0001 C CNN
 F 2 "PINTST" V -2270 4050 60  0001 C CNN
@@
 U 1 1 4BF650CE
 P 7500 2050
-F 0 "R1014" V 7440 2290 50  0000 C CNN
+F 0 "R1014" V 7450 2325 50  0000 C CNN
 F 1 "NA" V 7500 2050 50  0000 C CNN
 F 2 "SM0805" V 7680 2150 60  0001 C CNN
@@
 U 1 1 4BF507B3
 P 9000 3500
-F 0 "C1024" V 8930 3620 50  0000 L CNN
+F 0 "C1024" V 8825 3575 50  0000 L CNN
 F 1 "10nF" V 8925 3300 50  0000 L CNN
 F 2 "SM0805-C1" V 1130 2600 60  0001 C CNN
@@
 P 7875 3700
 F 0 "C1017" V 7905 3905 50  0000 L CNN
-F 1 "10nF" V 7800 3500 50  0000 L CNN
+F 1 "10nF" V 7800 3550 50  0000 L CNN
 F 2 "SM0805-C1" V 1130 2600 60  0001 C CNN
 F 4 "ill cap,106CKE200M" V 1130 2600 60  0001 C CNN "mfg,mfg#"
@@
 U 1 1 4BF3BF0A
 P 8350 2650
-F 0 "R1018" V 8300 2420 50  0000 C CNN
+F 0 "R1018" V 8400 2350 50  0000 C CNN
 F 1 "NA" V 8350 2650 50  0000 C CNN
 F 2 "SM0805" V 8530 2750 60  0001 C CNN
@@
 U 1 1 4E467DF8
 P 7350 4100
-F 0 "C1014" V 7280 4300 50  0000 L CNN
+F 0 "C1014" V 7275 4250 50  0000 L CNN
 F 1 "100nF" V 7400 3950 50  0000 L CNN
 F 2 "SM0805-C1" V 1130 2600 60  0001 C CNN
@@
 U 1 1 488A2BA8
 P 7350 4400
-F 0 "C1015" V 7390 4550 50  0000 L CNN
+F 0 "C1015" V 7475 4575 50  0000 L CNN
 F 1 "100nF" V 7400 4250 50  0000 L CNN
 F 2 "SM0805-C1" V 1130 2600 60  0001 C CNN
