File: KICAD_Project/sub_circuits/low_side_drive.sch (KiCad schematic (older format))
At the start: 79 parts, among them P1001 CONN_1, P1002 CONN_1, P1003 CONN_1, P1004 CONN_1, P1005 CONN_1, P1006 CONN_1, P1007 CONN_1, P1008 CONN_1, P1009 CONN_1, P1010 CONN_1, P1011 CONN_1, P1012 CONN_1, P1013 CONN_1, P1014 CONN_1, P1015 CONN_1, P1016 CONN_1, P1017 CONN_1, P1018 CONN_1, P1019 CONN_1, P1020 CONN_1, P1021 CONN_1, P1022 CONN_1, P1023 CONN_1, P1024 CONN_1, P1025 CONN_1, P1026 CONN_1, P1027 CONN_1, P1028 CONN_1, P1029 CONN_1, P1030 CONN_1, P1031 CONN_1, Q1001 IRF7341, Q1002 IRF7341, Q1003 IRF7341, U1001 MC33800

Commit message: Added some simulations for the AN protect lines
Signed-off-by: Jared Harvey <TortiseGIT@jaredharvey.com>
Connections:
- wire segments 220 -> 221

Commit message: Made more progress on the AN protects and LS drive 33800
Signed-off-by: Jared Harvey <TortiseGIT@jaredharvey.com>
Parts:
- removed C1002, C1005, C1007, C1008, C1010, C1011, C1016, C1017, C1019, C1020, C1021, C1022, C1023, C1024: 10nF, SM0805-C1, symbol C
- removed P1001, P1002, P1003, P1004, P1015, P1016, P1018, P1019, P1028, P1029, P1030, P1031: CONN_1, PINTST, symbol CONN_1
- removed R1009, R1012: 0R, SM0805, symbol R
- C1001, C1003, C1004, C1006, C1009, C1012, C1013, C1018: footprint SM0805-C1 -> SM0805; TOL (none) -> 10%; V 200V -> 50V; construct alum elec -> CERAMIC; mfg,mfg# ill cap,106CKE200M -> AVX,08055C103KAT2A; tolerance 10% -> (none); vend1,vend1# newark,69K7896 -> newark,07J3575
- C1014, C1015: footprint SM0805-C1 -> SM0805; TOL (none) -> 10%; V 100V -> 200V; construct ceramic -> CERAMIC; mfg,mfg# avx,08051C104KAT2A -> AVX,08055C104KAT2A; tolerance 10% -> (none); vend1,vend1# newark,96M1354 -> newark,27C8438
- D1001, D1002: footprint D4-SMA -> SMA
Connections:
- wire segments 221 -> 178
