File: KICAD_Project/sub_circuits/stepper_mc33879.sch (KiCad schematic (older format))
At the start: 21 parts

Commit message: Started laying out the harness in DXF, initial schematic capture complete, except for harness.
Signed-off-by: Jared Harvey <TortiseGIT@jaredharvey.com>
Connections:
- net labels added: GND_PWR8
- net labels removed: GND_PWR1, GND_PWR2
- wire segments 55 -> 54
Changed lines of the file:
@@
-EESchema Schematic File Version 2  date 8/6/2011 11:05:38 PM
+EESchema Schematic File Version 2  date 8/7/2011 7:33:14 PM
 LIBS:power
 LIBS:device
@@
 Wire Wire Line
 	6625 5400 7025 5400
-Wire Wire Line
-	6400 4650 6450 4650
 Wire Wire Line
 	10425 5525 10425 5300
@@
 	9750 6100 8800 6100
 Text Label 6950 6900 1    60   ~ 0
-GND_PWR2
+GND_PWR8
 Text Label 5550 5300 0    60   ~ 0
-GND_PWR1
+GND_PWR8
 Text Label 7125 5200 0    60   ~ 0
-GND_PWR1
-Text HLabel 6400 4650 0    60   Input ~ 0
-GND_PWR1
-Text Label 6450 4650 0    60   ~ 0
-GND_PWR1
+GND_PWR8
 Text Label 6625 5400 0    60   ~ 0
-GND_PWR2
+GND_PWR8
 Text Label 9625 6425 0    60   ~ 0
-GND_PWR2
+GND_PWR8
 Text Label 9425 5525 0    60   ~ 0
-GND_PWR2
+GND_PWR8
 Text Label 6525 6625 2    60   ~ 0
-GND_PWR2
+GND_PWR8
 Text Label 6525 6025 2    60   ~ 0
-GND_PWR2
+GND_PWR8
 Text Label 6450 4775 0    60   ~ 0
-GND_PWR2
+GND_PWR8
 Text HLabel 6400 4775 0    60   Input ~ 0
-GND_PWR2
+GND_PWR8
 Text HLabel 9750 6300 2    60   Input ~ 0
 D5_PIN

Commit message: About to runs scripts to scrub the BOM's, so here's a backup copy in case it goes wrong.
Signed-off-by: Jared Harvey <TortiseGIT@jaredharvey.com>
Parts:
- R701, R702, R703, R704, R705, R706, R707, R708, R709, R710, R711, R712: renamed from R?; footprint SM0805-R4 -> SM0805
- gave numbers to parts that had none: 9
Changed lines of the file:
@@
-EESchema Schematic File Version 2  date 8/7/2011 7:33:14 PM
+EESchema Schematic File Version 2  date 8/14/2011 3:32:14 PM
 LIBS:power
 LIBS:device
@@
 $Descr User 11000 8500
 encoding utf-8
-Sheet 7 14
+Sheet 7 13
 Title "freeEMS PLUS from Cinch template "
-Date "7 aug 2011"
+Date "14 aug 2011"
 Rev "A"
 Comp "diyefi.org/openecu.info"
@@
 D8_PIN
 $Comp
-L R R?
+L R R711
 U 1 1 4C1B4C13
 P 9250 5875
-F 0 "R?" V 9195 6125 50  0000 C CNN
+F 0 "R711" V 9195 6125 50  0000 C CNN
 F 1 "0R" V 9250 5875 50  0000 C CNN
-F 2 "SM0805-R4" H 9250 5875 60  0001 C CNN
+F 2 "SM0805" H 9250 5875 60  0001 C CNN
 F 4 "vishay,CRCW08050000ZSTA" V 3605 6900 60  0001 C CNN "mfg,#"
 F 5 "newark,36C9353" V 3605 6900 60  0001 C CNN "vend,#"
@@
 $EndComp
 $Comp
-L R R?
+L R R707
 U 1 1 4C1B4C00
 P 9100 6200
-F 0 "R?" V 9050 5930 50  0000 C CNN
+F 0 "R707" V 9050 5930 50  0000 C CNN
 F 1 "0R" V 9100 6200 50  0000 C CNN
-F 2 "SM0805-R4" H 9100 6200 60  0001 C CNN
+F 2 "SM0805" H 9100 6200 60  0001 C CNN
 F 4 "vishay,CRCW08050000ZSTA" V 3605 6900 60  0001 C CNN "mfg,#"
 F 5 "newark,36C9353" V 3605 6900 60  0001 C CNN "vend,#"
@@
 $EndComp
 $Comp
-L R R?
+L R R709
 U 1 1 4C1B4BAE
 P 9200 6400
-F 0 "R?" V 9260 6670 50  0000 C CNN
+F 0 "R709" V 9260 6670 50  0000 C CNN
 F 1 "0R" V 9200 6400 50  0000 C CNN
-F 2 "SM0805-R4" H 9200 6400 60  0001 C CNN
+F 2 "SM0805" H 9200 6400 60  0001 C CNN
 F 4 "vishay,CRCW08050000ZSTA" V 3605 6900 60  0001 C CNN "mfg,#"
 F 5 "newark,36C9353" V 3605 6900 60  0001 C CNN "vend,#"
@@
 $EndComp
 $Comp
-L R R?
+L R R708
 U 1 1 4C1B4B98
 P 9125 5500
-F 0 "R?" V 9035 5505 50  0000 C CNN
+F 0 "R708" V 9035 5505 50  0000 C CNN
 F 1 "0R" V 9125 5500 50  0000 C CNN
-F 2 "SM0805-R4" H 9125 5500 60  0001 C CNN
+F 2 "SM0805" H 9125 5500 60  0001 C CNN
 F 4 "vishay,CRCW08050000ZSTA" V 3605 6900 60  0001 C CNN "mfg,#"
 F 5 "newark,36C9353" V 3605 6900 60  0001 C CNN "vend,#"
@@
 $EndComp
 $Comp
-L R R?
+L R R706
 U 1 1 4C1B4B33
 P 7325 6400
-F 0 "R?" V 7375 6685 50  0000 C CNN
+F 0 "R706" V 7375 6685 50  0000 C CNN
 F 1 "0R" V 7325 6400 50  0000 C CNN
-F 2 "SM0805-R4" H 7325 6400 60  0001 C CNN
+F 2 "SM0805" H 7325 6400 60  0001 C CNN
 F 4 "vishay,CRCW08050000ZSTA" V 3605 6900 60  0001 C CNN "mfg,#"
 F 5 "newark,36C9353" V 3605 6900 60  0001 C CNN "vend,#"
@@
 $EndComp
 $Comp
-L R R?
+L R R703
 U 1 1 4C1B4A76
 P 7275 5400
-F 0 "R?" V 7355 5400 50  0000 C CNN
+F 0 "R703" V 7355 5400 50  0000 C CNN
 F 1 "0R" V 7275 5400 50  0000 C CNN
-F 2 "SM0805-R4" H 7275 5400 60  0001 C CNN
+F 2 "SM0805" H 7275 5400 60  0001 C CNN
 F 4 "vishay,CRCW08050000ZSTA" V 3605 6900 60  0001 C CNN "mfg,#"
 F 5 "newark,36C9353" V 3605 6900 60  0001 C CNN "vend,#"
@@
 $EndComp
 $Comp
-L R R?
+L R R705
 U 1 1 4C1B4A43
 P 7300 6200
-F 0 "R?" V 7350 6450 50  0000 C CNN
+F 0 "R705" V 7350 6450 50  0000 C CNN
 F 1 "0R" V 7300 6200 50  0000 C CNN
-F 2 "SM0805-R4" H 7300 6200 60  0001 C CNN
+F 2 "SM0805" H 7300 6200 60  0001 C CNN
 F 4 "vishay,CRCW08050000ZSTA" V 3605 6900 60  0001 C CNN "mfg,#"
 F 5 "newark,36C9353" V 3605 6900 60  0001 C CNN "vend,#"
@@
 $EndComp
 $Comp
-L R R?
+L R R704
 U 1 1 4C1B4A0A
 P 7300 5800
-F 0 "R?" V 7380 5800 50  0000 C CNN
+F 0 "R704" V 7380 5800 50  0000 C CNN
 F 1 "0R" V 7300 5800 50  0000 C CNN
-F 2 "SM0805-R4" H 7300 5800 60  0001 C CNN
+F 2 "SM0805" H 7300 5800 60  0001 C CNN
 F 4 "vishay,CRCW08050000ZSTA" V 3605 6900 60  0001 C CNN "mfg,#"
 F 5 "newark,36C9353" V 3605 6900 60  0001 C CNN "vend,#"
@@
 $EndComp
 $Comp
-L R R?
+L R R702
 U 1 1 4C1B47F7
 P 6900 6300
-F 0 "R?" V 6975 6175 50  0000 C CNN
+F 0 "R702" V 6975 6175 50  0000 C CNN
 F 1 "0R" V 6900 6300 50  0000 C CNN
-F 2 "SM0805-R4" H 6900 6300 60  0001 C CNN
+F 2 "SM0805" H 6900 6300 60  0001 C CNN
 F 4 "vishay,CRCW08050000ZSTA" V 3605 6900 60  0001 C CNN "mfg,#"
 F 5 "newark,36C9353" V 3605 6900 60  0001 C CNN "vend,#"
@@
 $EndComp
 $Comp
-L R R?
+L R R701
 U 1 1 4C1B47D6
 P 6875 5700
-F 0 "R?" V 6955 5700 50  0000 C CNN
+F 0 "R701" V 6955 5700 50  0000 C CNN
 F 1 "0R" V 6875 5700 50  0000 C CNN
-F 2 "SM0805-R4" H 6875 5700 60  0001 C CNN
+F 2 "SM0805" H 6875 5700 60  0001 C CNN
 F 4 "vishay,CRCW08050000ZSTA" V 3605 6900 60  0001 C CNN "mfg,#"
 F 5 "newark,36C9353" V 3605 6900 60  0001 C CNN "vend,#"
@@
 $EndComp
 $Comp
-L R R?
+L R R710
 U 1 1 4C1B4798
 P 9250 5700
-F 0 "R?" V 9300 5950 50  0000 C CNN
+F 0 "R710" V 9300 5950 50  0000 C CNN
 F 1 "0R" V 9250 5700 50  0000 C CNN
-F 2 "SM0805-R4" H 9250 5700 60  0001 C CNN
+F 2 "SM0805" H 9250 5700 60  0001 C CNN
 F 4 "vishay,CRCW08050000ZSTA" V 3605 6900 60  0001 C CNN "mfg,#"
 F 5 "newark,36C9353" V 3605 6900 60  0001 C CNN "vend,#"
@@
 $EndComp
 $Comp
-L R R?
+L R R712
 U 1 1 4C1B474F
 P 9325 6300
-F 0 "R?" V 9275 6600 50  0000 C CNN
+F 0 "R712" V 9275 6600 50  0000 C CNN
 F 1 "0R" V 9325 6300 50  0000 C CNN
-F 2 "SM0805-R4" H 9325 6300 60  0001 C CNN
+F 2 "SM0805" H 9325 6300 60  0001 C CNN
 F 4 "vishay,CRCW08050000ZSTA" V 3605 6900 60  0001 C CNN "mfg,#"
 F 5 "newark,36C9353" V 3605 6900 60  0001 C CNN "vend,#"
@@
 install or jumpers for stepper motor driver.
 $Comp
-L C C?
+L C C702
 U 1 1 4C0F6A72
 P 6525 5800
-F 0 "C?" H 6550 5900 50  0000 L CNN
+F 0 "C702" H 6550 5900 50  0000 L CNN
 F 1 "10uF" H 6275 5900 50  0000 L CNN
 F 2 "SM0805-C1" V 3605 6900 60  0001 C CNN
@@
 VBAT
 $Comp
-L CONN_1 P?
+L CONN_1 P701
 U 1 1 4C0F68D7
 P 6350 5600
-F 0 "P?" H 6430 5600 40  0000 L CNN
+F 0 "P701" H 6430 5600 40  0000 L CNN
 F 1 "CONN_1" H 6350 5655 30  0001 C CNN
 F 2 "PINTST" H 6350 5600 60  0001 C CNN
@@
 $EndComp
 $Comp
-L CONN_1 P?
+L CONN_1 P702
 U 1 1 4C0F68D6
 P 6350 6100
-F 0 "P?" H 6430 6100 40  0000 L CNN
+F 0 "P702" H 6430 6100 40  0000 L CNN
 F 1 "CONN_1" H 6350 6155 30  0001 C CNN
 F 2 "PINTST" H 6350 6100 60  0001 C CNN
@@
 $EndComp
 $Comp
-L C C?
+L C C701
 U 1 1 4C0F6880
 P 6200 5300
-F 0 "C?" V 6120 5160 50  0000 L CNN
+F 0 "C701" V 6120 5160 50  0000 L CNN
 F 1 "100nF" V 6125 5500 50  0000 L CNN
 F 2 "SM0805-C1" V 3280 6400 60  0001 C CNN
@@
 879_MOSI
 $Comp
-L MC33879 U??
+L MC33879 U701
 U 1 1 4C0F6129
 P 8200 5950
-F 0 "U??" H 8200 6800 70  0000 C CNN
+F 0 "U701" H 8200 6800 70  0000 C CNN
 F 1 "MC33879" H 8200 5100 70  0000 C CNN
 F 2 "SOIC32" H 8200 5950 60  0001 C CNN
@@
 879_SCLK
 $Comp
-L CONN_1 P?
+L CONN_1 P704
 U 1 1 4C0A3402
 P 9900 6100
-F 0 "P?" H 9980 6100 40  0000 L CNN
+F 0 "P704" H 9980 6100 40  0000 L CNN
 F 1 "CONN_1" H 9900 6155 30  0001 C CNN
 F 2 "PINTST" H 9900 6100 60  0001 C CNN
@@
 $EndComp
 $Comp
-L CONN_1 P?
+L CONN_1 P703
 U 1 1 4C0A2746
 P 9900 5600
-F 0 "P?" H 9980 5600 40  0000 L CNN
+F 0 "P703" H 9980 5600 40  0000 L CNN
 F 1 "CONN_1" H 9900 5655 30  0001 C CNN
 F 2 "PINTST" H 9900 5600 60  0001 C CNN
@@
 VBAT
 $Comp
-L C C?
+L C C704
 U 1 1 4BF507DC
 P 10125 5300
-F 0 "C?" V 10175 5495 50  0000 L CNN
+F 0 "C704" V 10175 5495 50  0000 L CNN
 F 1 "10uF" V 10050 5100 50  0000 L CNN
 F 2 "SM0805-C1" V 7205 6400 60  0001 C CNN
@@
 $EndComp
 $Comp
-L C C?
+L C C703
 U 1 1 4BF507A3
 P 6525 6375
-F 0 "C?" H 6620 6470 50  0000 L CNN
+F 0 "C703" H 6620 6470 50  0000 L CNN
 F 1 "10uF" H 6275 6475 50  0000 L CNN
 F 2 "SM0805-C1" V 3605 7475 60  0001 C CNN

Commit message: caps have been done with the scripts next up is the resistors.
Signed-off-by: Jared Harvey <TortiseGIT@jaredharvey.com>
Parts:
- C701: Field3 -,- -> (none); Field4 -,- -> (none); Field5 50,V -> (none); Field6 10,% -> (none); Field7 Ceramic -> (none); Field8 other,more,stuff -> (none); V (none) -> 100V; construct (none) -> ceramic; mfg,# murata,GRM21BR71H104KA01L -> (none); mfg,mfg# (none) -> avx,08051C104KAT2A; misc (none) -> other,more,stuff; tolerance (none) -> 10%; vend,# newark,38K1694 -> (none); vend1,vend1# (none) -> newark,96M1354
Changed lines of the file:
@@
-EESchema Schematic File Version 2  date 8/14/2011 3:32:14 PM
+EESchema Schematic File Version 2  date 8/14/2011 7:31:25 PM
 LIBS:power
 LIBS:device
@@
 F 0 "C701" V 6120 5160 50  0000 L CNN
 F 1 "100nF" V 6125 5500 50  0000 L CNN
-F 2 "SM0805-C1" V 3280 6400 60  0001 C CNN
-F 4 "murata,GRM21BR71H104KA01L " V 3280 6400 60  0001 C CNN "mfg,#"
-F 5 "newark,38K1694" V 3280 6400 60  0001 C CNN "vend,#"
-F 6 "-,-" V 3280 6400 60  0001 C CNN "Field3"
-F 7 "-,-" V 3280 6400 60  0001 C CNN "Field4"
-F 8 "50,V" V 3280 6400 60  0001 C CNN "Field5"
-F 9 "10,%" V 3280 6400 60  0001 C CNN "Field6"
-F 10 "Ceramic" V 3280 6400 60  0001 C CNN "Field7"
-F 11 "other,more,stuff" V 3280 6400 60  0001 C CNN "Field8"
+F 2 "SM0805-C1" V 1130 2600 60  0001 C CNN
+F 4 "avx,08051C104KAT2A" V 1130 2600 60  0001 C CNN "mfg,mfg#"
+F 5 "newark,96M1354" V 1130 2600 60  0001 C CNN "vend1,vend1#"
+F 6 "" V 1130 2600 60  0001 C CNN ""
+F 7 "" V 1130 2600 60  0001 C CNN ""
+F 8 "100V" V 1130 2600 60  0001 C CNN "V"
+F 9 "10%" V 1130 2600 60  0001 C CNN "tolerance"
+F 10 "ceramic" V 1130 2600 60  0001 C CNN "construct"
+F 11 "other,more,stuff" V 1130 2600 60  0001 C CNN "misc"
 	1    6200 5300
 	0    -1   -1   0

Commit message: Looks like the bulk components are golden now, there are still a couple straglers, mostly switch mode power supply stuff.
Signed-off-by: Jared Harvey <TortiseGIT@jaredharvey.com>
Parts:
- R701, R702, R703, R704, R705, R706, R707, R708, R709, R710, R711, R712: Field3 -,- -> (none); Field4 -,- -> (none); Field5 -,V -> (none); Field6 -,% -> (none); Field7 na -> (none); Field8 other,more,stuff -> (none); mfg,# vishay,CRCW08050000ZSTA -> (none); mfg,mfg# (none) -> vishay,CRCW08050000Z0EA; misc (none) -> other,more,stuff; tolerance (none) -> %; vend,# newark,36C9353 -> (none); vend1,vend1# (none) -> newark,52K9721; w (none) -> mW

Commit message: harness connector is much more ironed out now. CPU is not connected.
Signed-off-by: Jared Harvey <TortiseGIT@jaredharvey.com>
Connections:
- net labels added: GND_MC33879
Changed lines of the file:
@@
-EESchema Schematic File Version 2  date 8/14/2011 8:37:17 PM
+EESchema Schematic File Version 2  date 8/19/2011 6:13:41 AM
 LIBS:power
 LIBS:device
@@
 $Descr User 11000 8500
 encoding utf-8
-Sheet 7 13
+Sheet 8 13
 Title "freeEMS PLUS from Cinch template "
-Date "14 aug 2011"
-Rev "A"
+Date "19 aug 2011"
+Rev "A-DRAF"
 Comp "diyefi.org/openecu.info"
 Comment1 "Stepper motor control"
@@
 GND_PWR8
 Text Label 6450 4775 0    60   ~ 0
-GND_PWR8
+GND_MC33879
 Text HLabel 6400 4775 0    60   Input ~ 0
-GND_PWR8
+GND_MC33879
 Text HLabel 9750 6300 2    60   Input ~ 0
 D5_PIN

Commit message: several pins on the SOM are now connected.
Signed-off-by: Jared Harvey <TortiseGIT@jaredharvey.com>
Parts:
- renumbered C701 to C801, C702 to C802, C703 to C803, C704 to C804, P701 to P801, P702 to P802, P703 to P803, P704 to P804, R701 to R801, R702 to R802, R703 to R803, R704 to R804, R705 to R805, R706 to R806, R707 to R807, R708 to R808, R709 to R809, R710 to R810, R711 to R811, R712 to R812, U701 to U801
Changed lines of the file:
@@
-EESchema Schematic File Version 2  date 8/19/2011 6:13:41 AM
+EESchema Schematic File Version 2  date 8/20/2011 7:18:55 AM
 LIBS:power
 LIBS:device
@@
 Sheet 8 13
 Title "freeEMS PLUS from Cinch template "
-Date "19 aug 2011"
+Date "20 aug 2011"
 Rev "A-DRAF"
 Comp "diyefi.org/openecu.info"
@@
 D8_PIN
 $Comp
-L R R711
+L R R811
 U 1 1 4C1B4C13
 P 9250 5875
-F 0 "R711" V 9195 6125 50  0000 C CNN
+F 0 "R811" V 9195 6125 50  0000 C CNN
 F 1 "0R" V 9250 5875 50  0000 C CNN
 F 2 "SM0805" V 1130 2600 60  0001 C CNN
@@
 $EndComp
 $Comp
-L R R707
+L R R807
 U 1 1 4C1B4C00
 P 9100 6200
-F 0 "R707" V 9050 5930 50  0000 C CNN
+F 0 "R807" V 9050 5930 50  0000 C CNN
 F 1 "0R" V 9100 6200 50  0000 C CNN
 F 2 "SM0805" V 1130 2600 60  0001 C CNN
@@
 $EndComp
 $Comp
-L R R709
+L R R809
 U 1 1 4C1B4BAE
 P 9200 6400
-F 0 "R709" V 9260 6670 50  0000 C CNN
+F 0 "R809" V 9260 6670 50  0000 C CNN
 F 1 "0R" V 9200 6400 50  0000 C CNN
 F 2 "SM0805" V 1130 2600 60  0001 C CNN
@@
 $EndComp
 $Comp
-L R R708
+L R R808
 U 1 1 4C1B4B98
 P 9125 5500
-F 0 "R708" V 9035 5505 50  0000 C CNN
+F 0 "R808" V 9035 5505 50  0000 C CNN
 F 1 "0R" V 9125 5500 50  0000 C CNN
 F 2 "SM0805" V 1130 2600 60  0001 C CNN
@@
 $EndComp
 $Comp
-L R R706
+L R R806
 U 1 1 4C1B4B33
 P 7325 6400
-F 0 "R706" V 7375 6685 50  0000 C CNN
+F 0 "R806" V 7375 6685 50  0000 C CNN
 F 1 "0R" V 7325 6400 50  0000 C CNN
 F 2 "SM0805" V 1130 2600 60  0001 C CNN
@@
 $EndComp
 $Comp
-L R R703
+L R R803
 U 1 1 4C1B4A76
 P 7275 5400
-F 0 "R703" V 7355 5400 50  0000 C CNN
+F 0 "R803" V 7355 5400 50  0000 C CNN
 F 1 "0R" V 7275 5400 50  0000 C CNN
 F 2 "SM0805" V 1130 2600 60  0001 C CNN
@@
 $EndComp
 $Comp
-L R R705
+L R R805
 U 1 1 4C1B4A43
 P 7300 6200
-F 0 "R705" V 7350 6450 50  0000 C CNN
+F 0 "R805" V 7350 6450 50  0000 C CNN
 F 1 "0R" V 7300 6200 50  0000 C CNN
 F 2 "SM0805" V 1130 2600 60  0001 C CNN
@@
 $EndComp
 $Comp
-L R R704
+L R R804
 U 1 1 4C1B4A0A
 P 7300 5800
-F 0 "R704" V 7380 5800 50  0000 C CNN
+F 0 "R804" V 7380 5800 50  0000 C CNN
 F 1 "0R" V 7300 5800 50  0000 C CNN
 F 2 "SM0805" V 1130 2600 60  0001 C CNN
@@
 $EndComp
 $Comp
-L R R702
+L R R802
 U 1 1 4C1B47F7
 P 6900 6300
-F 0 "R702" V 6975 6175 50  0000 C CNN
+F 0 "R802" V 6975 6175 50  0000 C CNN
 F 1 "0R" V 6900 6300 50  0000 C CNN
 F 2 "SM0805" V 1130 2600 60  0001 C CNN
@@
 $EndComp
 $Comp
-L R R701
+L R R801
 U 1 1 4C1B47D6
 P 6875 5700
-F 0 "R701" V 6955 5700 50  0000 C CNN
+F 0 "R801" V 6955 5700 50  0000 C CNN
 F 1 "0R" V 6875 5700 50  0000 C CNN
 F 2 "SM0805" V 1130 2600 60  0001 C CNN
@@
 $EndComp
 $Comp
-L R R710
+L R R810
 U 1 1 4C1B4798
 P 9250 5700
-F 0 "R710" V 9300 5950 50  0000 C CNN
+F 0 "R810" V 9300 5950 50  0000 C CNN
 F 1 "0R" V 9250 5700 50  0000 C CNN
 F 2 "SM0805" V 1130 2600 60  0001 C CNN
@@
 $EndComp
 $Comp
-L R R712
+L R R812
 U 1 1 4C1B474F
 P 9325 6300
-F 0 "R712" V 9275 6600 50  0000 C CNN
+F 0 "R812" V 9275 6600 50  0000 C CNN
 F 1 "0R" V 9325 6300 50  0000 C CNN
 F 2 "SM0805" V 1130 2600 60  0001 C CNN
@@
 install or jumpers for stepper motor driver.
 $Comp
-L C C702
+L C C802
 U 1 1 4C0F6A72
 P 6525 5800
-F 0 "C702" H 6550 5900 50  0000 L CNN
+F 0 "C802" H 6550 5900 50  0000 L CNN
 F 1 "10uF" H 6275 5900 50  0000 L CNN
 F 2 "SM0805-C1" V 3605 6900 60  0001 C CNN
@@
 VBAT
 $Comp
-L CONN_1 P701
+L CONN_1 P801
 U 1 1 4C0F68D7
 P 6350 5600
-F 0 "P701" H 6430 5600 40  0000 L CNN
+F 0 "P801" H 6430 5600 40  0000 L CNN
 F 1 "CONN_1" H 6350 5655 30  0001 C CNN
 F 2 "PINTST" H 6350 5600 60  0001 C CNN
@@
 $EndComp
 $Comp
-L CONN_1 P702
+L CONN_1 P802
 U 1 1 4C0F68D6
 P 6350 6100
-F 0 "P702" H 6430 6100 40  0000 L CNN
+F 0 "P802" H 6430 6100 40  0000 L CNN
 F 1 "CONN_1" H 6350 6155 30  0001 C CNN
 F 2 "PINTST" H 6350 6100 60  0001 C CNN
@@
 $EndComp
 $Comp
-L C C701
+L C C801
 U 1 1 4C0F6880
 P 6200 5300
-F 0 "C701" V 6120 5160 50  0000 L CNN
+F 0 "C801" V 6120 5160 50  0000 L CNN
 F 1 "100nF" V 6125 5500 50  0000 L CNN
 F 2 "SM0805-C1" V 1130 2600 60  0001 C CNN
@@
 879_MOSI
 $Comp
-L MC33879 U701
+L MC33879 U801
 U 1 1 4C0F6129
 P 8200 5950
-F 0 "U701" H 8200 6800 70  0000 C CNN
+F 0 "U801" H 8200 6800 70  0000 C CNN
 F 1 "MC33879" H 8200 5100 70  0000 C CNN
 F 2 "SOIC32" H 8200 5950 60  0001 C CNN
@@
 879_SCLK
 $Comp
-L CONN_1 P704
+L CONN_1 P804
 U 1 1 4C0A3402
 P 9900 6100
-F 0 "P704" H 9980 6100 40  0000 L CNN
+F 0 "P804" H 9980 6100 40  0000 L CNN
 F 1 "CONN_1" H 9900 6155 30  0001 C CNN
 F 2 "PINTST" H 9900 6100 60  0001 C CNN
@@
 $EndComp
 $Comp
-L CONN_1 P703
+L CONN_1 P803
 U 1 1 4C0A2746
 P 9900 5600
-F 0 "P703" H 9980 5600 40  0000 L CNN
+F 0 "P803" H 9980 5600 40  0000 L CNN
 F 1 "CONN_1" H 9900 5655 30  0001 C CNN
 F 2 "PINTST" H 9900 5600 60  0001 C CNN
@@
 VBAT
 $Comp
-L C C704
+L C C804
 U 1 1 4BF507DC
 P 10125 5300
-F 0 "C704" V 10175 5495 50  0000 L CNN
+F 0 "C804" V 10175 5495 50  0000 L CNN
 F 1 "10uF" V 10050 5100 50  0000 L CNN
 F 2 "SM0805-C1" V 7205 6400 60  0001 C CNN
@@
 $EndComp
 $Comp
-L C C703
+L C C803
 U 1 1 4BF507A3
 P 6525 6375
-F 0 "C703" H 6620 6470 50  0000 L CNN
+F 0 "C803" H 6620 6470 50  0000 L CNN
 F 1 "10uF" H 6275 6475 50  0000 L CNN
 F 2 "SM0805-C1" V 3605 7475 60  0001 C CNN
