File: KICAD_Project/sub_circuits/stepper_mc33879.sch (KiCad schematic (older format))
At the start: 21 parts, among them P801 CONN_1, P802 CONN_1, P803 CONN_1, P804 CONN_1, U801 MC33879

Commit message: more stepper updates
Signed-off-by: Jared Harvey <TortiseGIT@jaredharvey.com>
Parts:
- C802, C803, C804: Field3 -,- -> (none); Field4 -,- -> (none); Field5 200,V -> (none); Field6 20,% -> (none); Field7 alum electro -> (none); Field8 other,more,stuff -> (none); V (none) -> 25V; construct (none) -> multi layer ceramic; mfg,# ill cap,106CKE200M -> (none); mfg,mfg# (none) -> AVX,08053C104KAT2A; misc (none) -> other,more,stuff; tolerance (none) -> 10%; vend,# newark,69K7896 -> (none); vend1,vend1# (none) -> newark,96M1381
Changed lines of the file:
@@
 F 0 "C802" H 6550 5900 50  0000 L CNN
 F 1 "10uF" H 6275 5900 50  0000 L CNN
-F 2 "SM0805-C1" V 3605 6900 60  0001 C CNN
-F 4 "ill cap,106CKE200M" V 3605 6900 60  0001 C CNN "mfg,#"
-F 5 "newark,69K7896" V 3605 6900 60  0001 C CNN "vend,#"
-F 6 "-,-" V 3605 6900 60  0001 C CNN "Field3"
-F 7 "-,-" V 3605 6900 60  0001 C CNN "Field4"
-F 8 "200,V" V 3605 6900 60  0001 C CNN "Field5"
-F 9 "20,%" V 3605 6900 60  0001 C CNN "Field6"
-F 10 "alum electro" V 3605 6900 60  0001 C CNN "Field7"
-F 11 "other,more,stuff" V 3605 6900 60  0001 C CNN "Field8"
+F 2 "SM0805-C1" V 1130 2600 60  0001 C CNN
+F 4 "AVX,08053C104KAT2A" V 1130 2600 60  0001 C CNN "mfg,mfg#"
+F 5 "newark,96M1381" V 1130 2600 60  0001 C CNN "vend1,vend1#"
+F 6 "" V 1130 2600 60  0001 C CNN ""
+F 7 "" V 1130 2600 60  0001 C CNN ""
+F 8 "25V" V 1130 2600 60  0001 C CNN "V"
+F 9 "10%" V 1130 2600 60  0001 C CNN "tolerance"
+F 10 "multi layer ceramic" V 1130 2600 60  0001 C CNN "construct"
+F 11 "other,more,stuff" V 1130 2600 60  0001 C CNN "misc"
 	1    6525 5800
 	1    0    0    1
@@
 F 0 "C804" V 10175 5495 50  0000 L CNN
 F 1 "10uF" V 10050 5100 50  0000 L CNN
-F 2 "SM0805-C1" V 7205 6400 60  0001 C CNN
-F 4 "ill cap,106CKE200M" V 3605 6900 60  0001 C CNN "mfg,#"
-F 5 "newark,69K7896" V 3605 6900 60  0001 C CNN "vend,#"
-F 6 "-,-" V 3605 6900 60  0001 C CNN "Field3"
-F 7 "-,-" V 3605 6900 60  0001 C CNN "Field4"
-F 8 "200,V" V 3605 6900 60  0001 C CNN "Field5"
-F 9 "20,%" V 3605 6900 60  0001 C CNN "Field6"
-F 10 "alum electro" V 3605 6900 60  0001 C CNN "Field7"
-F 11 "other,more,stuff" V 3605 6900 60  0001 C CNN "Field8"
+F 2 "SM0805-C1" V 1130 2600 60  0001 C CNN
+F 4 "AVX,08053C104KAT2A" V 1130 2600 60  0001 C CNN "mfg,mfg#"
+F 5 "newark,96M1381" V 1130 2600 60  0001 C CNN "vend1,vend1#"
+F 6 "" V 1130 2600 60  0001 C CNN ""
+F 7 "" V 1130 2600 60  0001 C CNN ""
+F 8 "25V" V 1130 2600 60  0001 C CNN "V"
+F 9 "10%" V 1130 2600 60  0001 C CNN "tolerance"
+F 10 "multi layer ceramic" V 1130 2600 60  0001 C CNN "construct"
+F 11 "other,more,stuff" V 1130 2600 60  0001 C CNN "misc"
 	1    10125 5300
 	0    1    -1   0
@@
 F 0 "C803" H 6620 6470 50  0000 L CNN
 F 1 "10uF" H 6275 6475 50  0000 L CNN
-F 2 "SM0805-C1" V 3605 7475 60  0001 C CNN
-F 4 "ill cap,106CKE200M" V 3605 6900 60  0001 C CNN "mfg,#"
-F 5 "newark,69K7896" V 3605 6900 60  0001 C CNN "vend,#"
-F 6 "-,-" V 3605 6900 60  0001 C CNN "Field3"
-F 7 "-,-" V 3605 6900 60  0001 C CNN "Field4"
-F 8 "200,V" V 3605 6900 60  0001 C CNN "Field5"
-F 9 "20,%" V 3605 6900 60  0001 C CNN "Field6"
-F 10 "alum electro" V 3605 6900 60  0001 C CNN "Field7"
-F 11 "other,more,stuff" V 3605 6900 60  0001 C CNN "Field8"
+F 2 "SM0805-C1" V 1130 2600 60  0001 C CNN
+F 4 "AVX,08053C104KAT2A" V 1130 2600 60  0001 C CNN "mfg,mfg#"
+F 5 "newark,96M1381" V 1130 2600 60  0001 C CNN "vend1,vend1#"
+F 6 "" V 1130 2600 60  0001 C CNN ""
+F 7 "" V 1130 2600 60  0001 C CNN ""
+F 8 "25V" V 1130 2600 60  0001 C CNN "V"
+F 9 "10%" V 1130 2600 60  0001 C CNN "tolerance"
+F 10 "multi layer ceramic" V 1130 2600 60  0001 C CNN "construct"
+F 11 "other,more,stuff" V 1130 2600 60  0001 C CNN "misc"
 	1    6525 6375
 	1    0    0    1

Commit message: Made more progress on the AN protects and LS drive 33800
Signed-off-by: Jared Harvey <TortiseGIT@jaredharvey.com>
Parts:
- C801: footprint SM0805-C1 -> SM0805; TOL (none) -> 10%; V 100V -> 200V; construct ceramic -> CERAMIC; mfg,mfg# avx,08051C104KAT2A -> AVX,08055C104KAT2A; tolerance 10% -> (none); vend1,vend1# newark,96M1354 -> newark,27C8438
Changed lines of the file:
@@
 F 0 "C801" V 6120 5160 50  0000 L CNN
 F 1 "100nF" V 6125 5500 50  0000 L CNN
-F 2 "SM0805-C1" V 1130 2600 60  0001 C CNN
-F 4 "avx,08051C104KAT2A" V 1130 2600 60  0001 C CNN "mfg,mfg#"
-F 5 "newark,96M1354" V 1130 2600 60  0001 C CNN "vend1,vend1#"
-F 6 "" V 1130 2600 60  0001 C CNN "Field6"
-F 7 "" V 1130 2600 60  0001 C CNN "Field7"
-F 8 "100V" V 1130 2600 60  0001 C CNN "V"
-F 9 "10%" V 1130 2600 60  0001 C CNN "tolerance"
-F 10 "ceramic" V 1130 2600 60  0001 C CNN "construct"
+F 2 "SM0805" V 1130 2600 60  0001 C CNN
+F 4 "AVX,08055C104KAT2A" V 1130 2600 60  0001 C CNN "mfg,mfg#"
+F 5 "newark,27C8438" V 1130 2600 60  0001 C CNN "vend1,vend1#"
+F 6 "" V 1130 2600 60  0001 C CNN ""
+F 7 "" V 1130 2600 60  0001 C CNN ""
+F 8 "200V" V 1130 2600 60  0001 C CNN "V"
+F 9 "10%" V 1130 2600 60  0001 C CNN "TOL"
+F 10 "CERAMIC" V 1130 2600 60  0001 C CNN "construct"
 F 11 "other,more,stuff" V 1130 2600 60  0001 C CNN "misc"
 	1    6200 5300
