File: KICAD_Project/sub_circuits/SENSOR_INPUTS.sch (KiCad schematic (older format))
At the start: 73 parts, among them U5 MPX4100A, U6 MPX4250A

Commit message: More work to capture, also I need it up there for collaboration purposes.
Signed-off-by: Jared Harvey <TortiseGIT@jaredharvey.com>
Parts:
- removed R? (x3): 1k, SM0805-R4, symbol R
- added C?: 15nf, SM0805-C1, symbol C
- added C?: .1uF, SM0805-C1, symbol C
- added D? (x2): MBR0520L, SOD123, symbol DIODE
- added R? (x4): 470R, SM0805-R4, symbol R
Connections:
- net labels added: AN_CPU_MISC2, AN_HARN_MISC2
- wire segments 138 -> 195
Other:
- moved on the sheet: C?, D?, R?

Commit message: About to runs scripts to scrub the BOM's, so here's a backup copy in case it goes wrong.
Signed-off-by: Jared Harvey <TortiseGIT@jaredharvey.com>
Parts:
- removed C? (x5): 15nf, SM0805-C1, symbol C
- removed C? (x2): 0.1uF, symbol C
- removed C? (x4): .1uF, SM0805-C1, symbol C
- removed D? (x10): MBR0520L, SOD123, symbol DIODE
- removed R? (x5): 470R, SM0805-R4, symbol R
- removed U?: MAX31855, symbol MAX31855
- added C1201, C1202: 0.1uF, SM0805, symbol C
- added C1203, C1204, C1205, C1206, C1207: 15nf, SM0805-C1, symbol C
- added C1209, C1210, C1211, C1212: .1uF, SM0805-C1, symbol C
- added D1201, D1202, D1203, D1204, D1205, D1206, D1207, D1208, D1209, D1210: MBR0520L, SOD-123, symbol DIODE
- added R1201, R1202, R1203, R1204, R1205: 470R, SM0805, symbol R
- added R1207: 2K4, SM0805-R4, symbol R
- added U1202: MAX31855, -SOIC8, symbol MAX31855
- C1208: renamed from C?; Field3 -,- -> (none); Field4 -,- -> (none); Field5 50,V -> (none); mfg (none) -> avx; mfg# (none) -> 08051C104KAT2A; vend,# newark, -> (none); vend1 (none) -> newark; vend1# (none) -> 96M1354
- R1210, R1211, R1214, R1216, R1218, R1219: renamed from R?; footprint SM0805-R4 -> SM0805
- R1212, R1213, R1215, R1217, R1220, R1221: renamed from R; footprint SM0805-R4 -> SM0805
- U1201: renamed from U?; footprint (none) -> -SOIC8; MFG (none) -> MAXIM; MFG# (none) -> MAX31855NASA+; VEND1 (none) -> MOUSER; VEND1# (none) -> 700-MAX31855NASA+
- gave numbers to parts that had none: 16
- renumbered C to C1215, C to C1216, C to C1218, C66 to C1219, C23 to C1221, C24 to C1222, C19 to C1225, C20 to C1226, C21 to C1227, C to C1230, C to C1231, C to C1234, C to C1235, P to P1203, P to P1204, R105 to R1208, R106 to R1209, R134 to R1222, U to U1204, U6 to U1205, U5 to U1207
Connections:
- wire segments 195 -> 143

Commit message: caps have been done with the scripts next up is the resistors.
Signed-off-by: Jared Harvey <TortiseGIT@jaredharvey.com>
Parts:
- C1201, C1202, C1221, C1223, C1225: footprint SM0805 -> SM0805-C1; V (none) -> 100V; Voltage 50v -> (none); mfg Murata -> (none); mfg# GRM21BR71H104KA01L -> (none); mfg,mfg# (none) -> avx,08051C104KAT2A; vend1 digikey -> (none); vend1# 490-1666-2-ND -> (none); vend1,vend1# (none) -> newark,96M1354
- C1208, C1209, C1210, C1211, C1212: value .1uF -> 0.1uF; Field6 10,% -> (none); Field7 Ceramic -> (none); Field8 other,more,stuff -> (none); V (none) -> 100V; construct (none) -> ceramic; mfg avx -> (none); mfg# 08051C104KAT2A -> (none); mfg,mfg# (none) -> avx,08051C104KAT2A; misc (none) -> other,more,stuff; tolerance (none) -> 10%; vend1 newark -> (none); vend1# 96M1354 -> (none); vend1,vend1# (none) -> newark,96M1354
- C1219, C1220: footprint SM0805 -> SM0805-C1; V (none) -> 25V; mfg AVX -> (none); mfg# 08055C333KAZ2A -> (none); mfg,mfg# (none) -> yageo,CC0805KRX7R8BB333; tol 10% -> (none); tolerance (none) -> 10%; vend1 digikey -> (none); vend1# 478-3550-1-ND -> (none); vend1,vend1# (none) -> newark,69C9599; voltage 50 -> (none)
- C1226: value .01uF -> 10nF; footprint SM0805 -> SM0805-C1; V (none) -> 200V; Voltate 50v -> (none); construct ??? -> alum elec; mfg Murata -> (none); mfg# GRM216R71H103KA01D -> (none); mfg,mfg# (none) -> ill cap,106CKE200M; tol 10% -> (none); tolerance (none) -> 10%; vend1 digikey -> (none); vend1# 490-1664-1-ND -> (none); vend1,vend1# (none) -> newark,69K7896
- C1229, C1231: value .1uF -> 0.1uF; Field3 - -> (none); Field4 - -> (none); Field5 100,v -> (none); Field6 10,% -> (none); Field7 ceramic -> (none); Field8 - -> (none); V (none) -> 100V; construct (none) -> ceramic; mfg,# avx,08051C104KAT2A -> (none); mfg,mfg# (none) -> avx,08051C104KAT2A; misc (none) -> other,more,stuff; tolerance (none) -> 10%; vend,# newark,96M1354 -> (none); vend1,vend1# (none) -> newark,96M1354
- C1232, C1234: Field3 - -> (none); Field4 - -> (none); Field5 50,v -> (none); Field6 10,% -> (none); Field7 ceramic -> (none); Field8 - -> (none); V (none) -> 100V; construct (none) -> ceramic; mfg,# murata,GRM21BR71H104KA01L -> (none); mfg,mfg# (none) -> avx,08051C104KAT2A; misc (none) -> other,more,stuff; tolerance (none) -> 10%; vend,# newark,38K1694 -> (none); vend1,vend1# (none) -> newark,96M1354

Commit message: Looks like the bulk components are golden now, there are still a couple straglers, mostly switch mode power supply stuff.
Signed-off-by: Jared Harvey <TortiseGIT@jaredharvey.com>
Parts:
- R1206, R1207: footprint SM0805-R4 -> SM0805; Field3 -,- -> (none); Field4 -,- -> (none); Field5 125,mW -> (none); Field6 1,% -> (none); Field7 thick film -> (none); Field8 other,more,stuff -> (none); construct (none) -> thin film; mfg,mfg# (none) -> vishay,TNPW08052K49BEEA; misc (none) -> other,more,stuff; tolerance (none) -> .1%; vend1,vend1# (none) -> newark,05R1646; w (none) -> 125mW
- R1209: mfg Stackpole -> (none); mfg# RMCF0805JT10K0CT -> (none); mfg,mfg# (none) -> BOURNS,CR0805-FX-1002ELF; power .125w -> (none); tol 5% -> (none); tolerance (none) -> 1%; vend1 digikey -> (none); vend1# RMCF0805JT10K0CT-ND -> (none); vend1,vend1# (none) -> newark,02J2368; w (none) -> 125mW
- R1214, R1215, R1216, R1217: Field3 - -> (none); Field4 - -> (none); Field5 125,mW -> (none); Field6 1,% -> (none); Field7 thick film -> (none); Field8 - -> (none); construct (none) -> thick film; mfg,# bourns,CR0805-FX-1002ELF -> (none); mfg,mfg# (none) -> BOURNS,CR0805-FX-1002ELF; misc (none) -> other,more,stuff; tolerance (none) -> 1%; vend,# newark,02J2368 -> (none); vend1,vend1# (none) -> newark,02J2368; w (none) -> 125mW

Commit message: harness connector is much more ironed out now. CPU is not connected.
Signed-off-by: Jared Harvey <TortiseGIT@jaredharvey.com>
Parts:
- removed C1205, C1206: 15nf, SM0805-C1, symbol C
- removed C1210, C1211: 0.1uF, SM0805-C1, symbol C
- removed D1205, D1206, D1207, D1208: MBR0520L, SOD-123, symbol DIODE
- removed R1203, R1204: 470R, SM0805, symbol R
Connections:
- net labels removed: AN_CPU_MISC, AN_CPU_MISC2, AN_HARN_MISC, AN_HARN_MISC2
- wire segments 143 -> 141

Commit message: several pins on the SOM are now connected.
Signed-off-by: Jared Harvey <TortiseGIT@jaredharvey.com>
Parts:
- renumbered C1201 to C1301, C1202 to C1302, C1203 to C1303, C1204 to C1304, C1207 to C1305, C1208 to C1306, C1209 to C1307, C1212 to C1308, C1213 to C1309, C1214 to C1310, C1215 to C1311, C1216 to C1312, C1217 to C1313, C1218 to C1314, C1219 to C1315, C1220 to C1316, C1221 to C1317, C1222 to C1318, C1223 to C1319, C1224 to C1320, C1225 to C1321, C1226 to C1322, C1227 to C1323, C1228 to C1324, C1229 to C1325, C1230 to C1326, C1231 to C1327, C1232 to C1328, C1233 to C1329, C1234 to C1330, C1235 to C1331, D1201 to D1301, D1202 to D1302, D1203 to D1303, D1204 to D1304, D1209 to D1305, D1210 to D1306, P1201 to P1301, P1202 to P1302, P1203 to P1303, P1204 to P1304, R1201 to R1301, R1202 to R1302, R1205 to R1303, R1206 to R1304, R1207 to R1305, R1208 to R1306, R1209 to R1307, R1210 to R1308, R1211 to R1309, R1212 to R1310, R1213 to R1311, R1214 to R1312, R1215 to R1313, R1216 to R1314, R1217 to R1315, R1218 to R1316, R1219 to R1317, R1220 to R1318, R1221 to R1319, R1222 to R1320, R1223 to R1321, U1201 to U1301, U1202 to U1302, U1203 to U1303, U1204 to U1304, U1205 to U1305, U1206 to U1306, U1207 to U1307

Commit message: routing has started
Signed-off-by: Jared Harvey <TortiseGIT@jaredharvey.com>
Changed lines of the file:
@@
-EESchema Schematic File Version 2  date 8/20/2011 7:18:56 AM
+EESchema Schematic File Version 2  date 8/20/2011 7:59:51 PM
 LIBS:power
 LIBS:device
@@
 U 1 1 4E39E4EC
 P 9975 4200
-F 0 "C1328" H 9850 4300 50  0000 L CNN
+F 0 "C1328" H 9700 4300 50  0000 L CNN
 F 1 "100nF" H 9700 4100 50  0000 L CNN
 F 2 "SM0805-C1" V 1130 2600 60  0001 C CNN
@@
 U 1 1 4C313468
 P 9975 5550
-F 0 "C1330" H 9850 5650 50  0000 L CNN
+F 0 "C1330" H 9700 5650 50  0000 L CNN
 F 1 "100nF" H 9700 5450 50  0000 L CNN
 F 2 "SM0805-C1" V 1130 2600 60  0001 C CNN
