File: KICAD_Project/sub_circuits/SENSOR_INPUTS.sch (KiCad schematic (older format))
At the start: 65 parts, among them U1301 MAX31855, U1302 MAX31855, U1303 MAX9939, U1304 MAX9939, U1305 MPX4250A, U1306 MPX4250A, U1307 MPX4100A

Commit message: Did a bit more layout work.
Signed-off-by: Jared Harvey <TortiseGIT@jaredharvey.com>
Parts:
- added U1203: SP723, SO8E, symbol SP723
Connections:
- wire segments 141 -> 162

Commit message: Changed AN protections to match QUCS simulation predictions.
Signed-off-by: Jared Harvey <TortiseGIT@jaredharvey.com>
Parts:
- C1303, C1304, C1305: value 15nf -> .01uf
- R1301, R1302, R1303: value 1k -> 2.2k
Changed lines of the file:
@@
-EESchema Schematic File Version 2  date 10/11/2011 7:34:30 AM
+EESchema Schematic File Version 2  date 10/14/2011 5:26:22 AM
 LIBS:power
 LIBS:device
@@
 Sheet 12 12
 Title "Open5xxxECU (o5e), an ECU that is no longer affiliated with freeEMS."
-Date "11 oct 2011"
+Date "14 oct 2011"
 Rev "A-DRAFT5"
 Comp "http://open5xxxecu.org/"
@@
 P 2450 5600
 F 0 "C1305" H 2500 5700 50  0000 L CNN
-F 1 "15nf" H 2500 5500 50  0000 L CNN
+F 1 ".01uf" H 2500 5500 50  0000 L CNN
 F 2 "SM0805-C1" V 280 6600 60  0001 C CNN
 F 4 "avx,08055C102KAT2A" V 130 10650 60  0001 C CNN "mfg,mfg#"
@@
 P 2450 2650
 F 0 "C1304" H 2500 2750 50  0000 L CNN
-F 1 "15nf" H 2500 2550 50  0000 L CNN
+F 1 ".01uf" H 2500 2550 50  0000 L CNN
 F 2 "SM0805-C1" V 280 3650 60  0001 C CNN
 F 4 "avx,08055C102KAT2A" V 130 7700 60  0001 C CNN "mfg,mfg#"
@@
 P 2750 5400
 F 0 "R1303" V 2830 5400 50  0000 C CNN
-F 1 "1k" V 2750 5400 50  0000 C CNN
+F 1 "2.2k" V 2750 5400 50  0000 C CNN
 F 2 "SM0805" V 1130 2600 60  0001 C CNN
 F 4 "vishay,CRCW08051K00FKTA" V 1130 2600 60  0001 C CNN "mfg,mfg#"
@@
 P 2750 2450
 F 0 "R1302" V 2830 2450 50  0000 C CNN
-F 1 "1k" V 2750 2450 50  0000 C CNN
+F 1 "2.2k" V 2750 2450 50  0000 C CNN
 F 2 "SM0805" V 1130 2600 60  0001 C CNN
 F 4 "vishay,CRCW08051K00FKTA" V 1130 2600 60  0001 C CNN "mfg,mfg#"
@@
 P 2750 1450
 F 0 "R1301" V 2830 1450 50  0000 C CNN
-F 1 "1k" V 2750 1450 50  0000 C CNN
+F 1 "2.2k" V 2750 1450 50  0000 C CNN
 F 2 "SM0805" V 1130 2600 60  0001 C CNN
 F 4 "vishay,CRCW08051K00FKTA" V 1130 2600 60  0001 C CNN "mfg,mfg#"
@@
 P 2450 1650
 F 0 "C1303" H 2500 1750 50  0000 L CNN
-F 1 "15nf" H 2500 1550 50  0000 L CNN
+F 1 ".01uf" H 2500 1550 50  0000 L CNN
 F 2 "SM0805-C1" V 280 2650 60  0001 C CNN
 F 4 "avx,08055C102KAT2A" V 130 6700 60  0001 C CNN "mfg,mfg#"

Commit message: Made more progress on the AN protects and LS drive 33800
Signed-off-by: Jared Harvey <TortiseGIT@jaredharvey.com>
Parts:
- removed D1302, D1304, D1306: ZENER, SOD-123, symbol ZENER
- added D1302, D1304, D1306: L-AN-D, SOD-123, symbol DIODE
- C1303, C1304, C1305: footprint SM0805-C1 -> SM0805; % (none) -> 10%; Field5 50,V -> (none); Field6 10,% -> (none); Field7 Ceramic -> (none); Field8 other,more,stuff -> (none); V (none) -> 50V; construct (none) -> ceramic; mfg,mfg# avx,08055C102KAT2A -> avx,08055C103KAT2A; misc (none) -> other,more,stuff; vend1,vend1# digi,478-1371-6-ND -> newark,07J3575
- C1306, C1307, C1308: footprint SM0805-C1 -> SM0805
- C1322: footprint SM0805-C1 -> SM0805; TOL (none) -> 10%; V 200V -> 50V; construct alum elec -> CERAMIC; mfg,mfg# ill cap,106CKE200M -> AVX,08055C103KAT2A; tolerance 10% -> (none); vend1,vend1# newark,69K7896 -> newark,07J3575
- C1328, C1330: TOL (none) -> 10%; V 100V -> 200V; construct ceramic -> CERAMIC; mfg,mfg# avx,08051C104KAT2A -> AVX,08055C104KAT2A; tolerance 10% -> (none); vend1,vend1# newark,96M1354 -> newark,27C8438
- D1301, D1303, D1305: value MBR0520L -> H-AN-D; Field3 -,- -> (none); Field4 -,- -> (none); Field5 20,V-reverse -> (none); Field6 .5,A-forward -> (none); Field7 SMT -> (none); Field8 other,more,stuff -> (none); construct (none) -> schottky; forward A (none) -> 200mA; mfg,# fairchild,MBR0520L -> (none); mfg,mfg# (none) -> ON-SEMI,BAT54T1G; misc (none) -> other,more,stuff; reverse V (none) -> 30V; vend,# mouser,512-MBR0520L -> (none); vend1,vend1# (none) -> NEWARK,67R1284
- R1301, R1302, R1303: % (none) -> 1%; TOL 1% -> (none); W 125mW -> .125W; construct THICK FILM -> thick film; mfg,mfg# vishay,CRCW08051K00FKTA -> vishay,CRCW08052K21FKEA; vend1,vend1# newark,05F1507 -> newark,52K9952
Other:
- note added: "TYP TPS wiper ranges from 1k, to 10k."

Commit message: about to position the regulators, save it as a backup copy
Signed-off-by: Jared Harvey <TortiseGIT@jaredharvey.com>
Parts:
- C1301, C1302, C1315, C1316, C1317, C1319, C1321: footprint SM0805-C1 -> SM0805
Changed lines of the file:
@@
-EESchema Schematic File Version 2  date 10/20/2011 5:18:40 AM
+EESchema Schematic File Version 2  date 10/21/2011 6:23:35 AM
 LIBS:power
 LIBS:device
@@
 Sheet 12 12
 Title "Open5xxxECU (o5e), an ECU that is no longer affiliated with freeEMS."
-Date "20 oct 2011"
-Rev "A-DRAFT6"
+Date "21 oct 2011"
+Rev "A-DRAFT7"
 Comp "http://open5xxxecu.org/"
 Comment1 "misc input signals"
@@
 F 0 "C1301" H 850 6750 50  0000 L CNN
 F 1 "0.1uF" H 850 6550 50  0000 L CNN
-F 2 "SM0805-C1" V 1130 2600 60  0001 C CNN
+F 2 "SM0805" V 1130 2600 60  0001 C CNN
 F 4 "avx,08051C104KAT2A" V 1130 2600 60  0001 C CNN "mfg,mfg#"
 F 5 "newark,96M1354" V 1130 2600 60  0001 C CNN "vend1,vend1#"
-F 6 "" V 1130 2600 60  0001 C CNN "Field6"
-F 7 "" V 1130 2600 60  0001 C CNN "Field7"
-F 8 "100V" V 1130 2600 60  0001 C CNN "V"
-F 9 "10%" V 1130 2600 60  0001 C CNN "tolerance"
-F 10 "ceramic" V 1130 2600 60  0001 C CNN "construct"
-F 11 "other,more,stuff" V 1130 2600 60  0001 C CNN "misc"
+F 6 "100V" V 1130 2600 60  0001 C CNN "V"
+F 7 "10%" V 1130 2600 60  0001 C CNN "tolerance"
+F 8 "ceramic" V 1130 2600 60  0001 C CNN "construct"
+F 9 "other,more,stuff" V 1130 2600 60  0001 C CNN "misc"
 	1    800  6650
 	1    0    0    -1
@@
 F 0 "C1302" H 1250 6750 50  0000 L CNN
 F 1 "0.1uF" H 1250 6550 50  0000 L CNN
-F 2 "SM0805-C1" V 1130 2600 60  0001 C CNN
+F 2 "SM0805" V 1130 2600 60  0001 C CNN
 F 4 "avx,08051C104KAT2A" V 1130 2600 60  0001 C CNN "mfg,mfg#"
 F 5 "newark,96M1354" V 1130 2600 60  0001 C CNN "vend1,vend1#"
-F 6 "" V 1130 2600 60  0001 C CNN "Field6"
-F 7 "" V 1130 2600 60  0001 C CNN "Field7"
-F 8 "100V" V 1130 2600 60  0001 C CNN "V"
-F 9 "10%" V 1130 2600 60  0001 C CNN "tolerance"
-F 10 "ceramic" V 1130 2600 60  0001 C CNN "construct"
-F 11 "other,more,stuff" V 1130 2600 60  0001 C CNN "misc"
+F 6 "100V" V 1130 2600 60  0001 C CNN "V"
+F 7 "10%" V 1130 2600 60  0001 C CNN "tolerance"
+F 8 "ceramic" V 1130 2600 60  0001 C CNN "construct"
+F 9 "other,more,stuff" V 1130 2600 60  0001 C CNN "misc"
 	1    1200 6650
 	1    0    0    -1
@@
 F 0 "C1319" H 7850 2000 50  0000 L CNN
 F 1 "0.1uF" H 7850 1800 50  0000 L CNN
-F 2 "SM0805-C1" V 1130 2600 60  0001 C CNN
+F 2 "SM0805" V 1130 2600 60  0001 C CNN
 F 4 "avx,08051C104KAT2A" V 1130 2600 60  0001 C CNN "mfg,mfg#"
 F 5 "newark,96M1354" V 1130 2600 60  0001 C CNN "vend1,vend1#"
-F 6 "" V 1130 2600 60  0001 C CNN "Field6"
-F 7 "" V 1130 2600 60  0001 C CNN "Field7"
-F 8 "100V" V 1130 2600 60  0001 C CNN "V"
-F 9 "10%" V 1130 2600 60  0001 C CNN "tolerance"
-F 10 "ceramic" V 1130 2600 60  0001 C CNN "construct"
-F 11 "other,more,stuff" V 1130 2600 60  0001 C CNN "misc"
+F 6 "100V" V 1130 2600 60  0001 C CNN "V"
+F 7 "10%" V 1130 2600 60  0001 C CNN "tolerance"
+F 8 "ceramic" V 1130 2600 60  0001 C CNN "construct"
+F 9 "other,more,stuff" V 1130 2600 60  0001 C CNN "misc"
 	1    7800 1900
 	1    0    0    -1
@@
 F 0 "C1316" H 7350 2400 50  0000 L CNN
 F 1 "33nF" H 7350 2200 50  0000 L CNN
-F 2 "SM0805-C1" V 1130 2600 60  0001 C CNN
+F 2 "SM0805" V 1130 2600 60  0001 C CNN
 F 4 "yageo,CC0805KRX7R8BB333" V 1130 2600 60  0001 C CNN "mfg,mfg#"
 F 5 "newark,69C9599" V 1130 2600 60  0001 C CNN "vend1,vend1#"
-F 6 "" V 1130 2600 60  0001 C CNN "Field6"
-F 7 "" V 1130 2600 60  0001 C CNN "Field7"
-F 8 "25V" V 1130 2600 60  0001 C CNN "V"
-F 9 "10%" V 1130 2600 60  0001 C CNN "tolerance"
-F 10 "ceramic" V 1130 2600 60  0001 C CNN "construct"
-F 11 "other,more,stuff" V 1130 2600 60  0001 C CNN "misc"
+F 6 "25V" V 1130 2600 60  0001 C CNN "V"
+F 7 "10%" V 1130 2600 60  0001 C CNN "tolerance"
+F 8 "ceramic" V 1130 2600 60  0001 C CNN "construct"
+F 9 "other,more,stuff" V 1130 2600 60  0001 C CNN "misc"
 	1    7300 2300
 	1    0    0    -1
@@
 F 0 "C1315" H 7350 1400 50  0000 L CNN
 F 1 "33nF" H 7350 1200 50  0000 L CNN
-F 2 "SM0805-C1" V 1130 2600 60  0001 C CNN
+F 2 "SM0805" V 1130 2600 60  0001 C CNN
 F 4 "yageo,CC0805KRX7R8BB333" V 1130 2600 60  0001 C CNN "mfg,mfg#"
 F 5 "newark,69C9599" V 1130 2600 60  0001 C CNN "vend1,vend1#"
-F 6 "" V 1130 2600 60  0001 C CNN "Field6"
-F 7 "" V 1130 2600 60  0001 C CNN "Field7"
-F 8 "25V" V 1130 2600 60  0001 C CNN "V"
-F 9 "10%" V 1130 2600 60  0001 C CNN "tolerance"
-F 10 "ceramic" V 1130 2600 60  0001 C CNN "construct"
-F 11 "other,more,stuff" V 1130 2600 60  0001 C CNN "misc"
+F 6 "25V" V 1130 2600 60  0001 C CNN "V"
+F 7 "10%" V 1130 2600 60  0001 C CNN "tolerance"
+F 8 "ceramic" V 1130 2600 60  0001 C CNN "construct"
+F 9 "other,more,stuff" V 1130 2600 60  0001 C CNN "misc"
 	1    7300 1300
 	1    0    0    -1
@@
 F 0 "C1317" H 7850 1000 50  0000 L CNN
 F 1 "0.1uF" H 7850 800 50  0000 L CNN
-F 2 "SM0805-C1" V 1130 2600 60  0001 C CNN
+F 2 "SM0805" V 1130 2600 60  0001 C CNN
 F 4 "avx,08051C104KAT2A" V 1130 2600 60  0001 C CNN "mfg,mfg#"
 F 5 "newark,96M1354" V 1130 2600 60  0001 C CNN "vend1,vend1#"
-F 6 "" V 1130 2600 60  0001 C CNN "Field6"
-F 7 "" V 1130 2600 60  0001 C CNN "Field7"
-F 8 "100V" V 1130 2600 60  0001 C CNN "V"
-F 9 "10%" V 1130 2600 60  0001 C CNN "tolerance"
-F 10 "ceramic" V 1130 2600 60  0001 C CNN "construct"
-F 11 "other,more,stuff" V 1130 2600 60  0001 C CNN "misc"
+F 6 "100V" V 1130 2600 60  0001 C CNN "V"
+F 7 "10%" V 1130 2600 60  0001 C CNN "tolerance"
+F 8 "ceramic" V 1130 2600 60  0001 C CNN "construct"
+F 9 "other,more,stuff" V 1130 2600 60  0001 C CNN "misc"
 	1    7800 900
 	1    0    0    -1
@@
 F 0 "C1321" H 7850 3000 50  0000 L CNN
 F 1 "0.1uF" H 7850 2800 50  0000 L CNN
-F 2 "SM0805-C1" V 1130 2600 60  0001 C CNN
+F 2 "SM0805" V 1130 2600 60  0001 C CNN
 F 4 "avx,08051C104KAT2A" V 1130 2600 60  0001 C CNN "mfg,mfg#"
 F 5 "newark,96M1354" V 1130 2600 60  0001 C CNN "vend1,vend1#"
-F 6 "" V 1130 2600 60  0001 C CNN "Field6"
-F 7 "" V 1130 2600 60  0001 C CNN "Field7"
-F 8 "100V" V 1130 2600 60  0001 C CNN "V"
-F 9 "10%" V 1130 2600 60  0001 C CNN "tolerance"
-F 10 "ceramic" V 1130 2600 60  0001 C CNN "construct"
-F 11 "other,more,stuff" V 1130 2600 60  0001 C CNN "misc"
+F 6 "100V" V 1130 2600 60  0001 C CNN "V"
+F 7 "10%" V 1130 2600 60  0001 C CNN "tolerance"
+F 8 "ceramic" V 1130 2600 60  0001 C CNN "construct"
+F 9 "other,more,stuff" V 1130 2600 60  0001 C CNN "misc"
 	1    7800 2900
 	1    0    0    -1
