File: KICAD_Project/sub_circuits/power_reg.sch (KiCad schematic (older format))
At the start: 43 parts, among them U2 LM2937, U35 L5973D, U4 MCP1826

Commit message: About to runs scripts to scrub the BOM's, so here's a backup copy in case it goes wrong.
Signed-off-by: Jared Harvey <TortiseGIT@jaredharvey.com>
Parts:
- C521: renamed from C140; value T495X337K010ATE035 -> 330uF; mfg,# T495X337K010ATE035 -> kemet,T495X337K010ATE035
- gave numbers to parts that had none: 6
- renumbered C2 to C501, C3 to C503, C134 to C505, C8 to C506, C9 to C507, C135 to C508, C138 to C509, C5 to C510, C6 to C512, C139 to C514, C141 to C515, C10 to C516, C12 to C517, C11 to C518, C136 to C519, C137 to C520, C143 to C522, C144 to C523, D113 to D501, D117 to D502, D118 to D503, D92 to D504, D114 to D506, D4 to D507, D119 to D508, L1 to L501, L2 to L502, R260 to R501, R226 to R502, R265 to R503, R272 to R504, R273 to R505, R274 to R506, U2 to U501, U4 to U503, U35 to U504

Commit message: caps have been done with the scripts next up is the resistors.
Signed-off-by: Jared Harvey <TortiseGIT@jaredharvey.com>
Parts:
- C503, C504, C507, C512, C513, C517: footprint SM0805 -> SM0805-C1; V (none) -> 100V; Voltage 50v -> (none); mfg Murata -> (none); mfg# GRM21BR71H104KA01L -> (none); mfg,mfg# (none) -> avx,08051C104KAT2A; vend1 digikey -> (none); vend1# 490-1666-2-ND -> (none); vend1,vend1# (none) -> newark,96M1354
- C505, C509, C515: Field3 -,- -> (none); Field4 -,- -> (none); Field5 50,V -> (none); Field6 10,% -> (none); Field7 ceramic -> (none); Field8 other,more,stuff -> (none); V (none) -> 100V; construct (none) -> ceramic; mfg,# murata,GRM21BR71H104KA01L -> (none); mfg,mfg# (none) -> avx,08051C104KAT2A; misc (none) -> other,more,stuff; tolerance (none) -> 10%; vend,# newark,38K1694 -> (none); vend1,vend1# (none) -> newark,96M1354
- C523: Field3 -,- -> (none); Field4 -,- -> (none); Field5 50,V -> (none); Field6 5,% -> (none); Field7 ceramic -> (none); Field8 other,more,stuff -> (none); V (none) -> 200V; construct (none) -> alum elec; mfg,# murata,GRM216R71H103JA01D -> (none); mfg,mfg# (none) -> ill cap,106CKE200M; misc (none) -> other,more,stuff; tolerance (none) -> 10%; vend,# newark,38K1697 -> (none); vend1,vend1# (none) -> newark,69K7896

Commit message: Looks like the bulk components are golden now, there are still a couple straglers, mostly switch mode power supply stuff.
Signed-off-by: Jared Harvey <TortiseGIT@jaredharvey.com>
Parts:
- L502: Field3 -,- -> (none); Field4 -,- -> (none); Field5 1,a -> (none); Field6 20,% -> (none); Field7 - -> (none); Field8 other,more,stuff -> (none); H (none) -> 33uH; construct (none) -> ferrite; mfg,# DR125-330-R -> (none); mfg,mfg# (none) -> coiltronics,DR125-330-R; misc (none) -> other,more,stuff; tolerance (none) -> 20%; vend,# newark,63K3559 -> (none); vend1,vend1# (none) -> digi,513-1528-6-ND
- R502: construct Thick Film -> thick film; mfg Stackpole Electronics Inc -> (none); mfg# RMCF0805JT22K0CT -> (none); mfg,mfg# (none) -> BOURNS,CR0805-FX-1002ELF; power .250mW -> (none); tol 5% -> (none); tolerance (none) -> 1%; vend1 digikey -> (none); vend1# RMCF0805JT22K0CT-ND -> (none); vend1,vend1# (none) -> newark,02J2368; w (none) -> 125mW
- R503: construct (none) -> thick film; mfg,mfg# (none) -> vishay,CRCW0805100KFKEA; misc (none) -> other,more,stuff; tolerance (none) -> 1%; vend1,vend1# (none) -> newark,52K9808; w (none) -> 125mW
- U503: A (none) -> 1A; construct (none) -> LINEAR; mfg,mfg# (none) -> MICROCHIP,MCP1826T-ADJE/DC; misc (none) -> other,more,stuff; vend1,vend1# (none) -> newark,08N6496
Changed lines of the file:
@@
-EESchema Schematic File Version 2  date 8/14/2011 7:31:24 PM
+EESchema Schematic File Version 2  date 8/14/2011 8:37:16 PM
 LIBS:power
 LIBS:device
@@
 F 4 "avx,08051C104KAT2A" V 1130 2600 60  0001 C CNN "mfg,mfg#"
 F 5 "newark,96M1354" V 1130 2600 60  0001 C CNN "vend1,vend1#"
-F 6 "" V 1130 2600 60  0001 C CNN ""
-F 7 "" V 1130 2600 60  0001 C CNN ""
+F 6 "" V 1130 2600 60  0001 C CNN "Field6"
+F 7 "" V 1130 2600 60  0001 C CNN "Field7"
 F 8 "100V" V 1130 2600 60  0001 C CNN "V"
 F 9 "10%" V 1130 2600 60  0001 C CNN "tolerance"
@@
 F 4 "avx,08051C104KAT2A" V 1130 2600 60  0001 C CNN "mfg,mfg#"
 F 5 "newark,96M1354" V 1130 2600 60  0001 C CNN "vend1,vend1#"
-F 6 "" V 1130 2600 60  0001 C CNN ""
-F 7 "" V 1130 2600 60  0001 C CNN ""
+F 6 "" V 1130 2600 60  0001 C CNN "Field6"
+F 7 "" V 1130 2600 60  0001 C CNN "Field7"
 F 8 "100V" V 1130 2600 60  0001 C CNN "V"
 F 9 "10%" V 1130 2600 60  0001 C CNN "tolerance"
@@
 F 0 "L502" V 7400 1550 40  0000 C CNN
 F 1 "DR125-330-R" V 7550 1550 40  0000 C CNN
-F 2 "SM100uH" H 7450 1550 60  0001 C CNN
-F 3 "PF0504.473NL Pulse Eng" H 7450 1550 60  0001 C CNN
-F 4 "DR125-330-R" H 7450 1550 60  0001 C CNN "mfg,#"
-F 5 "newark,63K3559" H 7450 1550 60  0001 C CNN "vend,#"
-F 6 "-,-" V 5080 100 60  0001 C CNN "Field3"
-F 7 "-,-" V 5080 100 60  0001 C CNN "Field4"
-F 8 "1,a" V 5080 100 60  0001 C CNN "Field5"
-F 9 "20,%" V 5080 100 60  0001 C CNN "Field6"
-F 10 "-" V 5080 100 60  0001 C CNN "Field7"
-F 11 "other,more,stuff" V 5080 100 60  0001 C CNN "Field8"
+F 2 "SM100uH" V 1130 2600 60  0001 C CNN
+F 4 "coiltronics,DR125-330-R" V 1130 2600 60  0001 C CNN "mfg,mfg#"
+F 5 "digi,513-1528-6-ND" V 1130 2600 60  0001 C CNN "vend1,vend1#"
+F 6 "" V 1130 2600 60  0001 C CNN "Field6"
+F 7 "" V 1130 2600 60  0001 C CNN "Field7"
+F 8 "33uH" V 1130 2600 60  0001 C CNN "H"
+F 9 "20%" V 1130 2600 60  0001 C CNN "tolerance"
+F 10 "ferrite" V 1130 2600 60  0001 C CNN "construct"
+F 11 "other,more,stuff" V 1130 2600 60  0001 C CNN "misc"
 	1    7450 1550
 	0    1    1    0
@@
 F 4 "ill cap,106CKE200M" V 1130 2600 60  0001 C CNN "mfg,mfg#"
 F 5 "newark,69K7896" V 1130 2600 60  0001 C CNN "vend1,vend1#"
-F 6 "" V 1130 2600 60  0001 C CNN ""
-F 7 "" V 1130 2600 60  0001 C CNN ""
+F 6 "" V 1130 2600 60  0001 C CNN "Field6"
+F 7 "" V 1130 2600 60  0001 C CNN "Field7"
 F 8 "200V" V 1130 2600 60  0001 C CNN "V"
 F 9 "10%" V 1130 2600 60  0001 C CNN "tolerance"
@@
 F 4 "avx,08051C104KAT2A" V 1130 2600 60  0001 C CNN "mfg,mfg#"
 F 5 "newark,96M1354" V 1130 2600 60  0001 C CNN "vend1,vend1#"
-F 6 "" V 1130 2600 60  0001 C CNN ""
-F 7 "" V 1130 2600 60  0001 C CNN ""
+F 6 "" V 1130 2600 60  0001 C CNN "Field6"
+F 7 "" V 1130 2600 60  0001 C CNN "Field7"
 F 8 "100V" V 1130 2600 60  0001 C CNN "V"
 F 9 "10%" V 1130 2600 60  0001 C CNN "tolerance"
@@
 F 4 "avx,08051C104KAT2A" V 1130 2600 60  0001 C CNN "mfg,mfg#"
 F 5 "newark,96M1354" V 1130 2600 60  0001 C CNN "vend1,vend1#"
-F 6 "" V 1130 2600 60  0001 C CNN ""
-F 7 "" V 1130 2600 60  0001 C CNN ""
+F 6 "" V 1130 2600 60  0001 C CNN "Field6"
+F 7 "" V 1130 2600 60  0001 C CNN "Field7"
 F 8 "100V" V 1130 2600 60  0001 C CNN "V"
 F 9 "10%" V 1130 2600 60  0001 C CNN "tolerance"
@@
 F 4 "avx,08051C104KAT2A" V 1130 2600 60  0001 C CNN "mfg,mfg#"
 F 5 "newark,96M1354" V 1130 2600 60  0001 C CNN "vend1,vend1#"
-F 6 "" V 1130 2600 60  0001 C CNN ""
-F 7 "" V 1130 2600 60  0001 C CNN ""
+F 6 "" V 1130 2600 60  0001 C CNN "Field6"
+F 7 "" V 1130 2600 60  0001 C CNN "Field7"
 F 8 "100V" V 1130 2600 60  0001 C CNN "V"
 F 9 "10%" V 1130 2600 60  0001 C CNN "tolerance"
@@
 F 4 "avx,08051C104KAT2A" V 1130 2600 60  0001 C CNN "mfg,mfg#"
 F 5 "newark,96M1354" V 1130 2600 60  0001 C CNN "vend1,vend1#"
-F 6 "" V 1130 2600 60  0001 C CNN ""
-F 7 "" V 1130 2600 60  0001 C CNN ""
+F 6 "" V 1130 2600 60  0001 C CNN "Field6"
+F 7 "" V 1130 2600 60  0001 C CNN "Field7"
 F 8 "100V" V 1130 2600 60  0001 C CNN "V"
 F 9 "10%" V 1130 2600 60  0001 C CNN "tolerance"
@@
 F 4 "avx,08051C104KAT2A" V 1130 2600 60  0001 C CNN "mfg,mfg#"
 F 5 "newark,96M1354" V 1130 2600 60  0001 C CNN "vend1,vend1#"
-F 6 "" V 1130 2600 60  0001 C CNN ""
-F 7 "" V 1130 2600 60  0001 C CNN ""
+F 6 "" V 1130 2600 60  0001 C CNN "Field6"
+F 7 "" V 1130 2600 60  0001 C CNN "Field7"
 F 8 "100V" V 1130 2600 60  0001 C CNN "V"
 F 9 "10%" V 1130 2600 60  0001 C CNN "tolerance"
@@
 F 0 "R503" V 4655 3525 50  0000 C CNN
 F 1 "100k" V 4575 3525 50  0000 C CNN
-F 2 "SM0805" H 4575 3525 60  0001 C CNN
+F 2 "SM0805" V 1130 2600 60  0001 C CNN
+F 4 "vishay,CRCW0805100KFKEA" V 1130 2600 60  0001 C CNN "mfg,mfg#"
+F 5 "newark,52K9808" V 1130 2600 60  0001 C CNN "vend1,vend1#"
+F 6 "" V 1130 2600 60  0001 C CNN "Field6"
+F 7 "" V 1130 2600 60  0001 C CNN "Field7"
+F 8 "125mW" V 1130 2600 60  0001 C CNN "w"
+F 9 "1%" V 1130 2600 60  0001 C CNN "tolerance"
+F 10 "thick film" V 1130 2600 60  0001 C CNN "construct"
+F 11 "other,more,stuff" V 1130 2600 60  0001 C CNN "misc"
 	1    4575 3525
 	1    0    0    -1
@@
 F 0 "U503" H 3875 3275 60  0000 C CNN
 F 1 "MCP1826" H 3725 3825 60  0000 C CNN
-F 2 "DPAK5" H 3725 3475 60  0001 C CNN
+F 2 "DPAK5" V 1130 2600 60  0001 C CNN
+F 4 "MICROCHIP,MCP1826T-ADJE/DC" V 1130 2600 60  0001 C CNN "mfg,mfg#"
+F 5 "newark,08N6496" V 1130 2600 60  0001 C CNN "vend1,vend1#"
+F 6 "" V 1130 2600 60  0001 C CNN "Field6"
+F 7 "" V 1130 2600 60  0001 C CNN "Field7"
+F 8 "1A" V 1130 2600 60  0001 C CNN "A"
+F 9 "" V 1130 2600 60  0001 C CNN "Field9"
+F 10 "LINEAR" V 1130 2600 60  0001 C CNN "construct"
+F 11 "other,more,stuff" V 1130 2600 60  0001 C CNN "misc"
 	1    3725 3475
 	1    0    0    -1
@@
 F 0 "R502" V 2855 3475 50  0000 C CNN
 F 1 "10k" V 2775 3475 50  0000 C CNN
-F 2 "SM0805" V 705 1475 60  0001 C CNN
-F 4 "Stackpole Electronics Inc" V 705 1475 60  0001 C CNN "mfg"
-F 5 "RMCF0805JT22K0CT" V 705 1475 60  0001 C CNN "mfg#"
-F 6 "digikey" V 705 1475 60  0001 C CNN "vend1"
-F 7 "RMCF0805JT22K0CT-ND" V 705 1475 60  0001 C CNN "vend1#"
-F 8 ".250mW" V 705 1475 60  0001 C CNN "power"
-F 9 "5%" V 705 1475 60  0001 C CNN "tol"
-F 10 "Thick Film" V 705 1475 60  0001 C CNN "construct"
-F 11 "other,more,stuff" V 705 1475 60  0001 C CNN "misc"
+F 2 "SM0805" V 1130 2600 60  0001 C CNN
+F 4 "BOURNS,CR0805-FX-1002ELF" V 1130 2600 60  0001 C CNN "mfg,mfg#"
+F 5 "newark,02J2368" V 1130 2600 60  0001 C CNN "vend1,vend1#"
+F 6 "" V 1130 2600 60  0001 C CNN "Field6"
+F 7 "" V 1130 2600 60  0001 C CNN "Field7"
+F 8 "125mW" V 1130 2600 60  0001 C CNN "w"
+F 9 "1%" V 1130 2600 60  0001 C CNN "tolerance"
+F 10 "thick film" V 1130 2600 60  0001 C CNN "construct"
+F 11 "other,more,stuff" V 1130 2600 60  0001 C CNN "misc"
 	1    2775 3475
 	0    1    1    0
@@
 F 4 "avx,08051C104KAT2A" V 1130 2600 60  0001 C CNN "mfg,mfg#"
 F 5 "newark,96M1354" V 1130 2600 60  0001 C CNN "vend1,vend1#"
-F 6 "" V 1130 2600 60  0001 C CNN ""
-F 7 "" V 1130 2600 60  0001 C CNN ""
+F 6 "" V 1130 2600 60  0001 C CNN "Field6"
+F 7 "" V 1130 2600 60  0001 C CNN "Field7"
 F 8 "100V" V 1130 2600 60  0001 C CNN "V"
 F 9 "10%" V 1130 2600 60  0001 C CNN "tolerance"
@@
 F 4 "avx,08051C104KAT2A" V 1130 2600 60  0001 C CNN "mfg,mfg#"
 F 5 "newark,96M1354" V 1130 2600 60  0001 C CNN "vend1,vend1#"
-F 6 "" V 1130 2600 60  0001 C CNN ""
-F 7 "" V 1130 2600 60  0001 C CNN ""
+F 6 "" V 1130 2600 60  0001 C CNN "Field6"
+F 7 "" V 1130 2600 60  0001 C CNN "Field7"
 F 8 "100V" V 1130 2600 60  0001 C CNN "V"
 F 9 "10%" V 1130 2600 60  0001 C CNN "tolerance"

Commit message: several pins on the SOM are now connected.
Signed-off-by: Jared Harvey <TortiseGIT@jaredharvey.com>
Parts:
- renumbered C501 to C701, C502 to C702, C503 to C703, C504 to C704, C505 to C705, C506 to C706, C507 to C707, C508 to C708, C509 to C709, C510 to C710, C511 to C711, C512 to C712, C513 to C713, C514 to C714, C515 to C715, C516 to C716, C517 to C717, C518 to C718, C519 to C719, C520 to C720, C521 to C721, C522 to C722, C523 to C723, D501 to D701, D502 to D702, D503 to D703, D504 to D704, D505 to D705, D506 to D706, D507 to D707, D508 to D708, L501 to L701, L502 to L702, R501 to R737, R502 to R738, R503 to R739, R504 to R740, R505 to R741, R506 to R742, U501 to U701, U502 to U702, U503 to U703, U504 to U704

Commit message: routing has started
Signed-off-by: Jared Harvey <TortiseGIT@jaredharvey.com>
Parts:
- removed U701: LM2937, DPAK2, symbol 7805
- removed U702: LM3940, DPAK2, symbol 7805
- added U701: LM2937, SOT223, symbol LM2937
- added U702: LM3940, SOT223, symbol LM3940
