File: KICAD_Project/sub_circuits/power_reg.sch (KiCad schematic (older format))
At the start: 43 parts, among them U701 LM2937, U702 LM3940, U703 MCP1826, U704 L5973D

Commit message: more stepper updates
Signed-off-by: Jared Harvey <TortiseGIT@jaredharvey.com>
Parts:
- C701, C702, C706: footprint SM1210 -> SM0805-C1; V (none) -> 25V; Voltate 16v -> (none); construct aluminum -> multi layer ceramic; mfg Nichicon -> (none); mfg# UVZ1C100MDD -> (none); mfg,mfg# (none) -> AVX,08053C104KAT2A; tol 20% -> (none); tolerance (none) -> 10%; vend1 digikey -> (none); vend1# 493-1279-ND -> (none); vend1,vend1# (none) -> newark,96M1381
- C708, C714: Field3 -,- -> (none); Field4 -,- -> (none); Field5 35,V -> (none); Field6 20,% -> (none); Field7 alum electro -> (none); Field8 other,more,stuff -> (none); V (none) -> 100V; construct (none) -> ceramic; mfg,# ill cap,107CKE035M -> (none); mfg,mfg# (none) -> avx,08051C104KAT2A; misc (none) -> other,more,stuff; tolerance (none) -> 10%; vend,# newark,69K7903 -> (none); vend1,vend1# (none) -> newark,96M1354
- C722: Field3 -,- -> (none); Field4 -,- -> (none); Field5 200,V -> (none); Field6 20,% -> (none); Field7 alum electro -> (none); Field8 other,more,stuff -> (none); V (none) -> 25V; construct (none) -> multi layer ceramic; mfg,# ill cap,106CKE200M -> (none); mfg,mfg# (none) -> AVX,08053C104KAT2A; misc (none) -> other,more,stuff; tolerance (none) -> 10%; vend,# newark,69K7896 -> (none); vend1,vend1# (none) -> newark,96M1381
- R739: W (none) -> 125mW; w 125mW -> (none)
Changed lines of the file:
@@
-EESchema Schematic File Version 2  date 8/27/2011 10:55:18 AM
+EESchema Schematic File Version 2  date 8/30/2011 5:58:29 AM
 LIBS:power
 LIBS:device
@@
 Sheet 7 13
 Title "freeEMS PLUS from Cinch template "
-Date "27 aug 2011"
+Date "30 aug 2011"
 Rev "A-DRAF"
 Comp "diyefi.org/openecu.info"
@@
 F 0 "C702" H 1025 6950 50  0000 L CNN
 F 1 "10uF" H 1025 6750 50  0000 L CNN
-F 2 "SM1210" V -2745 5950 60  0001 C CNN
-F 4 "Nichicon" V -2745 5950 60  0001 C CNN "mfg"
-F 5 "UVZ1C100MDD" V -2745 5950 60  0001 C CNN "mfg#"
-F 6 "digikey" V -2745 5950 60  0001 C CNN "vend1"
-F 7 "493-1279-ND" V -2745 5950 60  0001 C CNN "vend1#"
-F 8 "16v" V -2745 5950 60  0001 C CNN "Voltate"
-F 9 "20%" V -2745 5950 60  0001 C CNN "tol"
-F 10 "aluminum" V -2745 5950 60  0001 C CNN "construct"
-F 11 "other,more,stuff" V -2745 5950 60  0001 C CNN "misc"
+F 2 "SM0805-C1" V 1130 2600 60  0001 C CNN
+F 4 "AVX,08053C104KAT2A" V 1130 2600 60  0001 C CNN "mfg,mfg#"
+F 5 "newark,96M1381" V 1130 2600 60  0001 C CNN "vend1,vend1#"
+F 6 "" V 1130 2600 60  0001 C CNN ""
+F 7 "" V 1130 2600 60  0001 C CNN ""
+F 8 "25V" V 1130 2600 60  0001 C CNN "V"
+F 9 "10%" V 1130 2600 60  0001 C CNN "tolerance"
+F 10 "multi layer ceramic" V 1130 2600 60  0001 C CNN "construct"
+F 11 "other,more,stuff" V 1130 2600 60  0001 C CNN "misc"
 	1    975  6850
 	-1   0    0    -1
@@
 F 0 "C722" H 8200 1850 50  0000 L CNN
 F 1 "10uF" H 8200 1650 50  0000 L CNN
-F 2 "SM0805-C1" V 4680 850 60  0001 C CNN
-F 4 "ill cap,106CKE200M" V 4680 850 60  0001 C CNN "mfg,#"
-F 5 "newark,69K7896" V 4680 850 60  0001 C CNN "vend,#"
-F 6 "-,-" V 4680 850 60  0001 C CNN "Field3"
-F 7 "-,-" V 4680 850 60  0001 C CNN "Field4"
-F 8 "200,V" V 4680 850 60  0001 C CNN "Field5"
-F 9 "20,%" V 4680 850 60  0001 C CNN "Field6"
-F 10 "alum electro" V 4680 850 60  0001 C CNN "Field7"
-F 11 "other,more,stuff" V 4680 850 60  0001 C CNN "Field8"
+F 2 "SM0805-C1" V 1130 2600 60  0001 C CNN
+F 4 "AVX,08053C104KAT2A" V 1130 2600 60  0001 C CNN "mfg,mfg#"
+F 5 "newark,96M1381" V 1130 2600 60  0001 C CNN "vend1,vend1#"
+F 6 "" V 1130 2600 60  0001 C CNN ""
+F 7 "" V 1130 2600 60  0001 C CNN ""
+F 8 "25V" V 1130 2600 60  0001 C CNN "V"
+F 9 "10%" V 1130 2600 60  0001 C CNN "tolerance"
+F 10 "multi layer ceramic" V 1130 2600 60  0001 C CNN "construct"
+F 11 "other,more,stuff" V 1130 2600 60  0001 C CNN "misc"
 	1    8400 1750
 	-1   0    0    -1
@@
 F 0 "C708" H 2550 1850 50  0000 L CNN
 F 1 "100uF" H 2500 1650 50  0000 L CNN
-F 2 "SM0805-C1" V -1670 850 60  0001 C CNN
-F 4 "ill cap,107CKE035M" V -1670 850 60  0001 C CNN "mfg,#"
-F 5 "newark,69K7903" V -1670 850 60  0001 C CNN "vend,#"
-F 6 "-,-" V -1670 850 60  0001 C CNN "Field3"
-F 7 "-,-" V -1670 850 60  0001 C CNN "Field4"
-F 8 "35,V" V -1670 850 60  0001 C CNN "Field5"
-F 9 "20,%" V -1670 850 60  0001 C CNN "Field6"
-F 10 "alum electro" V -1670 850 60  0001 C CNN "Field7"
-F 11 "other,more,stuff" V -1670 850 60  0001 C CNN "Field8"
+F 2 "SM0805-C1" V 1130 2600 60  0001 C CNN
+F 4 "avx,08051C104KAT2A" V 1130 2600 60  0001 C CNN "mfg,mfg#"
+F 5 "newark,96M1354" V 1130 2600 60  0001 C CNN "vend1,vend1#"
+F 6 "" V 1130 2600 60  0001 C CNN ""
+F 7 "" V 1130 2600 60  0001 C CNN ""
+F 8 "100V" V 1130 2600 60  0001 C CNN "V"
+F 9 "10%" V 1130 2600 60  0001 C CNN "tolerance"
+F 10 "ceramic" V 1130 2600 60  0001 C CNN "construct"
+F 11 "other,more,stuff" V 1130 2600 60  0001 C CNN "misc"
 	1    2450 1750
 	-1   0    0    -1
@@
 F 0 "C714" H 3820 1850 50  0000 L CNN
 F 1 "100uF" H 3750 1650 50  0000 L CNN
-F 2 "SM0805-C1" V 1730 850 60  0001 C CNN
-F 4 "ill cap,107CKE035M" V -1670 850 60  0001 C CNN "mfg,#"
-F 5 "newark,69K7903" V -1670 850 60  0001 C CNN "vend,#"
-F 6 "-,-" V -1670 850 60  0001 C CNN "Field3"
-F 7 "-,-" V -1670 850 60  0001 C CNN "Field4"
-F 8 "35,V" V -1670 850 60  0001 C CNN "Field5"
-F 9 "20,%" V -1670 850 60  0001 C CNN "Field6"
-F 10 "alum electro" V -1670 850 60  0001 C CNN "Field7"
-F 11 "other,more,stuff" V -1670 850 60  0001 C CNN "Field8"
+F 2 "SM0805-C1" V 1130 2600 60  0001 C CNN
+F 4 "avx,08051C104KAT2A" V 1130 2600 60  0001 C CNN "mfg,mfg#"
+F 5 "newark,96M1354" V 1130 2600 60  0001 C CNN "vend1,vend1#"
+F 6 "" V 1130 2600 60  0001 C CNN ""
+F 7 "" V 1130 2600 60  0001 C CNN ""
+F 8 "100V" V 1130 2600 60  0001 C CNN "V"
+F 9 "10%" V 1130 2600 60  0001 C CNN "tolerance"
+F 10 "ceramic" V 1130 2600 60  0001 C CNN "construct"
+F 11 "other,more,stuff" V 1130 2600 60  0001 C CNN "misc"
 	1    3700 1750
 	-1   0    0    -1
@@
 F 0 "C701" H 1025 5900 50  0000 L CNN
 F 1 "10uF" H 1025 5700 50  0000 L CNN
-F 2 "SM1210" V -2745 4900 60  0001 C CNN
-F 4 "Nichicon" V -2745 4900 60  0001 C CNN "mfg"
-F 5 "UVZ1C100MDD" V -2745 4900 60  0001 C CNN "mfg#"
-F 6 "digikey" V -2745 4900 60  0001 C CNN "vend1"
-F 7 "493-1279-ND" V -2745 4900 60  0001 C CNN "vend1#"
-F 8 "16v" V -2745 4900 60  0001 C CNN "Voltate"
-F 9 "20%" V -2745 4900 60  0001 C CNN "tol"
-F 10 "aluminum" V -2745 4900 60  0001 C CNN "construct"
-F 11 "other,more,stuff" V -2745 4900 60  0001 C CNN "misc"
+F 2 "SM0805-C1" V 1130 2600 60  0001 C CNN
+F 4 "AVX,08053C104KAT2A" V 1130 2600 60  0001 C CNN "mfg,mfg#"
+F 5 "newark,96M1381" V 1130 2600 60  0001 C CNN "vend1,vend1#"
+F 6 "" V 1130 2600 60  0001 C CNN ""
+F 7 "" V 1130 2600 60  0001 C CNN ""
+F 8 "25V" V 1130 2600 60  0001 C CNN "V"
+F 9 "10%" V 1130 2600 60  0001 C CNN "tolerance"
+F 10 "multi layer ceramic" V 1130 2600 60  0001 C CNN "construct"
+F 11 "other,more,stuff" V 1130 2600 60  0001 C CNN "misc"
 	1    975  5800
 	-1   0    0    -1
@@
 F 4 "vishay,CRCW0805100KFKEA" V 1130 2600 60  0001 C CNN "mfg,mfg#"
 F 5 "newark,52K9808" V 1130 2600 60  0001 C CNN "vend1,vend1#"
-F 6 "" V 1130 2600 60  0001 C CNN "Field6"
-F 7 "" V 1130 2600 60  0001 C CNN "Field7"
-F 8 "125mW" V 1130 2600 60  0001 C CNN "w"
+F 6 "" V 1130 2600 60  0001 C CNN ""
+F 7 "" V 1130 2600 60  0001 C CNN ""
+F 8 "125mW" V 1130 2600 60  0001 C CNN "W"
 F 9 "1%" V 1130 2600 60  0001 C CNN "tolerance"
 F 10 "thick film" V 1130 2600 60  0001 C CNN "construct"
@@
 F 0 "C706" H 1550 3575 50  0000 L CNN
 F 1 "10uF" H 1550 3375 50  0000 L CNN
-F 2 "SM1210" V -2220 2575 60  0001 C CNN
-F 4 "Nichicon" V -2220 2575 60  0001 C CNN "mfg"
-F 5 "UVZ1C100MDD" V -2220 2575 60  0001 C CNN "mfg#"
-F 6 "digikey" V -2220 2575 60  0001 C CNN "vend1"
-F 7 "493-1279-ND" V -2220 2575 60  0001 C CNN "vend1#"
-F 8 "16v" V -2220 2575 60  0001 C CNN "Voltate"
-F 9 "20%" V -2220 2575 60  0001 C CNN "tol"
-F 10 "aluminum" V -2220 2575 60  0001 C CNN "construct"
-F 11 "other,more,stuff" V -2220 2575 60  0001 C CNN "misc"
+F 2 "SM0805-C1" V 1130 2600 60  0001 C CNN
+F 4 "AVX,08053C104KAT2A" V 1130 2600 60  0001 C CNN "mfg,mfg#"
+F 5 "newark,96M1381" V 1130 2600 60  0001 C CNN "vend1,vend1#"
+F 6 "" V 1130 2600 60  0001 C CNN ""
+F 7 "" V 1130 2600 60  0001 C CNN ""
+F 8 "25V" V 1130 2600 60  0001 C CNN "V"
+F 9 "10%" V 1130 2600 60  0001 C CNN "tolerance"
+F 10 "multi layer ceramic" V 1130 2600 60  0001 C CNN "construct"
+F 11 "other,more,stuff" V 1130 2600 60  0001 C CNN "misc"
 	1    1500 3475
 	-1   0    0    -1

Commit message: More work on footprints, and schematic BOM's.
Signed-off-by: Jared Harvey <TortiseGIT@jaredharvey.com>
Parts:
- D701: A (none) -> .02A; TOL (none) -> -%; current .02a -> (none); mfg OSRAM -> (none); mfg# LH R974-LP-1-0-20-R18 -> (none); mfg,mfg# (none) -> OSRAM,LH R974-LP-1-0-20-R18; tol -% -> (none); vend1 digikey -> (none); vend1# 475-1415-1-ND -> (none); vend1,vend1# (none) -> DIGI,475-1415-1-ND
Changed lines of the file:
@@
-EESchema Schematic File Version 2  date 9/1/2011 7:35:07 PM
+EESchema Schematic File Version 2  date 9/4/2011 3:29:41 PM
 LIBS:power
 LIBS:device
@@
 Sheet 7 13
 Title "freeEMS PLUS from Cinch template "
-Date "1 sep 2011"
+Date "4 sep 2011"
 Rev "A-DRAF"
 Comp "diyefi.org/openecu.info"
@@
 $EndComp
 $Comp
-L GND #PWR0138
+L GND #PWR702
 U 1 1 4E3DFCE8
 P 975 7100
-F 0 "#PWR0138" H 975 7100 30  0001 C CNN
+F 0 "#PWR702" H 975 7100 30  0001 C CNN
 F 1 "GND" H 975 7030 30  0001 C CNN
 	1    975  7100
@@
 $EndComp
 $Comp
-L GND #PWR0139
+L GND #PWR705
 U 1 1 4E3DFCE1
 P 3975 7100
-F 0 "#PWR0139" H 3975 7100 30  0001 C CNN
+F 0 "#PWR705" H 3975 7100 30  0001 C CNN
 F 1 "GND" H 3975 7030 30  0001 C CNN
 	1    3975 7100
@@
 F 0 "D701" H 1000 3700 50  0000 C CNN
 F 1 "LED" H 1000 3500 50  0000 C CNN
-F 2 "LED-0805" H 1000 3600 60  0001 C CNN
-F 4 "OSRAM" V -2470 2150 60  0001 C CNN "mfg"
-F 5 "LH R974-LP-1-0-20-R18" V -2470 2150 60  0001 C CNN "mfg#"
-F 6 "digikey" V -2470 2150 60  0001 C CNN "vend1"
-F 7 "475-1415-1-ND" V -2470 2150 60  0001 C CNN "vend1#"
-F 8 ".02a" V -2470 2150 60  0001 C CNN "current"
-F 9 "-%" V -2470 2150 60  0001 C CNN "tol"
-F 10 "RED" V -2470 2150 60  0001 C CNN "construct"
-F 11 "other,more,stuff" V -2470 2150 60  0001 C CNN "misc"
+F 2 "LED-0805" V 1130 2600 60  0001 C CNN
+F 4 "OSRAM,LH R974-LP-1-0-20-R18" V 1130 2600 60  0001 C CNN "mfg,mfg#"
+F 5 "DIGI,475-1415-1-ND" V 1130 2600 60  0001 C CNN "vend1,vend1#"
+F 6 "" V 1130 2600 60  0001 C CNN "Field6"
+F 7 "" V 1130 2600 60  0001 C CNN "Field7"
+F 8 ".02A" V 1130 2600 60  0001 C CNN "A"
+F 9 "-%" V 1130 2600 60  0001 C CNN "TOL"
+F 10 "RED" V 1130 2600 60  0001 C CNN "construct"
+F 11 "other,more,stuff" V 1130 2600 60  0001 C CNN "misc"
 	1    1000 3600
 	0    1    1    0
@@
 $EndComp
 $Comp
-L GND #PWR0140
+L GND #PWR708
 U 1 1 4E3DEE9D
 P 5325 3975
-F 0 "#PWR0140" H 5325 3975 30  0001 C CNN
+F 0 "#PWR708" H 5325 3975 30  0001 C CNN
 F 1 "GND" H 5325 3905 30  0001 C CNN
 	1    5325 3975
@@
 $EndComp
 $Comp
-L GND #PWR0141
+L GND #PWR704
 U 1 1 4E3DEE94
 P 3975 6050
-F 0 "#PWR0141" H 3975 6050 30  0001 C CNN
+F 0 "#PWR704" H 3975 6050 30  0001 C CNN
 F 1 "GND" H 3975 5980 30  0001 C CNN
 	1    3975 6050
@@
 $EndComp
 $Comp
-L GND #PWR0142
+L GND #PWR707
 U 1 1 4E3DEE87
 P 4950 2000
-F 0 "#PWR0142" H 4950 2000 30  0001 C CNN
+F 0 "#PWR707" H 4950 2000 30  0001 C CNN
 F 1 "GND" H 4950 1930 30  0001 C CNN
 	1    4950 2000
@@
 $EndComp
 $Comp
-L GND #PWR0143
+L GND #PWR706
 U 1 1 4BF26D5A
 P 4450 2000
-F 0 "#PWR0143" H 4450 2000 30  0001 C CNN
+F 0 "#PWR706" H 4450 2000 30  0001 C CNN
 F 1 "GND" H 4450 1930 30  0001 C CNN
 	1    4450 2000
@@
 $EndComp
 $Comp
-L GND #PWR0144
+L GND #PWR701
 U 1 1 486CA86E
 P 975 6050
-F 0 "#PWR0144" H 975 6050 30  0001 C CNN
+F 0 "#PWR701" H 975 6050 30  0001 C CNN
 F 1 "GND" H 975 5980 30  0001 C CNN
 	1    975  6050
@@
 $EndComp
 $Comp
-L GND #PWR0145
+L GND #PWR703
 U 1 1 4C2F529B
 P 3725 4025
-F 0 "#PWR0145" H 3725 4025 30  0001 C CNN
+F 0 "#PWR703" H 3725 4025 30  0001 C CNN
 F 1 "GND" H 3725 3955 30  0001 C CNN
 	1    3725 4025
