File: KICAD_Project/sub_circuits/power_reg.sch (KiCad schematic (older format))
At the start: 43 parts, among them U701 LM2937, U702 LM3940, U703 MCP1826, U704 L5973D

Commit message: Added some simulations for the AN protect lines
Signed-off-by: Jared Harvey <TortiseGIT@jaredharvey.com>
Parts:
- removed C719: 5.6nF, SM0805-C1, symbol C
- removed C720: 27pF, SM0805-C1, symbol C
- removed C721: 330uF, SM0805-C1, symbol CAPAPOL
- removed C722: 10uF, SM0805-C1, symbol C
- removed C723: 10nF, SM0805-C1, symbol C
- removed D708: STPS5L25, D4-SMB, symbol DIODE
- removed L702: DR125-330-R, SM100uH, symbol INDUCTOR
- removed R740: 3.6K 1%, SM0805, symbol R
- removed R741: 39k 1%, SM0805, symbol R
- removed R742: 13K 1%, SM0805, symbol R
- removed U704: L5973D, SO8E, symbol L5970D
Connections:
- wire segments 59 -> 44
- no-connect marks 2 -> 0
Other:
- note removed: "MBRA210LT3G"
- note removed: "THIS SECTION CONTAINS\n\nA 2 AMP SWITCHING 6V REGULATOR. THIS PREVENTS THE LINEARS FROM HEATING UP IN EXCESS."

Commit message: Made more progress on the AN protects and LS drive 33800
Signed-off-by: Jared Harvey <TortiseGIT@jaredharvey.com>
Parts:
- C705, C709, C715: footprint SM0805-C1 -> SM0805; TOL (none) -> 10%; V 100V -> 200V; construct ceramic -> CERAMIC; mfg,mfg# avx,08051C104KAT2A -> AVX,08055C104KAT2A; tolerance 10% -> (none); vend1,vend1# newark,96M1354 -> newark,27C8438
Changed lines of the file:
@@
-EESchema Schematic File Version 2  date 10/14/2011 5:26:22 AM
+EESchema Schematic File Version 2  date 10/16/2011 7:32:22 AM
 LIBS:power
 LIBS:device
@@
 Sheet 7 12
 Title "Open5xxxECU (o5e), an ECU that is no longer affiliated with freeEMS."
-Date "14 oct 2011"
+Date "16 oct 2011"
 Rev "A-DRAFT5"
 Comp "http://open5xxxecu.org/"
@@
 $EndComp
 $Comp
-L GND #PWR0134
+L GND #PWR0142
 U 1 1 4E3DFCE8
 P 975 7100
-F 0 "#PWR0134" H 975 7100 30  0001 C CNN
+F 0 "#PWR0142" H 975 7100 30  0001 C CNN
 F 1 "GND" H 975 7030 30  0001 C CNN
 	1    975  7100
@@
 $EndComp
 $Comp
-L GND #PWR0135
+L GND #PWR0143
 U 1 1 4E3DFCE1
 P 3975 7100
-F 0 "#PWR0135" H 3975 7100 30  0001 C CNN
+F 0 "#PWR0143" H 3975 7100 30  0001 C CNN
 F 1 "GND" H 3975 7030 30  0001 C CNN
 	1    3975 7100
@@
 $EndComp
 $Comp
-L GND #PWR0136
+L GND #PWR0144
 U 1 1 4E3DEE9D
 P 5325 3975
-F 0 "#PWR0136" H 5325 3975 30  0001 C CNN
+F 0 "#PWR0144" H 5325 3975 30  0001 C CNN
 F 1 "GND" H 5325 3905 30  0001 C CNN
 	1    5325 3975
@@
 $EndComp
 $Comp
-L GND #PWR0137
+L GND #PWR0145
 U 1 1 4E3DEE94
 P 3975 6050
-F 0 "#PWR0137" H 3975 6050 30  0001 C CNN
+F 0 "#PWR0145" H 3975 6050 30  0001 C CNN
 F 1 "GND" H 3975 5980 30  0001 C CNN
 	1    3975 6050
@@
 $EndComp
 $Comp
-L GND #PWR0138
+L GND #PWR0146
 U 1 1 4BF26D5A
 P 4450 2000
-F 0 "#PWR0138" H 4450 2000 30  0001 C CNN
+F 0 "#PWR0146" H 4450 2000 30  0001 C CNN
 F 1 "GND" H 4450 1930 30  0001 C CNN
 	1    4450 2000
@@
 F 0 "C705" H 1550 1850 50  0000 L CNN
 F 1 "100nF" H 1550 1650 50  0000 L CNN
-F 2 "SM0805-C1" V 1130 2600 60  0001 C CNN
-F 4 "avx,08051C104KAT2A" V 1130 2600 60  0001 C CNN "mfg,mfg#"
-F 5 "newark,96M1354" V 1130 2600 60  0001 C CNN "vend1,vend1#"
-F 6 "" V 1130 2600 60  0001 C CNN "Field6"
-F 7 "" V 1130 2600 60  0001 C CNN "Field7"
-F 8 "100V" V 1130 2600 60  0001 C CNN "V"
-F 9 "10%" V 1130 2600 60  0001 C CNN "tolerance"
-F 10 "ceramic" V 1130 2600 60  0001 C CNN "construct"
+F 2 "SM0805" V 1130 2600 60  0001 C CNN
+F 4 "AVX,08055C104KAT2A" V 1130 2600 60  0001 C CNN "mfg,mfg#"
+F 5 "newark,27C8438" V 1130 2600 60  0001 C CNN "vend1,vend1#"
+F 6 "" V 1130 2600 60  0001 C CNN "Field6"
+F 7 "" V 1130 2600 60  0001 C CNN "Field7"
+F 8 "200V" V 1130 2600 60  0001 C CNN "V"
+F 9 "10%" V 1130 2600 60  0001 C CNN "TOL"
+F 10 "CERAMIC" V 1130 2600 60  0001 C CNN "construct"
 F 11 "other,more,stuff" V 1130 2600 60  0001 C CNN "misc"
 	1    1500 1750
@@
 F 0 "C715" H 4010 1850 50  0000 L CNN
 F 1 "100nF" H 3950 1650 50  0000 L CNN
-F 2 "SM0805-C1" V 1130 2600 60  0001 C CNN
-F 4 "avx,08051C104KAT2A" V 1130 2600 60  0001 C CNN "mfg,mfg#"
-F 5 "newark,96M1354" V 1130 2600 60  0001 C CNN "vend1,vend1#"
-F 6 "" V 1130 2600 60  0001 C CNN "Field6"
-F 7 "" V 1130 2600 60  0001 C CNN "Field7"
-F 8 "100V" V 1130 2600 60  0001 C CNN "V"
-F 9 "10%" V 1130 2600 60  0001 C CNN "tolerance"
-F 10 "ceramic" V 1130 2600 60  0001 C CNN "construct"
+F 2 "SM0805" V 1130 2600 60  0001 C CNN
+F 4 "AVX,08055C104KAT2A" V 1130 2600 60  0001 C CNN "mfg,mfg#"
+F 5 "newark,27C8438" V 1130 2600 60  0001 C CNN "vend1,vend1#"
+F 6 "" V 1130 2600 60  0001 C CNN "Field6"
+F 7 "" V 1130 2600 60  0001 C CNN "Field7"
+F 8 "200V" V 1130 2600 60  0001 C CNN "V"
+F 9 "10%" V 1130 2600 60  0001 C CNN "TOL"
+F 10 "CERAMIC" V 1130 2600 60  0001 C CNN "construct"
 F 11 "other,more,stuff" V 1130 2600 60  0001 C CNN "misc"
 	1    4200 1750
@@
 F 0 "C709" H 2650 1860 50  0000 L CNN
 F 1 "100nF" H 2550 1650 50  0000 L CNN
-F 2 "SM0805-C1" V 1130 2600 60  0001 C CNN
-F 4 "avx,08051C104KAT2A" V 1130 2600 60  0001 C CNN "mfg,mfg#"
-F 5 "newark,96M1354" V 1130 2600 60  0001 C CNN "vend1,vend1#"
-F 6 "" V 1130 2600 60  0001 C CNN "Field6"
-F 7 "" V 1130 2600 60  0001 C CNN "Field7"
-F 8 "100V" V 1130 2600 60  0001 C CNN "V"
-F 9 "10%" V 1130 2600 60  0001 C CNN "tolerance"
-F 10 "ceramic" V 1130 2600 60  0001 C CNN "construct"
+F 2 "SM0805" V 1130 2600 60  0001 C CNN
+F 4 "AVX,08055C104KAT2A" V 1130 2600 60  0001 C CNN "mfg,mfg#"
+F 5 "newark,27C8438" V 1130 2600 60  0001 C CNN "vend1,vend1#"
+F 6 "" V 1130 2600 60  0001 C CNN "Field6"
+F 7 "" V 1130 2600 60  0001 C CNN "Field7"
+F 8 "200V" V 1130 2600 60  0001 C CNN "V"
+F 9 "10%" V 1130 2600 60  0001 C CNN "TOL"
+F 10 "CERAMIC" V 1130 2600 60  0001 C CNN "construct"
 F 11 "other,more,stuff" V 1130 2600 60  0001 C CNN "misc"
 	1    2800 1750
@@
 $EndComp
 $Comp
-L GND #PWR0139
+L GND #PWR0147
 U 1 1 486CA86E
 P 975 6050
-F 0 "#PWR0139" H 975 6050 30  0001 C CNN
+F 0 "#PWR0147" H 975 6050 30  0001 C CNN
 F 1 "GND" H 975 5980 30  0001 C CNN
 	1    975  6050
@@
 $EndComp
 $Comp
-L GND #PWR0140
+L GND #PWR0148
 U 1 1 4C2F529B
 P 3725 4025
-F 0 "#PWR0140" H 3725 4025 30  0001 C CNN
+F 0 "#PWR0148" H 3725 4025 30  0001 C CNN
 F 1 "GND" H 3725 3955 30  0001 C CNN
 	1    3725 4025

Commit message: AN/DIGI's now point at processor, LS now points at processor, reg schematic drafted
Signed-off-by: Jared Harvey <TortiseGIT@jaredharvey.com>
Parts:
- added C719: 100nF, SM0805, symbol C
- added D708: TPSMA27A, DO214, symbol DIODE
- added P701: CONN_1, PINTST, symbol CONN_1
- added R741: 215R, SM0805, symbol R
- added U704: 7812, DPAK2, symbol 7812
- added U705: OKR-T/3-W12-C, OKR-T/3, symbol OKR-T/3-W12-C
Connections:
- net labels added: 12V_BUF_BAT
- wire segments 44 -> 50
Other:
- note added: "*C717: aluminum\n*C718: tantalum, close to the regulator"
- note added: "1.182/(6-.591)=.2185kOhm trim\n(1.182/.215)+.591=6.08V"
- note added: "THIS SECTION CONTAINS\n\nFILTER/BULK CAPS\nREVERSE POLARITY PROTECTION DIODE\nREVERSE POLARITY SPIKE PROTECTION\nTRANSIENT INDUCTOR AND DIODE SHUNT\n\nEXPECTS AN UPSTREAM 10A FUSE"
- note removed: "*C10: aluminum\n*C11: tantalum, close to the regulator"
- note removed: "THIS SECTION CONTAINS\n\nFILTER/BULK CAPS\nREVERSE POLARITY PROTECTION DIODE\nREVERSE POLARITY SPIKE PROTECTION\nTRANSIENT INDUCTOR"
- moved on the sheet: C705, C708, D702, D703

Commit message: changed some file names removing spaces, added gen2 notes, and some minor board layout changes.
Signed-off-by: Jared Harvey <TortiseGIT@jaredharvey.com>
Parts:
- added D709: 1N4148, SOD-123, symbol DIODE
- added F701: 12A_FUSE, SIL-2, symbol FUSE
Connections:
- wire segments 50 -> 54
Other:
- note added: "THIS SECTION CONTAINS\n\nFILTER/BULK CAPS\nREVERSE POLARITY PROTECTION DIODE\nREVERSE POLARITY SPIKE PROTECTION\nTRANSIENT INDUCTOR AND DIODE SHUNT\n\nEXPECTS AN UPSTREAM 10A FUSE\nINCLUDED 12A FUSE IS FOR REVERSE PROTECTION ON OKR DEVICE"
- note removed: "THIS SECTION CONTAINS\n\nFILTER/BULK CAPS\nREVERSE POLARITY PROTECTION DIODE\nREVERSE POLARITY SPIKE PROTECTION\nTRANSIENT INDUCTOR AND DIODE SHUNT\n\nEXPECTS AN UPSTREAM 10A FUSE"
- moved on the sheet: C705, C708, C709, C714, C715, C719, D702, D703, D706, D708, L701, R738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

Commit message: about to position the regulators, save it as a backup copy
Signed-off-by: Jared Harvey <TortiseGIT@jaredharvey.com>
Parts:
- added P702, P703, P704, P705, P706: CONN_1, PINTST, symbol CONN_1
- C701, C702, C703, C704, C706, C707, C708, C712, C713, C714, C717: footprint SM0805-C1 -> SM0805
- C719: value 100nF -> 22uF; footprint SM0805 -> SM1210; V 200V -> 16V; construct CERAMIC -> multi layered CERAMIC; mfg,mfg# AVX,08055C104KAT2A -> Murata,GRM32ER61C226KE20L; vend1,vend1# newark,27C8438 -> digi,GRM32ER61C226KE20L
- R741: value 215R -> 220R; mfg,mfg# vishay,CRCW0805215RFKEA -> vishay,CRCW0805220RFKEA; vend1,vend1# newark,53K0018 -> digi,CRCW0805220RFKEA
Connections:
- wire segments 54 -> 55
Other:
- note added: "1.182/(6-.591)=.2185kOhm trim\n(1.182/.220)+.591=5.96V"
- note added: "THIS SECTION CONTAINS\n\nFILTER/BULK CAPS\nREVERSE POLARITY PROTECTION DIODE\nREVERSE POLARITY SPIKE PROTECTION\nTRANSIENT INDUCTOR AND DIODE SHUNT\n\nEXPECTS AN UPSTREAM 5A FUSE/CIRCUIT BREAKER\nINCLUDED 12A FUSE IS FOR REVERSE PROTECTION ON OKR DEVICE"
- note removed: "1.182/(6-.591)=.2185kOhm trim\n(1.182/.215)+.591=6.08V"
- note removed: "THIS SECTION CONTAINS\n\nFILTER/BULK CAPS\nREVERSE POLARITY PROTECTION DIODE\nREVERSE POLARITY SPIKE PROTECTION\nTRANSIENT INDUCTOR AND DIODE SHUNT\n\nEXPECTS AN UPSTREAM 10A FUSE\nINCLUDED 12A FUSE IS FOR REVERSE PROTECTION ON OKR DEVICE"
