File: KICAD_Project/sub_circuits/power_reg2.sch (KiCad schematic (older format))
At the start: 6 parts, among them U2 LM2937

Commit message: caps have been done with the scripts next up is the resistors.
Signed-off-by: Jared Harvey <TortiseGIT@jaredharvey.com>
Parts:
- C3, C6: footprint SM0805 -> SM0805-C1; V (none) -> 100V; Voltage 50v -> (none); mfg Murata -> (none); mfg# GRM21BR71H104KA01L -> (none); mfg,mfg# (none) -> avx,08051C104KAT2A; vend1 digikey -> (none); vend1# 490-1666-2-ND -> (none); vend1,vend1# (none) -> newark,96M1354
Changed lines of the file:
@@
 F 0 "C6" H 7500 3600 50  0000 L CNN
 F 1 "0.1uF" H 7500 3400 50  0000 L CNN
-F 2 "SM0805" V 1130 2600 60  0001 C CNN
-F 4 "Murata" V 1130 2600 60  0001 C CNN "mfg"
-F 5 "GRM21BR71H104KA01L" V 1130 2600 60  0001 C CNN "mfg#"
-F 6 "digikey" V 1130 2600 60  0001 C CNN "vend1"
-F 7 "490-1666-2-ND" V 1130 2600 60  0001 C CNN "vend1#"
-F 8 "50v" V 1130 2600 60  0001 C CNN "Voltage"
+F 2 "SM0805-C1" V 1130 2600 60  0001 C CNN
+F 4 "avx,08051C104KAT2A" V 1130 2600 60  0001 C CNN "mfg,mfg#"
+F 5 "newark,96M1354" V 1130 2600 60  0001 C CNN "vend1,vend1#"
+F 6 "" V 1130 2600 60  0001 C CNN ""
+F 7 "" V 1130 2600 60  0001 C CNN ""
+F 8 "100V" V 1130 2600 60  0001 C CNN "V"
 F 9 "10%" V 1130 2600 60  0001 C CNN "tolerance"
 F 10 "ceramic" V 1130 2600 60  0001 C CNN "construct"
@@
 F 0 "C3" H 5300 3600 50  0000 L CNN
 F 1 "0.1uF" H 5300 3400 50  0000 L CNN
-F 2 "SM0805" V 1130 2600 60  0001 C CNN
-F 4 "Murata" V 1130 2600 60  0001 C CNN "mfg"
-F 5 "GRM21BR71H104KA01L" V 1130 2600 60  0001 C CNN "mfg#"
-F 6 "digikey" V 1130 2600 60  0001 C CNN "vend1"
-F 7 "490-1666-2-ND" V 1130 2600 60  0001 C CNN "vend1#"
-F 8 "50v" V 1130 2600 60  0001 C CNN "Voltage"
+F 2 "SM0805-C1" V 1130 2600 60  0001 C CNN
+F 4 "avx,08051C104KAT2A" V 1130 2600 60  0001 C CNN "mfg,mfg#"
+F 5 "newark,96M1354" V 1130 2600 60  0001 C CNN "vend1,vend1#"
+F 6 "" V 1130 2600 60  0001 C CNN ""
+F 7 "" V 1130 2600 60  0001 C CNN ""
+F 8 "100V" V 1130 2600 60  0001 C CNN "V"
 F 9 "10%" V 1130 2600 60  0001 C CNN "tolerance"
 F 10 "ceramic" V 1130 2600 60  0001 C CNN "construct"

Commit message: routing has started
Signed-off-by: Jared Harvey <TortiseGIT@jaredharvey.com>
Parts:
- U2: footprint DPAK2 -> SOT223; V (none) -> 5V; construct (none) -> LINEAR; mfg national semi -> (none); mfg# LM2937IMP-5.0/NOPB -> (none); mfg,mfg# (none) -> NAT SEMI,LM2937IMP-5.0/NOPB; misc (none) -> other,more,stuff; tolerance (none) -> .05%; vend1 digikey -> (none); vend1# LM2937IMP-5.0CT-ND -> (none); vend1,vend1# (none) -> digi,LM2937IMP-5.0CT-ND
Changed lines of the file:
@@
 F 0 "U2" H 6200 3154 60  0000 C CNN
 F 1 "LM2937" H 6050 3550 60  0000 C CNN
-F 2 "DPAK2" H 6050 3350 60  0001 C CNN
-F 4 "national semi" H 6050 3350 60  0001 C CNN "mfg"
-F 5 "LM2937IMP-5.0/NOPB" H 6050 3350 60  0001 C CNN "mfg#"
-F 6 "digikey" H 6050 3350 60  0001 C CNN "vend1"
-F 7 "LM2937IMP-5.0CT-ND" H 6050 3350 60  0001 C CNN "vend1#"
+F 2 "SOT223" V 1130 2600 60  0001 C CNN
+F 4 "NAT SEMI,LM2937IMP-5.0/NOPB" V 1130 2600 60  0001 C CNN "mfg,mfg#"
+F 5 "digi,LM2937IMP-5.0CT-ND" V 1130 2600 60  0001 C CNN "vend1,vend1#"
+F 6 "" V 1130 2600 60  0001 C CNN ""
+F 7 "" V 1130 2600 60  0001 C CNN ""
+F 8 "5V" V 1130 2600 60  0001 C CNN "V"
+F 9 ".05%" V 1130 2600 60  0001 C CNN "tolerance"
+F 10 "LINEAR" V 1130 2600 60  0001 C CNN "construct"
+F 11 "other,more,stuff" V 1130 2600 60  0001 C CNN "misc"
 	1    6050 3350
 	1    0    0    -1

Commit message: more stepper updates
Signed-off-by: Jared Harvey <TortiseGIT@jaredharvey.com>
Parts:
- C2: footprint SM1210 -> SM0805-C1; V (none) -> 25V; Voltate 16v -> (none); construct aluminum -> multi layer ceramic; mfg Nichicon -> (none); mfg# UVZ1C100MDD -> (none); mfg,mfg# (none) -> AVX,08053C104KAT2A; tol 20% -> (none); tolerance (none) -> 10%; vend1 digikey -> (none); vend1# 493-1279-ND -> (none); vend1,vend1# (none) -> newark,96M1381
Changed lines of the file:
@@
 F 0 "C2" H 4900 3600 50  0000 L CNN
 F 1 "10uF" H 4900 3400 50  0000 L CNN
-F 2 "SM1210" V 1130 2600 60  0001 C CNN
-F 4 "Nichicon" V 1130 2600 60  0001 C CNN "mfg"
-F 5 "UVZ1C100MDD" V 1130 2600 60  0001 C CNN "mfg#"
-F 6 "digikey" V 1130 2600 60  0001 C CNN "vend1"
-F 7 "493-1279-ND" V 1130 2600 60  0001 C CNN "vend1#"
-F 8 "16v" V 1130 2600 60  0001 C CNN "Voltate"
-F 9 "20%" V 1130 2600 60  0001 C CNN "tol"
-F 10 "aluminum" V 1130 2600 60  0001 C CNN "construct"
+F 2 "SM0805-C1" V 1130 2600 60  0001 C CNN
+F 4 "AVX,08053C104KAT2A" V 1130 2600 60  0001 C CNN "mfg,mfg#"
+F 5 "newark,96M1381" V 1130 2600 60  0001 C CNN "vend1,vend1#"
+F 6 "" V 1130 2600 60  0001 C CNN ""
+F 7 "" V 1130 2600 60  0001 C CNN ""
+F 8 "25V" V 1130 2600 60  0001 C CNN "V"
+F 9 "10%" V 1130 2600 60  0001 C CNN "tolerance"
+F 10 "multi layer ceramic" V 1130 2600 60  0001 C CNN "construct"
 F 11 "other,more,stuff" V 1130 2600 60  0001 C CNN "misc"
 	1    4850 3500
