File: KICAD_Project/sub_circuits/pin_protect.sch (KiCad schematic (older format))
At the start: 84 parts

Commit message: More work on footprints, and schematic BOM's.
Signed-off-by: Jared Harvey <TortiseGIT@jaredharvey.com>
Parts:
- R401, R402, R403, R404, R405, R406, R407, R408, R409, R410, R411, R412, R413, R414, R415, R416, R417, R418, R419, R420, R421, R422, R423, R424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: W (none) -> 125mW; tol (none) -> 1%; tolerance 1% -> (none); w 125mW -> (none)
