File: KICAD_Project/sub_circuits/power_reg1.sch (KiCad schematic (older format))
At the start: 12 parts, among them U4 MCP1826

Commit message: caps have been done with the scripts next up is the resistors.
Signed-off-by: Jared Harvey <TortiseGIT@jaredharvey.com>
Parts:
- C12, C9: footprint SM0805 -> SM0805-C1; V (none) -> 100V; Voltage 50v -> (none); mfg Murata -> (none); mfg# GRM21BR71H104KA01L -> (none); mfg,mfg# (none) -> avx,08051C104KAT2A; vend1 digikey -> (none); vend1# 490-1666-2-ND -> (none); vend1,vend1# (none) -> newark,96M1354
Changed lines of the file:
@@
 F 0 "C12" H 8050 3600 50  0000 L CNN
 F 1 "0.1uF" H 8050 3400 50  0000 L CNN
-F 2 "SM0805" V 1680 2600 60  0001 C CNN
-F 4 "Murata" V 1680 2600 60  0001 C CNN "mfg"
-F 5 "GRM21BR71H104KA01L" V 1680 2600 60  0001 C CNN "mfg#"
-F 6 "digikey" V 1680 2600 60  0001 C CNN "vend1"
-F 7 "490-1666-2-ND" V 1680 2600 60  0001 C CNN "vend1#"
-F 8 "50v" V 1680 2600 60  0001 C CNN "Voltage"
-F 9 "10%" V 1680 2600 60  0001 C CNN "tolerance"
-F 10 "ceramic" V 1680 2600 60  0001 C CNN "construct"
-F 11 "other,more,stuff" V 1680 2600 60  0001 C CNN "misc"
+F 2 "SM0805-C1" V 1130 2600 60  0001 C CNN
+F 4 "avx,08051C104KAT2A" V 1130 2600 60  0001 C CNN "mfg,mfg#"
+F 5 "newark,96M1354" V 1130 2600 60  0001 C CNN "vend1,vend1#"
+F 6 "" V 1130 2600 60  0001 C CNN ""
+F 7 "" V 1130 2600 60  0001 C CNN ""
+F 8 "100V" V 1130 2600 60  0001 C CNN "V"
+F 9 "10%" V 1130 2600 60  0001 C CNN "tolerance"
+F 10 "ceramic" V 1130 2600 60  0001 C CNN "construct"
+F 11 "other,more,stuff" V 1130 2600 60  0001 C CNN "misc"
 	1    8000 3500
 	-1   0    0    -1
@@
 F 0 "C9" H 5300 3600 50  0000 L CNN
 F 1 "0.1uF" H 5300 3400 50  0000 L CNN
-F 2 "SM0805" V 1130 2600 60  0001 C CNN
-F 4 "Murata" V 1130 2600 60  0001 C CNN "mfg"
-F 5 "GRM21BR71H104KA01L" V 1130 2600 60  0001 C CNN "mfg#"
-F 6 "digikey" V 1130 2600 60  0001 C CNN "vend1"
-F 7 "490-1666-2-ND" V 1130 2600 60  0001 C CNN "vend1#"
-F 8 "50v" V 1130 2600 60  0001 C CNN "Voltage"
+F 2 "SM0805-C1" V 1130 2600 60  0001 C CNN
+F 4 "avx,08051C104KAT2A" V 1130 2600 60  0001 C CNN "mfg,mfg#"
+F 5 "newark,96M1354" V 1130 2600 60  0001 C CNN "vend1,vend1#"
+F 6 "" V 1130 2600 60  0001 C CNN ""
+F 7 "" V 1130 2600 60  0001 C CNN ""
+F 8 "100V" V 1130 2600 60  0001 C CNN "V"
 F 9 "10%" V 1130 2600 60  0001 C CNN "tolerance"
 F 10 "ceramic" V 1130 2600 60  0001 C CNN "construct"

Commit message: Looks like the bulk components are golden now, there are still a couple straglers, mostly switch mode power supply stuff.
Signed-off-by: Jared Harvey <TortiseGIT@jaredharvey.com>
Parts:
- R226: construct Thick Film -> thick film; mfg Stackpole Electronics Inc -> (none); mfg# RMCF0805JT22K0CT -> (none); mfg,mfg# (none) -> BOURNS,CR0805-FX-1002ELF; power .250mW -> (none); tol 5% -> (none); tolerance (none) -> 1%; vend1 digikey -> (none); vend1# RMCF0805JT22K0CT-ND -> (none); vend1,vend1# (none) -> newark,02J2368; w (none) -> 125mW
- R265: construct (none) -> thick film; mfg,mfg# (none) -> vishay,CRCW0805100KFKEA; misc (none) -> other,more,stuff; tolerance (none) -> 1%; vend1,vend1# (none) -> newark,52K9808; w (none) -> 125mW
- U4: A (none) -> 1A; construct (none) -> LINEAR; mfg,mfg# (none) -> MICROCHIP,MCP1826T-ADJE/DC; misc (none) -> other,more,stuff; vend1,vend1# (none) -> newark,08N6496
Changed lines of the file:
@@
 F 0 "R265" V 7330 3550 50  0000 C CNN
 F 1 "100k" V 7250 3550 50  0000 C CNN
-F 2 "SM0805" H 7250 3550 60  0001 C CNN
+F 2 "SM0805" V 1130 2600 60  0001 C CNN
+F 4 "vishay,CRCW0805100KFKEA" V 1130 2600 60  0001 C CNN "mfg,mfg#"
+F 5 "newark,52K9808" V 1130 2600 60  0001 C CNN "vend1,vend1#"
+F 6 "" V 1130 2600 60  0001 C CNN ""
+F 7 "" V 1130 2600 60  0001 C CNN ""
+F 8 "125mW" V 1130 2600 60  0001 C CNN "w"
+F 9 "1%" V 1130 2600 60  0001 C CNN "tolerance"
+F 10 "thick film" V 1130 2600 60  0001 C CNN "construct"
+F 11 "other,more,stuff" V 1130 2600 60  0001 C CNN "misc"
 	1    7250 3550
 	1    0    0    -1
@@
 F 0 "U4" H 6550 3300 60  0000 C CNN
 F 1 "MCP1826" H 6400 3850 60  0000 C CNN
-F 2 "DPAK5" H 6400 3500 60  0001 C CNN
+F 2 "DPAK5" V 1130 2600 60  0001 C CNN
+F 4 "MICROCHIP,MCP1826T-ADJE/DC" V 1130 2600 60  0001 C CNN "mfg,mfg#"
+F 5 "newark,08N6496" V 1130 2600 60  0001 C CNN "vend1,vend1#"
+F 6 "" V 1130 2600 60  0001 C CNN ""
+F 7 "" V 1130 2600 60  0001 C CNN ""
+F 8 "1A" V 1130 2600 60  0001 C CNN "A"
+F 9 "" V 1130 2600 60  0001 C CNN ""
+F 10 "LINEAR" V 1130 2600 60  0001 C CNN "construct"
+F 11 "other,more,stuff" V 1130 2600 60  0001 C CNN "misc"
 	1    6400 3500
 	1    0    0    -1
@@
 F 0 "R226" V 4930 5050 50  0000 C CNN
 F 1 "10k" V 4850 5050 50  0000 C CNN
-F 2 "SM0805" V 2780 3050 60  0001 C CNN
-F 4 "Stackpole Electronics Inc" V 2780 3050 60  0001 C CNN "mfg"
-F 5 "RMCF0805JT22K0CT" V 2780 3050 60  0001 C CNN "mfg#"
-F 6 "digikey" V 2780 3050 60  0001 C CNN "vend1"
-F 7 "RMCF0805JT22K0CT-ND" V 2780 3050 60  0001 C CNN "vend1#"
-F 8 ".250mW" V 2780 3050 60  0001 C CNN "power"
-F 9 "5%" V 2780 3050 60  0001 C CNN "tol"
-F 10 "Thick Film" V 2780 3050 60  0001 C CNN "construct"
-F 11 "other,more,stuff" V 2780 3050 60  0001 C CNN "misc"
+F 2 "SM0805" V 1130 2600 60  0001 C CNN
+F 4 "BOURNS,CR0805-FX-1002ELF" V 1130 2600 60  0001 C CNN "mfg,mfg#"
+F 5 "newark,02J2368" V 1130 2600 60  0001 C CNN "vend1,vend1#"
+F 6 "" V 1130 2600 60  0001 C CNN ""
+F 7 "" V 1130 2600 60  0001 C CNN ""
+F 8 "125mW" V 1130 2600 60  0001 C CNN "w"
+F 9 "1%" V 1130 2600 60  0001 C CNN "tolerance"
+F 10 "thick film" V 1130 2600 60  0001 C CNN "construct"
+F 11 "other,more,stuff" V 1130 2600 60  0001 C CNN "misc"
 	1    4850 5050
 	0    1    1    0

Commit message: more stepper updates
Signed-off-by: Jared Harvey <TortiseGIT@jaredharvey.com>
Parts:
- C8: footprint SM1210 -> SM0805-C1; V (none) -> 25V; Voltate 16v -> (none); construct aluminum -> multi layer ceramic; mfg Nichicon -> (none); mfg# UVZ1C100MDD -> (none); mfg,mfg# (none) -> AVX,08053C104KAT2A; tol 20% -> (none); tolerance (none) -> 10%; vend1 digikey -> (none); vend1# 493-1279-ND -> (none); vend1,vend1# (none) -> newark,96M1381
- R265: W (none) -> 125mW; w 125mW -> (none)
Changed lines of the file:
@@
 F 6 "" V 1130 2600 60  0001 C CNN ""
 F 7 "" V 1130 2600 60  0001 C CNN ""
-F 8 "125mW" V 1130 2600 60  0001 C CNN "w"
+F 8 "125mW" V 1130 2600 60  0001 C CNN "W"
 F 9 "1%" V 1130 2600 60  0001 C CNN "tolerance"
 F 10 "thick film" V 1130 2600 60  0001 C CNN "construct"
@@
 F 0 "C8" H 4900 3600 50  0000 L CNN
 F 1 "10uF" H 4900 3400 50  0000 L CNN
-F 2 "SM1210" V 1130 2600 60  0001 C CNN
-F 4 "Nichicon" V 1130 2600 60  0001 C CNN "mfg"
-F 5 "UVZ1C100MDD" V 1130 2600 60  0001 C CNN "mfg#"
-F 6 "digikey" V 1130 2600 60  0001 C CNN "vend1"
-F 7 "493-1279-ND" V 1130 2600 60  0001 C CNN "vend1#"
-F 8 "16v" V 1130 2600 60  0001 C CNN "Voltate"
-F 9 "20%" V 1130 2600 60  0001 C CNN "tol"
-F 10 "aluminum" V 1130 2600 60  0001 C CNN "construct"
+F 2 "SM0805-C1" V 1130 2600 60  0001 C CNN
+F 4 "AVX,08053C104KAT2A" V 1130 2600 60  0001 C CNN "mfg,mfg#"
+F 5 "newark,96M1381" V 1130 2600 60  0001 C CNN "vend1,vend1#"
+F 6 "" V 1130 2600 60  0001 C CNN ""
+F 7 "" V 1130 2600 60  0001 C CNN ""
+F 8 "25V" V 1130 2600 60  0001 C CNN "V"
+F 9 "10%" V 1130 2600 60  0001 C CNN "tolerance"
+F 10 "multi layer ceramic" V 1130 2600 60  0001 C CNN "construct"
 F 11 "other,more,stuff" V 1130 2600 60  0001 C CNN "misc"
 	1    4850 3500

Commit message: More work on footprints, and schematic BOM's.
Signed-off-by: Jared Harvey <TortiseGIT@jaredharvey.com>
Parts:
- D113: A (none) -> .02A; TOL (none) -> -%; current .02a -> (none); mfg OSRAM -> (none); mfg# LH R974-LP-1-0-20-R18 -> (none); mfg,mfg# (none) -> OSRAM,LH R974-LP-1-0-20-R18; tol -% -> (none); vend1 digikey -> (none); vend1# 475-1415-1-ND -> (none); vend1,vend1# (none) -> DIGI,475-1415-1-ND
Changed lines of the file:
@@
 F 0 "D113" H 4600 4150 50  0000 C CNN
 F 1 "LED" H 4600 3950 50  0000 C CNN
-F 2 "LED-0805" H 4600 4050 60  0001 C CNN
-F 4 "OSRAM" V 1130 2600 60  0001 C CNN "mfg"
-F 5 "LH R974-LP-1-0-20-R18" V 1130 2600 60  0001 C CNN "mfg#"
-F 6 "digikey" V 1130 2600 60  0001 C CNN "vend1"
-F 7 "475-1415-1-ND" V 1130 2600 60  0001 C CNN "vend1#"
-F 8 ".02a" V 1130 2600 60  0001 C CNN "current"
-F 9 "-%" V 1130 2600 60  0001 C CNN "tol"
+F 2 "LED-0805" V 1130 2600 60  0001 C CNN
+F 4 "OSRAM,LH R974-LP-1-0-20-R18" V 1130 2600 60  0001 C CNN "mfg,mfg#"
+F 5 "DIGI,475-1415-1-ND" V 1130 2600 60  0001 C CNN "vend1,vend1#"
+F 6 "" V 1130 2600 60  0001 C CNN ""
+F 7 "" V 1130 2600 60  0001 C CNN ""
+F 8 ".02A" V 1130 2600 60  0001 C CNN "A"
+F 9 "-%" V 1130 2600 60  0001 C CNN "TOL"
 F 10 "RED" V 1130 2600 60  0001 C CNN "construct"
 F 11 "other,more,stuff" V 1130 2600 60  0001 C CNN "misc"
