File: KICAD_Project/sub_circuits/stepper_L297.sch (KiCad schematic (older format))
At the start: 21 parts, among them P801 CONN_1, P802 CONN_1, P803 CONN_1, P804 CONN_1

Commit message: updates to the stepper
Signed-off-by: Jared Harvey <TortiseGIT@jaredharvey.com>
Parts:
- added P?: CONN_1, PINTST, symbol CONN_1
- added R? (x3): 100K, SM0805, symbol R
Connections:
- net labels added: L297_VREF
- wire segments 71 -> 85
- no-connect marks 5 -> 4
Other:
- moved on the sheet: R801, R803, R804

Commit message: more stepper updates
Signed-off-by: Jared Harvey <TortiseGIT@jaredharvey.com>
Parts:
- added C?: 470uF, SM0805-C1, symbol C
- added P?: CONN_1, PINTST, symbol CONN_1
- added R? (x3): 100K, SM0805, symbol R
- C804: Field3 -,- -> (none); Field4 -,- -> (none); Field5 200,V -> (none); Field6 20,% -> (none); Field7 alum electro -> (none); Field8 other,more,stuff -> (none); V (none) -> 25V; construct (none) -> multi layer ceramic; mfg,# ill cap,106CKE200M -> (none); mfg,mfg# (none) -> AVX,08053C104KAT2A; misc (none) -> other,more,stuff; tolerance (none) -> 10%; vend,# newark,69K7896 -> (none); vend1,vend1# (none) -> newark,96M1381
Connections:
- wire segments 85 -> 89
Changed lines of the file:
@@
-EESchema Schematic File Version 2  date 8/27/2011 10:55:18 AM
+EESchema Schematic File Version 2  date 8/30/2011 5:58:29 AM
 LIBS:power
 LIBS:device
@@
 Sheet 8 13
 Title "freeEMS PLUS from Cinch template "
-Date "27 aug 2011"
+Date "30 aug 2011"
 Rev "A-DRAF"
 Comp "diyefi.org/openecu.info"
@@
 Comment4 ""
 $EndDescr
+Connection ~ 4750 6350
+Wire Wire Line
+	4800 6350 4700 6350
+Wire Wire Line
+	5400 6700 5400 6350
+Wire Wire Line
+	5400 6350 5300 6350
 Connection ~ 8375 5650
 Wire Wire Line
@@
 Connection ~ 9100 6850
 Wire Wire Line
-	9100 6800 9100 6850
+	9100 6850 9100 6800
 Wire Wire Line
 	8850 6950 9300 6950
@@
 Connection ~ 9550 5650
 Wire Wire Line
-	10300 5650 8250 5650
+	8250 5650 10300 5650
 Connection ~ 10050 4650
 Wire Wire Line
@@
 	6850 5250 7050 5250
 Wire Wire Line
-	6200 4650 6850 4650
+	6850 4650 6200 4650
 Connection ~ 9850 6000
 Wire Wire Line
@@
 Connection ~ 6200 5150
 Wire Wire Line
-	6200 5250 6200 5050
+	6200 5050 6200 5250
 Wire Wire Line
 	9250 5250 9250 5050
@@
 Connection ~ 6500 5650
 Wire Wire Line
-	7050 5650 6200 5650
+	6200 5650 7050 5650
 Wire Wire Line
 	7050 4850 6900 4850
@@
 	6950 6450 7050 6450
 Wire Wire Line
-	8250 6850 9450 6850
+	9450 6850 8250 6850
 Wire Wire Line
 	10300 6850 9850 6850
@@
 	7050 5050 6500 5050
 Wire Wire Line
-	9550 5250 9550 5050
+	9550 5050 9550 5250
 Connection ~ 9550 5150
 Wire Wire Line
@@
 	6550 6150 6550 7100
 Wire Wire Line
-	6550 7100 10300 7100
-Wire Wire Line
-	10300 7100 10300 5050
+	10300 5050 10300 7100
 Connection ~ 10300 6850
 Connection ~ 10300 5650
@@
 Wire Wire Line
 	8325 6150 8250 6150
+Wire Wire Line
+	5300 6600 5650 6600
+Connection ~ 5400 6600
+Wire Wire Line
+	10300 7100 5400 7100
+Connection ~ 6550 7100
+Connection ~ 5650 7100
+$Comp
+L CONN_1 P?
+U 1 1 4E5CB382
+P 4750 6200
+F 0 "P?" H 4830 6200 40  0000 L CNN
+F 1 "CONN_1" H 4750 6255 30  0001 C CNN
+F 2 "PINTST" H 4750 6200 60  0001 C CNN
+	1    4750 6200
+	0    1    -1   0
+$EndComp
+Text Label 5650 6600 0    60   ~ 0
+L297_VREF
+$Comp
+L R R?
+U 1 1 4E5CB2D8
+P 5050 6350
+F 0 "R?" V 5130 6350 50  0000 C CNN
+F 1 "100K" V 5050 6350 50  0000 C CNN
+F 2 "SM0805" V -1095 3550 60  0001 C CNN
+F 4 "vishay,CRCW08050000Z0EA" V -1095 3550 60  0001 C CNN "mfg,mfg#"
+F 5 "newark,52K9721" V -1095 3550 60  0001 C CNN "vend1,vend1#"
+F 6 "" V -1095 3550 60  0001 C CNN "Field6"
+F 7 "" V -1095 3550 60  0001 C CNN "Field7"
+F 8 "mW" V -1095 3550 60  0001 C CNN "w"
+F 9 "%" V -1095 3550 60  0001 C CNN "tolerance"
+F 10 "" V -1095 3550 60  0001 C CNN "construct"
+F 11 "other,more,stuff" V -1095 3550 60  0001 C CNN "misc"
+	1    5050 6350
+	0    1    1    0
+$EndComp
+$Comp
+L R R?
+U 1 1 4E5CB275
+P 5650 6850
+F 0 "R?" V 5730 6850 50  0000 C CNN
+F 1 "100K" V 5650 6850 50  0000 C CNN
+F 2 "SM0805" V -495 4050 60  0001 C CNN
+F 4 "vishay,CRCW08050000Z0EA" V -495 4050 60  0001 C CNN "mfg,mfg#"
+F 5 "newark,52K9721" V -495 4050 60  0001 C CNN "vend1,vend1#"
+F 6 "" V -495 4050 60  0001 C CNN "Field6"
+F 7 "" V -495 4050 60  0001 C CNN "Field7"
+F 8 "mW" V -495 4050 60  0001 C CNN "w"
+F 9 "%" V -495 4050 60  0001 C CNN "tolerance"
+F 10 "" V -495 4050 60  0001 C CNN "construct"
+F 11 "other,more,stuff" V -495 4050 60  0001 C CNN "misc"
+	1    5650 6850
+	-1   0    0    1
+$EndComp
+$Comp
+L C C?
+U 1 1 4E5CB270
+P 5400 6900
+F 0 "C?" H 5425 7000 50  0000 L CNN
+F 1 "470uF" H 5150 7000 50  0000 L CNN
+F 2 "SM0805-C1" V 2480 8000 60  0001 C CNN
+F 4 "ill cap,106CKE200M" V 2480 8000 60  0001 C CNN "mfg,#"
+F 5 "newark,69K7896" V 2480 8000 60  0001 C CNN "vend,#"
+F 6 "-,-" V 2480 8000 60  0001 C CNN "Field3"
+F 7 "-,-" V 2480 8000 60  0001 C CNN "Field4"
+F 8 "200,V" V 2480 8000 60  0001 C CNN "Field5"
+F 9 "20,%" V 2480 8000 60  0001 C CNN "Field6"
+F 10 "alum electro" V 2480 8000 60  0001 C CNN "Field7"
+F 11 "other,more,stuff" V 2480 8000 60  0001 C CNN "Field8"
+	1    5400 6900
+	1    0    0    1
+$EndComp
+$Comp
+L R R?
+U 1 1 4E5CB26D
+P 5050 6600
+F 0 "R?" V 5130 6600 50  0000 C CNN
+F 1 "100K" V 5050 6600 50  0000 C CNN
+F 2 "SM0805" V -1095 3800 60  0001 C CNN
+F 4 "vishay,CRCW08050000Z0EA" V -1095 3800 60  0001 C CNN "mfg,mfg#"
+F 5 "newark,52K9721" V -1095 3800 60  0001 C CNN "vend1,vend1#"
+F 6 "" V -1095 3800 60  0001 C CNN "Field6"
+F 7 "" V -1095 3800 60  0001 C CNN "Field7"
+F 8 "mW" V -1095 3800 60  0001 C CNN "w"
+F 9 "%" V -1095 3800 60  0001 C CNN "tolerance"
+F 10 "" V -1095 3800 60  0001 C CNN "construct"
+F 11 "other,more,stuff" V -1095 3800 60  0001 C CNN "misc"
+	1    5050 6600
+	0    1    1    0
+$EndComp
+Text Label 4800 6600 2    60   ~ 0
+5V
+Text Label 8250 6550 0    60   ~ 0
+L297_VREF
 $Comp
 L R R?
@@
 $EndComp
 NoConn ~ 7050 6250
-Text HLabel 8250 6550 2    60   Input ~ 0
+Text HLabel 4700 6350 0    60   Input ~ 0
 L297_VREF
 $Comp
@@
 F 0 "C804" V 9700 6150 50  0000 L CNN
 F 1 "10uF" V 9575 6150 50  0000 L CNN
-F 2 "SM0805-C1" V 6730 7450 60  0001 C CNN
-F 4 "ill cap,106CKE200M" V 3130 7950 60  0001 C CNN "mfg,#"
-F 5 "newark,69K7896" V 3130 7950 60  0001 C CNN "vend,#"
-F 6 "-,-" V 3130 7950 60  0001 C CNN "Field3"
-F 7 "-,-" V 3130 7950 60  0001 C CNN "Field4"
-F 8 "200,V" V 3130 7950 60  0001 C CNN "Field5"
-F 9 "20,%" V 3130 7950 60  0001 C CNN "Field6"
-F 10 "alum electro" V 3130 7950 60  0001 C CNN "Field7"
-F 11 "other,more,stuff" V 3130 7950 60  0001 C CNN "Field8"
+F 2 "SM0805-C1" V 1130 2600 60  0001 C CNN
+F 4 "AVX,08053C104KAT2A" V 1130 2600 60  0001 C CNN "mfg,mfg#"
+F 5 "newark,96M1381" V 1130 2600 60  0001 C CNN "vend1,vend1#"
+F 6 "" V 1130 2600 60  0001 C CNN ""
+F 7 "" V 1130 2600 60  0001 C CNN ""
+F 8 "25V" V 1130 2600 60  0001 C CNN "V"
+F 9 "10%" V 1130 2600 60  0001 C CNN "tolerance"
+F 10 "multi layer ceramic" V 1130 2600 60  0001 C CNN "construct"
+F 11 "other,more,stuff" V 1130 2600 60  0001 C CNN "misc"
 	1    9650 6350
 	0    1    -1   0

Commit message: Changed over voltage protected MOSFETs to SO8 footprints.
Signed-off-by: Jared Harvey <TortiseGIT@jaredharvey.com>
Parts:
- removed P?: CONN_1, PINTST, symbol CONN_1
- removed R?: 100K, SM0805, symbol R
- gave numbers to parts that had none: 18
- renumbered C804 to C802, C801 to C803, C802 to C804, P802 to P801, P801 to P802, P803 to P804, P804 to P805, R801 to R805, R803 to R807, R804 to R808
Connections:
- wire segments 89 -> 87

Commit message: More work on footprints, and schematic BOM's.
Signed-off-by: Jared Harvey <TortiseGIT@jaredharvey.com>
Parts:
- D801, D802, D803, D804, D805, D806, D807, D808: footprint (none) -> D4-SMB; mfg,mfg# (none) -> stmicro,STPS340U; vend1,vend# (none) -> quest,STPS340U
- U801: footprint (none) -> SO20_POWER; MFG,MEG# (none) -> st,L298P013TR; VEND,VEND# (none) -> digi,497-3624-1-ND
- U802: footprint S020L -> SO20L; MFG,MFG# (none) -> st,L297D; VEND,VEND# (none) -> newark,89K0738
Changed lines of the file:
@@
-EESchema Schematic File Version 2  date 9/1/2011 7:35:07 PM
+EESchema Schematic File Version 2  date 9/4/2011 3:29:41 PM
 LIBS:power
 LIBS:device
@@
 Sheet 8 13
 Title "freeEMS PLUS from Cinch template "
-Date "1 sep 2011"
+Date "4 sep 2011"
 Rev "A-DRAF"
 Comp "diyefi.org/openecu.info"
@@
 Comment4 ""
 $EndDescr
+$Comp
+L DIODE D808
+U 1 1 4E63B087
+P 9550 5450
+F 0 "D808" H 9550 5550 40  0000 C CNN
+F 1 "DIODE" H 9550 5350 40  0000 C CNN
+F 2 "D4-SMB" H 9550 5450 60  0001 C CNN
+F 4 "stmicro,STPS340U" H 9550 5450 60  0001 C CNN "mfg,mfg#"
+F 5 "quest,STPS340U" H 9550 5450 60  0001 C CNN "vend1,vend#"
+	1    9550 5450
+	0    -1   -1   0
+$EndComp
+$Comp
+L DIODE D806
+U 1 1 4E63B084
+P 9250 5450
+F 0 "D806" H 9250 5550 40  0000 C CNN
+F 1 "DIODE" H 9250 5350 40  0000 C CNN
+F 2 "D4-SMB" H 9250 5450 60  0001 C CNN
+F 4 "stmicro,STPS340U" H 9250 5450 60  0001 C CNN "mfg,mfg#"
+F 5 "quest,STPS340U" H 9250 5450 60  0001 C CNN "vend1,vend#"
+	1    9250 5450
+	0    -1   -1   0
+$EndComp
+$Comp
+L DIODE D805
+U 1 1 4E63B07F
+P 9250 4850
+F 0 "D805" H 9250 4950 40  0000 C CNN
+F 1 "DIODE" H 9250 4750 40  0000 C CNN
+F 2 "D4-SMB" H 9250 4850 60  0001 C CNN
+F 4 "stmicro,STPS340U" H 9250 4850 60  0001 C CNN "mfg,mfg#"
+F 5 "quest,STPS340U" H 9250 4850 60  0001 C CNN "vend1,vend#"
+	1    9250 4850
+	0    -1   -1   0
+$EndComp
+$Comp
+L DIODE D807
+U 1 1 4E63B07C
+P 9550 4850
+F 0 "D807" H 9550 4950 40  0000 C CNN
+F 1 "DIODE" H 9550 4750 40  0000 C CNN
+F 2 "D4-SMB" H 9550 4850 60  0001 C CNN
+F 4 "stmicro,STPS340U" H 9550 4850 60  0001 C CNN "mfg,mfg#"
+F 5 "quest,STPS340U" H 9550 4850 60  0001 C CNN "vend1,vend#"
+	1    9550 4850
+	0    -1   -1   0
+$EndComp
+$Comp
+L DIODE D804
+U 1 1 4E63B07B
+P 6500 5450
+F 0 "D804" H 6500 5550 40  0000 C CNN
+F 1 "DIODE" H 6500 5350 40  0000 C CNN
+F 2 "D4-SMB" H 6500 5450 60  0001 C CNN
+F 4 "stmicro,STPS340U" H 6500 5450 60  0001 C CNN "mfg,mfg#"
+F 5 "quest,STPS340U" H 6500 5450 60  0001 C CNN "vend1,vend#"
+	1    6500 5450
+	0    -1   -1   0
+$EndComp
+$Comp
+L DIODE D802
+U 1 1 4E63B079
+P 6200 5450
+F 0 "D802" H 6200 5550 40  0000 C CNN
+F 1 "DIODE" H 6200 5350 40  0000 C CNN
+F 2 "D4-SMB" H 6200 5450 60  0001 C CNN
+F 4 "stmicro,STPS340U" H 6200 5450 60  0001 C CNN "mfg,mfg#"
+F 5 "quest,STPS340U" H 6200 5450 60  0001 C CNN "vend1,vend#"
+	1    6200 5450
+	0    -1   -1   0
+$EndComp
+$Comp
+L DIODE D803
+U 1 1 4E63B077
+P 6500 4850
+F 0 "D803" H 6500 4950 40  0000 C CNN
+F 1 "DIODE" H 6500 4750 40  0000 C CNN
+F 2 "D4-SMB" H 6500 4850 60  0001 C CNN
+F 4 "stmicro,STPS340U" H 6500 4850 60  0001 C CNN "mfg,mfg#"
+F 5 "quest,STPS340U" H 6500 4850 60  0001 C CNN "vend1,vend#"
+	1    6500 4850
+	0    -1   -1   0
+$EndComp
 Connection ~ 6200 5100
 Connection ~ 9550 5100
@@
 OUT4
 $Comp
-L DIODE D808
-U 1 1 4E58CFA4
-P 9550 5450
-F 0 "D808" H 9550 5550 40  0000 C CNN
-F 1 "DIODE" H 9550 5350 40  0000 C CNN
-	1    9550 5450
-	0    -1   -1   0
-$EndComp
-$Comp
-L DIODE D806
-U 1 1 4E58CFA3
-P 9250 5450
-F 0 "D806" H 9250 5550 40  0000 C CNN
-F 1 "DIODE" H 9250 5350 40  0000 C CNN
-	1    9250 5450
-	0    -1   -1   0
-$EndComp
-$Comp
-L DIODE D804
-U 1 1 4E58CFA2
-P 6500 5450
-F 0 "D804" H 6500 5550 40  0000 C CNN
-F 1 "DIODE" H 6500 5350 40  0000 C CNN
-	1    6500 5450
-	0    -1   -1   0
-$EndComp
-$Comp
-L DIODE D802
-U 1 1 4E58CFA1
-P 6200 5450
-F 0 "D802" H 6200 5550 40  0000 C CNN
-F 1 "DIODE" H 6200 5350 40  0000 C CNN
-	1    6200 5450
-	0    -1   -1   0
-$EndComp
-$Comp
 L DIODE D801
 U 1 1 4E58CF4A
@@
 F 0 "D801" H 6200 4950 40  0000 C CNN
 F 1 "DIODE" H 6200 4750 40  0000 C CNN
+F 2 "D4-SMB" H 6200 4850 60  0001 C CNN
+F 4 "stmicro,STPS340U" H 6200 4850 60  0001 C CNN "mfg,mfg#"
+F 5 "quest,STPS340U" H 6200 4850 60  0001 C CNN "vend1,vend#"
 	1    6200 4850
-	0    -1   -1   0
-$EndComp
-$Comp
-L DIODE D803
-U 1 1 4E58CF49
-P 6500 4850
-F 0 "D803" H 6500 4950 40  0000 C CNN
-F 1 "DIODE" H 6500 4750 40  0000 C CNN
-	1    6500 4850
-	0    -1   -1   0
-$EndComp
-$Comp
-L DIODE D805
-U 1 1 4E58CF41
-P 9250 4850
-F 0 "D805" H 9250 4950 40  0000 C CNN
-F 1 "DIODE" H 9250 4750 40  0000 C CNN
-	1    9250 4850
-	0    -1   -1   0
-$EndComp
-$Comp
-L DIODE D807
-U 1 1 4E58CF3B
-P 9550 4850
-F 0 "D807" H 9550 4950 40  0000 C CNN
-F 1 "DIODE" H 9550 4750 40  0000 C CNN
-	1    9550 4850
 	0    -1   -1   0
 $EndComp
@@
 F 0 "U801" H 7450 5750 70  0000 C CNN
 F 1 "L298N" H 7500 4650 70  0000 C CNN
+F 2 "SO20_POWER" H 7650 5200 60  0001 C CNN
+F 4 "st,L298P013TR" H 7650 5200 60  0001 C CNN "MFG,MEG#"
+F 5 "digi,497-3624-1-ND" H 7650 5200 60  0001 C CNN "VEND,VEND#"
 	1    7650 5200
 	1    0    0    -1
@@
 F 0 "U802" H 7450 7050 70  0000 C CNN
 F 1 "L297" H 7500 5950 70  0000 C CNN
-F 2 "S020L" H 7650 6500 60  0001 C CNN
+F 2 "SO20L" H 7650 6500 60  0001 C CNN
+F 4 "st,L297D" H 7650 6500 60  0001 C CNN "MFG,MFG#"
+F 5 "newark,89K0738" H 7650 6500 60  0001 C CNN "VEND,VEND#"
 	1    7650 6500
 	1    0    0    -1
