File: KICAD_Project/sub_circuits/stepper_L297.sch (KiCad schematic (older format))
At the start: 28 parts, among them P801 CONN_1, P802 CONN_1, P803 CONN_1, P804 CONN_1, P805 CONN_1, U801 L298N, U802 L297

Commit message: Made more progress on the AN protects and LS drive 33800
Signed-off-by: Jared Harvey <TortiseGIT@jaredharvey.com>
Parts:
- C803: footprint SM0805-C1 -> SM0805; TOL (none) -> 10%; V 100V -> 200V; construct ceramic -> CERAMIC; mfg,mfg# avx,08051C104KAT2A -> AVX,08055C104KAT2A; tolerance 10% -> (none); vend1,vend1# newark,96M1354 -> newark,27C8438
- C805: footprint SM0805-C1 -> SM0805; Field3 -,- -> (none); Field4 -,- -> (none); Field5 200,V -> (none); Field6 20,% -> (none); Field7 alum electro -> (none); Field8 other,more,stuff -> (none); TOL (none) -> 10%; V (none) -> 200V; construct (none) -> CERAMIC; mfg,# ill cap,106CKE200M -> (none); mfg,mfg# (none) -> AVX,08055C104KAT2A; misc (none) -> other,more,stuff; vend,# newark,69K7896 -> (none); vend1,vend1# (none) -> newark,27C8438
Changed lines of the file:
@@
 F 0 "C805" H 10325 4950 50  0000 L CNN
 F 1 "100nF" H 10050 4950 50  0000 L CNN
-F 2 "SM0805-C1" V 7380 5950 60  0001 C CNN
-F 4 "ill cap,106CKE200M" V 7380 5950 60  0001 C CNN "mfg,#"
-F 5 "newark,69K7896" V 7380 5950 60  0001 C CNN "vend,#"
-F 6 "-,-" V 7380 5950 60  0001 C CNN "Field3"
-F 7 "-,-" V 7380 5950 60  0001 C CNN "Field4"
-F 8 "200,V" V 7380 5950 60  0001 C CNN "Field5"
-F 9 "20,%" V 7380 5950 60  0001 C CNN "Field6"
-F 10 "alum electro" V 7380 5950 60  0001 C CNN "Field7"
-F 11 "other,more,stuff" V 7380 5950 60  0001 C CNN "Field8"
+F 2 "SM0805" V 1130 2600 60  0001 C CNN
+F 4 "AVX,08055C104KAT2A" V 1130 2600 60  0001 C CNN "mfg,mfg#"
+F 5 "newark,27C8438" V 1130 2600 60  0001 C CNN "vend1,vend1#"
+F 6 "" V 1130 2600 60  0001 C CNN ""
+F 7 "" V 1130 2600 60  0001 C CNN ""
+F 8 "200V" V 1130 2600 60  0001 C CNN "V"
+F 9 "10%" V 1130 2600 60  0001 C CNN "TOL"
+F 10 "CERAMIC" V 1130 2600 60  0001 C CNN "construct"
+F 11 "other,more,stuff" V 1130 2600 60  0001 C CNN "misc"
 	1    10300 4850
 	1    0    0    1
@@
 F 0 "C803" V 9570 6710 50  0000 L CNN
 F 1 "100nF" V 9575 7050 50  0000 L CNN
-F 2 "SM0805-C1" V 4580 4150 60  0001 C CNN
-F 4 "avx,08051C104KAT2A" V 4580 4150 60  0001 C CNN "mfg,mfg#"
-F 5 "newark,96M1354" V 4580 4150 60  0001 C CNN "vend1,vend1#"
-F 6 "" V 4580 4150 60  0001 C CNN "Field6"
-F 7 "" V 4580 4150 60  0001 C CNN "Field7"
-F 8 "100V" V 4580 4150 60  0001 C CNN "V"
-F 9 "10%" V 4580 4150 60  0001 C CNN "tolerance"
-F 10 "ceramic" V 4580 4150 60  0001 C CNN "construct"
-F 11 "other,more,stuff" V 4580 4150 60  0001 C CNN "misc"
+F 2 "SM0805" V 1130 2600 60  0001 C CNN
+F 4 "AVX,08055C104KAT2A" V 1130 2600 60  0001 C CNN "mfg,mfg#"
+F 5 "newark,27C8438" V 1130 2600 60  0001 C CNN "vend1,vend1#"
+F 6 "" V 1130 2600 60  0001 C CNN ""
+F 7 "" V 1130 2600 60  0001 C CNN ""
+F 8 "200V" V 1130 2600 60  0001 C CNN "V"
+F 9 "10%" V 1130 2600 60  0001 C CNN "TOL"
+F 10 "CERAMIC" V 1130 2600 60  0001 C CNN "construct"
+F 11 "other,more,stuff" V 1130 2600 60  0001 C CNN "misc"
 	1    9650 6850
 	0    1    -1   0
