File: KICAD_Project/sub_circuits/an_protect2.sch (KiCad schematic (older format))
At the start: 20 parts

Commit message: More work on footprints, and schematic BOM's.
Signed-off-by: Jared Harvey <TortiseGIT@jaredharvey.com>
Parts:
- R364, R365, R366, R367, R368, R369, R370, R371: W (none) -> 125mW; tol (none) -> 1%; tolerance 1% -> (none); w 125mW -> (none)
Changed lines of the file:
@@
 F 6 "" V 1130 2600 60  0001 C CNN ""
 F 7 "" V 1130 2600 60  0001 C CNN ""
-F 8 "125mW" V 1130 2600 60  0001 C CNN "w"
-F 9 "1%" V 1130 2600 60  0001 C CNN "tolerance"
+F 8 "125mW" V 1130 2600 60  0001 C CNN "W"
+F 9 "1%" V 1130 2600 60  0001 C CNN "tol"
 F 10 "thick film" V 1130 2600 60  0001 C CNN "construct"
 F 11 "other,more,stuff" V 1130 2600 60  0001 C CNN "misc"
@@
 F 6 "" V 1130 2600 60  0001 C CNN ""
 F 7 "" V 1130 2600 60  0001 C CNN ""
-F 8 "125mW" V 1130 2600 60  0001 C CNN "w"
-F 9 "1%" V 1130 2600 60  0001 C CNN "tolerance"
+F 8 "125mW" V 1130 2600 60  0001 C CNN "W"
+F 9 "1%" V 1130 2600 60  0001 C CNN "tol"
 F 10 "thick film" V 1130 2600 60  0001 C CNN "construct"
 F 11 "other,more,stuff" V 1130 2600 60  0001 C CNN "misc"
@@
 F 6 "" V 1130 2600 60  0001 C CNN ""
 F 7 "" V 1130 2600 60  0001 C CNN ""
-F 8 "125mW" V 1130 2600 60  0001 C CNN "w"
-F 9 "1%" V 1130 2600 60  0001 C CNN "tolerance"
+F 8 "125mW" V 1130 2600 60  0001 C CNN "W"
+F 9 "1%" V 1130 2600 60  0001 C CNN "tol"
 F 10 "thick film" V 1130 2600 60  0001 C CNN "construct"
 F 11 "other,more,stuff" V 1130 2600 60  0001 C CNN "misc"
@@
 F 6 "" V 1130 2600 60  0001 C CNN ""
 F 7 "" V 1130 2600 60  0001 C CNN ""
-F 8 "125mW" V 1130 2600 60  0001 C CNN "w"
-F 9 "1%" V 1130 2600 60  0001 C CNN "tolerance"
+F 8 "125mW" V 1130 2600 60  0001 C CNN "W"
+F 9 "1%" V 1130 2600 60  0001 C CNN "tol"
 F 10 "thick film" V 1130 2600 60  0001 C CNN "construct"
 F 11 "other,more,stuff" V 1130 2600 60  0001 C CNN "misc"
@@
 F 6 "" V 1130 2600 60  0001 C CNN ""
 F 7 "" V 1130 2600 60  0001 C CNN ""
-F 8 "125mW" V 1130 2600 60  0001 C CNN "w"
-F 9 "1%" V 1130 2600 60  0001 C CNN "tolerance"
+F 8 "125mW" V 1130 2600 60  0001 C CNN "W"
+F 9 "1%" V 1130 2600 60  0001 C CNN "tol"
 F 10 "thick film" V 1130 2600 60  0001 C CNN "construct"
 F 11 "other,more,stuff" V 1130 2600 60  0001 C CNN "misc"
@@
 F 6 "" V 1130 2600 60  0001 C CNN ""
 F 7 "" V 1130 2600 60  0001 C CNN ""
-F 8 "125mW" V 1130 2600 60  0001 C CNN "w"
-F 9 "1%" V 1130 2600 60  0001 C CNN "tolerance"
+F 8 "125mW" V 1130 2600 60  0001 C CNN "W"
+F 9 "1%" V 1130 2600 60  0001 C CNN "tol"
 F 10 "thick film" V 1130 2600 60  0001 C CNN "construct"
 F 11 "other,more,stuff" V 1130 2600 60  0001 C CNN "misc"
@@
 F 6 "" V 1130 2600 60  0001 C CNN ""
 F 7 "" V 1130 2600 60  0001 C CNN ""
-F 8 "125mW" V 1130 2600 60  0001 C CNN "w"
-F 9 "1%" V 1130 2600 60  0001 C CNN "tolerance"
+F 8 "125mW" V 1130 2600 60  0001 C CNN "W"
+F 9 "1%" V 1130 2600 60  0001 C CNN "tol"
 F 10 "thick film" V 1130 2600 60  0001 C CNN "construct"
 F 11 "other,more,stuff" V 1130 2600 60  0001 C CNN "misc"
@@
 F 6 "" V 1130 2600 60  0001 C CNN ""
 F 7 "" V 1130 2600 60  0001 C CNN ""
-F 8 "125mW" V 1130 2600 60  0001 C CNN "w"
-F 9 "1%" V 1130 2600 60  0001 C CNN "tolerance"
-F 10 "thick film" V 1130 2600 60  0001 C CNN "construct"
-F 11 "other,more,stuff" V 1130 2600 60  0001 C CNN "misc"
+F 8 "125mW" V 1130 2600 60  0001 C CNN "W"
+F 9 "1%" V 1130 2600 60  0001 C CNN "tol"
+F 10 "thick film" V 1130 2600 60  0001 C CNN "construct"
+F 11 "other,more,stuff" V 1130 2600 60  0001 C CNN "misc"

Commit message: routed all inj/ign's such that they simply need to be connected to the MCU pins.
Signed-off-by: Jared Harvey <TortiseGIT@jaredharvey.com>
Parts:
- R364, R365, R366, R367, R368, R369, R370, R371: TOL (none) -> 1%; construct thick film -> THICK FILM; tol 1% -> (none)
Changed lines of the file:
@@
 F 7 "" V 1130 2600 60  0001 C CNN ""
 F 8 "125mW" V 1130 2600 60  0001 C CNN "W"
-F 9 "1%" V 1130 2600 60  0001 C CNN "tol"
-F 10 "thick film" V 1130 2600 60  0001 C CNN "construct"
+F 9 "1%" V 1130 2600 60  0001 C CNN "TOL"
+F 10 "THICK FILM" V 1130 2600 60  0001 C CNN "construct"
 F 11 "other,more,stuff" V 1130 2600 60  0001 C CNN "misc"
 	1    6750 6450
@@
 F 7 "" V 1130 2600 60  0001 C CNN ""
 F 8 "125mW" V 1130 2600 60  0001 C CNN "W"
-F 9 "1%" V 1130 2600 60  0001 C CNN "tol"
-F 10 "thick film" V 1130 2600 60  0001 C CNN "construct"
+F 9 "1%" V 1130 2600 60  0001 C CNN "TOL"
+F 10 "THICK FILM" V 1130 2600 60  0001 C CNN "construct"
 F 11 "other,more,stuff" V 1130 2600 60  0001 C CNN "misc"
 	1    8450 6450
@@
 F 7 "" V 1130 2600 60  0001 C CNN ""
 F 8 "125mW" V 1130 2600 60  0001 C CNN "W"
-F 9 "1%" V 1130 2600 60  0001 C CNN "tol"
-F 10 "thick film" V 1130 2600 60  0001 C CNN "construct"
+F 9 "1%" V 1130 2600 60  0001 C CNN "TOL"
+F 10 "THICK FILM" V 1130 2600 60  0001 C CNN "construct"
 F 11 "other,more,stuff" V 1130 2600 60  0001 C CNN "misc"
 	1    8500 5050
@@
 F 7 "" V 1130 2600 60  0001 C CNN ""
 F 8 "125mW" V 1130 2600 60  0001 C CNN "W"
-F 9 "1%" V 1130 2600 60  0001 C CNN "tol"
-F 10 "thick film" V 1130 2600 60  0001 C CNN "construct"
+F 9 "1%" V 1130 2600 60  0001 C CNN "TOL"
+F 10 "THICK FILM" V 1130 2600 60  0001 C CNN "construct"
 F 11 "other,more,stuff" V 1130 2600 60  0001 C CNN "misc"
 	1    6800 5050
@@
 F 7 "" V 1130 2600 60  0001 C CNN ""
 F 8 "125mW" V 1130 2600 60  0001 C CNN "W"
-F 9 "1%" V 1130 2600 60  0001 C CNN "tol"
-F 10 "thick film" V 1130 2600 60  0001 C CNN "construct"
+F 9 "1%" V 1130 2600 60  0001 C CNN "TOL"
+F 10 "THICK FILM" V 1130 2600 60  0001 C CNN "construct"
 F 11 "other,more,stuff" V 1130 2600 60  0001 C CNN "misc"
 	1    6850 3750
@@
 F 7 "" V 1130 2600 60  0001 C CNN ""
 F 8 "125mW" V 1130 2600 60  0001 C CNN "W"
-F 9 "1%" V 1130 2600 60  0001 C CNN "tol"
-F 10 "thick film" V 1130 2600 60  0001 C CNN "construct"
+F 9 "1%" V 1130 2600 60  0001 C CNN "TOL"
+F 10 "THICK FILM" V 1130 2600 60  0001 C CNN "construct"
 F 11 "other,more,stuff" V 1130 2600 60  0001 C CNN "misc"
 	1    8550 3750
@@
 F 7 "" V 1130 2600 60  0001 C CNN ""
 F 8 "125mW" V 1130 2600 60  0001 C CNN "W"
-F 9 "1%" V 1130 2600 60  0001 C CNN "tol"
-F 10 "thick film" V 1130 2600 60  0001 C CNN "construct"
+F 9 "1%" V 1130 2600 60  0001 C CNN "TOL"
+F 10 "THICK FILM" V 1130 2600 60  0001 C CNN "construct"
 F 11 "other,more,stuff" V 1130 2600 60  0001 C CNN "misc"
 	1    8600 2400
@@
 F 7 "" V 1130 2600 60  0001 C CNN ""
 F 8 "125mW" V 1130 2600 60  0001 C CNN "W"
-F 9 "1%" V 1130 2600 60  0001 C CNN "tol"
-F 10 "thick film" V 1130 2600 60  0001 C CNN "construct"
+F 9 "1%" V 1130 2600 60  0001 C CNN "TOL"
+F 10 "THICK FILM" V 1130 2600 60  0001 C CNN "construct"
 F 11 "other,more,stuff" V 1130 2600 60  0001 C CNN "misc"
 	1    6900 2400
