File: KICAD_Project/sub_circuits/power_reg_s1.sch (KiCad schematic (older format))
At the start: 19 parts, among them U35 L5973D

Commit message: I did a fiar bit of work, and I want to be able to step back if I can, so this is a misc check in.
Signed-off-by: Jared Harvey <TortiseGIT@jaredharvey.com>
Other:
- moved on the sheet: C134, C135, C136, C137, C138, C139, C140, C141, C143, C144, D117, D118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

Commit message: caps have been done with the scripts next up is the resistors.
Signed-off-by: Jared Harvey <TortiseGIT@jaredharvey.com>
Parts:
- C134, C138, C141: Field3 -,- -> (none); Field4 -,- -> (none); Field5 50,V -> (none); Field6 10,% -> (none); Field7 ceramic -> (none); Field8 other,more,stuff -> (none); V (none) -> 100V; construct (none) -> ceramic; mfg,# murata,GRM21BR71H104KA01L -> (none); mfg,mfg# (none) -> avx,08051C104KAT2A; misc (none) -> other,more,stuff; tolerance (none) -> 10%; vend,# newark,38K1694 -> (none); vend1,vend1# (none) -> newark,96M1354
- C144: Field3 -,- -> (none); Field4 -,- -> (none); Field5 50,V -> (none); Field6 5,% -> (none); Field7 ceramic -> (none); Field8 other,more,stuff -> (none); V (none) -> 200V; construct (none) -> alum elec; mfg,# murata,GRM216R71H103JA01D -> (none); mfg,mfg# (none) -> ill cap,106CKE200M; misc (none) -> other,more,stuff; tolerance (none) -> 10%; vend,# newark,38K1697 -> (none); vend1,vend1# (none) -> newark,69K7896
Changed lines of the file:
@@
 F 0 "C144" H 4500 2550 50  0000 L CNN
 F 1 "10nF" H 4500 2350 50  0000 L CNN
-F 2 "SM0805-C1" V 980 1550 60  0001 C CNN
-F 4 "murata,GRM216R71H103JA01D" V 480 1150 60  0001 C CNN "mfg,#"
-F 5 "newark,38K1697" V 480 1150 60  0001 C CNN "vend,#"
-F 6 "-,-" V 480 1150 60  0001 C CNN "Field3"
-F 7 "-,-" V 480 1150 60  0001 C CNN "Field4"
-F 8 "50,V" V 480 1150 60  0001 C CNN "Field5"
-F 9 "5,%" V 480 1150 60  0001 C CNN "Field6"
-F 10 "ceramic" V 480 1150 60  0001 C CNN "Field7"
-F 11 "other,more,stuff" V 480 1150 60  0001 C CNN "Field8"
+F 2 "SM0805-C1" V 1130 2600 60  0001 C CNN
+F 4 "ill cap,106CKE200M" V 1130 2600 60  0001 C CNN "mfg,mfg#"
+F 5 "newark,69K7896" V 1130 2600 60  0001 C CNN "vend1,vend1#"
+F 6 "" V 1130 2600 60  0001 C CNN ""
+F 7 "" V 1130 2600 60  0001 C CNN ""
+F 8 "200V" V 1130 2600 60  0001 C CNN "V"
+F 9 "10%" V 1130 2600 60  0001 C CNN "tolerance"
+F 10 "alum elec" V 1130 2600 60  0001 C CNN "construct"
+F 11 "other,more,stuff" V 1130 2600 60  0001 C CNN "misc"
 	1    4700 2450
 	-1   0    0    -1
@@
 F 0 "C134" H 1250 950 50  0000 L CNN
 F 1 "100nF" H 1250 750 50  0000 L CNN
-F 2 "SM0805-C1" V -3370 -50 60  0001 C CNN
-F 4 "murata,GRM21BR71H104KA01L " V -3370 -50 60  0001 C CNN "mfg,#"
-F 5 "newark,38K1694" V -3370 -50 60  0001 C CNN "vend,#"
-F 6 "-,-" V -3370 -50 60  0001 C CNN "Field3"
-F 7 "-,-" V -3370 -50 60  0001 C CNN "Field4"
-F 8 "50,V" V -3370 -50 60  0001 C CNN "Field5"
-F 9 "10,%" V -3370 -50 60  0001 C CNN "Field6"
-F 10 "ceramic" V -3370 -50 60  0001 C CNN "Field7"
-F 11 "other,more,stuff" V -3370 -50 60  0001 C CNN "Field8"
+F 2 "SM0805-C1" V 1130 2600 60  0001 C CNN
+F 4 "avx,08051C104KAT2A" V 1130 2600 60  0001 C CNN "mfg,mfg#"
+F 5 "newark,96M1354" V 1130 2600 60  0001 C CNN "vend1,vend1#"
+F 6 "" V 1130 2600 60  0001 C CNN ""
+F 7 "" V 1130 2600 60  0001 C CNN ""
+F 8 "100V" V 1130 2600 60  0001 C CNN "V"
+F 9 "10%" V 1130 2600 60  0001 C CNN "tolerance"
+F 10 "ceramic" V 1130 2600 60  0001 C CNN "construct"
+F 11 "other,more,stuff" V 1130 2600 60  0001 C CNN "misc"
 	1    1200 850
 	-1   0    0    -1
@@
 F 0 "C141" H 3710 950 50  0000 L CNN
 F 1 "100nF" H 3650 750 50  0000 L CNN
-F 2 "SM0805-C1" V 1480 -50 60  0001 C CNN
-F 4 "murata,GRM21BR71H104KA01L " V -3370 -50 60  0001 C CNN "mfg,#"
-F 5 "newark,38K1694" V -3370 -50 60  0001 C CNN "vend,#"
-F 6 "-,-" V -3370 -50 60  0001 C CNN "Field3"
-F 7 "-,-" V -3370 -50 60  0001 C CNN "Field4"
-F 8 "50,V" V -3370 -50 60  0001 C CNN "Field5"
-F 9 "10,%" V -3370 -50 60  0001 C CNN "Field6"
-F 10 "ceramic" V -3370 -50 60  0001 C CNN "Field7"
-F 11 "other,more,stuff" V -3370 -50 60  0001 C CNN "Field8"
+F 2 "SM0805-C1" V 1130 2600 60  0001 C CNN
+F 4 "avx,08051C104KAT2A" V 1130 2600 60  0001 C CNN "mfg,mfg#"
+F 5 "newark,96M1354" V 1130 2600 60  0001 C CNN "vend1,vend1#"
+F 6 "" V 1130 2600 60  0001 C CNN ""
+F 7 "" V 1130 2600 60  0001 C CNN ""
+F 8 "100V" V 1130 2600 60  0001 C CNN "V"
+F 9 "10%" V 1130 2600 60  0001 C CNN "tolerance"
+F 10 "ceramic" V 1130 2600 60  0001 C CNN "construct"
+F 11 "other,more,stuff" V 1130 2600 60  0001 C CNN "misc"
 	1    3900 850
 	-1   0    0    -1
@@
 F 0 "C138" H 2350 960 50  0000 L CNN
 F 1 "100nF" H 2250 750 50  0000 L CNN
-F 2 "SM0805-C1" V -1220 -50 60  0001 C CNN
-F 4 "murata,GRM21BR71H104KA01L " V -3370 -50 60  0001 C CNN "mfg,#"
-F 5 "newark,38K1694" V -3370 -50 60  0001 C CNN "vend,#"
-F 6 "-,-" V -3370 -50 60  0001 C CNN "Field3"
-F 7 "-,-" V -3370 -50 60  0001 C CNN "Field4"
-F 8 "50,V" V -3370 -50 60  0001 C CNN "Field5"
-F 9 "10,%" V -3370 -50 60  0001 C CNN "Field6"
-F 10 "ceramic" V -3370 -50 60  0001 C CNN "Field7"
-F 11 "other,more,stuff" V -3370 -50 60  0001 C CNN "Field8"
+F 2 "SM0805-C1" V 1130 2600 60  0001 C CNN
+F 4 "avx,08051C104KAT2A" V 1130 2600 60  0001 C CNN "mfg,mfg#"
+F 5 "newark,96M1354" V 1130 2600 60  0001 C CNN "vend1,vend1#"
+F 6 "" V 1130 2600 60  0001 C CNN ""
+F 7 "" V 1130 2600 60  0001 C CNN ""
+F 8 "100V" V 1130 2600 60  0001 C CNN "V"
+F 9 "10%" V 1130 2600 60  0001 C CNN "tolerance"
+F 10 "ceramic" V 1130 2600 60  0001 C CNN "construct"
+F 11 "other,more,stuff" V 1130 2600 60  0001 C CNN "misc"
 	1    2500 850
 	-1   0    0    -1

Commit message: Looks like the bulk components are golden now, there are still a couple straglers, mostly switch mode power supply stuff.
Signed-off-by: Jared Harvey <TortiseGIT@jaredharvey.com>
Parts:
- L2: Field3 -,- -> (none); Field4 -,- -> (none); Field5 1,a -> (none); Field6 20,% -> (none); Field7 - -> (none); Field8 other,more,stuff -> (none); H (none) -> 33uH; construct (none) -> ferrite; mfg,# DR125-330-R -> (none); mfg,mfg# (none) -> coiltronics,DR125-330-R; misc (none) -> other,more,stuff; tolerance (none) -> 20%; vend,# newark,63K3559 -> (none); vend1,vend1# (none) -> digi,513-1528-6-ND
Changed lines of the file:
@@
 F 0 "L2" V 3200 2250 40  0000 C CNN
 F 1 "DR125-330-R" V 3350 2250 40  0000 C CNN
-F 2 "SM100uH" H 3250 2250 60  0001 C CNN
-F 3 "PF0504.473NL Pulse Eng" H 3250 2250 60  0001 C CNN
-F 4 "DR125-330-R" H 3250 2250 60  0001 C CNN "mfg,#"
-F 5 "newark,63K3559" H 3250 2250 60  0001 C CNN "vend,#"
-F 6 "-,-" V 880 800 60  0001 C CNN "Field3"
-F 7 "-,-" V 880 800 60  0001 C CNN "Field4"
-F 8 "1,a" V 880 800 60  0001 C CNN "Field5"
-F 9 "20,%" V 880 800 60  0001 C CNN "Field6"
-F 10 "-" V 880 800 60  0001 C CNN "Field7"
-F 11 "other,more,stuff" V 880 800 60  0001 C CNN "Field8"
+F 2 "SM100uH" V 1130 2600 60  0001 C CNN
+F 4 "coiltronics,DR125-330-R" V 1130 2600 60  0001 C CNN "mfg,mfg#"
+F 5 "digi,513-1528-6-ND" V 1130 2600 60  0001 C CNN "vend1,vend1#"
+F 6 "" V 1130 2600 60  0001 C CNN ""
+F 7 "" V 1130 2600 60  0001 C CNN ""
+F 8 "33uH" V 1130 2600 60  0001 C CNN "H"
+F 9 "20%" V 1130 2600 60  0001 C CNN "tolerance"
+F 10 "ferrite" V 1130 2600 60  0001 C CNN "construct"
+F 11 "other,more,stuff" V 1130 2600 60  0001 C CNN "misc"
 	1    3250 2250
 	0    1    1    0

Commit message: more stepper updates
Signed-off-by: Jared Harvey <TortiseGIT@jaredharvey.com>
Parts:
- C135, C139: Field3 -,- -> (none); Field4 -,- -> (none); Field5 35,V -> (none); Field6 20,% -> (none); Field7 alum electro -> (none); Field8 other,more,stuff -> (none); V (none) -> 100V; construct (none) -> ceramic; mfg,# ill cap,107CKE035M -> (none); mfg,mfg# (none) -> avx,08051C104KAT2A; misc (none) -> other,more,stuff; tolerance (none) -> 10%; vend,# newark,69K7903 -> (none); vend1,vend1# (none) -> newark,96M1354
- C143: Field3 -,- -> (none); Field4 -,- -> (none); Field5 200,V -> (none); Field6 20,% -> (none); Field7 alum electro -> (none); Field8 other,more,stuff -> (none); V (none) -> 25V; construct (none) -> multi layer ceramic; mfg,# ill cap,106CKE200M -> (none); mfg,mfg# (none) -> AVX,08053C104KAT2A; misc (none) -> other,more,stuff; tolerance (none) -> 10%; vend,# newark,69K7896 -> (none); vend1,vend1# (none) -> newark,96M1381
Changed lines of the file:
@@
 F 0 "C143" H 4000 2550 50  0000 L CNN
 F 1 "10uF" H 4000 2350 50  0000 L CNN
-F 2 "SM0805-C1" V 480 1550 60  0001 C CNN
-F 4 "ill cap,106CKE200M" V 480 1550 60  0001 C CNN "mfg,#"
-F 5 "newark,69K7896" V 480 1550 60  0001 C CNN "vend,#"
-F 6 "-,-" V 480 1550 60  0001 C CNN "Field3"
-F 7 "-,-" V 480 1550 60  0001 C CNN "Field4"
-F 8 "200,V" V 480 1550 60  0001 C CNN "Field5"
-F 9 "20,%" V 480 1550 60  0001 C CNN "Field6"
-F 10 "alum electro" V 480 1550 60  0001 C CNN "Field7"
-F 11 "other,more,stuff" V 480 1550 60  0001 C CNN "Field8"
+F 2 "SM0805-C1" V 1130 2600 60  0001 C CNN
+F 4 "AVX,08053C104KAT2A" V 1130 2600 60  0001 C CNN "mfg,mfg#"
+F 5 "newark,96M1381" V 1130 2600 60  0001 C CNN "vend1,vend1#"
+F 6 "" V 1130 2600 60  0001 C CNN ""
+F 7 "" V 1130 2600 60  0001 C CNN ""
+F 8 "25V" V 1130 2600 60  0001 C CNN "V"
+F 9 "10%" V 1130 2600 60  0001 C CNN "tolerance"
+F 10 "multi layer ceramic" V 1130 2600 60  0001 C CNN "construct"
+F 11 "other,more,stuff" V 1130 2600 60  0001 C CNN "misc"
 	1    4200 2450
 	-1   0    0    -1
@@
 F 0 "C135" H 2250 950 50  0000 L CNN
 F 1 "100uF" H 2200 750 50  0000 L CNN
-F 2 "SM0805-C1" V -1970 -50 60  0001 C CNN
-F 4 "ill cap,107CKE035M" V -1970 -50 60  0001 C CNN "mfg,#"
-F 5 "newark,69K7903" V -1970 -50 60  0001 C CNN "vend,#"
-F 6 "-,-" V -1970 -50 60  0001 C CNN "Field3"
-F 7 "-,-" V -1970 -50 60  0001 C CNN "Field4"
-F 8 "35,V" V -1970 -50 60  0001 C CNN "Field5"
-F 9 "20,%" V -1970 -50 60  0001 C CNN "Field6"
-F 10 "alum electro" V -1970 -50 60  0001 C CNN "Field7"
-F 11 "other,more,stuff" V -1970 -50 60  0001 C CNN "Field8"
+F 2 "SM0805-C1" V 1130 2600 60  0001 C CNN
+F 4 "avx,08051C104KAT2A" V 1130 2600 60  0001 C CNN "mfg,mfg#"
+F 5 "newark,96M1354" V 1130 2600 60  0001 C CNN "vend1,vend1#"
+F 6 "" V 1130 2600 60  0001 C CNN ""
+F 7 "" V 1130 2600 60  0001 C CNN ""
+F 8 "100V" V 1130 2600 60  0001 C CNN "V"
+F 9 "10%" V 1130 2600 60  0001 C CNN "tolerance"
+F 10 "ceramic" V 1130 2600 60  0001 C CNN "construct"
+F 11 "other,more,stuff" V 1130 2600 60  0001 C CNN "misc"
 	1    2150 850
 	-1   0    0    -1
@@
 F 0 "C139" H 3520 950 50  0000 L CNN
 F 1 "100uF" H 3450 750 50  0000 L CNN
-F 2 "SM0805-C1" V 1430 -50 60  0001 C CNN
-F 4 "ill cap,107CKE035M" V -1970 -50 60  0001 C CNN "mfg,#"
-F 5 "newark,69K7903" V -1970 -50 60  0001 C CNN "vend,#"
-F 6 "-,-" V -1970 -50 60  0001 C CNN "Field3"
-F 7 "-,-" V -1970 -50 60  0001 C CNN "Field4"
-F 8 "35,V" V -1970 -50 60  0001 C CNN "Field5"
-F 9 "20,%" V -1970 -50 60  0001 C CNN "Field6"
-F 10 "alum electro" V -1970 -50 60  0001 C CNN "Field7"
-F 11 "other,more,stuff" V -1970 -50 60  0001 C CNN "Field8"
+F 2 "SM0805-C1" V 1130 2600 60  0001 C CNN
+F 4 "avx,08051C104KAT2A" V 1130 2600 60  0001 C CNN "mfg,mfg#"
+F 5 "newark,96M1354" V 1130 2600 60  0001 C CNN "vend1,vend1#"
+F 6 "" V 1130 2600 60  0001 C CNN ""
+F 7 "" V 1130 2600 60  0001 C CNN ""
+F 8 "100V" V 1130 2600 60  0001 C CNN "V"
+F 9 "10%" V 1130 2600 60  0001 C CNN "tolerance"
+F 10 "ceramic" V 1130 2600 60  0001 C CNN "construct"
+F 11 "other,more,stuff" V 1130 2600 60  0001 C CNN "misc"
 	1    3400 850
 	-1   0    0    -1

Commit message: Made more progress on the AN protects and LS drive 33800
Signed-off-by: Jared Harvey <TortiseGIT@jaredharvey.com>
Parts:
- C134, C138, C141: footprint SM0805-C1 -> SM0805; TOL (none) -> 10%; V 100V -> 200V; construct ceramic -> CERAMIC; mfg,mfg# avx,08051C104KAT2A -> AVX,08055C104KAT2A; tolerance 10% -> (none); vend1,vend1# newark,96M1354 -> newark,27C8438
- C144: footprint SM0805-C1 -> SM0805; TOL (none) -> 10%; V 200V -> 50V; construct alum elec -> CERAMIC; mfg,mfg# ill cap,106CKE200M -> AVX,08055C103KAT2A; tolerance 10% -> (none); vend1,vend1# newark,69K7896 -> newark,07J3575
Changed lines of the file:
@@
 F 0 "C144" H 4500 2550 50  0000 L CNN
 F 1 "10nF" H 4500 2350 50  0000 L CNN
-F 2 "SM0805-C1" V 1130 2600 60  0001 C CNN
-F 4 "ill cap,106CKE200M" V 1130 2600 60  0001 C CNN "mfg,mfg#"
-F 5 "newark,69K7896" V 1130 2600 60  0001 C CNN "vend1,vend1#"
-F 6 "" V 1130 2600 60  0001 C CNN ""
-F 7 "" V 1130 2600 60  0001 C CNN ""
-F 8 "200V" V 1130 2600 60  0001 C CNN "V"
-F 9 "10%" V 1130 2600 60  0001 C CNN "tolerance"
-F 10 "alum elec" V 1130 2600 60  0001 C CNN "construct"
+F 2 "SM0805" V 1130 2600 60  0001 C CNN
+F 4 "AVX,08055C103KAT2A" V 1130 2600 60  0001 C CNN "mfg,mfg#"
+F 5 "newark,07J3575" V 1130 2600 60  0001 C CNN "vend1,vend1#"
+F 6 "" V 1130 2600 60  0001 C CNN ""
+F 7 "" V 1130 2600 60  0001 C CNN ""
+F 8 "50V" V 1130 2600 60  0001 C CNN "V"
+F 9 "10%" V 1130 2600 60  0001 C CNN "TOL"
+F 10 "CERAMIC" V 1130 2600 60  0001 C CNN "construct"
 F 11 "other,more,stuff" V 1130 2600 60  0001 C CNN "misc"
 	1    4700 2450
@@
 F 0 "C134" H 1250 950 50  0000 L CNN
 F 1 "100nF" H 1250 750 50  0000 L CNN
-F 2 "SM0805-C1" V 1130 2600 60  0001 C CNN
-F 4 "avx,08051C104KAT2A" V 1130 2600 60  0001 C CNN "mfg,mfg#"
-F 5 "newark,96M1354" V 1130 2600 60  0001 C CNN "vend1,vend1#"
-F 6 "" V 1130 2600 60  0001 C CNN ""
-F 7 "" V 1130 2600 60  0001 C CNN ""
-F 8 "100V" V 1130 2600 60  0001 C CNN "V"
-F 9 "10%" V 1130 2600 60  0001 C CNN "tolerance"
-F 10 "ceramic" V 1130 2600 60  0001 C CNN "construct"
+F 2 "SM0805" V 1130 2600 60  0001 C CNN
+F 4 "AVX,08055C104KAT2A" V 1130 2600 60  0001 C CNN "mfg,mfg#"
+F 5 "newark,27C8438" V 1130 2600 60  0001 C CNN "vend1,vend1#"
+F 6 "" V 1130 2600 60  0001 C CNN ""
+F 7 "" V 1130 2600 60  0001 C CNN ""
+F 8 "200V" V 1130 2600 60  0001 C CNN "V"
+F 9 "10%" V 1130 2600 60  0001 C CNN "TOL"
+F 10 "CERAMIC" V 1130 2600 60  0001 C CNN "construct"
 F 11 "other,more,stuff" V 1130 2600 60  0001 C CNN "misc"
 	1    1200 850
@@
 F 0 "C141" H 3710 950 50  0000 L CNN
 F 1 "100nF" H 3650 750 50  0000 L CNN
-F 2 "SM0805-C1" V 1130 2600 60  0001 C CNN
-F 4 "avx,08051C104KAT2A" V 1130 2600 60  0001 C CNN "mfg,mfg#"
-F 5 "newark,96M1354" V 1130 2600 60  0001 C CNN "vend1,vend1#"
-F 6 "" V 1130 2600 60  0001 C CNN ""
-F 7 "" V 1130 2600 60  0001 C CNN ""
-F 8 "100V" V 1130 2600 60  0001 C CNN "V"
-F 9 "10%" V 1130 2600 60  0001 C CNN "tolerance"
-F 10 "ceramic" V 1130 2600 60  0001 C CNN "construct"
+F 2 "SM0805" V 1130 2600 60  0001 C CNN
+F 4 "AVX,08055C104KAT2A" V 1130 2600 60  0001 C CNN "mfg,mfg#"
+F 5 "newark,27C8438" V 1130 2600 60  0001 C CNN "vend1,vend1#"
+F 6 "" V 1130 2600 60  0001 C CNN ""
+F 7 "" V 1130 2600 60  0001 C CNN ""
+F 8 "200V" V 1130 2600 60  0001 C CNN "V"
+F 9 "10%" V 1130 2600 60  0001 C CNN "TOL"
+F 10 "CERAMIC" V 1130 2600 60  0001 C CNN "construct"
 F 11 "other,more,stuff" V 1130 2600 60  0001 C CNN "misc"
 	1    3900 850
@@
 F 0 "C138" H 2350 960 50  0000 L CNN
 F 1 "100nF" H 2250 750 50  0000 L CNN
-F 2 "SM0805-C1" V 1130 2600 60  0001 C CNN
-F 4 "avx,08051C104KAT2A" V 1130 2600 60  0001 C CNN "mfg,mfg#"
-F 5 "newark,96M1354" V 1130 2600 60  0001 C CNN "vend1,vend1#"
-F 6 "" V 1130 2600 60  0001 C CNN ""
-F 7 "" V 1130 2600 60  0001 C CNN ""
-F 8 "100V" V 1130 2600 60  0001 C CNN "V"
-F 9 "10%" V 1130 2600 60  0001 C CNN "tolerance"
-F 10 "ceramic" V 1130 2600 60  0001 C CNN "construct"
+F 2 "SM0805" V 1130 2600 60  0001 C CNN
+F 4 "AVX,08055C104KAT2A" V 1130 2600 60  0001 C CNN "mfg,mfg#"
+F 5 "newark,27C8438" V 1130 2600 60  0001 C CNN "vend1,vend1#"
+F 6 "" V 1130 2600 60  0001 C CNN ""
+F 7 "" V 1130 2600 60  0001 C CNN ""
+F 8 "200V" V 1130 2600 60  0001 C CNN "V"
+F 9 "10%" V 1130 2600 60  0001 C CNN "TOL"
+F 10 "CERAMIC" V 1130 2600 60  0001 C CNN "construct"
 F 11 "other,more,stuff" V 1130 2600 60  0001 C CNN "misc"
 	1    2500 850
